Commit message: Rigid body dynamics back into trunk.
named coordinate frames for rigid body manipulators and the corresponding visualizers
fixed Pendulum.urdf
passed urdf dynamics tests for pendulum and acrobat.

git-svn-id: https://svn.csail.mit.edu/locomotion/robotlib/trunk@3385 c9849af7-e679-4ec6-a44e-fc146a885bd3

File: examples/Pendulum/Pendulum.urdf (robot description, URDF)
Before this commit: robot Pendulum, 4 links, 3 joints
Links:
- link arm_com: geometry visual sphere radius=.025
Joints:
- removed joint shoulder
- added joint theta: type continuous, parent base, child arm, axis 0 1 0

Commit message: updated Pendulum.urdf from Hongkai - this version works in gazebo. minor update to urdf parser: had to update the case where a root link was flagged as having no inertia, but obtained inertia via a fixed joint.
git-svn-id: https://svn.csail.mit.edu/locomotion/robotlib/trunk@3557 c9849af7-e679-4ec6-a44e-fc146a885bd3

File: examples/Pendulum/Pendulum.urdf (robot description, URDF)
Before this commit: robot Pendulum, 4 links, 3 joints
Links:
- removed link base
- added link world
- link arm: mass 1 -> 0.5; geometry collision cylinder length=.75 radius=.01; visual cylinder length=.75 radius=.01
- link arm_com: mass None -> 0.5; geometry collision sphere radius=.025; visual sphere radius=.025
- link base_part2: mass None -> 1; geometry collision sphere radius=.015; visual sphere radius=.015
Joints:
- joint base_weld: origin (none) -> xyz=0 0 1; parent base -> world
- joint theta: parent base -> base_part2
