Commit message: added value checking to simple four bar lcp test.  (but tolerance had to be quite high) added option to add additional floating base for urdf parsing. (implemented for planar only so far) redid rimless wheel urdf (via xacro) preparing for rimless wheel lcp test.
git-svn-id: https://svn.csail.mit.edu/locomotion/robotlib/trunk@3598 c9849af7-e679-4ec6-a44e-fc146a885bd3

File: examples/RimlessWheel/RimlessWheel.urdf (robot description, URDF)
Before this commit: robot RimlessWheel, 13 links, 12 joints
Links:
- removed link center
- removed link toe1
- removed link toe2
- removed link toe3
- removed link toe4
- removed link toe5
- removed link toe6
- removed link toe7
- removed link toe8
- added link hub, mass 1; visual cylinder length=.1 radius=.2
- added link spoke5; collision sphere radius=0; visual cylinder length=1 radius=0.0075
- added link spoke6; collision sphere radius=0; visual cylinder length=1 radius=0.0075
- added link spoke7; collision sphere radius=0; visual cylinder length=1 radius=0.0075
- added link spoke8; collision sphere radius=0; visual cylinder length=1 radius=0.0075
- link spoke1: geometry collision sphere radius=0; visual cylinder length=1 radius=0.0075
- link spoke2: geometry collision sphere radius=0; visual cylinder length=1 radius=0.0075
- link spoke3: geometry collision sphere radius=0; visual cylinder length=1 radius=0.0075
- link spoke4: geometry collision sphere radius=0; visual cylinder length=1 radius=0.0075
Joints:
- removed joint joint1
- removed joint joint2
- removed joint joint3
- removed joint joint4
- removed joint toejoint1
- removed joint toejoint2
- removed joint toejoint3
- removed joint toejoint4
- removed joint toejoint5
- removed joint toejoint6
- removed joint toejoint7
- removed joint toejoint8
- added joint spoke1_weld: type fixed, parent hub, child spoke1, origin xyz=0 0 0 rpy=0 0.0 0
- added joint spoke2_weld: type fixed, parent hub, child spoke2, origin xyz=0 0 0 rpy=0 0.7854 0
- added joint spoke3_weld: type fixed, parent hub, child spoke3, origin xyz=0 0 0 rpy=0 1.5708 0
- added joint spoke4_weld: type fixed, parent hub, child spoke4, origin xyz=0 0 0 rpy=0 2.3562 0
- added joint spoke5_weld: type fixed, parent hub, child spoke5, origin xyz=0 0 0 rpy=0 3.1416 0
- added joint spoke6_weld: type fixed, parent hub, child spoke6, origin xyz=0 0 0 rpy=0 3.927 0
- added joint spoke7_weld: type fixed, parent hub, child spoke7, origin xyz=0 0 0 rpy=0 4.7124 0
- added joint spoke8_weld: type fixed, parent hub, child spoke8, origin xyz=0 0 0 rpy=0 5.4978 0

Commit message: Updated RimlessWheel xacro / urdf;  it parses correctly and simulates as a PlanarRigidBodyManipulator with an error thrown for unsupported contacts.
git-svn-id: https://svn.csail.mit.edu/locomotion/robotlib/trunk@3599 c9849af7-e679-4ec6-a44e-fc146a885bd3

File: examples/RimlessWheel/RimlessWheel.urdf (robot description, URDF)
Before this commit: robot RimlessWheel, 9 links, 8 joints
Links:
- link hub: geometry visual cylinder length=.2 radius=.2

File: examples/RimlessWheel/RimlessWheel.xacro (robot description, xacro)
@@ -2,4 +2,6 @@
 <robot name="RimlessWheel" xmlns:xacro="http://ros.org/wiki/xacro">
   <xacro:property name="m" value="1" />
+  <!-- I have to add rotational inertia about the COM to the model to have a well-defined flight phase, even though the ideal rimless wheel model does not have it. -->
+  <xacro:property name="I" value="1" />
   <xacro:property name="l" value="1" />
   <xacro:property name="alpha" value="0.3927" />
@@ -7,5 +9,5 @@
     <inertial>
       <mass value="${m}"/>
-      <inertia ixx="0"  ixy="0"  ixz="0" iyy="0" iyz="0" izz="0" />
+      <inertia ixx="0"  ixy="0"  ixz="0" iyy="${I}" iyz="0" izz="0" />
     </inertial>
     <visual>
@@ -28,5 +30,5 @@
       </visual>
       <collision>
-        <origin xyz="0 0 ${l}" rpy="0 0 0"/>
+        <origin xyz="0 0 ${-l}" rpy="0 0 0"/>
         <geometry>
           <sphere radius="0"/>
