Commit message: clean up rimless wheel example (surpress warnings, fix zero inertias out of plane)
git-svn-id: https://svn.csail.mit.edu/locomotion/robotlib/trunk@7672 c9849af7-e679-4ec6-a44e-fc146a885bd3

File: examples/RimlessWheel/RimlessWheel.xacro (robot description, xacro)
@@ -12,5 +12,5 @@
     <inertial>
       <mass value="${m}"/>
-      <inertia ixx="0"  ixy="0"  ixz="0" iyy="${I}" iyz="0" izz="0" />
+      <inertia ixx="1"  ixy="0"  ixz="0" iyy="${I}" iyz="0" izz="1" />
     </inertial>
     <visual>
