Commit message: *finally* resolves 3D dynamics bug 1190.  sigh...
git-svn-id: https://svn.csail.mit.edu/locomotion/robotlib/trunk@4639 c9849af7-e679-4ec6-a44e-fc146a885bd3

File: examples/Pendulum/test/p11.urdf (robot description, URDF)
Before this commit: robot Pendulum, 3 links, 2 joints
Joints:
- joint theta: axis 0 1 0 -> 0 0 1

File: examples/Pendulum/test/p12.urdf (robot description, URDF)
Before this commit: robot Pendulum, 3 links, 2 joints
Links:
- link arm: geometry 
Joints:
- joint theta: axis 0 1 0 -> 0 0 1
