Commit message: committing Michael's patch, even though it won't pass unit tests yet.  the commit just got too complicated trying to do it in pieces (with git)
git-svn-id: https://svn.csail.mit.edu/locomotion/robotlib/trunk@4532 c9849af7-e679-4ec6-a44e-fc146a885bd3

File: examples/KneedCompassGait/KneedCompassGait.urdf (robot description, URDF)
Before this commit: robot KneedCompassGait, 10 links, 9 joints
Joints:
- joint left_knee_pin: limit lower=-Inf upper=0 effort=100 velocity=100 -> lower=0 upper=Inf effort=100 velocity=100
- joint right_knee_pin: limit lower=-Inf upper=0 effort=100 velocity=100 -> lower=0 upper=Inf effort=100 velocity=100

Commit message: *******  READ THIS *******
This is a major update to the rigid body manipulator classes.  (it will have many revision numbers because i'm pushing my git commit stack).  To update you will need to:

>> svn up
% configure
% make

You should look for out of date files that have been removed from the repo, but might not have been removed from your branch.  You can do this with
>> svn stat
and zap any files with a ? that you feel like you did not generate.  In particular, the rigid body mex files moved from util into their respective classes.

In order to update your own code, please note that:

* RigidBodyModel functionality has been merged into RigidBodyManipulator (same for the planar classes).  For the most part, code that you have which previously called the model functions can be redirected to the functionality on the manipulator class.   If you previously constructed a manipulator with
   m = RigidBodyModel('my.urdf',options);
   r = RigidBodyManipulator(m);
You should now use
   r = RigidBodyManipulator('my.urdf',options);

* The interface to the kinematics has changed a bit.  You should now do
  kinsol = doKinematics(r,q);
  pts_in_world_frame = forwardKin(r,kinsol,body_ind,pts_in_body_frame)

Let me know if you have any problems.  - Russ

****** END ESSENTIAL READ *****

fixed all unit tests.
moved HybridRigidBodyManipulator to dev (where it should have been until it's finished).

git-svn-id: https://svn.csail.mit.edu/locomotion/robotlib/trunk@4756 c9849af7-e679-4ec6-a44e-fc146a885bd3

File: examples/KneedCompassGait/KneedCompassGait.urdf (robot description, URDF)
Before this commit: robot KneedCompassGait, 10 links, 9 joints
Links:
- removed link world
Joints:
- removed joint floating_base

File: examples/KneedCompassGait/KneedCompassGait.xacro (robot description, xacro)
@@ -77,6 +77,4 @@
     </joint>
   </xacro:macro>
-  <link name="world">
-  </link>
   <link name="hip">
     <inertial>
@@ -93,9 +91,4 @@
     </visual>
   </link>
-  <joint name="floating_base" type="planar">
-    <parent link="world" />
-    <child link="hip" />
-    <axis xyz="0 1 0" />
-  </joint>
   <xacro:collisionlessleg lr="left_upper" cname="red" color="1 0 0 1" />
   <xacro:leg lr="left_lower" cname="red" color="1 0 0 1" />
