Commit message: fix state constraints logic in tiler. adds four bar demo from Andres. cute visualizer shows passive vs lqr response.
git-svn-id: https://svn.csail.mit.edu/locomotion/robotlib/trunk@5251 c9849af7-e679-4ec6-a44e-fc146a885bd3

File: examples/SimpleFourBar/FourBar2.urdf (robot description, URDF)
Before this commit: robot FourBar, 4 links, 3 joints
Links:
- link link_1: geometry visual cylinder length=4 radius=0.2
- link link_3: geometry visual cylinder length=5 radius=0.2
Joints:
- joint joint_0: limit (none) -> effort=100 velocity=100
- joint joint_1: limit effort=100 velocity=100 -> (none); origin xyz=0 0 1.8 rpy=0 0 0 -> xyz=0 0 4 rpy=0 0 0
