Commit message: sync w/ scott's branch.
git-svn-id: https://svn.csail.mit.edu/locomotion/robotlib/trunk@5557 c9849af7-e679-4ec6-a44e-fc146a885bd3

File: examples/Atlas/urdf/atlas_coffin_contact.urdf (robot description, URDF)
Before this commit: robot atlas, 29 links, 28 joints
Links:
- added link l_hand_point_mass, mass 2.9; visual sphere radius=0.03
- added link r_hand_point_mass, mass 2.9; visual sphere radius=0.03
- link l_foot: geometry collision sphere radius=0; collision sphere radius=0
- link r_foot: geometry collision sphere radius=0; collision sphere radius=0
Joints:
- added joint l_hand_joint: type fixed, parent l_hand, child l_hand_point_mass, origin xyz=0.0 0.15 0.0 rpy=0 0 0
- added joint r_hand_joint: type fixed, parent r_hand, child r_hand_point_mass, origin xyz=0.0 -0.15 0.0 rpy=0 0 0
