Commit message: updated atlas examples to use the new BDI joint names (hongkai ran into an issue with it being inconsistent with drc)
git-svn-id: https://svn.csail.mit.edu/locomotion/robotlib/trunk@6977 c9849af7-e679-4ec6-a44e-fc146a885bd3

File: examples/Atlas/urdf/atlas.urdf (robot description, URDF)
Before this commit: robot atlas, 29 links, 28 joints
Joints:
- removed joint back_lbz
- removed joint back_mby
- removed joint back_ubx
- removed joint l_leg_lax
- removed joint l_leg_lhy
- removed joint l_leg_mhx
- removed joint l_leg_uay
- removed joint l_leg_uhz
- removed joint r_leg_lax
- removed joint r_leg_lhy
- removed joint r_leg_mhx
- removed joint r_leg_uay
- removed joint r_leg_uhz
- added joint back_bkx: type revolute, parent mtorso, child utorso, origin xyz=0 0 0.05 rpy=0 -0 0, axis 1 0 0, limit lower=-0.790809 upper=0.790809 effort=94.91 velocity=12
- added joint back_bky: type revolute, parent ltorso, child mtorso, origin xyz=0 0 0.09 rpy=0 -0 0, axis 0 1 0, limit lower=-1.2 upper=1.28 effort=206.843 velocity=12
- added joint back_bkz: type revolute, parent pelvis, child ltorso, origin xyz=-0.0125 0 0 rpy=0 -0 0, axis 0 0 1, limit lower=-0.610865 upper=0.610865 effort=124.016 velocity=12
- added joint l_leg_akx: type revolute, parent l_talus, child l_foot, origin xyz=0 0 0 rpy=0 -0 0, axis 1 0 0, limit lower=-0.436 upper=0.436 effort=90 velocity=12
- added joint l_leg_aky: type revolute, parent l_lleg, child l_talus, origin xyz=0 0 -0.422 rpy=0 -0 0, axis 0 1 0, limit lower=-0.698 upper=0.698 effort=220 velocity=12
- added joint l_leg_hpx: type revolute, parent l_uglut, child l_lglut, origin xyz=0 0 0 rpy=0 -0 0, axis 1 0 0, limit lower=-0.47 upper=0.495 effort=180 velocity=12
- added joint l_leg_hpy: type revolute, parent l_lglut, child l_uleg, origin xyz=0.05 0 -0.05 rpy=0 -0 0, axis 0 1 0, limit lower=-1.75 upper=0.524 effort=260 velocity=12
- added joint l_leg_hpz: type revolute, parent pelvis, child l_uglut, origin xyz=0 0.089 0 rpy=0 -0 0, axis 0 0 1, limit lower=-0.32 upper=1.14 effort=110 velocity=12
- added joint r_leg_akx: type revolute, parent r_talus, child r_foot, origin xyz=0 0 0 rpy=0 -0 0, axis 1 0 0, limit lower=-0.436 upper=0.436 effort=90 velocity=12
- added joint r_leg_aky: type revolute, parent r_lleg, child r_talus, origin xyz=0 0 -0.422 rpy=0 -0 0, axis 0 1 0, limit lower=-0.698 upper=0.698 effort=220 velocity=12
- added joint r_leg_hpx: type revolute, parent r_uglut, child r_lglut, origin xyz=0 0 0 rpy=0 -0 0, axis 1 0 0, limit lower=-0.495 upper=0.47 effort=180 velocity=12
- added joint r_leg_hpy: type revolute, parent r_lglut, child r_uleg, origin xyz=0.05 0 -0.05 rpy=0 -0 0, axis 0 1 0, limit lower=-1.745 upper=0.524 effort=260 velocity=12
- added joint r_leg_hpz: type revolute, parent pelvis, child r_uglut, origin xyz=0 -0.089 0 rpy=0 -0 0, axis 0 0 1, limit lower=-1.14 upper=0.32 effort=260 velocity=12

File: examples/Atlas/urdf/atlas_coffin_contact.urdf (robot description, URDF)
Before this commit: robot atlas, 31 links, 30 joints
Joints:
- removed joint back_lbz
- removed joint back_mby
- removed joint back_ubx
- removed joint l_leg_lax
- removed joint l_leg_lhy
- removed joint l_leg_mhx
- removed joint l_leg_uay
- removed joint l_leg_uhz
- removed joint r_leg_lax
- removed joint r_leg_lhy
- removed joint r_leg_mhx
- removed joint r_leg_uay
- removed joint r_leg_uhz
- added joint back_bkx: type revolute, parent mtorso, child utorso, origin xyz=0 0 0.05 rpy=0 -0 0, axis 1 0 0, limit lower=-0.790809 upper=0.790809 effort=94.91 velocity=12
- added joint back_bky: type revolute, parent ltorso, child mtorso, origin xyz=0 0 0.09 rpy=0 -0 0, axis 0 1 0, limit lower=-1.2 upper=1.28 effort=206.843 velocity=12
- added joint back_bkz: type revolute, parent pelvis, child ltorso, origin xyz=-0.0125 0 0 rpy=0 -0 0, axis 0 0 1, limit lower=-0.610865 upper=0.610865 effort=124.016 velocity=12
- added joint l_leg_akx: type revolute, parent l_talus, child l_foot, origin xyz=0 0 0 rpy=0 -0 0, axis 1 0 0, limit lower=-0.436 upper=0.436 effort=90 velocity=12
- added joint l_leg_aky: type revolute, parent l_lleg, child l_talus, origin xyz=0 0 -0.422 rpy=0 -0 0, axis 0 1 0, limit lower=-0.698 upper=0.698 effort=220 velocity=12
- added joint l_leg_hpx: type revolute, parent l_uglut, child l_lglut, origin xyz=0 0 0 rpy=0 -0 0, axis 1 0 0, limit lower=-0.47 upper=0.495 effort=180 velocity=12
- added joint l_leg_hpy: type revolute, parent l_lglut, child l_uleg, origin xyz=0.05 0 -0.05 rpy=0 -0 0, axis 0 1 0, limit lower=-1.75 upper=0.524 effort=260 velocity=12
- added joint l_leg_hpz: type revolute, parent pelvis, child l_uglut, origin xyz=0 0.089 0 rpy=0 -0 0, axis 0 0 1, limit lower=-0.32 upper=1.14 effort=110 velocity=12
- added joint r_leg_akx: type revolute, parent r_talus, child r_foot, origin xyz=0 0 0 rpy=0 -0 0, axis 1 0 0, limit lower=-0.436 upper=0.436 effort=90 velocity=12
- added joint r_leg_aky: type revolute, parent r_lleg, child r_talus, origin xyz=0 0 -0.422 rpy=0 -0 0, axis 0 1 0, limit lower=-0.698 upper=0.698 effort=220 velocity=12
- added joint r_leg_hpx: type revolute, parent r_uglut, child r_lglut, origin xyz=0 0 0 rpy=0 -0 0, axis 1 0 0, limit lower=-0.495 upper=0.47 effort=180 velocity=12
- added joint r_leg_hpy: type revolute, parent r_lglut, child r_uleg, origin xyz=0.05 0 -0.05 rpy=0 -0 0, axis 0 1 0, limit lower=-1.745 upper=0.524 effort=260 velocity=12
- added joint r_leg_hpz: type revolute, parent pelvis, child r_uglut, origin xyz=0 -0.089 0 rpy=0 -0 0, axis 0 0 1, limit lower=-1.14 upper=0.32 effort=260 velocity=12

File: examples/Atlas/urdf/atlas_minimal_contact.urdf (robot description, URDF)
Before this commit: robot atlas, 29 links, 28 joints
Joints:
- removed joint back_lbz
- removed joint back_mby
- removed joint back_ubx
- removed joint l_leg_lax
- removed joint l_leg_lhy
- removed joint l_leg_mhx
- removed joint l_leg_uay
- removed joint l_leg_uhz
- removed joint r_leg_lax
- removed joint r_leg_lhy
- removed joint r_leg_mhx
- removed joint r_leg_uay
- removed joint r_leg_uhz
- added joint back_bkx: type revolute, parent mtorso, child utorso, origin xyz=0 0 0.05 rpy=0 -0 0, axis 1 0 0, limit lower=-0.790809 upper=0.790809 effort=94.91 velocity=12
- added joint back_bky: type revolute, parent ltorso, child mtorso, origin xyz=0 0 0.09 rpy=0 -0 0, axis 0 1 0, limit lower=-1.2 upper=1.28 effort=206.843 velocity=12
- added joint back_bkz: type revolute, parent pelvis, child ltorso, origin xyz=-0.0125 0 0 rpy=0 -0 0, axis 0 0 1, limit lower=-0.610865 upper=0.610865 effort=124.016 velocity=12
- added joint l_leg_akx: type revolute, parent l_talus, child l_foot, origin xyz=0 0 0 rpy=0 -0 0, axis 1 0 0, limit lower=-0.436 upper=0.436 effort=90 velocity=12
- added joint l_leg_aky: type revolute, parent l_lleg, child l_talus, origin xyz=0 0 -0.422 rpy=0 -0 0, axis 0 1 0, limit lower=-0.698 upper=0.698 effort=220 velocity=12
- added joint l_leg_hpx: type revolute, parent l_uglut, child l_lglut, origin xyz=0 0 0 rpy=0 -0 0, axis 1 0 0, limit lower=-0.47 upper=0.495 effort=180 velocity=12
- added joint l_leg_hpy: type revolute, parent l_lglut, child l_uleg, origin xyz=0.05 0 -0.05 rpy=0 -0 0, axis 0 1 0, limit lower=-1.75 upper=0.524 effort=260 velocity=12
- added joint l_leg_hpz: type revolute, parent pelvis, child l_uglut, origin xyz=0 0.089 0 rpy=0 -0 0, axis 0 0 1, limit lower=-0.32 upper=1.14 effort=110 velocity=12
- added joint r_leg_akx: type revolute, parent r_talus, child r_foot, origin xyz=0 0 0 rpy=0 -0 0, axis 1 0 0, limit lower=-0.436 upper=0.436 effort=90 velocity=12
- added joint r_leg_aky: type revolute, parent r_lleg, child r_talus, origin xyz=0 0 -0.422 rpy=0 -0 0, axis 0 1 0, limit lower=-0.698 upper=0.698 effort=220 velocity=12
- added joint r_leg_hpx: type revolute, parent r_uglut, child r_lglut, origin xyz=0 0 0 rpy=0 -0 0, axis 1 0 0, limit lower=-0.495 upper=0.47 effort=180 velocity=12
- added joint r_leg_hpy: type revolute, parent r_lglut, child r_uleg, origin xyz=0.05 0 -0.05 rpy=0 -0 0, axis 0 1 0, limit lower=-1.745 upper=0.524 effort=260 velocity=12
- added joint r_leg_hpz: type revolute, parent pelvis, child r_uglut, origin xyz=0 -0.089 0 rpy=0 -0 0, axis 0 0 1, limit lower=-1.14 upper=0.32 effort=260 velocity=12
