Commit message: Move chull Atlas to examples/Atlas and add meshes

File: examples/Atlas/urdf/atlas_chull.urdf (robot description, URDF)
Before this commit: robot atlas, 29 links, 28 joints
Links:
- link l_clav: geometry collision mesh filename=meshes/l_clav_chull.wrl scale=1 1 1; visual mesh filename=meshes/l_clav_chull.wrl scale=1 1 1
- link l_farm: geometry collision mesh filename=meshes/l_farm_chull.wrl scale=1 1 1; visual mesh filename=meshes/l_farm_chull.wrl scale=1 1 1
- link l_foot: geometry collision mesh filename=meshes/l_foot_chull.wrl scale=1 1 1; visual mesh filename=meshes/l_foot_chull.wrl scale=1 1 1
- link l_hand: geometry collision mesh filename=meshes/l_hand_chull.wrl scale=1 1 1; visual mesh filename=meshes/l_hand_chull.wrl scale=1 1 1
- link l_larm: geometry collision mesh filename=meshes/l_elbow_rx_chull.wrl scale=1 1 1; visual mesh filename=meshes/l_elbow_rx_chull.wrl scale=1 1 1
- link l_lglut: geometry visual mesh filename=meshes/l_lglut_chull.wrl scale=1 1 1
- link l_lleg: geometry collision mesh filename=meshes/l_lleg_chull.wrl scale=1 1 1; visual mesh filename=meshes/l_lleg_chull.wrl scale=1 1 1
- link l_scap: geometry collision mesh filename=meshes/l_sh_rx_chull.wrl scale=1 1 1; visual mesh filename=meshes/l_sh_rx_chull.wrl scale=1 1 1
- link l_talus: geometry visual mesh filename=meshes/l_talus_chull.wrl scale=1 1 1
- link l_uarm: geometry collision mesh filename=meshes/l_elbow_ry_chull.wrl scale=1 1 1; visual mesh filename=meshes/l_elbow_ry_chull.wrl scale=1 1 1
- link l_uglut: geometry visual mesh filename=meshes/l_uglut_chull.wrl scale=1 1 1
- link l_uleg: geometry collision mesh filename=meshes/l_uleg_chull.wrl scale=1 1 1; visual mesh filename=meshes/l_uleg_chull.wrl scale=1 1 1
- link ltorso: geometry visual mesh filename=meshes/ltorso_chull.wrl scale=1 1 1
- link mtorso: geometry visual mesh filename=meshes/mtorso_chull.wrl scale=1 1 1
- link pelvis: geometry collision mesh filename=meshes/pelvis_chull.wrl scale=1 1 1; visual mesh filename=meshes/pelvis_chull.wrl scale=1 1 1
- link r_clav: geometry collision mesh filename=meshes/r_clav_chull.wrl scale=1 1 1; visual mesh filename=meshes/r_clav_chull.wrl scale=1 1 1
- link r_farm: geometry collision mesh filename=meshes/r_farm_chull.wrl scale=1 1 1; visual mesh filename=meshes/r_farm_chull.wrl scale=1 1 1
- link r_foot: geometry collision mesh filename=meshes/r_foot_chull.wrl scale=1 1 1; visual mesh filename=meshes/r_foot_chull.wrl scale=1 1 1
- link r_hand: geometry collision mesh filename=meshes/r_hand_chull.wrl scale=1 1 1; visual mesh filename=meshes/r_hand_chull.wrl scale=1 1 1
- link r_larm: geometry collision mesh filename=meshes/r_elbow_rx_chull.wrl scale=1 1 1; visual mesh filename=meshes/r_elbow_rx_chull.wrl scale=1 1 1
- link r_lglut: geometry visual mesh filename=meshes/r_lglut_chull.wrl scale=1 1 1
- link r_lleg: geometry collision mesh filename=meshes/r_lleg_chull.wrl scale=1 1 1; visual mesh filename=meshes/r_lleg_chull.wrl scale=1 1 1
- link r_scap: geometry collision mesh filename=meshes/r_sh_rx_chull.wrl scale=1 1 1; visual mesh filename=meshes/r_sh_rx_chull.wrl scale=1 1 1
- link r_talus: geometry visual mesh filename=meshes/r_talus_chull.wrl scale=1 1 1
- link r_uarm: geometry collision mesh filename=meshes/r_elbow_ry_chull.wrl scale=1 1 1; visual mesh filename=meshes/r_elbow_ry_chull.wrl scale=1 1 1
- link r_uglut: geometry visual mesh filename=meshes/r_uglut_chull.wrl scale=1 1 1
- link r_uleg: geometry collision mesh filename=meshes/r_uleg_chull.wrl scale=1 1 1; visual mesh filename=meshes/r_uleg_chull.wrl scale=1 1 1
- link utorso: geometry collision mesh filename=meshes/utorso_chull.wrl scale=1 1 1; collision mesh filename=meshes/utorso_pack_chull.wrl scale=1 1 1

Commit message: removes reference to drcsim package.

File: examples/Atlas/urdf/atlas_chull.urdf (robot description, URDF)
Before this commit: robot atlas, 29 links, 28 joints
Links:
- link head: geometry visual mesh filename=meshes/head.wrl
