Commit message: add traj stabilization script for atlas passive ankle

File: examples/Atlas/urdf/atlas_simple_spring_ankle.urdf (robot description, URDF)
Before this commit: robot atlas, 16 links, 15 joints
Links:
- link l_foot: geometry collision sphere radius=0; collision sphere radius=0
- link r_foot: geometry collision sphere radius=0; collision sphere radius=0
