Commit message: cleaning atlas traj opt up a little

File: examples/Atlas/urdf/atlas_simple_planar_contact.urdf (robot description, URDF)
Before this commit: robot atlas, 16 links, 15 joints
Joints:
- joint l_leg_aky: limit lower=-1 upper=0.7 effort=350 velocity=12 -> lower=-1.3 upper=1 effort=70 velocity=12
- joint r_leg_aky: limit lower=-1 upper=0.7 effort=350 velocity=12 -> lower=-1.3 upper=1 effort=70 velocity=12
