Commit message: added joint limits

File: examples/Atlas/urdf/door.urdf (robot description, URDF)
Before this commit: robot door, 5 links, 4 joints
Joints:
- joint hinge: limit (none) -> lower=0 upper=3/4*pi

Commit message: changed joint types for the door hinge and handle to revolute

File: examples/Atlas/urdf/door.urdf (robot description, URDF)
Before this commit: robot door, 5 links, 4 joints
Joints:
- joint handle_turn: type continuous -> revolute
- joint hinge: type continuous -> revolute
