Commit message: add package.xml in Atlas folder, use 'package' syntax in the urdf in Atlas folder

File: examples/Atlas/urdf/robotiq.urdf (robot description, URDF)
Before this commit: robot s-model_articulated, 34 links, 33 joints
Links:
- link finger_1_link_0: geometry visual mesh filename=package://Atlas/urdf/meshes/s-model_articulated/visual/link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
- link finger_1_link_1: geometry collision box size=.028 .01 .03; visual mesh filename=package://Atlas/urdf/meshes/s-model_articulated/visual/link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
- link finger_1_link_2: geometry collision box size=.018 .01 .03; visual mesh filename=package://Atlas/urdf/meshes/s-model_articulated/visual/link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
- link finger_1_link_3: geometry collision box size=.025 .01 .03; visual mesh filename=package://Atlas/urdf/meshes/s-model_articulated/visual/link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
- link finger_2_link_0: geometry visual mesh filename=package://Atlas/urdf/meshes/s-model_articulated/visual/link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
- link finger_2_link_1: geometry collision box size=.028 .01 .03; visual mesh filename=package://Atlas/urdf/meshes/s-model_articulated/visual/link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
- link finger_2_link_2: geometry collision box size=.018 .01 .03; visual mesh filename=package://Atlas/urdf/meshes/s-model_articulated/visual/link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
- link finger_2_link_3: geometry collision box size=.025 .01 .03; visual mesh filename=package://Atlas/urdf/meshes/s-model_articulated/visual/link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
- link finger_middle_link_0: geometry visual mesh filename=package://Atlas/urdf/meshes/s-model_articulated/visual/link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
- link finger_middle_link_1: geometry collision box size=.028 .01 .03; visual mesh filename=package://Atlas/urdf/meshes/s-model_articulated/visual/link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
- link finger_middle_link_2: geometry collision box size=.018 .01 .03; visual mesh filename=package://Atlas/urdf/meshes/s-model_articulated/visual/link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
- link finger_middle_link_3: geometry collision box size=.025 .01 .03; visual mesh filename=package://Atlas/urdf/meshes/s-model_articulated/visual/link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
- link palm: geometry collision box size=.1 .01 .1; visual mesh filename=package://Atlas/urdf/meshes/s-model_articulated/visual/palm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
