Commit message: removed joint limits, fixed damping threshold

File: examples/Atlas/urdf/robotiq_limp.urdf (robot description, URDF)
Before this commit: robot s-model_articulated, 13 links, 12 joints
Joints:
- joint finger_1_joint_0: limit lower=0 upper=1.055 effort=100 -> (none)
- joint finger_1_joint_1: limit lower=0 upper=1.5708 effort=100 -> (none)
- joint finger_1_joint_2: limit lower=-0.7854 upper=3.1416 effort=100 -> (none)
- joint finger_2_joint_0: limit lower=0 upper=1.055 effort=100 -> (none)
- joint finger_2_joint_1: limit lower=0 upper=1.5708 effort=100 -> (none)
- joint finger_2_joint_2: limit lower=-0.7854 upper=3.1416 effort=100 -> (none)
- joint finger_middle_joint_0: limit lower=0 upper=1.055 effort=100 -> (none)
- joint finger_middle_joint_1: limit lower=0 upper=1.5708 effort=100 -> (none)
- joint finger_middle_joint_2: limit lower=-0.7854 upper=3.1416 effort=100 -> (none)

File: examples/Atlas/urdf/robotiq_springs.urdf (robot description, URDF)
Before this commit: robot s-model_articulated, 13 links, 12 joints
Joints:
- joint finger_1_joint_0: limit lower=0 upper=1.055 effort=100 -> (none)
- joint finger_1_joint_1: limit lower=0 upper=1.5708 effort=100 -> (none)
- joint finger_1_joint_2: limit lower=-0.7854 upper=3.1416 effort=100 -> (none)
- joint finger_2_joint_0: limit lower=0 upper=1.055 effort=100 -> (none)
- joint finger_2_joint_1: limit lower=0 upper=1.5708 effort=100 -> (none)
- joint finger_2_joint_2: limit lower=-0.7854 upper=3.1416 effort=100 -> (none)
- joint finger_middle_joint_0: limit lower=0 upper=1.055 effort=100 -> (none)
- joint finger_middle_joint_1: limit lower=0 upper=1.5708 effort=100 -> (none)
- joint finger_middle_joint_2: limit lower=-0.7854 upper=3.1416 effort=100 -> (none)

File: examples/Atlas/urdf/robotiq_springs_damping.urdf (robot description, URDF)
Before this commit: robot s-model_articulated, 13 links, 12 joints
Joints:
- joint finger_1_joint_0: limit lower=0 upper=1.055 effort=100 -> (none)
- joint finger_1_joint_1: limit lower=0 upper=1.5708 effort=100 -> (none)
- joint finger_1_joint_2: limit lower=-0.7854 upper=3.1416 effort=100 -> (none)
- joint finger_2_joint_0: limit lower=0 upper=1.055 effort=100 -> (none)
- joint finger_2_joint_1: limit lower=0 upper=1.5708 effort=100 -> (none)
- joint finger_2_joint_2: limit lower=-0.7854 upper=3.1416 effort=100 -> (none)
- joint finger_middle_joint_0: limit lower=0 upper=1.055 effort=100 -> (none)
- joint finger_middle_joint_1: limit lower=0 upper=1.5708 effort=100 -> (none)
- joint finger_middle_joint_2: limit lower=-0.7854 upper=3.1416 effort=100 -> (none)
