Commit message: added tendon actuated robotiq hand

File: examples/Atlas/urdf/robotiq_tendons.urdf (robot description, URDF)
Before this commit: robot s-model_articulated, 13 links, 12 joints
Links:
- added link finger_tensioner, mass 0.1; visual sphere radius=0.01
Joints:
- added joint finger_tensioner: type prismatic, parent palm, child finger_tensioner, origin xyz=0 0 0, axis 0 1 0, limit lower=-0.02 upper=0.1
