Commit message: added PD controlled hand and example scripts for PD control and tendons

File: examples/Atlas/urdf/robotiq_simple.urdf (robot description, URDF)
Before this commit: robot s-model_articulated, 13 links, 12 joints
Joints:
- joint finger_1_joint_0: type continuous -> revolute
- joint finger_1_joint_1: type continuous -> revolute
- joint finger_1_joint_2: type continuous -> revolute
- joint finger_2_joint_0: type continuous -> revolute
- joint finger_2_joint_1: type continuous -> revolute
- joint finger_2_joint_2: type continuous -> revolute
- joint finger_middle_joint_0: type continuous -> revolute
- joint finger_middle_joint_1: type continuous -> revolute
- joint finger_middle_joint_2: type continuous -> revolute
