Commit message: fixed atlas head mesh reference

File: examples/Atlas/urdf/atlas_convex_hull.urdf (robot description, URDF)
Before this commit: robot atlas, 29 links, 28 joints
Links:
- link head: geometry visual mesh filename=meshes/head.wrl

File: examples/Atlas/urdf/atlas_minimal_contact.urdf (robot description, URDF)
Before this commit: robot atlas, 29 links, 28 joints
Links:
- link head: geometry visual mesh filename=meshes/head.wrl

Commit message: increased radius of contact spheres in Atlas contact geometry for better numerical stability in bullet

File: examples/Atlas/urdf/atlas_convex_hull.urdf (robot description, URDF)
Before this commit: robot atlas, 29 links, 28 joints
Links:
- link l_foot: geometry collision mesh filename=package://Atlas/urdf/meshes/l_foot_chull.wrl scale=1 1 1; collision sphere radius=1e-7
- link r_foot: geometry collision mesh filename=package://Atlas/urdf/meshes/r_foot_chull.wrl scale=1 1 1; collision sphere radius=1e-7

File: examples/Atlas/urdf/atlas_minimal_contact.urdf (robot description, URDF)
Before this commit: robot atlas, 29 links, 28 joints
Links:
- link l_foot: geometry collision sphere radius=1e-7; collision sphere radius=1e-7
- link l_hand: geometry collision sphere radius=1e-7; collision sphere radius=1e-7
- link l_lleg: geometry collision sphere radius=1e-7; visual mesh filename=package://Atlas/urdf/meshes/l_lleg.wrl scale=1 1 1
- link l_uleg: geometry collision sphere radius=1e-7; collision sphere radius=1e-7
- link pelvis: geometry collision sphere radius=1e-7; collision sphere radius=1e-7
- link r_foot: geometry collision sphere radius=1e-7; collision sphere radius=1e-7
- link r_hand: geometry collision sphere radius=1e-7; collision sphere radius=1e-7
- link r_lleg: geometry collision sphere radius=1e-7; visual mesh filename=package://Atlas/urdf/meshes/r_lleg.wrl scale=1 1 1
- link r_uleg: geometry collision sphere radius=1e-7; collision sphere radius=1e-7
- link utorso: geometry collision sphere radius=1e-7; collision sphere radius=1e-7

Commit message: moved zero radius sphere handling into the geometry parser

File: examples/Atlas/urdf/atlas_convex_hull.urdf (robot description, URDF)
Before this commit: robot atlas, 29 links, 28 joints
Links:
- link l_foot: geometry collision mesh filename=package://Atlas/urdf/meshes/l_foot_chull.wrl scale=1 1 1; collision sphere radius=0
- link r_foot: geometry collision mesh filename=package://Atlas/urdf/meshes/r_foot_chull.wrl scale=1 1 1; collision sphere radius=0

Commit message: replaced atlas v3 with atlas v5

File: examples/Atlas/urdf/atlas_convex_hull.urdf (robot description, URDF)
Before this commit: robot atlas, 29 links, 28 joints
Links:
- removed link l_farm
- removed link r_farm
- added link center_bottom_led_frame, mass 0.1
- added link center_top_led_frame, mass 0.1
- added link head_hokuyo_frame, mass 0.01
- added link hokuyo_link, mass 0.057664; collision mesh filename=package://Atlas/urdf/meshes/head_camera_chull.obj; visual mesh filename=package://Atlas/urdf/meshes/head_camera_chull.obj
- added link l_hand_camera_link
- added link l_hand_camera_optical_frame
- added link l_hand_face
- added link l_hand_force_torque, mass 0.1; visual box size=0.01 0.01 0.01
- added link l_hand_gripper
- added link l_lfarm, mass 0.648; collision mesh filename=package://Atlas/urdf/meshes/r_hand_chull.obj; visual mesh filename=package://Atlas/urdf/meshes/r_hand.obj
- added link l_ufarm, mass 2.4798; collision mesh filename=package://Atlas/urdf/meshes/r_farm_chull.obj; visual mesh filename=package://Atlas/urdf/meshes/r_farm.obj
- added link left_camera_frame, mass 0.1
- added link left_led_frame, mass 0.1
- added link left_palm; collision mesh filename=package://Atlas/urdf/meshes/GRIPPER_OPEN_chull.obj scale=1 1 1; visual mesh filename=package://Atlas/urdf/meshes/GRIPPER_OPEN_chull.obj scale=1 1 1
- added link post_spindle
- added link post_spindle_cal_pitch
- added link post_spindle_cal_roll
- added link post_spindle_cal_x
- added link post_spindle_cal_y
- added link post_spindle_cal_z
- added link pre_spindle
- added link pre_spindle_cal_pitch
- added link pre_spindle_cal_roll
- added link pre_spindle_cal_x
- added link pre_spindle_cal_y
- added link pre_spindle_cal_yaw
- added link pre_spindle_cal_z
- added link r_hand_camera_link
- added link r_hand_camera_optical_frame
- added link r_hand_face
- added link r_hand_force_torque, mass 0.1; visual box size=0.01 0.01 0.01
- added link r_hand_gripper
- added link r_lfarm, mass 0.648; collision mesh filename=package://Atlas/urdf/meshes/r_hand_chull.obj; visual mesh filename=package://Atlas/urdf/meshes/r_hand.obj
- added link r_ufarm, mass 2.4798; collision mesh filename=package://Atlas/urdf/meshes/r_farm_chull.obj; visual mesh filename=package://Atlas/urdf/meshes/r_farm.obj
- added link right_led_frame, mass 0.1
- added link right_palm; collision mesh filename=package://Atlas/urdf/meshes/GRIPPER_OPEN_chull.obj scale=1 1 1; visual mesh filename=package://Atlas/urdf/meshes/GRIPPER_OPEN_chull.obj scale=1 1 1
- link head: mass 1.477574 -> 1.4199; geometry collision mesh filename=package://Atlas/urdf/meshes/head_chull.obj; visual mesh filename=package://Atlas/urdf/meshes/head_chull.obj
- link l_clav: mass 3.45 -> 4.466; geometry collision mesh filename=package://Atlas/urdf/meshes/r_clav_chull.obj; visual mesh filename=package://Atlas/urdf/meshes/r_clav.obj
- link l_foot: mass 2.05 -> 2.410; geometry collision mesh filename=package://Atlas/urdf/meshes/l_foot_chull.obj; collision sphere radius=0.0
- link l_hand: mass 2.509 -> 0.5839; geometry 
- link l_larm: mass 2.509 -> 3.248; geometry collision mesh filename=package://Atlas/urdf/meshes/r_larm_chull.obj; visual mesh filename=package://Atlas/urdf/meshes/r_larm.obj
- link l_lglut: mass 0.866 -> 0.898; geometry collision mesh filename=package://Atlas/urdf/meshes/l_lglut_chull.obj; visual mesh filename=package://Atlas/urdf/meshes/l_lglut.obj
- link l_lleg: mass 5.479 -> 4.515; geometry collision mesh filename=package://Atlas/urdf/meshes/l_lleg_chull.obj; visual mesh filename=package://Atlas/urdf/meshes/l_lleg.obj
- link l_scap: mass 3.012 -> 3.899; geometry collision mesh filename=package://Atlas/urdf/meshes/r_scap_chull.obj; visual mesh filename=package://Atlas/urdf/meshes/r_scap.obj
- link l_talus: geometry visual mesh filename=package://Atlas/urdf/meshes/l_talus.obj
- link l_uarm: mass 3.388 -> 4.386; geometry collision mesh filename=package://Atlas/urdf/meshes/r_uarm_chull.obj; visual mesh filename=package://Atlas/urdf/meshes/r_uarm.obj
- link l_uglut: mass 0.648 -> 1.959; geometry collision mesh filename=package://Atlas/urdf/meshes/l_uglut_chull.obj; visual mesh filename=package://Atlas/urdf/meshes/l_uglut.obj
- link l_uleg: mass 9.209 -> 8.204; geometry collision mesh filename=package://Atlas/urdf/meshes/l_uleg_chull.obj; visual mesh filename=package://Atlas/urdf/meshes/l_uleg.obj
- link ltorso: mass 2.409 -> 2.270; geometry visual mesh filename=package://Atlas/urdf/meshes/ltorso.obj
- link mtorso: mass 0.69 -> 0.799; geometry visual mesh filename=package://Atlas/urdf/meshes/mtorso.obj
- link pelvis: mass 17.882 -> 9.509; geometry collision mesh filename=package://Atlas/urdf/meshes/pelvis_chull.obj; visual mesh filename=package://Atlas/urdf/meshes/pelvis.obj
- link r_clav: mass 3.45 -> 4.466; geometry collision mesh filename=package://Atlas/urdf/meshes/r_clav_chull.obj; visual mesh filename=package://Atlas/urdf/meshes/r_clav.obj
- link r_foot: mass 2.05 -> 2.41; geometry collision mesh filename=package://Atlas/urdf/meshes/r_foot_chull.obj; collision sphere radius=0.0
- link r_hand: mass 2.509 -> 0.5839; geometry 
- link r_larm: mass 2.509 -> 3.248; geometry collision mesh filename=package://Atlas/urdf/meshes/r_larm_chull.obj; visual mesh filename=package://Atlas/urdf/meshes/r_larm.obj
- link r_lglut: mass 0.866 -> 0.898; geometry collision mesh filename=package://Atlas/urdf/meshes/r_lglut_chull.obj; visual mesh filename=package://Atlas/urdf/meshes/r_lglut.obj
- link r_lleg: mass 5.479 -> 4.515; geometry collision mesh filename=package://Atlas/urdf/meshes/r_lleg_chull.obj; visual mesh filename=package://Atlas/urdf/meshes/r_lleg.obj
- link r_scap: mass 3.012 -> 3.899; geometry collision mesh filename=package://Atlas/urdf/meshes/r_scap_chull.obj; visual mesh filename=package://Atlas/urdf/meshes/r_scap.obj
- link r_talus: geometry visual mesh filename=package://Atlas/urdf/meshes/r_talus.obj
- link r_uarm: mass 3.388 -> 4.386; geometry collision mesh filename=package://Atlas/urdf/meshes/r_uarm_chull.obj; visual mesh filename=package://Atlas/urdf/meshes/r_uarm.obj
- link r_uglut: mass 0.648 -> 1.959; geometry collision mesh filename=package://Atlas/urdf/meshes/r_uglut_chull.obj; visual mesh filename=package://Atlas/urdf/meshes/r_uglut.obj
- link r_uleg: mass 9.209 -> 8.204; geometry collision mesh filename=package://Atlas/urdf/meshes/r_uleg_chull.obj; visual mesh filename=package://Atlas/urdf/meshes/r_uleg.obj
- link utorso: mass 52 -> 84.409; geometry collision mesh filename=package://Atlas/urdf/meshes/utorso_chull.obj; visual mesh filename=package://Atlas/urdf/meshes/utorso.obj
Joints:
- removed joint l_arm_usy
- removed joint r_arm_usy
- added joint center_bottom_led_frame_joint: type fixed, parent head, child center_bottom_led_frame, origin xyz=0.01125 0.0 -0.0155
- added joint center_top_led_frame_joint: type fixed, parent head, child center_top_led_frame, origin xyz=0.01125 0.0 0.0105
- added joint head_hokuyo_fixed_joint: type fixed, parent hokuyo_link, child head_hokuyo_frame, origin xyz=0.03 0 0.015 rpy=0 0 0, axis 0 1 0
- added joint hokuyo_joint: type fixed, parent pre_spindle_cal_yaw, child post_spindle, origin xyz=0 0 0 rpy=0 0 0, axis 1 0 0
- added joint l_arm_lwy: type revolute, parent l_lfarm, child l_hand, origin xyz=0 0 0 rpy=0 3.14159265359 0, axis -0.0 -1.0 -0.0, limit lower=-2.9671 upper=2.9671 effort=25 velocity=10
- added joint l_arm_shz: type revolute, parent utorso, child l_clav, origin xyz=0.1406 0.2256 0.4776 rpy=0 0 3.14159265359, axis 0 0 1, limit lower=-1.5708 upper=0.785398 effort=87 velocity=12
- added joint l_hand_camera_joint: type fixed, parent l_hand_force_torque, child l_hand_camera_link, origin xyz=-0.09892  0.01431 0.0 rpy= -1.57079 0  1.5708
- added joint l_hand_camera_optical_frame_joint: type fixed, parent l_hand_camera_link, child l_hand_camera_optical_frame, origin xyz=0 0 0 rpy=-1.57079 0.0 -1.57079
- added joint l_hand_face_joint: type fixed, parent l_hand_force_torque, child l_hand_face, origin xyz=0 0.12 0 rpy=0.0 0.0 0.0
- added joint l_hand_force_torque_joint: type fixed, parent l_hand, child l_hand_force_torque, origin xyz=0 -0.1245 0 rpy=0 0 3.141592
- added joint l_hand_gripper_joint: type fixed, parent l_hand_force_torque, child l_hand_gripper, origin xyz=0 0.18 0 rpy=0.0 0.0 0.0
- added joint left_camera_frame_joint: type fixed, parent head, child left_camera_frame, origin xyz=0.0 0.035 -0.002
- added joint left_led_frame_joint: type fixed, parent head, child left_led_frame, origin xyz=-0.01443 0.07452 0.050346 rpy=0 -0.15 0.53
- added joint left_palm_joint: type fixed, parent l_hand_force_torque, child left_palm
- added joint post_spindle_cal_pitch_joint: type fixed, parent post_spindle_cal_roll, child post_spindle_cal_pitch, axis 0 1 0
- added joint post_spindle_cal_roll_joint: type fixed, parent post_spindle_cal_z, child post_spindle_cal_roll, axis 1 0 0
- added joint post_spindle_cal_x_joint: type fixed, parent post_spindle, child post_spindle_cal_x, axis 1 0 0, limit lower=-0.5 upper=0.5 effort=0.0 velocity=0.0
- added joint post_spindle_cal_y_joint: type fixed, parent post_spindle_cal_x, child post_spindle_cal_y, axis 0 1 0, limit lower=-0.5 upper=0.5 effort=0.0 velocity=0.0
- added joint post_spindle_cal_yaw_joint: type fixed, parent post_spindle_cal_pitch, child hokuyo_link, axis 0 0 1
- added joint post_spindle_cal_z_joint: type fixed, parent post_spindle_cal_y, child post_spindle_cal_z, axis 0 0 1, limit lower=-0.5 upper=0.5 effort=0.0 velocity=0.0
- added joint pre_spindle_cal_pitch_joint: type fixed, parent pre_spindle_cal_roll, child pre_spindle_cal_pitch, axis 0 1 0
- added joint pre_spindle_cal_roll_joint: type fixed, parent pre_spindle_cal_z, child pre_spindle_cal_roll, axis 1 0 0
- added joint pre_spindle_cal_x_joint: type fixed, parent pre_spindle, child pre_spindle_cal_x, axis 1 0 0, limit lower=-0.5 upper=0.5 effort=0.0 velocity=0.0
- added joint pre_spindle_cal_y_joint: type fixed, parent pre_spindle_cal_x, child pre_spindle_cal_y, axis 0 1 0, limit lower=-0.5 upper=0.5 effort=0.0 velocity=0.0
- added joint pre_spindle_cal_yaw_joint: type fixed, parent pre_spindle_cal_pitch, child pre_spindle_cal_yaw, axis 0 0 1
- added joint pre_spindle_cal_z_joint: type fixed, parent pre_spindle_cal_y, child pre_spindle_cal_z, axis 0 0 1, limit lower=-0.5 upper=0.5 effort=0.0 velocity=0.0
- added joint pre_spindle_joint: type fixed, parent head, child pre_spindle, origin xyz=-0.0446 0 0.0880 rpy=0 0 0, axis 0 1 0
- added joint r_arm_lwy: type revolute, parent r_lfarm, child r_hand, origin xyz=0 0 0 rpy=0 0 0, axis 0 1 0, limit lower=-2.9671 upper=2.9671 effort=25 velocity=10
- added joint r_arm_shz: type revolute, parent utorso, child r_clav, origin xyz=0.1406 -0.2256 0.4776 rpy=0 0 0, axis 0 0 1, limit lower=-0.785398 upper=1.5708 effort=87 velocity=12
- added joint r_hand_camera_joint: type fixed, parent r_hand_force_torque, child r_hand_camera_link, origin xyz=0.09892  0.01431 0.0 rpy= 1.57079 0  1.5708
- added joint r_hand_camera_optical_frame_joint: type fixed, parent r_hand_camera_link, child r_hand_camera_optical_frame, origin xyz=0 0 0 rpy=-1.57079 0.0 -1.57079
- added joint r_hand_face_joint: type fixed, parent r_hand_force_torque, child r_hand_face, origin xyz=0 0.12 0 rpy=0.0 0.0 0.0
- added joint r_hand_force_torque_joint: type fixed, parent r_hand, child r_hand_force_torque, origin xyz=0 -0.1245 0 rpy=0 0 3.141592
- added joint r_hand_gripper_joint: type fixed, parent r_hand_force_torque, child r_hand_gripper, origin xyz=0 0.18 0 rpy=0.0 0.0 0.0
- added joint right_led_frame_joint: type fixed, parent head, child right_led_frame, origin xyz=-0.01443 -0.07452 0.050346 rpy=0 -0.15 -0.53
- added joint right_palm_joint: type fixed, parent r_hand_force_torque, child right_palm
- joint back_bkx: limit lower=-0.698132 upper=0.698132 effort=200 velocity=12 -> lower=-0.523599 upper=0.523599 effort=300 velocity=12; origin xyz=0 0 0.05 rpy=0 -0 0 -> xyz=0 0 0.05 rpy=0 0 0
- joint back_bky: limit lower=-0.262 upper=0.524 effort=206.843 velocity=12 -> lower=-0.219388 upper=0.538783 effort=445 velocity=9; origin xyz=0 0 0.16197 rpy=0 -0 0 -> xyz=0 0 0.162 rpy=0 0 0
- joint back_bkz: limit lower=-0.663225 upper=0.663225 effort=114 velocity=12 -> lower=-0.663225 upper=0.663225 effort=106 velocity=12; origin xyz=-0.0125 0 0 rpy=0 -0 0 -> xyz=-0.0125 0 0 rpy=0 0 0
- joint l_arm_elx: axis 1 0 0 -> -1.0 -0.0 -0.0; limit lower=0 upper=2.35619 effort=55 velocity=12 -> lower=0 upper=2.35619 effort=112 velocity=12; origin xyz=0 0.119 0.00921 rpy=0 -0 0 -> xyz=0 -0.119 0.0092 rpy=0 0 0
- joint l_arm_ely: axis 0 1 0 -> -0.0 -1.0 -0.0; limit lower=0 upper=3.14159 effort=55 velocity=12 -> lower=0 upper=3.14159 effort=63 velocity=12; origin xyz=0 0.187 0.016 rpy=0 -0 0 -> xyz=0 -0.187 -0.016 rpy=0 0 0
- joint l_arm_mwx: child l_hand -> l_lfarm; limit lower=-1.1781 upper=1.1781 effort=55 velocity=12 -> lower=-1.7628 upper=1.7628 effort=25 velocity=10; origin xyz=0 0.119 0.00921 rpy=0 -0 0 -> xyz=0 0 0 rpy=0 0 0; parent l_farm -> l_ufarm
- joint l_arm_shx: axis 1 0 0 -> -1.0 -0.0 -0.0; limit lower=-1.5708 upper=1.5708 effort=107 velocity=12 -> lower=-1.5708 upper=1.5708 effort=99 velocity=12; origin xyz=0 0.14035 0.19609 rpy=0 -0 0 -> xyz=0 -0.11 -0.245 rpy=0 0 0
- joint l_arm_uwy: axis 0 1 0 -> -0.0 -1.0 -0.0; child l_farm -> l_ufarm; limit lower=0 upper=3.14159 effort=55 velocity=12 -> lower=-3.011 upper=3.011 effort=25 velocity=10; origin xyz=0 0.187 -0.00921 rpy=0 -0 0 -> xyz=0 -0.29955 -0.00921 rpy=0 3.14159265359 0
- joint l_leg_akx: limit lower=-0.8 upper=0.8 effort=130 velocity=12 -> lower=-0.8 upper=0.8 effort=360 velocity=12; origin xyz=0 0 0 rpy=0 -0 0 -> xyz=0 0 0 rpy=0 0 0
- joint l_leg_aky: limit lower=-1 upper=0.7 effort=350 velocity=12 -> lower=-1 upper=0.7 effort=740 velocity=12; origin xyz=0 0 -0.422 rpy=0 -0 0 -> xyz=0 0 -0.422 rpy=0 0 0
- joint l_leg_hpx: limit lower=-0.523599 upper=0.523599 effort=250 velocity=12 -> lower=-0.523599 upper=0.523599 effort=530 velocity=12; origin xyz=0 0 0 rpy=0 -0 0 -> xyz=0 0 0 rpy=0 0 0
- joint l_leg_hpy: limit lower=-1.72072 upper=0.524821 effort=260 velocity=12 -> lower=-1.61234 upper=0.65764 effort=840 velocity=12; origin xyz=0.05 0 -0.05 rpy=0 -0 0 -> xyz=0.05 0.0225 -0.066 rpy=0 0 0
- joint l_leg_hpz: limit lower=-0.174533 upper=1.22173 effort=68 velocity=12 -> lower=-0.174358 upper=0.786794 effort=275 velocity=12; origin xyz=0 0.089 0 rpy=0 -0 0 -> xyz=0 0.089 0 rpy=0 0 0
- joint l_leg_kny: limit lower=0 upper=2.38569 effort=220 velocity=12 -> lower=0 upper=2.35637 effort=890 velocity=12; origin xyz=-0.05 0 -0.374 rpy=0 -0 0 -> xyz=-0.05 0 -0.374 rpy=0 0 0
- joint neck_ay: limit lower=-0.602139 upper=1.14494 effort=5 velocity=12 -> lower=-0.602139 upper=1.14319 effort=25 velocity=6.28; origin xyz=0.21672 0 0.53796 rpy=0 -0 0 -> xyz=0.2546 0 0.6215 rpy=0 0 0
- joint r_arm_elx: limit lower=-2.35619 upper=0 effort=55 velocity=12 -> lower=-2.35619 upper=0 effort=112 velocity=12; origin xyz=0 -0.119 0.00921 rpy=0 -0 0 -> xyz=0 -0.119 0.0092 rpy=0 0 0
- joint r_arm_ely: limit lower=0 upper=3.14159 effort=55 velocity=12 -> lower=0 upper=3.14159 effort=63 velocity=12; origin xyz=0 -0.187 0.016 rpy=0 -0 0 -> xyz=0 -0.187 -0.016 rpy=0 0 0
- joint r_arm_mwx: child r_hand -> r_lfarm; limit lower=-1.1781 upper=1.1781 effort=55 velocity=12 -> lower=-1.7628 upper=1.7628 effort=25 velocity=10; origin xyz=0 -0.119 0.00921 rpy=0 -0 0 -> xyz=0 0 0 rpy=0 0 0; parent r_farm -> r_ufarm
- joint r_arm_shx: limit lower=-1.5708 upper=1.5708 effort=107 velocity=12 -> lower=-1.5708 upper=1.5708 effort=99 velocity=12; origin xyz=0 -0.14035 0.19609 rpy=0 -0 0 -> xyz=0 -0.11 -0.245 rpy=0 0 0
- joint r_arm_uwy: child r_farm -> r_ufarm; limit lower=0 upper=3.14159 effort=55 velocity=12 -> lower=-3.011 upper=3.011 effort=25 velocity=10; origin xyz=0 -0.187 -0.00921 rpy=0 -0 0 -> xyz=0 -0.29955 -0.00921 rpy=0 0 0
- joint r_leg_akx: limit lower=-0.8 upper=0.8 effort=130 velocity=12 -> lower=-0.8 upper=0.8 effort=360 velocity=12; origin xyz=0 0 0 rpy=0 -0 0 -> xyz=0 0 0 rpy=0 0 0
- joint r_leg_aky: limit lower=-1 upper=0.7 effort=350 velocity=12 -> lower=-1 upper=0.7 effort=740 velocity=12; origin xyz=0 0 -0.422 rpy=0 -0 0 -> xyz=0 0 -0.422 rpy=0 0 0
- joint r_leg_hpx: limit lower=-0.523599 upper=0.523599 effort=250 velocity=12 -> lower=-0.523599 upper=0.523599 effort=530 velocity=12; origin xyz=0 0 0 rpy=0 -0 0 -> xyz=0 0 0 rpy=0 0 0
- joint r_leg_hpy: limit lower=-1.72072 upper=0.524821 effort=260 velocity=12 -> lower=-1.61234 upper=0.65764 effort=840 velocity=12; origin xyz=0.05 0 -0.05 rpy=0 -0 0 -> xyz=0.05 -0.0225 -0.066 rpy=0 0 0
- joint r_leg_hpz: limit lower=-1.22173 upper=0.174533 effort=68 velocity=12 -> lower=-0.786794 upper=0.174358 effort=275 velocity=12; origin xyz=0 -0.089 0 rpy=0 -0 0 -> xyz=0 -0.089 0 rpy=0 0 0
- joint r_leg_kny: limit lower=0 upper=2.38569 effort=220 velocity=12 -> lower=0 upper=2.35637 effort=890 velocity=12; origin xyz=-0.05 0 -0.374 rpy=0 -0 0 -> xyz=-0.05 0 -0.374 rpy=0 0 0
