Commit message: fixed textures, removed spurious contact points, fixed unit test bugs

File: examples/Atlas/urdf/atlas_convex_hull.urdf (robot description, URDF)
Before this commit: robot atlas, 63 links, 62 joints
Links:
- added link l_situational_awareness_camera_link, mass 0.1; collision box size=0.01 0.01 0.01; visual box size=0.01 0.01 0.01
- added link l_situational_awareness_camera_optical_frame
- added link left_camera_optical_frame
- added link r_situational_awareness_camera_link, mass 0.1; collision box size=0.01 0.01 0.01; visual box size=0.01 0.01 0.01
- added link r_situational_awareness_camera_optical_frame
- added link right_camera_frame, mass 0.1
- added link right_camera_optical_frame
Joints:
- added joint l_situational_awareness_camera_joint: type fixed, parent utorso, child l_situational_awareness_camera_link, origin xyz=0.155 0.121 0.785 rpy=0 0 1.309
- added joint l_situational_awareness_camera_optical_frame_joint: type fixed, parent l_situational_awareness_camera_link, child l_situational_awareness_camera_optical_frame, origin xyz=0 0 0 rpy=-1.5708 0.0 -1.5708
- added joint left_camera_optical_frame_joint: type fixed, parent left_camera_frame, child left_camera_optical_frame, origin xyz=0 0 0 rpy=-1.5708 0.0 -1.5708
- added joint r_situational_awareness_camera_joint: type fixed, parent utorso, child r_situational_awareness_camera_link, origin xyz=0.155 -0.121 0.785 rpy=0 0 -1.309
- added joint r_situational_awareness_camera_optical_frame_joint: type fixed, parent r_situational_awareness_camera_link, child r_situational_awareness_camera_optical_frame, origin xyz=0 0 0 rpy=-1.5708 0.0 -1.5708
- added joint right_camera_frame_joint: type fixed, parent head, child right_camera_frame, origin xyz=0.0 -0.035 -0.002
- added joint right_camera_optical_frame_joint: type fixed, parent right_camera_frame, child right_camera_optical_frame, origin xyz=0 0 0 rpy=-1.5708 0.0 -1.5708

File: examples/Atlas/urdf/atlas_minimal_contact.urdf (robot description, URDF)
Before this commit: robot atlas, 81 links, 80 joints
Links:
- removed link l_hand_camera_link
- removed link l_hand_camera_optical_frame
- removed link l_hand_face
- removed link l_hand_gripper
- removed link left_finger_1_link_0
- removed link left_finger_1_link_1
- removed link left_finger_1_link_2
- removed link left_finger_1_link_3
- removed link left_finger_2_link_0
- removed link left_finger_2_link_1
- removed link left_finger_2_link_2
- removed link left_finger_2_link_3
- removed link left_finger_middle_link_0
- removed link left_finger_middle_link_1
- removed link left_finger_middle_link_2
- removed link left_finger_middle_link_3
- removed link left_palm
- removed link r_hand_camera_link
- removed link r_hand_camera_optical_frame
- removed link r_hand_face
- removed link r_hand_gripper
- removed link right_finger_1_link_0
- removed link right_finger_1_link_1
- removed link right_finger_1_link_2
- removed link right_finger_1_link_3
- removed link right_finger_2_link_0
- removed link right_finger_2_link_1
- removed link right_finger_2_link_2
- removed link right_finger_2_link_3
- removed link right_finger_middle_link_0
- removed link right_finger_middle_link_1
- removed link right_finger_middle_link_2
- removed link right_finger_middle_link_3
- removed link right_palm
- added link center_bottom_led_frame, mass 0.1
- added link center_top_led_frame, mass 0.1
- added link head_hokuyo_frame, mass 0.01
- added link l_situational_awareness_camera_link, mass 0.1; visual box size=0.01 0.01 0.01
- added link l_situational_awareness_camera_optical_frame
- added link left_camera_frame, mass 0.1
- added link left_camera_optical_frame
- added link left_led_frame, mass 0.1
- added link r_situational_awareness_camera_link, mass 0.1; visual box size=0.01 0.01 0.01
- added link r_situational_awareness_camera_optical_frame
- added link right_camera_frame, mass 0.1
- added link right_camera_optical_frame
- added link right_led_frame, mass 0.1
- link l_hand: geometry 
- link l_lleg: geometry visual mesh filename=package://Atlas/urdf/meshes/l_lleg.obj
- link l_uleg: geometry visual mesh filename=package://Atlas/urdf/meshes/l_uleg.obj
- link pelvis: geometry visual mesh filename=package://Atlas/urdf/meshes/pelvis.obj
- link r_hand: geometry 
- link r_lleg: geometry visual mesh filename=package://Atlas/urdf/meshes/r_lleg.obj
- link r_uleg: geometry visual mesh filename=package://Atlas/urdf/meshes/r_uleg.obj
- link utorso: geometry visual mesh filename=package://Atlas/urdf/meshes/utorso.obj
Joints:
- removed joint l_hand_camera_joint
- removed joint l_hand_camera_optical_frame_joint
- removed joint l_hand_face_joint
- removed joint l_hand_gripper_joint
- removed joint left_finger_1_joint_1
- removed joint left_finger_1_joint_2
- removed joint left_finger_1_joint_3
- removed joint left_finger_2_joint_1
- removed joint left_finger_2_joint_2
- removed joint left_finger_2_joint_3
- removed joint left_finger_middle_joint_1
- removed joint left_finger_middle_joint_2
- removed joint left_finger_middle_joint_3
- removed joint left_palm_finger_1_joint
- removed joint left_palm_finger_2_joint
- removed joint left_palm_finger_middle_joint
- removed joint left_robotiq_hand_joint
- removed joint r_hand_camera_joint
- removed joint r_hand_camera_optical_frame_joint
- removed joint r_hand_face_joint
- removed joint r_hand_gripper_joint
- removed joint right_finger_1_joint_1
- removed joint right_finger_1_joint_2
- removed joint right_finger_1_joint_3
- removed joint right_finger_2_joint_1
- removed joint right_finger_2_joint_2
- removed joint right_finger_2_joint_3
- removed joint right_finger_middle_joint_1
- removed joint right_finger_middle_joint_2
- removed joint right_finger_middle_joint_3
- removed joint right_palm_finger_1_joint
- removed joint right_palm_finger_2_joint
- removed joint right_palm_finger_middle_joint
- removed joint right_robotiq_hand_joint
- added joint center_bottom_led_frame_joint: type fixed, parent head, child center_bottom_led_frame, origin xyz=0.01125 0.0 -0.0155
- added joint center_top_led_frame_joint: type fixed, parent head, child center_top_led_frame, origin xyz=0.01125 0.0 0.0105
- added joint head_hokuyo_fixed_joint: type fixed, parent hokuyo_link, child head_hokuyo_frame, origin xyz=0.03 0 0.015 rpy=0 0 0, axis 0 1 0
- added joint l_situational_awareness_camera_joint: type fixed, parent utorso, child l_situational_awareness_camera_link, origin xyz=0.155 0.121 0.785 rpy=0 0 1.309
- added joint l_situational_awareness_camera_optical_frame_joint: type fixed, parent l_situational_awareness_camera_link, child l_situational_awareness_camera_optical_frame, origin xyz=0 0 0 rpy=-1.5708 0.0 -1.5708
- added joint left_camera_frame_joint: type fixed, parent head, child left_camera_frame, origin xyz=0.0 0.035 -0.002
- added joint left_camera_optical_frame_joint: type fixed, parent left_camera_frame, child left_camera_optical_frame, origin xyz=0 0 0 rpy=-1.5708 0.0 -1.5708
- added joint left_led_frame_joint: type fixed, parent head, child left_led_frame, origin xyz=-0.01443 0.07452 0.050346 rpy=0 -0.15 0.53
- added joint r_situational_awareness_camera_joint: type fixed, parent utorso, child r_situational_awareness_camera_link, origin xyz=0.155 -0.121 0.785 rpy=0 0 -1.309
- added joint r_situational_awareness_camera_optical_frame_joint: type fixed, parent r_situational_awareness_camera_link, child r_situational_awareness_camera_optical_frame, origin xyz=0 0 0 rpy=-1.5708 0.0 -1.5708
- added joint right_camera_frame_joint: type fixed, parent head, child right_camera_frame, origin xyz=0.0 -0.035 -0.002
- added joint right_camera_optical_frame_joint: type fixed, parent right_camera_frame, child right_camera_optical_frame, origin xyz=0 0 0 rpy=-1.5708 0.0 -1.5708
- added joint right_led_frame_joint: type fixed, parent head, child right_led_frame, origin xyz=-0.01443 -0.07452 0.050346 rpy=0 -0.15 -0.53

Commit message: add forefoot-only support for narrow stairs

File: examples/Atlas/urdf/atlas_convex_hull.urdf (robot description, URDF)
Before this commit: robot atlas, 70 links, 69 joints
Links:
- link l_foot: geometry collision mesh filename=package://Atlas/urdf/meshes/l_foot_chull.obj; collision sphere radius=0.0
- link r_foot: geometry collision mesh filename=package://Atlas/urdf/meshes/r_foot_chull.obj; collision sphere radius=0.0

File: examples/Atlas/urdf/atlas_minimal_contact.urdf (robot description, URDF)
Before this commit: robot atlas, 60 links, 59 joints
Links:
- link l_foot: geometry collision sphere radius=0.0; collision sphere radius=0.0
- link r_foot: geometry collision sphere radius=0.0; collision sphere radius=0.0
