Commit message: merge from Hongkai and Andres for ik sequences.  Added Atlas example. Updated atlas_minimal_contact.urdf to the model with contact points on the knees and hands. (and made the corresponding mods)
git-svn-id: https://svn.csail.mit.edu/locomotion/robotlib/trunk@5657 c9849af7-e679-4ec6-a44e-fc146a885bd3

File: examples/Atlas/urdf/atlas_minimal_contact.urdf (robot description, URDF)
Before this commit: robot atlas, 29 links, 28 joints
Links:
- link head: geometry visual mesh filename=package://mit_drcsim_scripts/models/multisense_sl/meshes/ba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
- link l_clav: geometry visual mesh filename=package://mit_drcsim_scripts/models/mit_robot/meshes/l_clav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 scale=1 1 1
- link l_farm: geometry visual mesh filename=package://mit_drcsim_scripts/models/mit_robot/meshes/l_farm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 scale=1 1 1
- link l_foot: mass 1.634 -> 0.817; geometry collision sphere radius=0; collision sphere radius=0
- link l_hand: geometry collision sphere radius=0; visual mesh filename=package://mit_drcsim_scripts/models/mit_robot/meshes/l_hand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 scale=1 1 1
- link l_larm: geometry visual mesh filename=package://mit_drcsim_scripts/models/mit_robot/meshes/l_larm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 scale=1 1 1
- link l_lglut: geometry visual mesh filename=package://mit_drcsim_scripts/models/mit_robot/meshes/l_lglu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 scale=1 1 1
- link l_lleg: geometry collision sphere radius=0; visual mesh filename=package://mit_drcsim_scripts/models/mit_robot/meshes/l_lleg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 scale=1 1 1
- link l_scap: geometry visual mesh filename=package://mit_drcsim_scripts/models/mit_robot/meshes/l_scap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 scale=1 1 1
- link l_talus: mass 0.1 -> 0.817; geometry visual mesh filename=package://mit_drcsim_scripts/models/mit_robot/meshes/l_talu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 scale=1 1 1
- link l_uarm: geometry visual mesh filename=package://mit_drcsim_scripts/models/mit_robot/meshes/l_uarm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 scale=1 1 1
- link l_uglut: geometry visual mesh filename=package://mit_drcsim_scripts/models/mit_robot/meshes/l_uglu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 scale=1 1 1
- link l_uleg: geometry visual mesh filename=package://mit_drcsim_scripts/models/mit_robot/meshes/l_uleg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 scale=1 1 1
- link ltorso: geometry visual mesh filename=package://mit_drcsim_scripts/models/mit_robot/meshes/ltorso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 scale=1 1 1
- link mtorso: geometry visual mesh filename=package://mit_drcsim_scripts/models/mit_robot/meshes/mtorso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 scale=1 1 1
- link pelvis: geometry visual mesh filename=package://mit_drcsim_scripts/models/mit_robot/meshes/pelvis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 scale=1 1 1
- link r_clav: geometry visual mesh filename=package://mit_drcsim_scripts/models/mit_robot/meshes/r_clav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 scale=1 1 1
- link r_farm: geometry visual mesh filename=package://mit_drcsim_scripts/models/mit_robot/meshes/r_farm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 scale=1 1 1
- link r_foot: mass 1.634 -> 0.817; geometry collision sphere radius=0; collision sphere radius=0
- link r_hand: geometry collision sphere radius=0; visual mesh filename=package://mit_drcsim_scripts/models/mit_robot/meshes/r_hand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 scale=1 1 1
- link r_larm: geometry visual mesh filename=package://mit_drcsim_scripts/models/mit_robot/meshes/r_larm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 scale=1 1 1
- link r_lglut: geometry visual mesh filename=package://mit_drcsim_scripts/models/mit_robot/meshes/r_lglu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 scale=1 1 1
- link r_lleg: geometry collision sphere radius=0; visual mesh filename=package://mit_drcsim_scripts/models/mit_robot/meshes/r_lleg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 scale=1 1 1
- link r_scap: geometry visual mesh filename=package://mit_drcsim_scripts/models/mit_robot/meshes/r_scap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 scale=1 1 1
- link r_talus: mass 0.1 -> 0.817; geometry visual mesh filename=package://mit_drcsim_scripts/models/mit_robot/meshes/r_talu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 scale=1 1 1
- link r_uarm: geometry visual mesh filename=package://mit_drcsim_scripts/models/mit_robot/meshes/r_uarm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 scale=1 1 1
- link r_uglut: geometry visual mesh filename=package://mit_drcsim_scripts/models/mit_robot/meshes/r_uglu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 scale=1 1 1
- link r_uleg: geometry visual mesh filename=package://mit_drcsim_scripts/models/mit_robot/meshes/r_uleg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 scale=1 1 1
- link utorso: geometry visual mesh filename=package://mit_drcsim_scripts/models/mit_robot/meshes/utorso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 scale=1 1 1

Commit message: accidentally committed atlas model which pointed to the drc version of the meshes.  should be resolved here.
git-svn-id: https://svn.csail.mit.edu/locomotion/robotlib/trunk@5660 c9849af7-e679-4ec6-a44e-fc146a885bd3

File: examples/Atlas/urdf/atlas_minimal_contact.urdf (robot description, URDF)
Before this commit: robot atlas, 29 links, 28 joints
Links:
- link head: geometry visual mesh filename=meshes/base_link.wrl
- link l_clav: geometry visual mesh filename=meshes/l_clav.wrl scale=1 1 1
- link l_farm: geometry visual mesh filename=meshes/l_farm.wrl scale=1 1 1
- link l_foot: geometry collision sphere radius=0; collision sphere radius=0
- link l_hand: geometry collision sphere radius=0; visual mesh filename=meshes/l_hand.wrl scale=1 1 1
- link l_larm: geometry visual mesh filename=meshes/l_larm.wrl scale=1 1 1
- link l_lglut: geometry visual mesh filename=meshes/l_lglut.wrl scale=1 1 1
- link l_lleg: geometry collision sphere radius=0; visual mesh filename=meshes/l_lleg.wrl scale=1 1 1
- link l_scap: geometry visual mesh filename=meshes/l_scap.wrl scale=1 1 1
- link l_talus: geometry visual mesh filename=meshes/l_talus.wrl scale=1 1 1
- link l_uarm: geometry visual mesh filename=meshes/l_uarm.wrl scale=1 1 1
- link l_uglut: geometry visual mesh filename=meshes/l_uglut.wrl scale=1 1 1
- link l_uleg: geometry visual mesh filename=meshes/l_uleg.wrl scale=1 1 1
- link ltorso: geometry visual mesh filename=meshes/ltorso.wrl scale=1 1 1
- link mtorso: geometry visual mesh filename=meshes/mtorso.wrl scale=1 1 1
- link pelvis: geometry visual mesh filename=meshes/pelvis.wrl scale=1 1 1
- link r_clav: geometry visual mesh filename=meshes/r_clav.wrl scale=1 1 1
- link r_farm: geometry visual mesh filename=meshes/r_farm.wrl scale=1 1 1
- link r_foot: geometry collision sphere radius=0; collision sphere radius=0
- link r_hand: geometry collision sphere radius=0; visual mesh filename=meshes/r_hand.wrl scale=1 1 1
- link r_larm: geometry visual mesh filename=meshes/r_larm.wrl scale=1 1 1
- link r_lglut: geometry visual mesh filename=meshes/r_lglut.wrl scale=1 1 1
- link r_lleg: geometry collision sphere radius=0; visual mesh filename=meshes/r_lleg.wrl scale=1 1 1
- link r_scap: geometry visual mesh filename=meshes/r_scap.wrl scale=1 1 1
- link r_talus: geometry visual mesh filename=meshes/r_talus.wrl scale=1 1 1
- link r_uarm: geometry visual mesh filename=meshes/r_uarm.wrl scale=1 1 1
- link r_uglut: geometry visual mesh filename=meshes/r_uglut.wrl scale=1 1 1
- link r_uleg: geometry visual mesh filename=meshes/r_uleg.wrl scale=1 1 1
- link utorso: geometry visual mesh filename=meshes/utorso.wrl scale=1 1 1

Commit message: put zero radius spheres back into the atlas_minimal_contact urdf

File: examples/Atlas/urdf/atlas_minimal_contact.urdf (robot description, URDF)
Before this commit: robot atlas, 29 links, 28 joints
Links:
- link l_foot: geometry collision sphere radius=0; collision sphere radius=0
- link l_hand: geometry collision sphere radius=0; collision sphere radius=0
- link l_lleg: geometry collision sphere radius=0; visual mesh filename=package://Atlas/urdf/meshes/l_lleg.wrl scale=1 1 1
- link l_uleg: geometry collision sphere radius=0; collision sphere radius=0
- link pelvis: geometry collision sphere radius=0; collision sphere radius=0
- link r_foot: geometry collision sphere radius=0; collision sphere radius=0
- link r_hand: geometry collision sphere radius=0; collision sphere radius=0
- link r_lleg: geometry collision sphere radius=0; visual mesh filename=package://Atlas/urdf/meshes/r_lleg.wrl scale=1 1 1
- link r_uleg: geometry collision sphere radius=0; collision sphere radius=0
- link utorso: geometry collision sphere radius=0; collision sphere radius=0

Commit message: split midfoot contacts into front and rear, and move y positions inward

File: examples/Atlas/urdf/atlas_minimal_contact.urdf (robot description, URDF)
Before this commit: robot atlas, 60 links, 59 joints
Links:
- link l_foot: geometry collision sphere radius=0.0; collision sphere radius=0.0
- link r_foot: geometry collision sphere radius=0.0; collision sphere radius=0.0
