Commit message: Added kanako's urdf edits for effort and contact points. hubo_traj.mat contains the tunePD trajectory from Kanako's code. Updated SimpleWave and HuboPlant.
git-svn-id: https://svn.csail.mit.edu/locomotion/robotlib/trunk@5643 c9849af7-e679-4ec6-a44e-fc146a885bd3

File: examples/Hubo/model/huboplus.urdf (robot description, URDF)
Before this commit: robot huboplus, 59 links, 58 joints
Links:
- link Body_LAR: geometry collision sphere radius=0; collision sphere radius=0
- link Body_RAR: geometry collision sphere radius=0; collision sphere radius=0
Joints:
- joint HNP: limit lower=-0.523599 upper=0.523599 effort=10.0 velocity=1.0 -> lower=-0.523599 upper=0.523599 effort=1000.0 velocity=1.0
- joint HNR: limit lower=-0.523599 upper=0.523599 effort=10.0 velocity=1.0 -> lower=-0.523599 upper=0.523599 effort=1000.0 velocity=1.0
- joint HipYaw: limit lower=-3.14158 upper=3.14158 effort=10.0 velocity=1.0 -> lower=-3.14158 upper=3.14158 effort=1000.0 velocity=1.0
- joint Knuckle2: limit lower=-3.14 upper=3.14 effort=10.0 velocity=1.0 -> lower=-3.14 upper=3.14 effort=1000.0 velocity=1.0
- joint Knuckle212: limit lower=-3.14 upper=3.14 effort=10.0 velocity=1.0 -> lower=-3.14 upper=3.14 effort=1000.0 velocity=1.0
- joint Knuckle215: limit lower=-3.14 upper=3.14 effort=10.0 velocity=1.0 -> lower=-3.14 upper=3.14 effort=1000.0 velocity=1.0
- joint Knuckle218: limit lower=-3.14 upper=3.14 effort=10.0 velocity=1.0 -> lower=-3.14 upper=3.14 effort=1000.0 velocity=1.0
- joint Knuckle221: limit lower=-3.14 upper=3.14 effort=10.0 velocity=1.0 -> lower=-3.14 upper=3.14 effort=1000.0 velocity=1.0
- joint Knuckle230: limit lower=-3.14 upper=3.14 effort=10.0 velocity=1.0 -> lower=-3.14 upper=3.14 effort=1000.0 velocity=1.0
- joint Knuckle233: limit lower=-3.14 upper=3.14 effort=10.0 velocity=1.0 -> lower=-3.14 upper=3.14 effort=1000.0 velocity=1.0
- joint Knuckle236: limit lower=-3.14 upper=3.14 effort=10.0 velocity=1.0 -> lower=-3.14 upper=3.14 effort=1000.0 velocity=1.0
- joint Knuckle239: limit lower=-3.14 upper=3.14 effort=10.0 velocity=1.0 -> lower=-3.14 upper=3.14 effort=1000.0 velocity=1.0
- joint Knuckle29: limit lower=-3.14 upper=3.14 effort=10.0 velocity=1.0 -> lower=-3.14 upper=3.14 effort=1000.0 velocity=1.0
- joint Knuckle3: limit lower=-3.14 upper=3.14 effort=10.0 velocity=1.0 -> lower=-3.14 upper=3.14 effort=1000.0 velocity=1.0
- joint Knuckle310: limit lower=-3.14 upper=3.14 effort=10.0 velocity=1.0 -> lower=-3.14 upper=3.14 effort=1000.0 velocity=1.0
- joint Knuckle313: limit lower=-3.14 upper=3.14 effort=10.0 velocity=1.0 -> lower=-3.14 upper=3.14 effort=1000.0 velocity=1.0
- joint Knuckle316: limit lower=-3.14 upper=3.14 effort=10.0 velocity=1.0 -> lower=-3.14 upper=3.14 effort=1000.0 velocity=1.0
- joint Knuckle319: limit lower=-3.14 upper=3.14 effort=10.0 velocity=1.0 -> lower=-3.14 upper=3.14 effort=1000.0 velocity=1.0
- joint Knuckle322: limit lower=-3.14 upper=3.14 effort=10.0 velocity=1.0 -> lower=-3.14 upper=3.14 effort=1000.0 velocity=1.0
- joint Knuckle331: limit lower=-3.14 upper=3.14 effort=10.0 velocity=1.0 -> lower=-3.14 upper=3.14 effort=1000.0 velocity=1.0
- joint Knuckle334: limit lower=-3.14 upper=3.14 effort=10.0 velocity=1.0 -> lower=-3.14 upper=3.14 effort=1000.0 velocity=1.0
- joint Knuckle337: limit lower=-3.14 upper=3.14 effort=10.0 velocity=1.0 -> lower=-3.14 upper=3.14 effort=1000.0 velocity=1.0
- joint Knuckle340: limit lower=-3.14 upper=3.14 effort=10.0 velocity=1.0 -> lower=-3.14 upper=3.14 effort=1000.0 velocity=1.0
- joint LeftAnklePitch: limit lower=-1.29154 upper=1.69297 effort=10.0 velocity=1.0 -> lower=-1.29154 upper=1.69297 effort=1000.0 velocity=1.0
- joint LeftAnkleRoll: limit lower=-0.191986 upper=0.191986 effort=10.0 velocity=1.0 -> lower=-0.191986 upper=0.191986 effort=1000.0 velocity=1.0
- joint LeftElbowPitch: limit lower=-2.49582 upper=0.0698132 effort=10.0 velocity=1.0 -> lower=-2.49582 upper=0.0698132 effort=1000.0 velocity=1.0
- joint LeftHipPitch: limit lower=-1.48353 upper=1.6057 effort=10.0 velocity=1.0 -> lower=-1.48353 upper=1.6057 effort=1000.0 velocity=1.0
- joint LeftHipRoll: limit lower=-0.488692 upper=0.488692 effort=10.0 velocity=1.0 -> lower=-0.488692 upper=0.488692 effort=1000.0 velocity=1.0
- joint LeftHipYaw: limit lower=-1.5708 upper=1.5708 effort=10.0 velocity=1.0 -> lower=-1.5708 upper=1.5708 effort=1000.0 velocity=1.0
- joint LeftKneePitch: limit lower=-0.0698132 upper=2.60054 effort=10.0 velocity=1.0 -> lower=-0.0698132 upper=2.60054 effort=1000.0 velocity=1.0
- joint LeftShoulderPitch: limit lower=-3.14158 upper=3.14158 effort=10.0 velocity=1.0 -> lower=-3.14158 upper=3.14158 effort=1000.0 velocity=1.0
- joint LeftShoulderRoll: limit lower=-1.5708 upper=1.5708 effort=10.0 velocity=1.0 -> lower=-1.5708 upper=1.5708 effort=1000.0 velocity=1.0
- joint LeftShoulderYaw: limit lower=-3.14158 upper=3.14158 effort=10.0 velocity=1.0 -> lower=-3.14158 upper=3.14158 effort=1000.0 velocity=1.0
- joint LeftWristPitch: limit lower=-1.64061 upper=1.01229 effort=10.0 velocity=1.0 -> lower=-1.64061 upper=1.01229 effort=1000.0 velocity=1.0
- joint LeftWristYaw: limit lower=-3.14158 upper=3.14158 effort=10.0 velocity=1.0 -> lower=-3.14158 upper=3.14158 effort=1000.0 velocity=1.0
- joint RightAnklePitch: limit lower=-1.29154 upper=1.69297 effort=10.0 velocity=1.0 -> lower=-1.29154 upper=1.69297 effort=1000.0 velocity=1.0
- joint RightAnkleRoll: limit lower=-0.191986 upper=0.191986 effort=10.0 velocity=1.0 -> lower=-0.191986 upper=0.191986 effort=1000.0 velocity=1.0
- joint RightElbowPitch: limit lower=-2.49582 upper=0.0698132 effort=10.0 velocity=1.0 -> lower=-2.49582 upper=0.0698132 effort=1000.0 velocity=1.0
- joint RightHipPitch: limit lower=-1.48353 upper=1.6057 effort=10.0 velocity=1.0 -> lower=-1.48353 upper=1.6057 effort=1000.0 velocity=1.0
- joint RightHipRoll: limit lower=-0.488692 upper=0.488692 effort=10.0 velocity=1.0 -> lower=-0.488692 upper=0.488692 effort=1000.0 velocity=1.0
- joint RightHipYaw: limit lower=-1.5708 upper=1.5708 effort=10.0 velocity=1.0 -> lower=-1.5708 upper=1.5708 effort=1000.0 velocity=1.0
- joint RightKneePitch: limit lower=-0.0698132 upper=2.60054 effort=10.0 velocity=1.0 -> lower=-0.0698132 upper=2.60054 effort=1000.0 velocity=1.0
- joint RightShoulderPitch: limit lower=-3.14158 upper=3.14158 effort=10.0 velocity=1.0 -> lower=-3.14158 upper=3.14158 effort=1000.0 velocity=1.0
- joint RightShoulderRoll: limit lower=-1.5708 upper=1.5708 effort=10.0 velocity=1.0 -> lower=-1.5708 upper=1.5708 effort=1000.0 velocity=1.0
- joint RightShoulderYaw: limit lower=-3.14158 upper=3.14158 effort=10.0 velocity=1.0 -> lower=-3.14158 upper=3.14158 effort=1000.0 velocity=1.0
- joint RightWristPitch: limit lower=-1.64061 upper=1.01229 effort=10.0 velocity=1.0 -> lower=-1.64061 upper=1.01229 effort=1000.0 velocity=1.0
- joint RightWristYaw: limit lower=-3.14158 upper=3.14158 effort=10.0 velocity=1.0 -> lower=-3.14158 upper=3.14158 effort=1000.0 velocity=1.0
- joint leftIndexKnuckle1: limit lower=-3.14 upper=3.14 effort=10.0 velocity=1.0 -> lower=-3.14 upper=3.14 effort=1000.0 velocity=1.0
- joint leftMiddleKnuckle1: limit lower=-3.14 upper=3.14 effort=10.0 velocity=1.0 -> lower=-3.14 upper=3.14 effort=1000.0 velocity=1.0
- joint leftPinkyKnuckle1: limit lower=-3.14 upper=3.14 effort=10.0 velocity=1.0 -> lower=-3.14 upper=3.14 effort=1000.0 velocity=1.0
- joint leftRingKnuckle1: limit lower=-3.14 upper=3.14 effort=10.0 velocity=1.0 -> lower=-3.14 upper=3.14 effort=1000.0 velocity=1.0
- joint leftThumbKnuckle1: limit lower=-3.14 upper=3.14 effort=10.0 velocity=1.0 -> lower=-3.14 upper=3.14 effort=1000.0 velocity=1.0
- joint rightIndexKnuckle1: limit lower=-3.14 upper=3.14 effort=10.0 velocity=1.0 -> lower=-3.14 upper=3.14 effort=1000.0 velocity=1.0
- joint rightMiddleKnuckle1: limit lower=-3.14 upper=3.14 effort=10.0 velocity=1.0 -> lower=-3.14 upper=3.14 effort=1000.0 velocity=1.0
- joint rightPinkyKnuckle1: limit lower=-3.14 upper=3.14 effort=10.0 velocity=1.0 -> lower=-3.14 upper=3.14 effort=1000.0 velocity=1.0
- joint rightRingKnuckle1: limit lower=-3.14 upper=3.14 effort=10.0 velocity=1.0 -> lower=-3.14 upper=3.14 effort=1000.0 velocity=1.0
- joint rightThumbKnuckle1: limit lower=-3.14 upper=3.14 effort=10.0 velocity=1.0 -> lower=-3.14 upper=3.14 effort=1000.0 velocity=1.0
