Commit message: added drawing logic for sphere, box, and cylinder primitives. viewer compiles but crashes on brick example.
git-svn-id: https://svn.csail.mit.edu/locomotion/robotlib/trunk@5794 c9849af7-e679-4ec6-a44e-fc146a885bd3

File: systems/plants/test/brick1.urdf (robot description, URDF)
Before this commit: robot myfirst, 1 links, 0 joints
Links:
- removed link base_link
- added link brick, mass 10; collision box size=0.06 0.06 1.176; visual box size=0.06 0.06 1.176
