Commit message: adding pairwise contact constraints with point specification and body-to-world collision checking. fixing bullet_collision_normals unit test
git-svn-id: https://svn.csail.mit.edu/locomotion/robotlib/trunk@6278 c9849af7-e679-4ec6-a44e-fc146a885bd3

File: systems/plants/test/ground_plane.urdf (robot description, URDF)
Before this commit: robot ground_plane, 1 links, 0 joints
Links:
- link ground_plane: mass 10 -> None; geometry collision box size=10 10 1; visual box size=10 10 0
