Commit message: patch from Tim with minor edits from me on the way in.
git-svn-id: https://svn.csail.mit.edu/locomotion/robotlib/trunk@6888 c9849af7-e679-4ec6-a44e-fc146a885bd3

File: systems/plants/test/TestWing.urdf (robot description, URDF)
Before this commit: robot Test_3D_Glider, 1 links, 0 joints
Links:
- removed link Wing3D
- added link Wing, mass .13; collision box size=.4 1 .04; visual box size=.4 1 .01
