Commit message: working through implementation of hybrid manipulators (joint limits first)
git-svn-id: https://svn.csail.mit.edu/locomotion/robotlib/trunk@3548 c9849af7-e679-4ec6-a44e-fc146a885bd3

File: examples/Acrobot/Acrobot.urdf (robot description, URDF)
Before this commit: robot Acrobot, 3 links, 2 joints
Joints:
- joint elbow: limit (none) -> lower=-1.5 upper=1.5; type continuous -> revolute

Commit message: acrobat test with joint limits works.
git-svn-id: https://svn.csail.mit.edu/locomotion/robotlib/trunk@3559 c9849af7-e679-4ec6-a44e-fc146a885bd3

File: examples/Acrobot/Acrobot.urdf (robot description, URDF)
Before this commit: robot Acrobot, 3 links, 2 joints
Joints:
- joint elbow: limit lower=-1.5 upper=1.5 -> (none)

Commit message: viewer show brick and acrobot urdfs.  needs lighting/shading and probably debugging.
git-svn-id: https://svn.csail.mit.edu/locomotion/robotlib/trunk@5795 c9849af7-e679-4ec6-a44e-fc146a885bd3

File: examples/Acrobot/Acrobot.urdf (robot description, URDF)
Before this commit: robot Acrobot, 3 links, 2 joints
Joints:
- joint elbow: type revolute -> continuous
