Commit message: implemented quick version of rospack for urdf parser.  drc drake unit tests work in the drake_viewer now. sets drake_viewer to default on mac (not on linux, until I fix the autolaunch).
git-svn-id: https://svn.csail.mit.edu/locomotion/robotlib/trunk@6474 c9849af7-e679-4ec6-a44e-fc146a885bd3

File: examples/PR2/pr2.urdf (robot description, URDF)
Before this commit: robot pr2, 82 links, 81 joints
Links:
- link base_link: geometry collision mesh filename=pr2_description/meshes/base_v0/base_L.stl; visual mesh filename=pr2_description/meshes/base_v0/base.stl
- link bl_caster_l_wheel_link: geometry collision cylinder length=0.034 radius=0.074792; visual mesh filename=pr2_description/meshes/base_v0/wheel.stl
- link bl_caster_r_wheel_link: geometry collision cylinder length=0.034 radius=0.074792; visual mesh filename=pr2_description/meshes/base_v0/wheel.stl
- link bl_caster_rotation_link: geometry collision mesh filename=pr2_description/meshes/base_v0/caster_L.stl; visual mesh filename=pr2_description/meshes/base_v0/caster.stl
- link br_caster_l_wheel_link: geometry collision cylinder length=0.034 radius=0.074792; visual mesh filename=pr2_description/meshes/base_v0/wheel.stl
- link br_caster_r_wheel_link: geometry collision cylinder length=0.034 radius=0.074792; visual mesh filename=pr2_description/meshes/base_v0/wheel.stl
- link br_caster_rotation_link: geometry collision mesh filename=pr2_description/meshes/base_v0/caster_L.stl; visual mesh filename=pr2_description/meshes/base_v0/caster.stl
- link fl_caster_l_wheel_link: geometry collision cylinder length=0.034 radius=0.074792; visual mesh filename=pr2_description/meshes/base_v0/wheel.stl
- link fl_caster_r_wheel_link: geometry collision cylinder length=0.034 radius=0.074792; visual mesh filename=pr2_description/meshes/base_v0/wheel.stl
- link fl_caster_rotation_link: geometry collision mesh filename=pr2_description/meshes/base_v0/caster_L.stl; visual mesh filename=pr2_description/meshes/base_v0/caster.stl
- link fr_caster_l_wheel_link: geometry collision cylinder length=0.034 radius=0.074792; visual mesh filename=pr2_description/meshes/base_v0/wheel.stl
- link fr_caster_r_wheel_link: geometry collision cylinder length=0.034 radius=0.074792; visual mesh filename=pr2_description/meshes/base_v0/wheel.stl
- link fr_caster_rotation_link: geometry collision mesh filename=pr2_description/meshes/base_v0/caster_L.stl; visual mesh filename=pr2_description/meshes/base_v0/caster.stl
- link head_pan_link: geometry collision mesh filename=pr2_description/meshes/head_v0/head_pan_L.stl; visual mesh filename=pr2_description/meshes/head_v0/head_pan.stl
- link head_tilt_link: geometry collision mesh filename=pr2_description/meshes/head_v0/head_tilt_L.stl; visual mesh filename=pr2_description/meshes/head_v0/head_tilt.stl
- link l_elbow_flex_link: geometry collision mesh filename=pr2_description/meshes/upper_arm_v0/elbow_flex.stl; visual mesh filename=pr2_description/meshes/upper_arm_v0/elbow_flex.stl
- link l_forearm_link: geometry collision mesh filename=pr2_description/meshes/forearm_v0/forearm.stl; visual mesh filename=pr2_description/meshes/forearm_v0/forearm.stl
- link l_forearm_roll_link: geometry collision mesh filename=pr2_description/meshes/upper_arm_v0/forearm_roll_L.stl; visual mesh filename=pr2_description/meshes/upper_arm_v0/forearm_roll.stl
- link l_gripper_l_finger_link: geometry collision mesh filename=pr2_description/meshes/gripper_v0/l_finger.stl; visual mesh filename=pr2_description/meshes/gripper_v0/l_finger.stl
- link l_gripper_l_finger_tip_link: geometry collision mesh filename=pr2_description/meshes/gripper_v0/l_finger_tip.stl; visual mesh filename=pr2_description/meshes/gripper_v0/l_finger_tip.stl
- link l_gripper_palm_link: geometry collision mesh filename=pr2_description/meshes/gripper_v0/gripper_palm.stl; visual mesh filename=pr2_description/meshes/gripper_v0/gripper_palm.stl
- link l_gripper_r_finger_link: geometry collision mesh filename=pr2_description/meshes/gripper_v0/l_finger.stl; visual mesh filename=pr2_description/meshes/gripper_v0/l_finger.stl
- link l_gripper_r_finger_tip_link: geometry collision mesh filename=pr2_description/meshes/gripper_v0/l_finger_tip.stl; visual mesh filename=pr2_description/meshes/gripper_v0/l_finger_tip.stl
- link l_shoulder_lift_link: geometry collision mesh filename=pr2_description/meshes/shoulder_v0/shoulder_lift.stl; visual mesh filename=pr2_description/meshes/shoulder_v0/shoulder_lift.stl
- link l_shoulder_pan_link: geometry collision mesh filename=pr2_description/meshes/shoulder_v0/shoulder_pan.stl; visual mesh filename=pr2_description/meshes/shoulder_v0/shoulder_pan.stl
- link l_upper_arm_link: geometry collision mesh filename=pr2_description/meshes/upper_arm_v0/upper_arm.stl; visual mesh filename=pr2_description/meshes/upper_arm_v0/upper_arm.stl
- link l_upper_arm_roll_link: geometry collision mesh filename=pr2_description/meshes/shoulder_v0/upper_arm_roll_L.stl; visual mesh filename=pr2_description/meshes/shoulder_v0/upper_arm_roll.stl
- link l_wrist_flex_link: geometry collision mesh filename=pr2_description/meshes/forearm_v0/wrist_flex.stl; visual mesh filename=pr2_description/meshes/forearm_v0/wrist_flex.stl
- link l_wrist_roll_link: geometry collision mesh filename=pr2_description/meshes/forearm_v0/wrist_roll_L.stl; visual mesh filename=pr2_description/meshes/forearm_v0/wrist_roll.stl
- link laser_tilt_mount_link: geometry collision mesh filename=pr2_description/meshes/tilting_laser_v0/tilting_hokuyo_L.stl; visual mesh filename=pr2_description/meshes/tilting_laser_v0/tilting_hokuyo.stl
- link r_elbow_flex_link: geometry collision mesh filename=pr2_description/meshes/upper_arm_v0/elbow_flex.stl; visual mesh filename=pr2_description/meshes/upper_arm_v0/elbow_flex.stl
- link r_forearm_link: geometry collision mesh filename=pr2_description/meshes/forearm_v0/forearm.stl; visual mesh filename=pr2_description/meshes/forearm_v0/forearm.stl
- link r_forearm_roll_link: geometry collision mesh filename=pr2_description/meshes/upper_arm_v0/forearm_roll_L.stl; visual mesh filename=pr2_description/meshes/upper_arm_v0/forearm_roll.stl
- link r_gripper_l_finger_link: geometry collision mesh filename=pr2_description/meshes/gripper_v0/l_finger.stl; visual mesh filename=pr2_description/meshes/gripper_v0/l_finger.stl
- link r_gripper_l_finger_tip_link: geometry collision mesh filename=pr2_description/meshes/gripper_v0/l_finger_tip.stl; visual mesh filename=pr2_description/meshes/gripper_v0/l_finger_tip.stl
- link r_gripper_palm_link: geometry collision mesh filename=pr2_description/meshes/gripper_v0/gripper_palm.stl; visual mesh filename=pr2_description/meshes/gripper_v0/gripper_palm.stl
- link r_gripper_r_finger_link: geometry collision mesh filename=pr2_description/meshes/gripper_v0/l_finger.stl; visual mesh filename=pr2_description/meshes/gripper_v0/l_finger.stl
- link r_gripper_r_finger_tip_link: geometry collision mesh filename=pr2_description/meshes/gripper_v0/l_finger_tip.stl; visual mesh filename=pr2_description/meshes/gripper_v0/l_finger_tip.stl
- link r_shoulder_lift_link: geometry collision mesh filename=pr2_description/meshes/shoulder_v0/shoulder_lift.stl; visual mesh filename=pr2_description/meshes/shoulder_v0/shoulder_lift.stl
- link r_shoulder_pan_link: geometry collision mesh filename=pr2_description/meshes/shoulder_v0/shoulder_pan.stl; visual mesh filename=pr2_description/meshes/shoulder_v0/shoulder_pan.stl
- link r_upper_arm_link: geometry collision mesh filename=pr2_description/meshes/upper_arm_v0/upper_arm.stl; visual mesh filename=pr2_description/meshes/upper_arm_v0/upper_arm.stl
- link r_upper_arm_roll_link: geometry collision mesh filename=pr2_description/meshes/shoulder_v0/upper_arm_roll_L.stl; visual mesh filename=pr2_description/meshes/shoulder_v0/upper_arm_roll.stl
- link r_wrist_flex_link: geometry collision mesh filename=pr2_description/meshes/forearm_v0/wrist_flex.stl; visual mesh filename=pr2_description/meshes/forearm_v0/wrist_flex.stl
- link r_wrist_roll_link: geometry collision mesh filename=pr2_description/meshes/forearm_v0/wrist_roll_L.stl; visual mesh filename=pr2_description/meshes/forearm_v0/wrist_roll.stl
- link torso_lift_link: geometry collision mesh filename=pr2_description/meshes/torso_v0/torso_lift_L.stl; visual mesh filename=pr2_description/meshes/torso_v0/torso_lift.stl
