Commit message: puts zmp riccati equation into relative coordinates. i don't like the wiggles when the translation is set to 1000, but it appears to be just a numerical artifact.
git-svn-id: https://svn.csail.mit.edu/locomotion/robotlib/trunk@6131 c9849af7-e679-4ec6-a44e-fc146a885bd3

File: examples/ZMP/CartTable.urdf (robot description, URDF)
Before this commit: robot CartTable, 5 links, 3 joints
Links:
- link base: geometry visual box size=.2 .2 .01

Commit message: fix urdf parser error reporting. make carttable.urdf compatible with ROS urdf parser.
git-svn-id: https://svn.csail.mit.edu/locomotion/robotlib/trunk@6469 c9849af7-e679-4ec6-a44e-fc146a885bd3

File: examples/ZMP/CartTable.urdf (robot description, URDF)
Before this commit: robot CartTable, 5 links, 3 joints
Joints:
- added joint base_weld2: type fixed, parent base_part2, child base_part3, origin xyz=0 0 0
- joint base_weld: child base_part3 -> base_part2; parent base_part2 -> base

Commit message: add a few checkDependency's for sedumi fix scope lcm ref fix caretable example
git-svn-id: https://svn.csail.mit.edu/locomotion/robotlib/trunk@6624 c9849af7-e679-4ec6-a44e-fc146a885bd3

File: examples/ZMP/CartTable.urdf (robot description, URDF)
Before this commit: robot CartTable, 5 links, 4 joints
Links:
- link base: geometry collision box size=.2 .2 .01; visual box size=.2 .2 .01
