Commit message: fix from Andres for bug 1749 - support points with radius zero in bullet collision checking
git-svn-id: https://svn.csail.mit.edu/locomotion/robotlib/trunk@7020 c9849af7-e679-4ec6-a44e-fc146a885bd3

File: systems/plants/Constraint/test/model_simple_visuals.urdf (robot description, URDF)
Before this commit: robot atlas, 33 links, 32 joints
Links:
- removed link left_hook
- removed link right_hook
Joints:
- removed joint left_hook_joint
- removed joint right_hook_joint
