Commit message: fixes from Tim plus a new runDircolPerchingURDF
git-svn-id: https://svn.csail.mit.edu/locomotion/robotlib/trunk@7032 c9849af7-e679-4ec6-a44e-fc146a885bd3

File: examples/Glider/GliderBalanced.URDF (robot description, URDF)
Before this commit: robot Glider, 2 links, 1 joints
Links:
- link Elevator: mass 0.00000001 -> 1e-9

Commit message: more fixes from Tim
git-svn-id: https://svn.csail.mit.edu/locomotion/robotlib/trunk@7033 c9849af7-e679-4ec6-a44e-fc146a885bd3

File: examples/Glider/GliderBalanced.URDF (robot description, URDF)
Before this commit: robot Glider, 2 links, 1 joints
Links:
- link Elevator: mass 1e-9 -> .00001; geometry collision mesh filename=meshes/GliderElevator.STL; visual box size=.08 .1 .01
- link fuselage: geometry collision mesh filename=meshes/GliderFuselage.STL; visual box size=.3 .1 .03
