Commit message: remove the mat files in trajectoryOptimization/dev

File: solvers/trajectoryOptimization/dev/ground.urdf (robot description, URDF)
Before this commit: robot stage, 1 links, 0 joints
Links:
- removed link stage
- added link ground, mass 0; collision box size=2 2 0.05; visual box size=2 2 0.05
