Commit message: working edits on hopper example

File: examples/test/OneLegHopper.urdf (robot description, URDF)
Before this commit: robot hopper, 3 links, 2 joints
Links:
- link foot: mass 1 -> 0.5; geometry collision sphere radius=0; collision sphere radius=0
- link shin: mass 1 -> 0.5

Commit message: various minor edits/fixes. adds script for running LQR solution

File: examples/test/OneLegHopper.urdf (robot description, URDF)
Before this commit: robot hopper, 3 links, 2 joints
Joints:
- joint ankle: limit (none) -> effort=400
- joint knee: limit (none) -> effort=400

Commit message: working QP stabilization for hopper

File: examples/test/OneLegHopper.urdf (robot description, URDF)
Before this commit: robot hopper, 3 links, 2 joints
Joints:
- joint ankle: limit effort=400 -> effort=100
- joint knee: limit effort=400 -> effort=100
