Commit message: update irb140 urdf

File: examples/IRB140/irb_140.urdf (robot description, URDF)
Before this commit: robot IRB140_-_M2004C_Complete_base.SLDASM, 7 links, 6 joints
Joints:
- joint joint1: limit lower=-2.88 upper=2.88 effort=300 velocity=4.36 -> lower=-3.14159265359 upper=3.14159265359 effort=300 velocity=4.36; origin xyz=0 0 0 rpy=0 0 0 -> xyz=0 -0.1095 0 rpy=0 0 0
- joint joint2: limit lower=-1.92 upper=1.92 effort=300 velocity=4.36 -> lower=-1.57079633 upper=1.91986218 effort=300 velocity=4.36; origin xyz=0 -0.352 0 rpy=0 0 0 -> xyz=0.07 -0.2425 0 rpy=0 0 0
- joint joint3: limit lower=-1.575 upper=1.23 effort=300 velocity=4.36 -> lower=-4.01425728 upper=0.87266463 effort=300 velocity=4.36
- joint joint4: limit lower=-2.80 upper=2.80 effort=300 velocity=5.58 -> lower=-3.49065850 upper=3.49065850 effort=300 velocity=5.58; origin xyz=0 0 0 rpy=0 0 0 -> xyz=0.2185 0 0 rpy=0 0 0
- joint joint5: limit lower=-2.10 upper=2.10 effort=300 velocity=5.58 -> lower=-2.09439510 upper=2.09439510 effort=300 velocity=5.58; origin xyz=0.45 0 0 rpy=0 0 0 -> xyz=0.1615 0 0 rpy=0 0 0
- joint joint6: limit lower=-6.985 upper=6.985 effort=300 velocity=7.33 -> lower=-6.98131701 upper=-6.98131701 effort=300 velocity=7.33

Commit message: The rotation axis of of joint1 and joint3 in the URDF are in the opposite direction as the real robot, change the direction of their rotation axis

File: examples/IRB140/irb_140.urdf (robot description, URDF)
Before this commit: robot IRB140_-_M2004C_Complete_base.SLDASM, 7 links, 6 joints
Joints:
- joint joint1: axis 0 1 0 -> 0 -1 0
- joint joint3: axis 0 0 -1 -> 0 0 1

File: examples/IRB140/irb_140_convhull.urdf (robot description, URDF)
Before this commit: robot IRB140_-_M2004C_Complete_base.SLDASM, 7 links, 6 joints
Joints:
- joint joint1: axis 0 1 0 -> 0 -1 0
- joint joint3: axis 0 0 -1 -> 0 0 1

Commit message: remove the collision geometry in the base link of IRB140, otherwise RigidBodyManipulator will check collision between world+base link and link1, and it would always fail

File: examples/IRB140/irb_140.urdf (robot description, URDF)
Before this commit: robot IRB140_-_M2004C_Complete_base.SLDASM, 7 links, 6 joints
Links:
- link base_link: geometry collision mesh filename=meshes/base_link.stl

File: examples/IRB140/irb_140_convhull.urdf (robot description, URDF)
Before this commit: robot IRB140_-_M2004C_Complete_base.SLDASM, 7 links, 6 joints
Links:
- link base_link: geometry visual mesh filename=meshes/base_link_chull.wrl
