Commit message: add the transformation from the arm to the hand palm

File: examples/IRB140/irb_140_robotiq.urdf (robot description, URDF)
Before this commit: robot IRB140_-_M2004C_Complete_base.SLDASM, 30 links, 29 joints
Links:
- removed link ATI_sensor
Joints:
- removed joint ATI_sensor_joint
- joint robotiq_hand_joint: origin xyz=0.0 0.07459 0.0 rpy=0.0 0.0 0 -> xyz=0.11904 0 0 rpy=0.0 0.0 -1.57079; parent ATI_sensor -> link_6
