Commit message: add IRB140 package in examples/IRB140 directory

File: examples/IRB140/urdf/ATI_sensor.urdf (robot description, URDF)
Before this commit: robot ATI-sensor, 1 links, 0 joints
Links:
- link ATI_sensor: geometry collision mesh filename=package://IRB140/urdf/meshes/ATI_sensor.STL; visual mesh filename=package://IRB140/urdf/meshes/ATI_sensor.STL

File: examples/IRB140/urdf/irb_140.urdf (robot description, URDF)
Before this commit: robot IRB140_-_M2004C_Complete_base.SLDASM, 7 links, 6 joints
Links:
- link base_link: geometry collision mesh filename=package://IRB140/urdf/meshes/base_link.stl
- link link_1: geometry collision mesh filename=package://IRB140/urdf/meshes/link1.stl; visual mesh filename=package://IRB140/urdf/meshes/link1.stl
- link link_2: geometry collision mesh filename=package://IRB140/urdf/meshes/link2.stl; visual mesh filename=package://IRB140/urdf/meshes/link2.stl
- link link_3: geometry collision mesh filename=package://IRB140/urdf/meshes/link3.stl; visual mesh filename=package://IRB140/urdf/meshes/link3.stl
- link link_4: geometry collision mesh filename=package://IRB140/urdf/meshes/link4.stl; visual mesh filename=package://IRB140/urdf/meshes/link4.stl
- link link_5: geometry collision mesh filename=package://IRB140/urdf/meshes/link5.stl; visual mesh filename=package://IRB140/urdf/meshes/link5.stl
- link link_6: geometry collision mesh filename=package://IRB140/urdf/meshes/link6.stl; visual mesh filename=package://IRB140/urdf/meshes/link6.stl

File: examples/IRB140/urdf/irb_140_convhull.urdf (robot description, URDF)
Before this commit: robot IRB140_-_M2004C_Complete_base.SLDASM, 7 links, 6 joints
Links:
- link base_link: geometry visual mesh filename=package://IRB140/urdf/meshes/base_link_chull.wrl
- link link_1: geometry collision mesh filename=package://IRB140/urdf/meshes/link1_chull.wrl; visual mesh filename=package://IRB140/urdf/meshes/link1_chull.wrl
- link link_2: geometry collision mesh filename=package://IRB140/urdf/meshes/link2_chull.wrl; visual mesh filename=package://IRB140/urdf/meshes/link2_chull.wrl
- link link_3: geometry collision mesh filename=package://IRB140/urdf/meshes/link3_chull.wrl; visual mesh filename=package://IRB140/urdf/meshes/link3_chull.wrl
- link link_4: geometry collision mesh filename=package://IRB140/urdf/meshes/link4_chull.wrl; visual mesh filename=package://IRB140/urdf/meshes/link4_chull.wrl
- link link_5: geometry collision mesh filename=package://IRB140/urdf/meshes/link5_chull.wrl; visual mesh filename=package://IRB140/urdf/meshes/link5_chull.wrl
- link link_6: geometry collision mesh filename=package://IRB140/urdf/meshes/link6_chull.wrl; visual mesh filename=package://IRB140/urdf/meshes/link6_chull.wrl

File: examples/IRB140/urdf/irb_140_robotiq.urdf (robot description, URDF)
Before this commit: robot IRB140_-_M2004C_Complete_base.SLDASM, 29 links, 28 joints
Links:
- removed link finger_1_fourbar_0_link_0
- removed link finger_2_fourbar_0_link_0
- removed link finger_middle_fourbar_0_link_0
- added link finger_1_fourbar_0_link_3, mass 0.00001; visual cylinder length=.01473 radius=0.001
- added link finger_1_fourbar_3_link_1, mass 0.00001; visual cylinder length=.02222 radius=0.001
- added link finger_1_fourbar_3_link_2, mass 0.00001; visual cylinder length=.03810 radius=0.001
- added link finger_1_fourbar_3_link_3, mass 0.00001; visual cylinder length=.01270 radius=0.001
- added link finger_1_fourbar_linkage, mass 0.00001; visual cylinder length=.015236 radius=0.001
- added link finger_2_fourbar_0_link_3, mass 0.00001; visual cylinder length=.01473 radius=0.001
- added link finger_2_fourbar_3_link_1, mass 0.00001; visual cylinder length=.02222 radius=0.001
- added link finger_2_fourbar_3_link_2, mass 0.00001; visual cylinder length=.03810 radius=0.001
- added link finger_2_fourbar_3_link_3, mass 0.00001; visual cylinder length=.01270 radius=0.001
- added link finger_2_fourbar_linkage, mass 0.00001; visual cylinder length=.015236 radius=0.001
- added link finger_middle_fourbar_0_link_3, mass 0.00001; visual cylinder length=.01473 radius=0.001
- added link finger_middle_fourbar_3_link_1, mass 0.00001; visual cylinder length=.02222 radius=0.001
- added link finger_middle_fourbar_3_link_2, mass 0.00001; visual cylinder length=.03810 radius=0.001
- added link finger_middle_fourbar_3_link_3, mass 0.00001; visual cylinder length=.01270 radius=0.001
- added link finger_middle_fourbar_linkage, mass 0.00001; visual cylinder length=.015236 radius=0.001
- link base_link: geometry collision mesh filename=package://IRB140/urdf/meshes/base_link.stl
- link finger_1_fourbar_0_link_1: mass 0.000001 -> 0.00001; geometry visual cylinder length=.02858 radius=0.001
- link finger_1_fourbar_0_link_2: mass 0.000001 -> 0.00001; geometry visual cylinder length=.05398 radius=0.001
- link finger_1_link_0: geometry visual mesh filename=package://Atlas/urdf/meshes/s-model_articulated/visual/link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
- link finger_1_link_1: geometry collision box size=.028 .01 .03; visual mesh filename=package://Atlas/urdf/meshes/s-model_articulated/visual/link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
- link finger_1_link_2: geometry collision box size=.018 .01 .03; visual mesh filename=package://Atlas/urdf/meshes/s-model_articulated/visual/link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
- link finger_1_link_3: geometry collision box size=.025 .01 .03; visual mesh filename=package://Atlas/urdf/meshes/s-model_articulated/visual/link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
- link finger_2_fourbar_0_link_1: mass 0.000001 -> 0.00001; geometry visual cylinder length=.02858 radius=0.001
- link finger_2_fourbar_0_link_2: mass 0.000001 -> 0.00001; geometry visual cylinder length=.05398 radius=0.001
- link finger_2_link_0: geometry visual mesh filename=package://Atlas/urdf/meshes/s-model_articulated/visual/link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
- link finger_2_link_1: geometry collision box size=.028 .01 .03; visual mesh filename=package://Atlas/urdf/meshes/s-model_articulated/visual/link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
- link finger_2_link_2: geometry collision box size=.018 .01 .03; visual mesh filename=package://Atlas/urdf/meshes/s-model_articulated/visual/link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
- link finger_2_link_3: geometry collision box size=.025 .01 .03; visual mesh filename=package://Atlas/urdf/meshes/s-model_articulated/visual/link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
- link finger_middle_fourbar_0_link_1: mass 0.000001 -> 0.00001; geometry visual cylinder length=.02858 radius=0.001
- link finger_middle_fourbar_0_link_2: mass 0.000001 -> 0.00001; geometry visual cylinder length=.05398 radius=0.001
- link finger_middle_link_0: geometry visual mesh filename=package://Atlas/urdf/meshes/s-model_articulated/visual/link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
- link finger_middle_link_1: geometry collision box size=.028 .01 .03; visual mesh filename=package://Atlas/urdf/meshes/s-model_articulated/visual/link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
- link finger_middle_link_2: geometry collision box size=.018 .01 .03; visual mesh filename=package://Atlas/urdf/meshes/s-model_articulated/visual/link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
- link finger_middle_link_3: geometry collision box size=.025 .01 .03; visual mesh filename=package://Atlas/urdf/meshes/s-model_articulated/visual/link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
- link link_1: geometry collision mesh filename=package://IRB140/urdf/meshes/link1.stl; visual mesh filename=package://IRB140/urdf/meshes/link1.stl
- link link_2: geometry collision mesh filename=package://IRB140/urdf/meshes/link2.stl; visual mesh filename=package://IRB140/urdf/meshes/link2.stl
- link link_3: geometry collision mesh filename=package://IRB140/urdf/meshes/link3.stl; visual mesh filename=package://IRB140/urdf/meshes/link3.stl
- link link_4: geometry collision mesh filename=package://IRB140/urdf/meshes/link4.stl; visual mesh filename=package://IRB140/urdf/meshes/link4.stl
- link link_5: geometry collision mesh filename=package://IRB140/urdf/meshes/link5.stl; visual mesh filename=package://IRB140/urdf/meshes/link5.stl
- link link_6: geometry collision mesh filename=package://IRB140/urdf/meshes/link6.stl; visual mesh filename=package://IRB140/urdf/meshes/link6.stl
- link palm: geometry collision box size=.1 .01 .1; visual mesh filename=package://Atlas/urdf/meshes/s-model_articulated/visual/palm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
Joints:
- removed joint finger_1_fourbar_0_joint_3
- removed joint finger_1_joint_3
- removed joint finger_2_fourbar_0_joint_3
- removed joint finger_2_joint_3
- removed joint finger_middle_fourbar_0_joint_3
- removed joint finger_middle_joint_3
- added joint finger_1_fourbar_0_joint_0: type revolute, parent finger_1_link_0, child finger_1_fourbar_0_link_1, origin xyz=0.020 0 0 rpy=0 0 0, axis 0 0 1, limit lower=-2.10 upper=-0.255 effort=100 velocity=100
- added joint finger_1_fourbar_3_joint_0: type continuous, parent finger_1_link_2, child finger_1_fourbar_3_link_1, origin xyz=0 0 0 rpy=0 0 0, axis 0 0 1, limit lower=-1.367 upper=-0.945 effort=100 velocity=100
- added joint finger_1_fourbar_3_joint_1: type continuous, parent finger_1_fourbar_3_link_1, child finger_1_fourbar_3_link_2, origin xyz=0.02222 0 0 rpy=0 0 0, axis 0 0 1, limit lower=1.235 upper=1.613 effort=100 velocity=100
- added joint finger_1_fourbar_3_joint_2: type continuous, parent finger_1_link_3, child finger_1_fourbar_3_link_3, origin xyz=0 0 0 rpy=0 0 0, axis 0 0 1, limit lower=-1.367 upper=-0.995 effort=100 velocity=100
- added joint finger_1_fourbar_linkage_joint_0: type continuous, parent finger_1_fourbar_0_link_3, child finger_1_fourbar_linkage, origin xyz=.01473 0 0 rpy=0 0 0, axis 0 0 1, limit lower=1.4 upper=1.5 effort=100 velocity=100
- added joint finger_1_joint_0: type revolute, parent finger_1_link_0, child finger_1_link_1, origin xyz=0.020 0 0 rpy=0 0 0, axis 0 0 1, limit lower=0 upper=1.055 effort=100 velocity=100
- added joint finger_2_fourbar_0_joint_0: type revolute, parent finger_2_link_0, child finger_2_fourbar_0_link_1, origin xyz=0.020 0 0 rpy=0 0 0, axis 0 0 1, limit lower=-2.10 upper=-0.255 effort=100 velocity=100
- added joint finger_2_fourbar_3_joint_0: type continuous, parent finger_2_link_2, child finger_2_fourbar_3_link_1, origin xyz=0 0 0 rpy=0 0 0, axis 0 0 1, limit lower=-1.367 upper=-0.945 effort=100 velocity=100
- added joint finger_2_fourbar_3_joint_1: type continuous, parent finger_2_fourbar_3_link_1, child finger_2_fourbar_3_link_2, origin xyz=0.02222 0 0 rpy=0 0 0, axis 0 0 1, limit lower=1.235 upper=1.613 effort=100 velocity=100
- added joint finger_2_fourbar_3_joint_2: type continuous, parent finger_2_link_3, child finger_2_fourbar_3_link_3, origin xyz=0 0 0 rpy=0 0 0, axis 0 0 1, limit lower=-1.367 upper=-0.995 effort=100 velocity=100
- added joint finger_2_fourbar_linkage_joint_0: type continuous, parent finger_2_fourbar_0_link_3, child finger_2_fourbar_linkage, origin xyz=.01473 0 0 rpy=0 0 0, axis 0 0 1, limit lower=1.4 upper=1.5 effort=100 velocity=100
- added joint finger_2_joint_0: type revolute, parent finger_2_link_0, child finger_2_link_1, origin xyz=0.020 0 0 rpy=0 0 0, axis 0 0 1, limit lower=0 upper=1.055 effort=100 velocity=100
- added joint finger_middle_fourbar_0_joint_0: type revolute, parent finger_middle_link_0, child finger_middle_fourbar_0_link_1, origin xyz=0.020 0 0 rpy=0 0 0, axis 0 0 1, limit lower=-2.10 upper=-0.255 effort=100 velocity=100
- added joint finger_middle_fourbar_3_joint_0: type continuous, parent finger_middle_link_2, child finger_middle_fourbar_3_link_1, origin xyz=0 0 0 rpy=0 0 0, axis 0 0 1, limit lower=-1.367 upper=-0.945 effort=100 velocity=100
- added joint finger_middle_fourbar_3_joint_1: type continuous, parent finger_middle_fourbar_3_link_1, child finger_middle_fourbar_3_link_2, origin xyz=0.02222 0 0 rpy=0 0 0, axis 0 0 1, limit lower=1.235 upper=1.613 effort=100 velocity=100
- added joint finger_middle_fourbar_3_joint_2: type continuous, parent finger_middle_link_3, child finger_middle_fourbar_3_link_3, origin xyz=0 0 0 rpy=0 0 0, axis 0 0 1, limit lower=-1.367 upper=-0.995 effort=100 velocity=100
- added joint finger_middle_fourbar_linkage_joint_0: type continuous, parent finger_middle_fourbar_0_link_3, child finger_middle_fourbar_linkage, origin xyz=.01473 0 0 rpy=0 0 0, axis 0 0 1, limit lower=1.4 upper=1.5 effort=100 velocity=100
- added joint finger_middle_joint_0: type revolute, parent finger_middle_link_0, child finger_middle_link_1, origin xyz=0.020 0 0 rpy=0 0 0, axis 0 0 1, limit lower=0 upper=1.055 effort=100 velocity=100
- joint finger_1_fourbar_0_joint_1: child finger_1_fourbar_0_link_0 -> finger_1_fourbar_0_link_2; limit (none) -> lower=1.092 upper=1.940 effort=100 velocity=100; origin xyz=0 0 0 rpy=0 0 0 -> xyz=.02858 0 0 rpy=0 0 0; parent finger_1_link_1 -> finger_1_fourbar_0_link_1
- joint finger_1_fourbar_0_joint_2: child finger_1_fourbar_0_link_1 -> finger_1_fourbar_0_link_3; limit (none) -> lower=-2.111 upper=-0.199 effort=100 velocity=100; origin xyz=0.02858 0 0 rpy=0 0 0 -> xyz=0.050 -.028 0 rpy=0 0 -0.52; parent finger_1_fourbar_0_link_0 -> finger_1_link_1
- joint finger_1_joint_1: child finger_1_link_1 -> finger_1_link_2; limit lower=0 upper=3.1416 effort=100 velocity=100 -> lower=0 upper=1.5708 effort=100 velocity=100; origin xyz=0.020 0 0 rpy=0 0 0 -> xyz=0.050 -.028 0 rpy=0 0 -0.52; parent finger_1_link_0 -> finger_1_link_1
- joint finger_1_joint_2: child finger_1_link_2 -> finger_1_link_3; limit lower=0 upper=3.1416 effort=100 velocity=100 -> lower=-0.7854 upper=3.1416 effort=100 velocity=100; origin xyz=0.050 -.028 0 rpy=0 0 -0.52 -> xyz=0.039 0 0 rpy=0 0 0; parent finger_1_link_1 -> finger_1_link_2
- joint finger_2_fourbar_0_joint_1: child finger_2_fourbar_0_link_0 -> finger_2_fourbar_0_link_2; limit (none) -> lower=1.092 upper=1.940 effort=100 velocity=100; origin xyz=0 0 0 rpy=0 0 0 -> xyz=.02858 0 0 rpy=0 0 0; parent finger_2_link_1 -> finger_2_fourbar_0_link_1
- joint finger_2_fourbar_0_joint_2: child finger_2_fourbar_0_link_1 -> finger_2_fourbar_0_link_3; limit (none) -> lower=-2.111 upper=-0.199 effort=100 velocity=100; origin xyz=0.02858 0 0 rpy=0 0 0 -> xyz=0.050 -.028 0 rpy=0 0 -0.52; parent finger_2_fourbar_0_link_0 -> finger_2_link_1
- joint finger_2_joint_1: child finger_2_link_1 -> finger_2_link_2; limit lower=0 upper=3.1416 effort=100 velocity=100 -> lower=0 upper=1.5708 effort=100 velocity=100; origin xyz=0.020 0 0 rpy=0 0 0 -> xyz=0.050 -.028 0 rpy=0 0 -0.52; parent finger_2_link_0 -> finger_2_link_1
- joint finger_2_joint_2: child finger_2_link_2 -> finger_2_link_3; limit lower=0 upper=3.1416 effort=100 velocity=100 -> lower=-0.7854 upper=3.1416 effort=100 velocity=100; origin xyz=0.050 -.028 0 rpy=0 0 -0.52 -> xyz=0.039 0 0 rpy=0 0 0; parent finger_2_link_1 -> finger_2_link_2
- joint finger_middle_fourbar_0_joint_1: child finger_middle_fourbar_0_link_0 -> finger_middle_fourbar_0_link_2; limit (none) -> lower=1.092 upper=1.940 effort=100 velocity=100; origin xyz=0 0 0 rpy=0 0 0 -> xyz=.02858 0 0 rpy=0 0 0; parent finger_middle_link_1 -> finger_middle_fourbar_0_link_1
- joint finger_middle_fourbar_0_joint_2: child finger_middle_fourbar_0_link_1 -> finger_middle_fourbar_0_link_3; limit (none) -> lower=-2.111 upper=-0.199 effort=100 velocity=100; origin xyz=0.02858 0 0 rpy=0 0 0 -> xyz=0.050 -.028 0 rpy=0 0 -0.52; parent finger_middle_fourbar_0_link_0 -> finger_middle_link_1
- joint finger_middle_joint_1: child finger_middle_link_1 -> finger_middle_link_2; limit lower=0 upper=3.1416 effort=100 velocity=100 -> lower=0 upper=1.5708 effort=100 velocity=100; origin xyz=0.020 0 0 rpy=0 0 0 -> xyz=0.050 -.028 0 rpy=0 0 -0.52; parent finger_middle_link_0 -> finger_middle_link_1
- joint finger_middle_joint_2: child finger_middle_link_2 -> finger_middle_link_3; limit lower=0 upper=3.1416 effort=100 velocity=100 -> lower=-0.7854 upper=3.1416 effort=100 velocity=100; origin xyz=0.050 -.028 0 rpy=0 0 -0.52 -> xyz=0.039 0 0 rpy=0 0 0; parent finger_middle_link_1 -> finger_middle_link_2
- joint palm_finger_1_joint: limit lower=-0.16 upper=0.25 effort=100 velocity=100 -> (none); type revolute -> fixed
- joint palm_finger_2_joint: limit lower=-0.25 upper=0.16 effort=100 velocity=100 -> (none); type revolute -> fixed
