Commit message: add the convex hull obj in IRB140

File: examples/IRB140/urdf/irb_140.urdf (robot description, URDF)
Before this commit: robot IRB140_-_M2004C_Complete_base.SLDASM, 7 links, 6 joints
Links:
- link base_link: geometry visual mesh filename=package://IRB140/urdf/meshes/base_link.stl

File: examples/IRB140/urdf/irb_140_convhull.urdf (robot description, URDF)
Before this commit: robot IRB140_-_M2004C_Complete_base.SLDASM, 7 links, 6 joints
Links:
- link base_link: geometry visual mesh filename=package://IRB140/urdf/meshes/base_link_chull.stl
- link link_1: geometry collision mesh filename=package://IRB140/urdf/meshes/link1_chull.stl; visual mesh filename=package://IRB140/urdf/meshes/link1_chull.stl
- link link_2: geometry collision mesh filename=package://IRB140/urdf/meshes/link2_chull.stl; visual mesh filename=package://IRB140/urdf/meshes/link2_chull.stl
- link link_3: geometry collision mesh filename=package://IRB140/urdf/meshes/link3_chull.stl; visual mesh filename=package://IRB140/urdf/meshes/link3_chull.stl
- link link_4: geometry collision mesh filename=package://IRB140/urdf/meshes/link4_chull.stl; visual mesh filename=package://IRB140/urdf/meshes/link4_chull.stl
- link link_5: geometry collision mesh filename=package://IRB140/urdf/meshes/link5_chull.stl; visual mesh filename=package://IRB140/urdf/meshes/link5_chull.stl
- link link_6: geometry collision mesh filename=package://IRB140/urdf/meshes/link6_chull.stl; visual mesh filename=package://IRB140/urdf/meshes/link6_chull.stl

Commit message: add collision filter group in IRB140 urdf, change the joint limit of joint6 in IRB140

File: examples/IRB140/urdf/irb_140.urdf (robot description, URDF)
Before this commit: robot IRB140_-_M2004C_Complete_base.SLDASM, 7 links, 6 joints
Links:
- link base_link: geometry collision mesh filename=package://IRB140/urdf/meshes/base_link.stl; visual mesh filename=package://IRB140/urdf/meshes/base_link.stl
Joints:
- joint joint6: limit lower=-6.98131701 upper=-6.98131701 effort=300 velocity=7.33 -> lower=-6.98131701 upper=6.98131701 effort=300 velocity=7.33

File: examples/IRB140/urdf/irb_140_convhull.urdf (robot description, URDF)
Before this commit: robot IRB140_-_M2004C_Complete_base.SLDASM, 7 links, 6 joints
Links:
- link base_link: geometry collision mesh filename=package://IRB140/urdf/meshes/base_link_chull.stl; visual mesh filename=package://IRB140/urdf/meshes/base_link_chull.stl
Joints:
- joint joint6: limit lower=-6.98131701 upper=-6.98131701 effort=300 velocity=7.33 -> lower=-6.98131701 upper=6.98131701 effort=300 velocity=7.33
