Commit message: add joint limits in robotiq_simple.urdf

File: examples/IRB140/urdf/irb_140_robotiq_simple_ati.urdf (robot description, URDF)
Before this commit: robot s-model_articulated, 13 links, 12 joints
Links:
- added link ATI_sensor, mass 0.68252; collision mesh filename=package://IRB140/urdf/meshes/ATI_sensor.stl; visual mesh filename=package://IRB140/urdf/meshes/ATI_sensor.stl
- added link base_link, mass 12.409016159487; collision mesh filename=package://IRB140/urdf/meshes/base_link.stl; visual mesh filename=package://IRB140/urdf/meshes/base_link.stl
- added link link_1, mass 16.287755696602; collision mesh filename=package://IRB140/urdf/meshes/link1.stl; visual mesh filename=package://IRB140/urdf/meshes/link1.stl
- added link link_2, mass 7.58037424484438; collision mesh filename=package://IRB140/urdf/meshes/link2.stl; visual mesh filename=package://IRB140/urdf/meshes/link2.stl
- added link link_3, mass 8.03072730997701; collision mesh filename=package://IRB140/urdf/meshes/link3.stl; visual mesh filename=package://IRB140/urdf/meshes/link3.stl
- added link link_4, mass 1.7702548022269; collision mesh filename=package://IRB140/urdf/meshes/link4.stl; visual mesh filename=package://IRB140/urdf/meshes/link4.stl
- added link link_5, mass 0.145550520315438; collision mesh filename=package://IRB140/urdf/meshes/link5.stl; visual mesh filename=package://IRB140/urdf/meshes/link5.stl
- added link link_6, mass 0.0258654328719498; collision mesh filename=package://IRB140/urdf/meshes/link6.stl; visual mesh filename=package://IRB140/urdf/meshes/link6.stl
Joints:
- added joint ati_joint: type fixed, parent link_6, child ATI_sensor, origin xyz=0.00953 0 0 rpy=0.0 0.0 -1.57079
- added joint joint1: type revolute, parent base_link, child link_1, origin xyz=0 0 0.1095 rpy=-1.57079 0 0, axis 0 -1 0, limit lower=-3.14159265359 upper=3.14159265359 effort=300 velocity=4.36
- added joint joint2: type revolute, parent link_1, child link_2, origin xyz=0.07 -0.2425 0 rpy=0 0 0, axis 0 0 1, limit lower=-1.57079633 upper=1.91986218 effort=300 velocity=4.36
- added joint joint3: type revolute, parent link_2, child link_3, origin xyz=0 -0.360 0 rpy=0 0 0, axis 0 0 1, limit lower=-4.01425728 upper=0.87266463 effort=300 velocity=4.36
- added joint joint4: type revolute, parent link_3, child link_4, origin xyz=0.2185 0 0 rpy=0 0 0, axis 1 0 0, limit lower=-3.49065850 upper=3.49065850 effort=300 velocity=5.58
- added joint joint5: type revolute, parent link_4, child link_5, origin xyz=0.1615 0 0 rpy=0 0 0, axis 0 0 -1, limit lower=-2.09439510 upper=2.09439510 effort=300 velocity=5.58
- added joint joint6: type revolute, parent link_5, child link_6, origin xyz=0.065 0 0 rpy=0 0 0, axis 1 0 0, limit lower=-6.98131701 upper=6.98131701 effort=300 velocity=7.33
- added joint robotiq_hand_joint: type fixed, parent link_6, child palm, origin xyz=0.11904 0 0 rpy=0.0 0.0 -1.57079
