Commit message: Reverted Atlasv4 to pre-merge

File: examples/Atlasv4/urdf/atlas_convex_hull.urdf (robot description, URDF)
Before this commit: robot atlas, 70 links, 69 joints
Links:
- removed link center_bottom_led_frame
- removed link center_top_led_frame
- removed link head_hokuyo_frame
- removed link hokuyo_link
- removed link l_hand_camera_link
- removed link l_hand_camera_optical_frame
- removed link l_hand_face
- removed link l_hand_force_torque
- removed link l_hand_gripper
- removed link l_lfarm
- removed link l_situational_awareness_camera_link
- removed link l_situational_awareness_camera_optical_frame
- removed link l_ufarm
- removed link left_camera_frame
- removed link left_camera_optical_frame
- removed link left_led_frame
- removed link left_palm
- removed link post_spindle
- removed link post_spindle_cal_pitch
- removed link post_spindle_cal_roll
- removed link post_spindle_cal_x
- removed link post_spindle_cal_y
- removed link post_spindle_cal_z
- removed link pre_spindle
- removed link pre_spindle_cal_pitch
- removed link pre_spindle_cal_roll
- removed link pre_spindle_cal_x
- removed link pre_spindle_cal_y
- removed link pre_spindle_cal_yaw
- removed link pre_spindle_cal_z
- removed link r_hand_camera_link
- removed link r_hand_camera_optical_frame
- removed link r_hand_face
- removed link r_hand_force_torque
- removed link r_hand_gripper
- removed link r_lfarm
- removed link r_situational_awareness_camera_link
- removed link r_situational_awareness_camera_optical_frame
- removed link r_ufarm
- removed link right_camera_frame
- removed link right_camera_optical_frame
- removed link right_led_frame
- removed link right_palm
- added link l_farm, mass 3.388; collision mesh filename=meshes/l_farm_chull.wrl scale=1 1 1; visual mesh filename=meshes/l_farm.wrl scale=1 1 1
- added link r_farm, mass 3.388; collision mesh filename=meshes/r_farm_chull.wrl scale=1 1 1; visual mesh filename=meshes/r_farm.wrl scale=1 1 1
- link head: mass 1.4199 -> 1.477574; geometry visual mesh filename=meshes/head.wrl
- link l_clav: mass 4.466 -> 3.45; geometry collision mesh filename=meshes/l_clav_chull.wrl scale=1 1 1; visual mesh filename=meshes/l_clav.wrl scale=1 1 1
- link l_foot: mass 2.410 -> 2.05; geometry collision mesh filename=meshes/l_foot_chull.wrl scale=1 1 1; collision sphere radius=0
- link l_hand: mass 0.5839 -> 2.509; geometry collision mesh filename=meshes/GRIPPER_OPEN_chull.wrl scale=1 1 1; collision mesh filename=meshes/l_hand_chull.wrl scale=1 1 1
- link l_larm: mass 3.248 -> 2.509; geometry collision mesh filename=meshes/l_elbow_rx_chull.wrl scale=1 1 1; visual mesh filename=meshes/l_elbow_rx.wrl scale=1 1 1
- link l_lglut: mass 0.898 -> 0.866; geometry visual mesh filename=meshes/l_lglut.wrl scale=1 1 1
- link l_lleg: mass 4.515 -> 5.479; geometry collision mesh filename=meshes/l_lleg_chull.wrl scale=1 1 1; visual mesh filename=meshes/l_lleg.wrl scale=1 1 1
- link l_scap: mass 3.899 -> 3.012; geometry collision mesh filename=meshes/l_sh_rx_chull.wrl scale=1 1 1; visual mesh filename=meshes/l_sh_rx.wrl scale=1 1 1
- link l_talus: geometry visual mesh filename=meshes/l_talus.wrl scale=1 1 1
- link l_uarm: mass 4.386 -> 3.388; geometry collision mesh filename=meshes/l_elbow_ry_chull.wrl scale=1 1 1; visual mesh filename=meshes/l_elbow_ry.wrl scale=1 1 1
- link l_uglut: mass 1.959 -> 0.648; geometry visual mesh filename=meshes/l_uglut.wrl scale=1 1 1
- link l_uleg: mass 8.204 -> 9.209; geometry collision mesh filename=meshes/l_uleg_chull.wrl scale=1 1 1; visual mesh filename=meshes/l_uleg.wrl scale=1 1 1
- link ltorso: mass 2.270 -> 2.409; geometry visual mesh filename=meshes/ltorso.wrl scale=1 1 1
- link mtorso: mass 0.799 -> 0.69; geometry visual mesh filename=meshes/mtorso.wrl scale=1 1 1
- link pelvis: mass 9.509 -> 17.882; geometry collision mesh filename=meshes/pelvis_chull.wrl scale=1 1 1; visual mesh filename=meshes/pelvis.wrl scale=1 1 1
- link r_clav: mass 4.466 -> 3.45; geometry collision mesh filename=meshes/r_clav_chull.wrl scale=1 1 1; visual mesh filename=meshes/r_clav.wrl scale=1 1 1
- link r_foot: mass 2.41 -> 2.05; geometry collision mesh filename=meshes/r_foot_chull.wrl scale=1 1 1; collision sphere radius=0
- link r_hand: mass 0.5839 -> 2.509; geometry collision mesh filename=meshes/GRIPPER_OPEN_chull.wrl scale=1 1 1; collision mesh filename=meshes/r_hand_chull.wrl scale=1 1 1
- link r_larm: mass 3.248 -> 2.509; geometry collision mesh filename=meshes/r_elbow_rx_chull.wrl scale=1 1 1; visual mesh filename=meshes/r_elbow_rx.wrl scale=1 1 1
- link r_lglut: mass 0.898 -> 0.866; geometry visual mesh filename=meshes/r_lglut.wrl scale=1 1 1
- link r_lleg: mass 4.515 -> 5.479; geometry collision mesh filename=meshes/r_lleg_chull.wrl scale=1 1 1; visual mesh filename=meshes/r_lleg.wrl scale=1 1 1
- link r_scap: mass 3.899 -> 3.012; geometry collision mesh filename=meshes/r_sh_rx_chull.wrl scale=1 1 1; visual mesh filename=meshes/r_sh_rx.wrl scale=1 1 1
- link r_talus: geometry visual mesh filename=meshes/r_talus.wrl scale=1 1 1
- link r_uarm: mass 4.386 -> 3.388; geometry collision mesh filename=meshes/r_elbow_ry_chull.wrl scale=1 1 1; visual mesh filename=meshes/r_elbow_ry.wrl scale=1 1 1
- link r_uglut: mass 1.959 -> 0.648; geometry visual mesh filename=meshes/r_uglut.wrl scale=1 1 1
- link r_uleg: mass 8.204 -> 9.209; geometry collision mesh filename=meshes/r_uleg_chull.wrl scale=1 1 1; visual mesh filename=meshes/r_uleg.wrl scale=1 1 1
- link utorso: mass 84.409 -> 52; geometry collision mesh filename=meshes/utorso_chull.wrl scale=1 1 1; collision mesh filename=meshes/utorso_pack_chull.wrl scale=1 1 1
Joints:
- removed joint center_bottom_led_frame_joint
- removed joint center_top_led_frame_joint
- removed joint head_hokuyo_fixed_joint
- removed joint hokuyo_joint
- removed joint l_arm_lwy
- removed joint l_arm_shz
- removed joint l_hand_camera_joint
- removed joint l_hand_camera_optical_frame_joint
- removed joint l_hand_face_joint
- removed joint l_hand_force_torque_joint
- removed joint l_hand_gripper_joint
- removed joint l_situational_awareness_camera_joint
- removed joint l_situational_awareness_camera_optical_frame_joint
- removed joint left_camera_frame_joint
- removed joint left_camera_optical_frame_joint
- removed joint left_led_frame_joint
- removed joint left_palm_joint
- removed joint post_spindle_cal_pitch_joint
- removed joint post_spindle_cal_roll_joint
- removed joint post_spindle_cal_x_joint
- removed joint post_spindle_cal_y_joint
- removed joint post_spindle_cal_yaw_joint
- removed joint post_spindle_cal_z_joint
- removed joint pre_spindle_cal_pitch_joint
- removed joint pre_spindle_cal_roll_joint
- removed joint pre_spindle_cal_x_joint
- removed joint pre_spindle_cal_y_joint
- removed joint pre_spindle_cal_yaw_joint
- removed joint pre_spindle_cal_z_joint
- removed joint pre_spindle_joint
- removed joint r_arm_lwy
- removed joint r_arm_shz
- removed joint r_hand_camera_joint
- removed joint r_hand_camera_optical_frame_joint
- removed joint r_hand_face_joint
- removed joint r_hand_force_torque_joint
- removed joint r_hand_gripper_joint
- removed joint r_situational_awareness_camera_joint
- removed joint r_situational_awareness_camera_optical_frame_joint
- removed joint right_camera_frame_joint
- removed joint right_camera_optical_frame_joint
- removed joint right_led_frame_joint
- removed joint right_palm_joint
- added joint l_arm_usy: type revolute, parent utorso, child l_clav, origin xyz=0.06441 0.13866 0.10718 rpy=0 -0 0, axis 0 0.5 0.866025, limit lower=-1.5708 upper=0.785398 effort=75 velocity=12
- added joint r_arm_usy: type revolute, parent utorso, child r_clav, origin xyz=0.06441 -0.13866 0.10718 rpy=0 -0 0, axis 0 0.5 -0.866025, limit lower=-1.5708 upper=0.785398 effort=75 velocity=12
- joint back_bkx: limit lower=-0.523599 upper=0.523599 effort=300 velocity=12 -> lower=-0.698132 upper=0.698132 effort=200 velocity=12; origin xyz=0 0 0.05 rpy=0 0 0 -> xyz=0 0 0.05 rpy=0 -0 0
- joint back_bky: limit lower=-0.219388 upper=0.538783 effort=445 velocity=9 -> lower=-0.262 upper=0.524 effort=206.843 velocity=12; origin xyz=0 0 0.162 rpy=0 0 0 -> xyz=0 0 0.16197 rpy=0 -0 0
- joint back_bkz: limit lower=-0.663225 upper=0.663225 effort=106 velocity=12 -> lower=-0.663225 upper=0.663225 effort=114 velocity=12; origin xyz=-0.0125 0 0 rpy=0 0 0 -> xyz=-0.0125 0 0 rpy=0 -0 0
- joint l_arm_elx: axis -1.0 -0.0 -0.0 -> 1 0 0; limit lower=0 upper=2.35619 effort=112 velocity=12 -> lower=0 upper=2.35619 effort=55 velocity=12; origin xyz=0 -0.119 0.0092 rpy=0 0 0 -> xyz=0 0.119 0.00921 rpy=0 -0 0
- joint l_arm_ely: axis -0.0 -1.0 -0.0 -> 0 1 0; limit lower=0 upper=3.14159 effort=63 velocity=12 -> lower=0 upper=3.14159 effort=55 velocity=12; origin xyz=0 -0.187 -0.016 rpy=0 0 0 -> xyz=0 0.187 0.016 rpy=0 -0 0
- joint l_arm_mwx: child l_lfarm -> l_hand; limit lower=-1.7628 upper=1.7628 effort=25 velocity=10 -> lower=-1.1781 upper=1.1781 effort=55 velocity=12; origin xyz=0 0 0 rpy=0 0 0 -> xyz=0 0.119 0.00921 rpy=0 -0 0; parent l_ufarm -> l_farm
- joint l_arm_shx: axis -1.0 -0.0 -0.0 -> 1 0 0; limit lower=-1.5708 upper=1.5708 effort=99 velocity=12 -> lower=-1.5708 upper=1.5708 effort=107 velocity=12; origin xyz=0 -0.11 -0.245 rpy=0 0 0 -> xyz=0 0.14035 0.19609 rpy=0 -0 0
- joint l_arm_uwy: axis -0.0 -1.0 -0.0 -> 0 1 0; child l_ufarm -> l_farm; limit lower=-3.011 upper=3.011 effort=25 velocity=10 -> lower=0 upper=3.14159 effort=55 velocity=12; origin xyz=0 -0.29955 -0.00921 rpy=0 3.14159265359 0 -> xyz=0 0.187 -0.00921 rpy=0 -0 0
- joint l_leg_akx: limit lower=-0.8 upper=0.8 effort=360 velocity=12 -> lower=-0.8 upper=0.8 effort=130 velocity=12; origin xyz=0 0 0 rpy=0 0 0 -> xyz=0 0 0 rpy=0 -0 0
- joint l_leg_aky: limit lower=-1 upper=0.7 effort=740 velocity=12 -> lower=-1 upper=0.7 effort=350 velocity=12; origin xyz=0 0 -0.422 rpy=0 0 0 -> xyz=0 0 -0.422 rpy=0 -0 0
- joint l_leg_hpx: limit lower=-0.523599 upper=0.523599 effort=530 velocity=12 -> lower=-0.523599 upper=0.523599 effort=250 velocity=12; origin xyz=0 0 0 rpy=0 0 0 -> xyz=0 0 0 rpy=0 -0 0
- joint l_leg_hpy: limit lower=-1.61234 upper=0.65764 effort=840 velocity=12 -> lower=-1.72072 upper=0.524821 effort=260 velocity=12; origin xyz=0.05 0.0225 -0.066 rpy=0 0 0 -> xyz=0.05 0 -0.05 rpy=0 -0 0
- joint l_leg_hpz: limit lower=-0.174358 upper=0.786794 effort=275 velocity=12 -> lower=-0.174533 upper=1.22173 effort=68 velocity=12; origin xyz=0 0.089 0 rpy=0 0 0 -> xyz=0 0.089 0 rpy=0 -0 0
- joint l_leg_kny: limit lower=0 upper=2.35637 effort=890 velocity=12 -> lower=0 upper=2.38569 effort=220 velocity=12; origin xyz=-0.05 0 -0.374 rpy=0 0 0 -> xyz=-0.05 0 -0.374 rpy=0 -0 0
- joint neck_ay: limit lower=-0.602139 upper=1.14319 effort=25 velocity=6.28 -> lower=-0.602139 upper=1.14494 effort=5 velocity=12; origin xyz=0.2546 0 0.6215 rpy=0 0 0 -> xyz=0.21672 0 0.53796 rpy=0 -0 0
- joint r_arm_elx: limit lower=-2.35619 upper=0 effort=112 velocity=12 -> lower=-2.35619 upper=0 effort=55 velocity=12; origin xyz=0 -0.119 0.0092 rpy=0 0 0 -> xyz=0 -0.119 0.00921 rpy=0 -0 0
- joint r_arm_ely: limit lower=0 upper=3.14159 effort=63 velocity=12 -> lower=0 upper=3.14159 effort=55 velocity=12; origin xyz=0 -0.187 -0.016 rpy=0 0 0 -> xyz=0 -0.187 0.016 rpy=0 -0 0
- joint r_arm_mwx: child r_lfarm -> r_hand; limit lower=-1.7628 upper=1.7628 effort=25 velocity=10 -> lower=-1.1781 upper=1.1781 effort=55 velocity=12; origin xyz=0 0 0 rpy=0 0 0 -> xyz=0 -0.119 0.00921 rpy=0 -0 0; parent r_ufarm -> r_farm
- joint r_arm_shx: limit lower=-1.5708 upper=1.5708 effort=99 velocity=12 -> lower=-1.5708 upper=1.5708 effort=107 velocity=12; origin xyz=0 -0.11 -0.245 rpy=0 0 0 -> xyz=0 -0.14035 0.19609 rpy=0 -0 0
- joint r_arm_uwy: child r_ufarm -> r_farm; limit lower=-3.011 upper=3.011 effort=25 velocity=10 -> lower=0 upper=3.14159 effort=55 velocity=12; origin xyz=0 -0.29955 -0.00921 rpy=0 0 0 -> xyz=0 -0.187 -0.00921 rpy=0 -0 0
- joint r_leg_akx: limit lower=-0.8 upper=0.8 effort=360 velocity=12 -> lower=-0.8 upper=0.8 effort=130 velocity=12; origin xyz=0 0 0 rpy=0 0 0 -> xyz=0 0 0 rpy=0 -0 0
- joint r_leg_aky: limit lower=-1 upper=0.7 effort=740 velocity=12 -> lower=-1 upper=0.7 effort=350 velocity=12; origin xyz=0 0 -0.422 rpy=0 0 0 -> xyz=0 0 -0.422 rpy=0 -0 0
- joint r_leg_hpx: limit lower=-0.523599 upper=0.523599 effort=530 velocity=12 -> lower=-0.523599 upper=0.523599 effort=250 velocity=12; origin xyz=0 0 0 rpy=0 0 0 -> xyz=0 0 0 rpy=0 -0 0
- joint r_leg_hpy: limit lower=-1.61234 upper=0.65764 effort=840 velocity=12 -> lower=-1.72072 upper=0.524821 effort=260 velocity=12; origin xyz=0.05 -0.0225 -0.066 rpy=0 0 0 -> xyz=0.05 0 -0.05 rpy=0 -0 0
- joint r_leg_hpz: limit lower=-0.786794 upper=0.174358 effort=275 velocity=12 -> lower=-1.22173 upper=0.174533 effort=68 velocity=12; origin xyz=0 -0.089 0 rpy=0 0 0 -> xyz=0 -0.089 0 rpy=0 -0 0
- joint r_leg_kny: limit lower=0 upper=2.35637 effort=890 velocity=12 -> lower=0 upper=2.38569 effort=220 velocity=12; origin xyz=-0.05 0 -0.374 rpy=0 0 0 -> xyz=-0.05 0 -0.374 rpy=0 -0 0
