Commit message: Working commit.

File: examples/Atlasv4/urdf/atlas_planar_one_arm.urdf (robot description, URDF)
Before this commit: robot atlas, 28 links, 27 joints
Links:
- removed link l_clav
- removed link l_farm
- removed link l_hand
- removed link l_larm
- removed link l_scap
- removed link l_uarm
Joints:
- removed joint l_arm_elx
- removed joint l_arm_ely
- removed joint l_arm_mwx
- removed joint l_arm_shx
- removed joint l_arm_usy
- removed joint l_arm_uwy

File: examples/Atlasv4/urdf/atlas_planar_one_arm_noback.urdf (robot description, URDF)
Before this commit: robot atlas, 28 links, 27 joints
Links:
- removed link l_clav
- removed link l_farm
- removed link l_hand
- removed link l_larm
- removed link l_scap
- removed link l_uarm
Joints:
- removed joint l_arm_elx
- removed joint l_arm_ely
- removed joint l_arm_mwx
- removed joint l_arm_shx
- removed joint l_arm_usy
- removed joint l_arm_uwy
- joint back_bky: axis 0 1 0 -> (none); limit lower=-0.262 upper=0.524 effort=206.843 velocity=12 -> (none); type revolute -> fixed
