Commit message: six leg pairs

File: drake/examples/Strandbeest/Strandbeest.xacro (robot description, xacro)
@@ -5,12 +5,13 @@
  xmlns:xacro="http://ros.org/wiki/xacro" name="Strandbeest">
  <xacro:include filename="LegPair.xacro" />
+ <xacro:property name="pi" value="3.1415926535897931" />
  <link name="crank_axle">
     <inertial>
-      <origin xyz="0 0 0" rpy="1.5708 0 0"/>
+      <origin xyz="0 0 0" rpy="${pi/2} 0 0"/>
       <mass value="1"/>
         <inertia ixx="1"  ixy="0"  ixz="0" iyy="1" iyz="0" izz="1" />
     </inertial>
     <visual>
-      <origin xyz="0 0 0" rpy="1.5708 0 0"/>
+      <origin xyz="0 0 0" rpy="${pi/2} 0 0"/>
       <geometry>
         <cylinder length="1" radius="0.02"/>
@@ -21,17 +22,31 @@
     </visual>
   </link>
-  <xacro:strandbeest_leg_pair prefix="pair01">
-  </xacro:strandbeest_leg_pair>
-  <joint name="joint_crank_axle_l" type="fixed">
-    <axis xyz="0 1 0"/>
-    <parent link="crank_axle"/>
-    <child link="pair01_bar_l"/>
-    <origin rpy="0 3.14159 0" xyz="0 0 0"/>
-  </joint>
-  <joint name="joint_crank_axle_m" type="continuous">
-    <axis xyz="0 1 0"/>
-    <parent link="crank_axle"/>
-    <child link="pair01_bar_m"/>
-    <origin rpy="0 0 0" xyz="0 0 0"/>
-  </joint>
+  <xacro:macro name="positioned_leg_pair" params="name offset angle">
+	  <xacro:strandbeest_leg_pair prefix="${name}">
+	  </xacro:strandbeest_leg_pair>
+	  <joint name="joint_crank_axle_l" type="fixed">
+	    <axis xyz="0 1 0"/>
+	    <parent link="crank_axle"/>
+	    <child link="${name}_bar_l"/>
+	    <origin rpy="0 ${pi} 0" xyz="0 ${offset} 0"/>
+	  </joint>
+	  <joint name="joint_crank_axle_m" type="fixed">
+	    <axis xyz="0 1 0"/>
+	    <parent link="crank_axle"/>
+	    <child link="${name}_bar_m"/>
+	    <origin rpy="0 ${angle} 0" xyz="0 ${offset} 0"/>
+	  </joint>
+	</xacro:macro>
+	<xacro:positioned_leg_pair name="pair01" offset="-0.5" angle="0">
+	</xacro:positioned_leg_pair>
+	<xacro:positioned_leg_pair name="pair02" offset="-0.3" angle="${2*pi/3}">
+	</xacro:positioned_leg_pair>
+	<xacro:positioned_leg_pair name="pair03" offset="-0.1" angle="${4*pi/3}">
+	</xacro:positioned_leg_pair>
+	<xacro:positioned_leg_pair name="pair04" offset="0.1" angle="${pi/3}">
+	</xacro:positioned_leg_pair>
+	<xacro:positioned_leg_pair name="pair05" offset="0.3" angle="${3*pi/3}">
+	</xacro:positioned_leg_pair>
+	<xacro:positioned_leg_pair name="pair06" offset="0.5" angle="${5*pi/3}">
+	</xacro:positioned_leg_pair>
 </robot>

Commit message: add a basic controller (untested)

File: drake/examples/Strandbeest/Strandbeest.xacro (robot description, xacro)
@@ -44,4 +44,9 @@
     <origin rpy="0 0 0" xyz="0 0 0.078"/>
   </joint>
+  <transmission name="crossbar_crank_transmission" type="pr2_mechanism_model/SimpleTransmission">
+    <joint name="joint_crossbar_crank"/>
+    <actuator name="crossbar_crank_motor"/>
+    <mechanicalReduction>1</mechanicalReduction>
+  </transmission>
   <xacro:macro name="positioned_leg_pair" params="name offset angle">
 	  <xacro:strandbeest_leg_pair prefix="${name}">
@@ -67,8 +72,7 @@
 	<xacro:positioned_leg_pair name="pair01" offset="-0.5" angle="0">
 	</xacro:positioned_leg_pair>
-<!-- 	<xacro:positioned_leg_pair name="pair02" offset="-0.3" angle="${2*pi/3}">
+	<xacro:positioned_leg_pair name="pair02" offset="-0.3" angle="${2*pi/3}">
 	</xacro:positioned_leg_pair>
- -->
-<!-- 	<xacro:positioned_leg_pair name="pair03" offset="-0.1" angle="${4*pi/3}">
+	<xacro:positioned_leg_pair name="pair03" offset="-0.1" angle="${4*pi/3}">
 	</xacro:positioned_leg_pair>
 	<xacro:positioned_leg_pair name="pair04" offset="0.1" angle="${pi/3}">
@@ -78,4 +82,3 @@
 	<xacro:positioned_leg_pair name="pair06" offset="0.5" angle="${5*pi/3}">
 	</xacro:positioned_leg_pair>
- -->
 </robot>
