Commit message: working leg pair

File: drake/examples/Strandbeest/LegAssembly.xacro (robot description, xacro)
@@ -4,4 +4,5 @@
  xsi:schemaLocation="http://drake.mit.edu ../../doc/drakeURDF.xsd"
  xmlns:xacro="http://ros.org/wiki/xacro" name="LegAssembly">
+ <xacro:property name="pi" value="3.1415926535897931" />
 <xacro:macro name="strandbeest_leg" params="prefix">
   <link name="${prefix}_bar_j">
@@ -65,5 +66,5 @@
     <child link="${prefix}_bar_c"/>
     <origin rpy="0 0 0" xyz="0 0 0.619"/>
-    <limit lower="1.5708" upper="3.14159" effort="0" velocity="1000"/>
+    <limit lower="${pi/2}" upper="${pi}" effort="0" velocity="1000"/>
   </joint>
   <link name="${prefix}_bars_g_h_i">

File: drake/examples/Strandbeest/Strandbeest.xacro (robot description, xacro)
@@ -4,5 +4,5 @@
  xsi:schemaLocation="http://drake.mit.edu ../../doc/drakeURDF.xsd"
  xmlns:xacro="http://ros.org/wiki/xacro" name="Strandbeest">
- <xacro:include filename="LegAssembly.xacro" />
+ <xacro:include filename="LegPair.xacro" />
  <link name="crank_axle">
     <inertial>
@@ -21,82 +21,17 @@
     </visual>
   </link>
-  <link name="bar_l">
-    <inertial>
-      <origin xyz="0 0 0.039" rpy="0 0 0"/>
-      <mass value="1"/>
-        <inertia ixx="1"  ixy="0"  ixz="0" iyy="1" iyz="0" izz="1" />
-    </inertial>
-    <visual>
-      <origin xyz="0 0 0.039" rpy="0 0 0"/>
-      <geometry>
-        <cylinder length="0.078" radius="0.01"/>
-      </geometry>
-      <material>
-        <color rgba=".6353 0 0 1"/>
-      </material>
-    </visual>
-  </link>
+  <xacro:strandbeest_leg_pair prefix="pair01">
+  </xacro:strandbeest_leg_pair>
   <joint name="joint_crank_axle_l" type="fixed">
     <axis xyz="0 1 0"/>
     <parent link="crank_axle"/>
-    <child link="bar_l"/>
+    <child link="pair01_bar_l"/>
     <origin rpy="0 3.14159 0" xyz="0 0 0"/>
   </joint>
-  <link name="bar_a">
-    <inertial>
-      <origin xyz="0 0 0.19" rpy="0 0 0"/>
-      <mass value="1"/>
-        <inertia ixx="1"  ixy="0"  ixz="0" iyy="1" iyz="0" izz="1" />
-    </inertial>
-    <visual>
-      <origin xyz="0 0 0.19" rpy="0 0 0"/>
-      <geometry>
-        <cylinder length="0.38" radius="0.01"/>
-      </geometry>
-      <material>
-        <color rgba="0 .6353 0 1"/>
-      </material>
-    </visual>
-  </link>
-  <joint name="joint_l_a" type="fixed">
-    <axis xyz="0 1 0"/>
-    <parent link="bar_l"/>
-    <child link="bar_a"/>
-    <origin rpy="0 1.5708 0" xyz="0 0 0.078"/>
-  </joint>
-  <link name="bar_m">
-    <inertial>
-      <origin xyz="0 0 0.075" rpy="0 0 0"/>
-      <mass value="1"/>
-        <inertia ixx="1"  ixy="0"  ixz="0" iyy="1" iyz="0" izz="1" />
-    </inertial>
-    <visual>
-      <origin xyz="0 0 0.075" rpy="0 0 0"/>
-      <geometry>
-        <cylinder length="0.15" radius="0.01"/>
-      </geometry>
-      <material>
-        <color rgba=".6353 .6353 .6353 1"/>
-      </material>
-    </visual>
-  </link>
   <joint name="joint_crank_axle_m" type="continuous">
     <axis xyz="0 1 0"/>
     <parent link="crank_axle"/>
-    <child link="bar_m"/>
+    <child link="pair01_bar_m"/>
     <origin rpy="0 0 0" xyz="0 0 0"/>
   </joint>
-  <loop_joint name="leg01_loop_a_c" type="continuous">
-    <axis xyz="0 1 0"/>
-    <link1 link="bar_a" rpy="0 0 0" xyz="0 0 0.38"/>
-    <link2 link="leg01_bar_c" rpy="0 0 0" xyz="0 0 0.393"/>
-  </loop_joint>
-  <joint name="leg01_joint_m_j" type="continuous">
-    <axis xyz="0 1 0"/>
-    <parent link="bar_m"/>
-    <child link="leg01_bar_j"/>
-    <origin rpy="0 0 0" xyz="0 0 0.15"/>
-  </joint>
-  <xacro:strandbeest_leg prefix="leg01">
-  </xacro:strandbeest_leg>
 </robot>

Commit message: functioning crankshaft

File: drake/examples/Strandbeest/LegAssembly.xacro (robot description, xacro)
@@ -101,4 +101,10 @@
       </material>
     </visual>
+    <collision>
+      <origin rpy="0 0 0" xyz="0 0 0.49"/>
+      <geometry>
+        <sphere radius="0.01"/>
+      </geometry>
+    </collision>
   </link>
   <joint name="${prefix}_joint_k_i" type="revolute">

File: drake/examples/Strandbeest/LegPair.xacro (robot description, xacro)
@@ -43,5 +43,5 @@
     <parent link="${prefix}_bar_l"/>
     <child link="${prefix}_bar_a"/>
-    <origin rpy="0 ${pi/2} 0" xyz="0 0 0.078"/>
+    <origin rpy="0 ${-pi/2} 0" xyz="0 0 0"/>
   </joint>
   <link name="${prefix}_bar_m">

File: drake/examples/Strandbeest/Strandbeest.xacro (robot description, xacro)
@@ -6,4 +6,20 @@
  <xacro:include filename="LegPair.xacro" />
  <xacro:property name="pi" value="3.1415926535897931" />
+ <link name="crossbar">
+    <inertial>
+      <origin xyz="0 0 0" rpy="${pi/2} 0 0"/>
+      <mass value="1"/>
+        <inertia ixx="1"  ixy="0"  ixz="0" iyy="1" iyz="0" izz="1" />
+    </inertial>
+    <visual>
+      <origin xyz="0 0 0" rpy="${pi/2} 0 0"/>
+      <geometry>
+        <cylinder length="1" radius="0.01"/>
+      </geometry>
+      <material>
+        <color rgba="0 0 .6353 1"/>
+      </material>
+    </visual>
+  </link>
  <link name="crank_axle">
     <inertial>
@@ -22,14 +38,20 @@
     </visual>
   </link>
+  <joint name="joint_crossbar_crank" type="continuous">
+    <axis xyz="0 1 0"/>
+    <parent link="crossbar"/>
+    <child link="crank_axle"/>
+    <origin rpy="0 0 0" xyz="0 0 0.078"/>
+  </joint>
   <xacro:macro name="positioned_leg_pair" params="name offset angle">
 	  <xacro:strandbeest_leg_pair prefix="${name}">
 	  </xacro:strandbeest_leg_pair>
-	  <joint name="joint_crank_axle_l" type="fixed">
+	  <joint name="${name}_joint_crossbar_l" type="fixed">
 	    <axis xyz="0 1 0"/>
-	    <parent link="crank_axle"/>
+	    <parent link="crossbar"/>
 	    <child link="${name}_bar_l"/>
-	    <origin rpy="0 ${pi} 0" xyz="0 ${offset} 0"/>
+	    <origin rpy="0 0 0" xyz="0 ${offset} 0"/>
 	  </joint>
-	  <joint name="joint_crank_axle_m" type="fixed">
+	  <joint name="${name}_joint_crank_axle_m" type="fixed">
 	    <axis xyz="0 1 0"/>
 	    <parent link="crank_axle"/>
@@ -37,10 +59,16 @@
 	    <origin rpy="0 ${angle} 0" xyz="0 ${offset} 0"/>
 	  </joint>
+  <loop_joint name="${name}_loop_crank_l" type="continuous">
+    <axis xyz="0 1 0"/>
+    <link1 link="crank_axle" rpy="0 0 0" xyz="0 ${offset} 0"/>
+    <link2 link="${name}_bar_l" rpy="0 0 0" xyz="0 0 0.078"/>
+  </loop_joint>
 	</xacro:macro>
 	<xacro:positioned_leg_pair name="pair01" offset="-0.5" angle="0">
 	</xacro:positioned_leg_pair>
-	<xacro:positioned_leg_pair name="pair02" offset="-0.3" angle="${2*pi/3}">
+<!-- 	<xacro:positioned_leg_pair name="pair02" offset="-0.3" angle="${2*pi/3}">
 	</xacro:positioned_leg_pair>
-	<xacro:positioned_leg_pair name="pair03" offset="-0.1" angle="${4*pi/3}">
+ -->
+<!-- 	<xacro:positioned_leg_pair name="pair03" offset="-0.1" angle="${4*pi/3}">
 	</xacro:positioned_leg_pair>
 	<xacro:positioned_leg_pair name="pair04" offset="0.1" angle="${pi/3}">
@@ -50,3 +78,4 @@
 	<xacro:positioned_leg_pair name="pair06" offset="0.5" angle="${5*pi/3}">
 	</xacro:positioned_leg_pair>
+ -->
 </robot>

Commit message: add strandbeest to the gallery and update its colors

File: drake/examples/Strandbeest/LegAssembly.xacro (robot description, xacro)
@@ -18,6 +18,6 @@
         <cylinder length="0.50" radius="0.01"/>
       </geometry>
-      <material>
-        <color rgba=".6353 .6353 .6353 1"/>
+      <material name="orange">
+        <color rgba="1 .6392 .0980 1"/>
       </material>
     </visual>
@@ -34,7 +34,5 @@
         <cylinder length="0.619" radius="0.01"/>
       </geometry>
-      <material>
-        <color rgba=".6353 .6353 .6353 1"/>
-      </material>
+      <material name="orange"/>
     </visual>
   </link>
@@ -57,7 +55,5 @@
         <cylinder length="0.393" radius="0.01"/>
       </geometry>
-      <material>
-        <color rgba=".6353 .6353 .6353 1"/>
-      </material>
+      <material name="orange"/>
     </visual>
   </link>
@@ -80,7 +76,5 @@
         <cylinder length="0.49" radius="0.01"/>
       </geometry>
-      <material>
-        <color rgba=".6353 0.6353 0.6353 1"/>
-      </material>
+      <material name="orange"/>
     </visual>
     <visual>
@@ -89,7 +83,5 @@
         <cylinder length="0.367" radius="0.01"/>
       </geometry>
-      <material>
-        <color rgba=".6353 0.6353 0.6353 1"/>
-      </material>
+      <material name="orange"/>
     </visual>
     <visual>
@@ -98,7 +90,5 @@
         <cylinder length="0.657" radius="0.01"/>
       </geometry>
-      <material>
-        <color rgba=".6353 0.6353 0.6353 1"/>
-      </material>
+      <material name="orange"/>
     </visual>
     <collision>
@@ -132,7 +122,5 @@
         <cylinder length="0.558" radius="0.01"/>
       </geometry>
-      <material>
-        <color rgba=".6353 0.6353 0.6353 1"/>
-      </material>
+      <material name="orange"/>
     </visual>
     <visual>
@@ -141,7 +129,5 @@
         <cylinder length="0.401" radius="0.01"/>
       </geometry>
-      <material>
-        <color rgba=".6353 0.6353 0.6353 1"/>
-      </material>
+      <material name="orange"/>
     </visual>
     <visual>
@@ -150,7 +136,5 @@
         <cylinder length="0.415" radius="0.01"/>
       </geometry>
-      <material>
-        <color rgba=".6353 0.6353 0.6353 1"/>
-      </material>
+      <material name="orange"/>
     </visual>
   </link>
@@ -178,7 +162,5 @@
         <cylinder length="0.394" radius="0.01"/>
       </geometry>
-      <material>
-        <color rgba=".6353 .6353 .6353 1"/>
-      </material>
+      <material name="orange"/>
     </visual>
   </link>

File: drake/examples/Strandbeest/LegPair.xacro (robot description, xacro)
@@ -19,7 +19,5 @@
         <cylinder length="0.078" radius="0.01"/>
       </geometry>
-      <material>
-        <color rgba=".6353 .6353 .6353 1"/>
-      </material>
+      <material name="orange"/>
     </visual>
   </link>
@@ -35,7 +33,5 @@
         <cylinder length="0.76" radius="0.01"/>
       </geometry>
-      <material>
-        <color rgba=".6353 .6353 .6353 1"/>
-      </material>
+      <material name="orange"/>
     </visual>
   </link>
@@ -57,7 +53,5 @@
         <cylinder length="0.15" radius="0.01"/>
       </geometry>
-      <material>
-        <color rgba=".6353 .6353 .6353 1"/>
-      </material>
+      <material name="orange"/>
     </visual>
   </link>

File: drake/examples/Strandbeest/Strandbeest.xacro (robot description, xacro)
@@ -17,6 +17,6 @@
         <cylinder length="1" radius="0.01"/>
       </geometry>
-      <material>
-        <color rgba="0 0 .6353 1"/>
+      <material name="orange">
+        <color rgba="1 .6392 .0980 1"/>
       </material>
     </visual>
@@ -33,7 +33,5 @@
         <cylinder length="1" radius="0.02"/>
       </geometry>
-      <material>
-        <color rgba=".6353 .6353 .6353 1"/>
-      </material>
+      <material name="orange"/>
     </visual>
   </link>
