Commit message: rename torso

File: drake/examples/Valkyrie/urdf/urdf/valkyrie_A_sim_drake.urdf (robot description, URDF)
Before this commit: robot valkyrie, 87 links, 86 joints
Links:
- removed link torso
- removed link torsoPitchLink
- removed link torsoYawLink
- added link ltorso, mass 0.5; collision mesh filename=package://val_description/model/meshes/torso/torsoyaw.dae; visual mesh filename=package://val_description/model/meshes/torso/torsoyaw.dae
- added link mtorso, mass 0.1; collision mesh filename=package://val_description/model/meshes/torso/torsopitch.dae; visual mesh filename=package://val_description/model/meshes/torso/torsopitch.dae
- added link utorso, mass 39.47; collision mesh filename=package://val_description/model/meshes/torso/torso.dae; visual mesh filename=package://val_description/model/meshes/torso/torso.dae
Joints:
- joint leftHazardCamera_Offset: parent torso -> utorso
- joint leftShoulderPitch: parent torso -> utorso
- joint leftTorsoIMU_Offset: parent torso -> utorso
- joint lowerNeckPitch: parent torso -> utorso
- joint rightHazardCamera_Offset: parent torso -> utorso
- joint rightShoulderPitch: parent torso -> utorso
- joint rightTorsoIMU_Offset: parent torso -> utorso
- joint torsoPitch: child torsoPitchLink -> mtorso; parent torsoYawLink -> ltorso
- joint torsoRoll: child torso -> utorso; parent torsoPitchLink -> mtorso
- joint torsoYaw: child torsoYawLink -> ltorso

Commit message: legs

File: drake/examples/Valkyrie/urdf/urdf/valkyrie_A_sim_drake.urdf (robot description, URDF)
Before this commit: robot valkyrie, 87 links, 86 joints
Links:
- removed link leftAnklePitchLink
- removed link leftFoot
- removed link leftHipPitchLink
- removed link leftHipRollLink
- removed link leftHipYawLink
- removed link leftKneePitchLink
- removed link rightAnklePitchLink
- removed link rightFoot
- removed link rightHipPitchLink
- removed link rightHipRollLink
- removed link rightHipYawLink
- removed link rightKneePitchLink
- added link l_foot, mass 3.255; collision box size=0.27 0.16 0.064; collision sphere radius=0.0
- added link l_lglut, mass 3.665; collision mesh filename=package://val_description/model/meshes/legs/lj2_left.dae; visual mesh filename=package://val_description/model/meshes/legs/lj2_left.dae
- added link l_lleg, mass 6.6; collision mesh filename=package://val_description/model/meshes/legs/lj4_left.dae; visual mesh filename=package://val_description/model/meshes/legs/lj4_left.dae
- added link l_talus, mass 0.06; collision mesh filename=package://val_description/model/meshes/legs/lj5.dae; visual mesh filename=package://val_description/model/meshes/legs/lj5.dae
- added link l_uglut, mass 2.39; collision mesh filename=package://val_description/model/meshes/legs/lj1_left.dae; visual mesh filename=package://val_description/model/meshes/legs/lj1_left.dae
- added link l_uleg, mass 10.2; collision mesh filename=package://val_description/model/meshes/legs/lj3_left.dae; visual mesh filename=package://val_description/model/meshes/legs/lj3_left.dae
- added link r_foot, mass 3.255; collision box size=0.27 0.16 0.064; collision sphere radius=0.0
- added link r_lglut, mass 3.665; collision mesh filename=package://val_description/model/meshes/legs/lj2_right.dae; visual mesh filename=package://val_description/model/meshes/legs/lj2_right.dae
- added link r_lleg, mass 6.6; collision mesh filename=package://val_description/model/meshes/legs/lj4_right.dae; visual mesh filename=package://val_description/model/meshes/legs/lj4_right.dae
- added link r_talus, mass 0.06; collision mesh filename=package://val_description/model/meshes/legs/lj5.dae; visual mesh filename=package://val_description/model/meshes/legs/lj5.dae
- added link r_uglut, mass 2.39; collision mesh filename=package://val_description/model/meshes/legs/lj1_right.dae; visual mesh filename=package://val_description/model/meshes/legs/lj1_right.dae
- added link r_uleg, mass 10.2; collision mesh filename=package://val_description/model/meshes/legs/lj3_right.dae; visual mesh filename=package://val_description/model/meshes/legs/lj3_right.dae
Joints:
- joint leftAnklePitch: child leftAnklePitchLink -> l_talus; parent leftKneePitchLink -> l_lleg
- joint leftAnkleRoll: child leftFoot -> l_foot; parent leftAnklePitchLink -> l_talus
- joint leftCOP_Offset: parent leftFoot -> l_foot
- joint leftHipPitch: child leftHipPitchLink -> l_uleg; parent leftHipRollLink -> l_lglut
- joint leftHipRoll: child leftHipRollLink -> l_lglut; parent leftHipYawLink -> l_uglut
- joint leftHipYaw: child leftHipYawLink -> l_uglut
- joint leftKneePitch: child leftKneePitchLink -> l_lleg; parent leftHipPitchLink -> l_uleg
- joint leftLegSixAxis_Offset: parent leftFoot -> l_foot
- joint rightAnklePitch: child rightAnklePitchLink -> r_talus; parent rightKneePitchLink -> r_lleg
- joint rightAnkleRoll: child rightFoot -> r_foot; parent rightAnklePitchLink -> r_talus
- joint rightCOP_Offset: parent rightFoot -> r_foot
- joint rightHipPitch: child rightHipPitchLink -> r_uleg; parent rightHipRollLink -> r_lglut
- joint rightHipRoll: child rightHipRollLink -> r_lglut; parent rightHipYawLink -> r_uglut
- joint rightHipYaw: child rightHipYawLink -> r_uglut
- joint rightKneePitch: child rightKneePitchLink -> r_lleg; parent rightHipPitchLink -> r_uleg
- joint rightLegSixAxis_Offset: parent rightFoot -> r_foot

Commit message: arms

File: drake/examples/Valkyrie/urdf/urdf/valkyrie_A_sim_drake.urdf (robot description, URDF)
Before this commit: robot valkyrie, 87 links, 86 joints
Links:
- removed link leftElbowPitchLink
- removed link leftForearmLink
- removed link leftPalm
- removed link leftShoulderPitchLink
- removed link leftShoulderRollLink
- removed link leftShoulderYawLink
- removed link leftWristRollLink
- removed link rightElbowPitchLink
- removed link rightForearmLink
- removed link rightPalm
- removed link rightShoulderPitchLink
- removed link rightShoulderRollLink
- removed link rightShoulderYawLink
- removed link rightWristRollLink
- added link l_clav, mass 2.65; collision mesh filename=package://val_description/model/meshes/arms/aj1_left.dae; visual mesh filename=package://val_description/model/meshes/arms/aj1_left.dae
- added link l_farm, mass 2.476; collision mesh filename=package://val_description/model/meshes/arms/aj5_left.dae; visual mesh filename=package://val_description/model/meshes/arms/aj5_left.dae
- added link l_hand, mass 0.712; collision mesh filename=package://val_description/model/meshes/arms/palm_left.dae; visual mesh filename=package://val_description/model/meshes/arms/palm_left.dae
- added link l_larm, mass 1.83; collision mesh filename=package://val_description/model/meshes/arms/aj4_left.dae; visual mesh filename=package://val_description/model/meshes/arms/aj4_left.dae
- added link l_scap, mass 3.97; collision mesh filename=package://val_description/model/meshes/arms/aj2_left.dae; visual mesh filename=package://val_description/model/meshes/arms/aj2_left.dae
- added link l_uarm, mass 3.085; collision mesh filename=package://val_description/model/meshes/arms/aj3_left.dae; visual mesh filename=package://val_description/model/meshes/arms/aj3_left.dae
- added link l_uhand, mass 0.14; collision mesh filename=package://val_description/model/meshes/arms/aj6_left.dae; visual mesh filename=package://val_description/model/meshes/arms/aj6_left.dae
- added link r_clav, mass 2.65; collision mesh filename=package://val_description/model/meshes/arms/aj1_right.dae; visual mesh filename=package://val_description/model/meshes/arms/aj1_right.dae
- added link r_farm, mass 2.476; collision mesh filename=package://val_description/model/meshes/arms/aj5_right.dae; visual mesh filename=package://val_description/model/meshes/arms/aj5_right.dae
- added link r_hand, mass 0.712; collision mesh filename=package://val_description/model/meshes/arms/palm_right.dae; visual mesh filename=package://val_description/model/meshes/arms/palm_right.dae
- added link r_larm, mass 1.83; collision mesh filename=package://val_description/model/meshes/arms/aj4_right.dae; visual mesh filename=package://val_description/model/meshes/arms/aj4_right.dae
- added link r_scap, mass 3.97; collision mesh filename=package://val_description/model/meshes/arms/aj2_right.dae; visual mesh filename=package://val_description/model/meshes/arms/aj2_right.dae
- added link r_uarm, mass 3.085; collision mesh filename=package://val_description/model/meshes/arms/aj3_right.dae; visual mesh filename=package://val_description/model/meshes/arms/aj3_right.dae
- added link r_uhand, mass 0.14; collision mesh filename=package://val_description/model/meshes/arms/aj6_right.dae; visual mesh filename=package://val_description/model/meshes/arms/aj6_right.dae
Joints:
- joint l_hand_force_torque_joint: parent leftPalm -> l_hand
- joint leftElbowPitch: child leftElbowPitchLink -> l_larm; parent leftShoulderYawLink -> l_uarm
- joint leftForearmYaw: child leftForearmLink -> l_farm; parent leftElbowPitchLink -> l_larm
- joint leftIndexFingerPitch1: parent leftPalm -> l_hand
- joint leftMiddleFingerPitch1: parent leftPalm -> l_hand
- joint leftPinkyPitch1: parent leftPalm -> l_hand
- joint leftShoulderPitch: child leftShoulderPitchLink -> l_clav
- joint leftShoulderRoll: child leftShoulderRollLink -> l_scap; parent leftShoulderPitchLink -> l_clav
- joint leftShoulderYaw: child leftShoulderYawLink -> l_uarm; parent leftShoulderRollLink -> l_scap
- joint leftThumbRoll: parent leftPalm -> l_hand
- joint leftWristPitch: child leftPalm -> l_hand; parent leftWristRollLink -> l_uhand
- joint leftWristRoll: child leftWristRollLink -> l_uhand; parent leftForearmLink -> l_farm
- joint r_hand_force_torque_joint: parent rightPalm -> r_hand
- joint rightElbowPitch: child rightElbowPitchLink -> r_larm; parent rightShoulderYawLink -> r_uarm
- joint rightForearmYaw: child rightForearmLink -> r_farm; parent rightElbowPitchLink -> r_larm
- joint rightIndexFingerPitch1: parent rightPalm -> r_hand
- joint rightMiddleFingerPitch1: parent rightPalm -> r_hand
- joint rightPinkyPitch1: parent rightPalm -> r_hand
- joint rightShoulderPitch: child rightShoulderPitchLink -> r_clav
- joint rightShoulderRoll: child rightShoulderRollLink -> r_scap; parent rightShoulderPitchLink -> r_clav
- joint rightShoulderYaw: child rightShoulderYawLink -> r_uarm; parent rightShoulderRollLink -> r_scap
- joint rightThumbRoll: parent rightPalm -> r_hand
- joint rightWristPitch: child rightPalm -> r_hand; parent rightWristRollLink -> r_uhand
- joint rightWristRoll: child rightWristRollLink -> r_uhand; parent rightForearmLink -> r_farm

Commit message: rename joints except neck

File: drake/examples/Valkyrie/urdf/urdf/valkyrie_A_sim_drake.urdf (robot description, URDF)
Before this commit: robot valkyrie, 87 links, 86 joints
Joints:
- removed joint leftAnklePitch
- removed joint leftAnkleRoll
- removed joint leftElbowPitch
- removed joint leftForearmYaw
- removed joint leftHipPitch
- removed joint leftHipRoll
- removed joint leftHipYaw
- removed joint leftKneePitch
- removed joint leftShoulderPitch
- removed joint leftShoulderRoll
- removed joint leftShoulderYaw
- removed joint leftWristPitch
- removed joint leftWristRoll
- removed joint rightAnklePitch
- removed joint rightAnkleRoll
- removed joint rightElbowPitch
- removed joint rightForearmYaw
- removed joint rightHipPitch
- removed joint rightHipRoll
- removed joint rightHipYaw
- removed joint rightKneePitch
- removed joint rightShoulderPitch
- removed joint rightShoulderRoll
- removed joint rightShoulderYaw
- removed joint rightWristPitch
- removed joint rightWristRoll
- removed joint torsoPitch
- removed joint torsoRoll
- removed joint torsoYaw
- added joint back_bkx: type revolute, parent mtorso, child utorso, origin xyz=0.0 0.0 0.0203 rpy=0.0 0.0 0.0, axis 1 0 0, limit lower=-0.23 upper=0.255 effort=150 velocity=9
- added joint back_bky: type revolute, parent ltorso, child mtorso, origin xyz=0.04191 0.0 0.0 rpy=0.0 0.0 0.0, axis 0 1 0, limit lower=-0.13 upper=0.666 effort=150 velocity=9
- added joint back_bkz: type revolute, parent pelvis, child ltorso, origin xyz=0.0 0.0 0.0 rpy=0.0 0.0 0.0, axis 0 0 1, limit lower=-1.329 upper=1.181 effort=190 velocity=5.89
- added joint l_arm_elx: type revolute, parent l_uarm, child l_larm, origin xyz=0.0254 0.33 0.0 rpy=0.0 0.0 0.0, axis 0 0 1, limit lower=-2.174 upper=0.12 effort=65 velocity=11.5
- added joint l_arm_ely: type revolute, parent l_scap, child l_uarm, origin xyz=0.0 0.0 0.0 rpy=0.0 0.0 0.0, axis 0 1 0, limit lower=-3.1 upper=2.18 effort=65 velocity=11.5
- added joint l_arm_lwy: type revolute, parent l_uhand, child l_hand, origin xyz=0.0 0.0 0.0 rpy=0.0 0.0 0.0, axis 0 0 1, limit lower=-0.36 upper=0.49 effort=14 velocity=1
- added joint l_arm_mwx: type revolute, parent l_farm, child l_uhand, origin xyz=0.0 0.2871 0.0 rpy=0.0 0.0 0.0, axis 1 0 0, limit lower=-0.62 upper=0.625 effort=14 velocity=1
- added joint l_arm_shx: type revolute, parent l_clav, child l_scap, origin xyz=0.0 0.2499 0.0 rpy=0.0 0.0 0.0, axis 1 0 0, limit lower=-1.519 upper=1.266 effort=190 velocity=5.89
- added joint l_arm_shz: type revolute, parent utorso, child l_clav, origin xyz=-0.0316 0.0 0.2984 rpy=0.0 0.0 0.0, axis 0 1 0, limit lower=-2.85 upper=2.0 effort=190 velocity=5.89
- added joint l_arm_uwyYaw: type revolute, parent l_larm, child l_farm, origin xyz=-0.0254 0 0 rpy=0.0 0.0 0.0, axis 0 1 0, limit lower=-2.019 upper=3.14 effort=26 velocity=5
- added joint l_leg_akx: type revolute, parent l_talus, child l_foot, origin xyz=0.0 0.0 0.0 rpy=0.0 0.0 0.0, axis 1 0 0, limit lower=-0.349 upper=0.348 effort=205 velocity=11
- added joint l_leg_aky: type revolute, parent l_lleg, child l_talus, origin xyz=-0.0102381 0.0 -0.40627 rpy=0.0 0.0 0.0, axis 0 1 0, limit lower=-0.8644 upper=0.875 effort=205 velocity=11
- added joint l_leg_hpx: type revolute, parent l_uglut, child l_lglut, origin xyz=0.0 0.0 0.0 rpy=0.0 0.0 0.0, axis 1 0 0, limit lower=-0.467 upper=0.5515 effort=350 velocity=7
- added joint l_leg_hpy: type revolute, parent l_lglut, child l_uleg, origin xyz=0.0 0.0 -0.0609 rpy=0.0 0.0 0.0, axis 0 1 0, limit lower=-2.42 upper=1.619 effort=350 velocity=6.11
- added joint l_leg_hpz: type revolute, parent pelvis, child l_uglut, origin xyz=0.0 0.1016 -0.1853 rpy=0.0 0.0 0.0, axis 0 0 1, limit lower=-0.4141 upper=1.1 effort=190 velocity=5.89
- added joint l_leg_kny: type revolute, parent l_uleg, child l_lleg, origin xyz=0.000112225 0.0361046 -0.430959 rpy=0.0 0.0 0.0, axis 0 1 0, limit lower=-0.083 upper=2.057 effort=350 velocity=6.11
- added joint r_arm_elx: type revolute, parent r_uarm, child r_larm, origin xyz=0.0254 -0.33 0.0 rpy=0.0 0.0 0.0, axis 0 0 1, limit lower=-0.12 upper=2.174 effort=65 velocity=11.5
- added joint r_arm_ely: type revolute, parent r_scap, child r_uarm, origin xyz=0.0 0.0 0.0 rpy=0.0 0.0 0.0, axis 0 1 0, limit lower=-3.1 upper=2.18 effort=65 velocity=11.5
- added joint r_arm_lwy: type revolute, parent r_uhand, child r_hand, origin xyz=0.0 0.0 0.0 rpy=0.0 0.0 0.0, axis 0 0 1, limit lower=-0.49 upper=0.36 effort=14 velocity=1
- added joint r_arm_mwx: type revolute, parent r_farm, child r_uhand, origin xyz=0.0 -0.2871 0.0 rpy=0.0 0.0 0.0, axis 1 0 0, limit lower=-0.625 upper=0.62 effort=14 velocity=1
- added joint r_arm_shx: type revolute, parent r_clav, child r_scap, origin xyz=0.0 -0.2499 0.0 rpy=0.0 0.0 0.0, axis 1 0 0, limit lower=-1.266 upper=1.519 effort=190 velocity=5.89
- added joint r_arm_shz: type revolute, parent utorso, child r_clav, origin xyz=-0.0316 0.0 0.2984 rpy=0.0 0.0 0.0, axis 0 1 0, limit lower=-2.85 upper=2.0 effort=190 velocity=5.89
- added joint r_arm_uwyYaw: type revolute, parent r_larm, child r_farm, origin xyz=-0.0254 0 0 rpy=0.0 0.0 0.0, axis 0 1 0, limit lower=-2.019 upper=3.14 effort=26 velocity=5
- added joint r_leg_akx: type revolute, parent r_talus, child r_foot, origin xyz=0.0 0.0 0.0 rpy=0.0 0.0 0.0, axis 1 0 0, limit lower=-0.349 upper=0.348 effort=205 velocity=11
- added joint r_leg_aky: type revolute, parent r_lleg, child r_talus, origin xyz=-0.0102381 0.0 -0.40627 rpy=0.0 0.0 0.0, axis 0 1 0, limit lower=-0.8644 upper=0.875 effort=205 velocity=11
- added joint r_leg_hpx: type revolute, parent r_uglut, child r_lglut, origin xyz=0.0 0.0 0.0 rpy=0.0 0.0 0.0, axis 1 0 0, limit lower=-0.5515 upper=0.467 effort=350 velocity=7
- added joint r_leg_hpy: type revolute, parent r_lglut, child r_uleg, origin xyz=0.0 0.0 -0.0609 rpy=0.0 0.0 0.0, axis 0 1 0, limit lower=-2.42 upper=1.619 effort=350 velocity=6.11
- added joint r_leg_hpz: type revolute, parent pelvis, child r_uglut, origin xyz=0.0 -0.1016 -0.1853 rpy=0.0 0.0 0.0, axis 0 0 1, limit lower=-1.1 upper=0.4141 effort=190 velocity=5.89
- added joint r_leg_kny: type revolute, parent r_uleg, child r_lleg, origin xyz=0.000112225 -0.0361046 -0.430959 rpy=0.0 0.0 0.0, axis 0 1 0, limit lower=-0.083 upper=2.057 effort=350 velocity=6.11

Commit message: balancing test works

File: drake/examples/Valkyrie/urdf/urdf/valkyrie_A_sim_drake.urdf (robot description, URDF)
Before this commit: robot valkyrie, 87 links, 86 joints
Joints:
- removed joint l_arm_uwyYaw
- removed joint lowerNeckPitch
- removed joint r_arm_uwyYaw
- added joint l_arm_uwy: type revolute, parent l_larm, child l_farm, origin xyz=-0.0254 0 0 rpy=0.0 0.0 0.0, axis 0 1 0, limit lower=-2.019 upper=3.14 effort=26 velocity=5
- added joint neck_ay: type revolute, parent utorso, child lowerNeckPitchLink, origin xyz=0.0203518 0.0 0.33845 rpy=0.0 0.0 0.0, axis 0 1 0, limit lower=0 upper=1.162 effort=26 velocity=5
- added joint r_arm_uwy: type revolute, parent r_larm, child r_farm, origin xyz=-0.0254 0 0 rpy=0.0 0.0 0.0, axis 0 1 0, limit lower=-2.019 upper=3.14 effort=26 velocity=5
- joint neckYaw: type revolute -> fixed
- joint upperNeckPitch: type revolute -> fixed

Commit message: valkyrie walks just fine in drake
major changes:
- made all back and leg joint torque limits huge
- make ankle joint position limits huge
- changed the height of the walking gait in LIP & pelvis_height_about_sole
- made neck joints fixed except for one

File: drake/examples/Valkyrie/urdf/urdf/valkyrie_A_sim_drake.urdf (robot description, URDF)
Before this commit: robot valkyrie, 87 links, 86 joints
Joints:
- joint back_bkx: limit lower=-0.23 upper=0.255 effort=150 velocity=9 -> lower=-0.23 upper=0.255 effort=800 velocity=9
- joint back_bky: limit lower=-0.13 upper=0.666 effort=150 velocity=9 -> lower=-0.13 upper=0.666 effort=800 velocity=9
- joint back_bkz: limit lower=-1.329 upper=1.181 effort=190 velocity=5.89 -> lower=-1.329 upper=1.181 effort=800 velocity=5.89
- joint l_leg_akx: limit lower=-0.349 upper=0.348 effort=205 velocity=11 -> lower=-1.349 upper=1.348 effort=805 velocity=11
- joint l_leg_aky: limit lower=-0.8644 upper=0.875 effort=205 velocity=11 -> lower=-1.8644 upper=1.875 effort=805 velocity=11
- joint l_leg_hpx: limit lower=-0.467 upper=0.5515 effort=350 velocity=7 -> lower=-0.467 upper=0.5515 effort=840 velocity=7
- joint l_leg_hpy: limit lower=-2.42 upper=1.619 effort=350 velocity=6.11 -> lower=-2.42 upper=1.619 effort=840 velocity=6.11
- joint l_leg_hpz: limit lower=-0.4141 upper=1.1 effort=190 velocity=5.89 -> lower=-0.4141 upper=1.1 effort=840 velocity=5.89
- joint l_leg_kny: limit lower=-0.083 upper=2.057 effort=350 velocity=6.11 -> lower=-0.083 upper=2.057 effort=950 velocity=6.11
- joint r_leg_akx: limit lower=-0.349 upper=0.348 effort=205 velocity=11 -> lower=-1.349 upper=1.348 effort=805 velocity=11
- joint r_leg_aky: limit lower=-0.8644 upper=0.875 effort=205 velocity=11 -> lower=-1.8644 upper=1.875 effort=805 velocity=11
- joint r_leg_hpx: limit lower=-0.5515 upper=0.467 effort=350 velocity=7 -> lower=-0.5515 upper=0.467 effort=840 velocity=7
- joint r_leg_hpy: limit lower=-2.42 upper=1.619 effort=350 velocity=6.11 -> lower=-2.42 upper=1.619 effort=840 velocity=6.11
- joint r_leg_hpz: limit lower=-1.1 upper=0.4141 effort=190 velocity=5.89 -> lower=-1.1 upper=0.4141 effort=840 velocity=5.89
- joint r_leg_kny: limit lower=-0.083 upper=2.057 effort=350 velocity=6.11 -> lower=-0.083 upper=2.057 effort=950 velocity=6.11
