Commit message: Val desc uses obj and wrl

File: drake/examples/Valkyrie/urdf/urdf/valkyrie_A_sim_drake.urdf (robot description, URDF)
Before this commit: robot valkyrie, 87 links, 86 joints
Links:
- link hokuyo_link: geometry collision box size=0.08 0.06 0.04238; collision cylinder length=0.047 radius=0.024425
- link l_clav: geometry collision mesh filename=package://Valkyrie/urdf/model/meshes/arms/aj1_left.obj; visual mesh filename=package://Valkyrie/urdf/model/meshes/arms/aj1_left.obj
- link l_farm: geometry collision mesh filename=package://Valkyrie/urdf/model/meshes/arms/aj5_left.obj; visual mesh filename=package://Valkyrie/urdf/model/meshes/arms/aj5_left.obj
- link l_foot: geometry collision box size=0.27 0.16 0.064; collision sphere radius=0.0
- link l_hand: geometry collision mesh filename=package://Valkyrie/urdf/model/meshes/arms/palm_left.obj; visual mesh filename=package://Valkyrie/urdf/model/meshes/arms/palm_left.obj
- link l_larm: geometry collision mesh filename=package://Valkyrie/urdf/model/meshes/arms/aj4_left.obj; visual mesh filename=package://Valkyrie/urdf/model/meshes/arms/aj4_left.obj
- link l_lglut: geometry collision mesh filename=package://Valkyrie/urdf/model/meshes/legs/lj2_left.obj; visual mesh filename=package://Valkyrie/urdf/model/meshes/legs/lj2_left.obj
- link l_lleg: geometry collision mesh filename=package://Valkyrie/urdf/model/meshes/legs/lj4_left.obj; visual mesh filename=package://Valkyrie/urdf/model/meshes/legs/lj4_left.obj
- link l_scap: geometry collision mesh filename=package://Valkyrie/urdf/model/meshes/arms/aj2_left.obj; visual mesh filename=package://Valkyrie/urdf/model/meshes/arms/aj2_left.obj
- link l_talus: geometry collision mesh filename=package://Valkyrie/urdf/model/meshes/legs/lj5.obj; visual mesh filename=package://Valkyrie/urdf/model/meshes/legs/lj5.obj
- link l_uarm: geometry collision mesh filename=package://Valkyrie/urdf/model/meshes/arms/aj3_left.obj; visual mesh filename=package://Valkyrie/urdf/model/meshes/arms/aj3_left.obj
- link l_uglut: geometry collision mesh filename=package://Valkyrie/urdf/model/meshes/legs/lj1_left.obj; visual mesh filename=package://Valkyrie/urdf/model/meshes/legs/lj1_left.obj
- link l_uhand: geometry collision mesh filename=package://Valkyrie/urdf/model/meshes/arms/aj6_left.obj; visual mesh filename=package://Valkyrie/urdf/model/meshes/arms/aj6_left.obj
- link l_uleg: geometry collision mesh filename=package://Valkyrie/urdf/model/meshes/legs/lj3_left.obj; visual mesh filename=package://Valkyrie/urdf/model/meshes/legs/lj3_left.obj
- link leftIndexFingerPitch1Link: geometry collision mesh filename=package://Valkyrie/urdf/model/meshes/fingers/indexj1_left.o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; visual mesh filename=package://Valkyrie/urdf/model/meshes/fingers/indexj1_left.o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
- link leftIndexFingerPitch2Link: geometry collision mesh filename=package://Valkyrie/urdf/model/meshes/fingers/indexj2_left.o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; visual mesh filename=package://Valkyrie/urdf/model/meshes/fingers/indexj2_left.o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
- link leftIndexFingerPitch3Link: geometry collision mesh filename=package://Valkyrie/urdf/model/meshes/fingers/indexj3_left.o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; visual mesh filename=package://Valkyrie/urdf/model/meshes/fingers/indexj3_left.o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
- link leftMiddleFingerPitch1Link: geometry collision mesh filename=package://Valkyrie/urdf/model/meshes/fingers/middlej1_left.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; visual mesh filename=package://Valkyrie/urdf/model/meshes/fingers/middlej1_left.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
- link leftMiddleFingerPitch2Link: geometry collision mesh filename=package://Valkyrie/urdf/model/meshes/fingers/middlej2_left.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; visual mesh filename=package://Valkyrie/urdf/model/meshes/fingers/middlej2_left.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
- link leftMiddleFingerPitch3Link: geometry collision mesh filename=package://Valkyrie/urdf/model/meshes/fingers/middlej3_left.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; visual mesh filename=package://Valkyrie/urdf/model/meshes/fingers/middlej3_left.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
- link leftPinkyPitch1Link: geometry collision mesh filename=package://Valkyrie/urdf/model/meshes/fingers/pinkyj1_left.o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; visual mesh filename=package://Valkyrie/urdf/model/meshes/fingers/pinkyj1_left.o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
- link leftPinkyPitch2Link: geometry collision mesh filename=package://Valkyrie/urdf/model/meshes/fingers/pinkyj2_left.o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; visual mesh filename=package://Valkyrie/urdf/model/meshes/fingers/pinkyj2_left.o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
- link leftPinkyPitch3Link: geometry collision mesh filename=package://Valkyrie/urdf/model/meshes/fingers/pinkyj3_left.o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; visual mesh filename=package://Valkyrie/urdf/model/meshes/fingers/pinkyj3_left.o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
- link leftThumbPitch1Link: geometry collision mesh filename=package://Valkyrie/urdf/model/meshes/fingers/thumbj2_left.o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; visual mesh filename=package://Valkyrie/urdf/model/meshes/fingers/thumbj2_left.o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
- link leftThumbPitch2Link: geometry collision mesh filename=package://Valkyrie/urdf/model/meshes/fingers/thumbj3_left.o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; visual mesh filename=package://Valkyrie/urdf/model/meshes/fingers/thumbj3_left.o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
- link leftThumbPitch3Link: geometry collision mesh filename=package://Valkyrie/urdf/model/meshes/fingers/thumbj4_left.o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; visual mesh filename=package://Valkyrie/urdf/model/meshes/fingers/thumbj4_left.o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
- link leftThumbRollLink: geometry collision mesh filename=package://Valkyrie/urdf/model/meshes/fingers/thumbj1_left.o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; visual mesh filename=package://Valkyrie/urdf/model/meshes/fingers/thumbj1_left.o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
- link lowerNeckPitchLink: geometry collision mesh filename=package://Valkyrie/urdf/model/meshes/head/neckj1.obj; visual mesh filename=package://Valkyrie/urdf/model/meshes/head/neckj1.obj
- link ltorso: geometry collision mesh filename=package://Valkyrie/urdf/model/meshes/torso/torsoyaw.obj; visual mesh filename=package://Valkyrie/urdf/model/meshes/torso/torsoyaw.obj
- link mtorso: geometry collision mesh filename=package://Valkyrie/urdf/model/meshes/torso/torsopitch.obj; visual mesh filename=package://Valkyrie/urdf/model/meshes/torso/torsopitch.obj
- link neckYawLink: geometry collision mesh filename=package://Valkyrie/urdf/model/meshes/head/neckj2.obj; visual mesh filename=package://Valkyrie/urdf/model/meshes/head/neckj2.obj
- link pelvis: geometry collision mesh filename=package://Valkyrie/urdf/model/meshes/pelvis/pelvis.obj; visual mesh filename=package://Valkyrie/urdf/model/meshes/pelvis/pelvis.obj
- link r_clav: geometry collision mesh filename=package://Valkyrie/urdf/model/meshes/arms/aj1_right.obj; visual mesh filename=package://Valkyrie/urdf/model/meshes/arms/aj1_right.obj
- link r_farm: geometry collision mesh filename=package://Valkyrie/urdf/model/meshes/arms/aj5_right.obj; visual mesh filename=package://Valkyrie/urdf/model/meshes/arms/aj5_right.obj
- link r_foot: geometry collision box size=0.27 0.16 0.064; collision sphere radius=0.0
- link r_hand: geometry collision mesh filename=package://Valkyrie/urdf/model/meshes/arms/palm_right.obj; visual mesh filename=package://Valkyrie/urdf/model/meshes/arms/palm_right.obj
- link r_larm: geometry collision mesh filename=package://Valkyrie/urdf/model/meshes/arms/aj4_right.obj; visual mesh filename=package://Valkyrie/urdf/model/meshes/arms/aj4_right.obj
- link r_lglut: geometry collision mesh filename=package://Valkyrie/urdf/model/meshes/legs/lj2_right.obj; visual mesh filename=package://Valkyrie/urdf/model/meshes/legs/lj2_right.obj
- link r_lleg: geometry collision mesh filename=package://Valkyrie/urdf/model/meshes/legs/lj4_right.obj; visual mesh filename=package://Valkyrie/urdf/model/meshes/legs/lj4_right.obj
- link r_scap: geometry collision mesh filename=package://Valkyrie/urdf/model/meshes/arms/aj2_right.obj; visual mesh filename=package://Valkyrie/urdf/model/meshes/arms/aj2_right.obj
- link r_talus: geometry collision mesh filename=package://Valkyrie/urdf/model/meshes/legs/lj5.obj; visual mesh filename=package://Valkyrie/urdf/model/meshes/legs/lj5.obj
- link r_uarm: geometry collision mesh filename=package://Valkyrie/urdf/model/meshes/arms/aj3_right.obj; visual mesh filename=package://Valkyrie/urdf/model/meshes/arms/aj3_right.obj
- link r_uglut: geometry collision mesh filename=package://Valkyrie/urdf/model/meshes/legs/lj1_right.obj; visual mesh filename=package://Valkyrie/urdf/model/meshes/legs/lj1_right.obj
- link r_uhand: geometry collision mesh filename=package://Valkyrie/urdf/model/meshes/arms/aj6_right.obj; visual mesh filename=package://Valkyrie/urdf/model/meshes/arms/aj6_right.obj
- link r_uleg: geometry collision mesh filename=package://Valkyrie/urdf/model/meshes/legs/lj3_right.obj; visual mesh filename=package://Valkyrie/urdf/model/meshes/legs/lj3_right.obj
- link rightIndexFingerPitch1Link: geometry collision mesh filename=package://Valkyrie/urdf/model/meshes/fingers/indexj1_right.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; visual mesh filename=package://Valkyrie/urdf/model/meshes/fingers/indexj1_right.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
- link rightIndexFingerPitch2Link: geometry collision mesh filename=package://Valkyrie/urdf/model/meshes/fingers/indexj2_right.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; visual mesh filename=package://Valkyrie/urdf/model/meshes/fingers/indexj2_right.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
- link rightIndexFingerPitch3Link: geometry collision mesh filename=package://Valkyrie/urdf/model/meshes/fingers/indexj3_right.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; visual mesh filename=package://Valkyrie/urdf/model/meshes/fingers/indexj3_right.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
- link rightMiddleFingerPitch1Link: geometry collision mesh filename=package://Valkyrie/urdf/model/meshes/fingers/middlej1_right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; visual mesh filename=package://Valkyrie/urdf/model/meshes/fingers/middlej1_right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
- link rightMiddleFingerPitch2Link: geometry collision mesh filename=package://Valkyrie/urdf/model/meshes/fingers/middlej2_right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; visual mesh filename=package://Valkyrie/urdf/model/meshes/fingers/middlej2_right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
- link rightMiddleFingerPitch3Link: geometry collision mesh filename=package://Valkyrie/urdf/model/meshes/fingers/middlej3_right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; visual mesh filename=package://Valkyrie/urdf/model/meshes/fingers/middlej3_right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
- link rightPinkyPitch1Link: geometry collision mesh filename=package://Valkyrie/urdf/model/meshes/fingers/pinkyj1_right.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; visual mesh filename=package://Valkyrie/urdf/model/meshes/fingers/pinkyj1_right.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
- link rightPinkyPitch2Link: geometry collision mesh filename=package://Valkyrie/urdf/model/meshes/fingers/pinkyj2_right.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; visual mesh filename=package://Valkyrie/urdf/model/meshes/fingers/pinkyj2_right.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
- link rightPinkyPitch3Link: geometry collision mesh filename=package://Valkyrie/urdf/model/meshes/fingers/pinkyj3_right.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; visual mesh filename=package://Valkyrie/urdf/model/meshes/fingers/pinkyj3_right.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
- link rightThumbPitch1Link: geometry collision mesh filename=package://Valkyrie/urdf/model/meshes/fingers/thumbj2_right.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; visual mesh filename=package://Valkyrie/urdf/model/meshes/fingers/thumbj2_right.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
- link rightThumbPitch2Link: geometry collision mesh filename=package://Valkyrie/urdf/model/meshes/fingers/thumbj3_right.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; visual mesh filename=package://Valkyrie/urdf/model/meshes/fingers/thumbj3_right.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
- link rightThumbPitch3Link: geometry collision mesh filename=package://Valkyrie/urdf/model/meshes/fingers/thumbj4_right.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; visual mesh filename=package://Valkyrie/urdf/model/meshes/fingers/thumbj4_right.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
- link rightThumbRollLink: geometry collision mesh filename=package://Valkyrie/urdf/model/meshes/fingers/thumbj1_right.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; visual mesh filename=package://Valkyrie/urdf/model/meshes/fingers/thumbj1_right.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
- link upperNeckPitchLink: geometry collision mesh filename=package://Valkyrie/urdf/model/meshes/head/head_multisense_n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; visual mesh filename=package://Valkyrie/urdf/model/meshes/head/head_multisense_n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
- link utorso: geometry collision mesh filename=package://Valkyrie/urdf/model/meshes/torso/torso.obj; visual mesh filename=package://Valkyrie/urdf/model/meshes/torso/torso.obj

Commit message: use fp locally

File: drake/examples/Valkyrie/urdf/urdf/valkyrie_A_sim_drake.urdf (robot description, URDF)
Before this commit: robot valkyrie, 87 links, 86 joints
Links:
- link l_clav: geometry collision mesh filename=package://Valkyrie/urdf/model/meshes/arms/aj1_left.dae; visual mesh filename=package://Valkyrie/urdf/model/meshes/arms/aj1_left.dae
- link l_farm: geometry collision mesh filename=package://Valkyrie/urdf/model/meshes/arms/aj5_left.dae; visual mesh filename=package://Valkyrie/urdf/model/meshes/arms/aj5_left.dae
- link l_foot: geometry collision box size=0.27 0.16 0.064; collision sphere radius=0.0
- link l_hand: geometry collision mesh filename=package://Valkyrie/urdf/model/meshes/arms/palm_left.dae; visual mesh filename=package://Valkyrie/urdf/model/meshes/arms/palm_left.dae
- link l_larm: geometry collision mesh filename=package://Valkyrie/urdf/model/meshes/arms/aj4_left.dae; visual mesh filename=package://Valkyrie/urdf/model/meshes/arms/aj4_left.dae
- link l_lglut: geometry collision mesh filename=package://Valkyrie/urdf/model/meshes/legs/lj2_left.dae; visual mesh filename=package://Valkyrie/urdf/model/meshes/legs/lj2_left.dae
- link l_lleg: geometry collision mesh filename=package://Valkyrie/urdf/model/meshes/legs/lj4_left.dae; visual mesh filename=package://Valkyrie/urdf/model/meshes/legs/lj4_left.dae
- link l_scap: geometry collision mesh filename=package://Valkyrie/urdf/model/meshes/arms/aj2_left.dae; visual mesh filename=package://Valkyrie/urdf/model/meshes/arms/aj2_left.dae
- link l_talus: geometry collision mesh filename=package://Valkyrie/urdf/model/meshes/legs/lj5.dae; visual mesh filename=package://Valkyrie/urdf/model/meshes/legs/lj5.dae
- link l_uarm: geometry collision mesh filename=package://Valkyrie/urdf/model/meshes/arms/aj3_left.dae; visual mesh filename=package://Valkyrie/urdf/model/meshes/arms/aj3_left.dae
- link l_uglut: geometry collision mesh filename=package://Valkyrie/urdf/model/meshes/legs/lj1_left.dae; visual mesh filename=package://Valkyrie/urdf/model/meshes/legs/lj1_left.dae
- link l_uhand: geometry collision mesh filename=package://Valkyrie/urdf/model/meshes/arms/aj6_left.dae; visual mesh filename=package://Valkyrie/urdf/model/meshes/arms/aj6_left.dae
- link l_uleg: geometry collision mesh filename=package://Valkyrie/urdf/model/meshes/legs/lj3_left.dae; visual mesh filename=package://Valkyrie/urdf/model/meshes/legs/lj3_left.dae
- link leftIndexFingerPitch1Link: geometry collision mesh filename=package://Valkyrie/urdf/model/meshes/fingers/indexj1_left.d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; visual mesh filename=package://Valkyrie/urdf/model/meshes/fingers/indexj1_left.d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
- link leftIndexFingerPitch2Link: geometry collision mesh filename=package://Valkyrie/urdf/model/meshes/fingers/indexj2_left.d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; visual mesh filename=package://Valkyrie/urdf/model/meshes/fingers/indexj2_left.d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
- link leftIndexFingerPitch3Link: geometry collision mesh filename=package://Valkyrie/urdf/model/meshes/fingers/indexj3_left.d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; visual mesh filename=package://Valkyrie/urdf/model/meshes/fingers/indexj3_left.d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
- link leftPinkyPitch1Link: geometry collision mesh filename=package://Valkyrie/urdf/model/meshes/fingers/pinkyj1_left.d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; visual mesh filename=package://Valkyrie/urdf/model/meshes/fingers/pinkyj1_left.d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
- link leftPinkyPitch2Link: geometry collision mesh filename=package://Valkyrie/urdf/model/meshes/fingers/pinkyj2_left.d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; visual mesh filename=package://Valkyrie/urdf/model/meshes/fingers/pinkyj2_left.d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
- link leftPinkyPitch3Link: geometry collision mesh filename=package://Valkyrie/urdf/model/meshes/fingers/pinkyj3_left.d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; visual mesh filename=package://Valkyrie/urdf/model/meshes/fingers/pinkyj3_left.d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
- link leftThumbPitch1Link: geometry collision mesh filename=package://Valkyrie/urdf/model/meshes/fingers/thumbj2_left.d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; visual mesh filename=package://Valkyrie/urdf/model/meshes/fingers/thumbj2_left.d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
- link leftThumbPitch2Link: geometry collision mesh filename=package://Valkyrie/urdf/model/meshes/fingers/thumbj3_left.d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; visual mesh filename=package://Valkyrie/urdf/model/meshes/fingers/thumbj3_left.d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
- link leftThumbPitch3Link: geometry collision mesh filename=package://Valkyrie/urdf/model/meshes/fingers/thumbj4_left.d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; visual mesh filename=package://Valkyrie/urdf/model/meshes/fingers/thumbj4_left.d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
- link leftThumbRollLink: geometry collision mesh filename=package://Valkyrie/urdf/model/meshes/fingers/thumbj1_left.d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; visual mesh filename=package://Valkyrie/urdf/model/meshes/fingers/thumbj1_left.d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
- link lowerNeckPitchLink: geometry collision mesh filename=package://Valkyrie/urdf/model/meshes/head/neckj1.dae; visual mesh filename=package://Valkyrie/urdf/model/meshes/head/neckj1.dae
- link ltorso: geometry collision mesh filename=package://Valkyrie/urdf/model/meshes/torso/torsoyaw.dae; visual mesh filename=package://Valkyrie/urdf/model/meshes/torso/torsoyaw.dae
- link mtorso: geometry collision mesh filename=package://Valkyrie/urdf/model/meshes/torso/torsopitch.dae; visual mesh filename=package://Valkyrie/urdf/model/meshes/torso/torsopitch.dae
- link neckYawLink: geometry collision mesh filename=package://Valkyrie/urdf/model/meshes/head/neckj2.dae; visual mesh filename=package://Valkyrie/urdf/model/meshes/head/neckj2.dae
- link pelvis: geometry collision mesh filename=package://Valkyrie/urdf/model/meshes/pelvis/pelvis.dae; visual mesh filename=package://Valkyrie/urdf/model/meshes/pelvis/pelvis.dae
- link r_clav: geometry collision mesh filename=package://Valkyrie/urdf/model/meshes/arms/aj1_right.dae; visual mesh filename=package://Valkyrie/urdf/model/meshes/arms/aj1_right.dae
- link r_farm: geometry collision mesh filename=package://Valkyrie/urdf/model/meshes/arms/aj5_right.dae; visual mesh filename=package://Valkyrie/urdf/model/meshes/arms/aj5_right.dae
- link r_foot: geometry collision box size=0.27 0.16 0.064; collision sphere radius=0.0
- link r_hand: geometry collision mesh filename=package://Valkyrie/urdf/model/meshes/arms/palm_right.dae; visual mesh filename=package://Valkyrie/urdf/model/meshes/arms/palm_right.dae
- link r_larm: geometry collision mesh filename=package://Valkyrie/urdf/model/meshes/arms/aj4_right.dae; visual mesh filename=package://Valkyrie/urdf/model/meshes/arms/aj4_right.dae
- link r_lglut: geometry collision mesh filename=package://Valkyrie/urdf/model/meshes/legs/lj2_right.dae; visual mesh filename=package://Valkyrie/urdf/model/meshes/legs/lj2_right.dae
- link r_lleg: geometry collision mesh filename=package://Valkyrie/urdf/model/meshes/legs/lj4_right.dae; visual mesh filename=package://Valkyrie/urdf/model/meshes/legs/lj4_right.dae
- link r_scap: geometry collision mesh filename=package://Valkyrie/urdf/model/meshes/arms/aj2_right.dae; visual mesh filename=package://Valkyrie/urdf/model/meshes/arms/aj2_right.dae
- link r_talus: geometry collision mesh filename=package://Valkyrie/urdf/model/meshes/legs/lj5.dae; visual mesh filename=package://Valkyrie/urdf/model/meshes/legs/lj5.dae
- link r_uarm: geometry collision mesh filename=package://Valkyrie/urdf/model/meshes/arms/aj3_right.dae; visual mesh filename=package://Valkyrie/urdf/model/meshes/arms/aj3_right.dae
- link r_uglut: geometry collision mesh filename=package://Valkyrie/urdf/model/meshes/legs/lj1_right.dae; visual mesh filename=package://Valkyrie/urdf/model/meshes/legs/lj1_right.dae
- link r_uhand: geometry collision mesh filename=package://Valkyrie/urdf/model/meshes/arms/aj6_right.dae; visual mesh filename=package://Valkyrie/urdf/model/meshes/arms/aj6_right.dae
- link r_uleg: geometry collision mesh filename=package://Valkyrie/urdf/model/meshes/legs/lj3_right.dae; visual mesh filename=package://Valkyrie/urdf/model/meshes/legs/lj3_right.dae
- link utorso: geometry collision mesh filename=package://Valkyrie/urdf/model/meshes/torso/torso.dae; visual mesh filename=package://Valkyrie/urdf/model/meshes/torso/torso.dae
