Commit message: revert name changes

File: drake/examples/Valkyrie/urdf/urdf/valkyrie_A_sim_drake.urdf (robot description, URDF)
Before this commit: robot valkyrie, 87 links, 86 joints
Links:
- removed link l_clav
- removed link l_farm
- removed link l_foot
- removed link l_hand
- removed link l_larm
- removed link l_lglut
- removed link l_lleg
- removed link l_scap
- removed link l_talus
- removed link l_uarm
- removed link l_uglut
- removed link l_uhand
- removed link l_uleg
- removed link ltorso
- removed link mtorso
- removed link r_clav
- removed link r_farm
- removed link r_foot
- removed link r_hand
- removed link r_larm
- removed link r_lglut
- removed link r_lleg
- removed link r_scap
- removed link r_talus
- removed link r_uarm
- removed link r_uglut
- removed link r_uhand
- removed link r_uleg
- removed link utorso
- added link leftAnklePitchLink, mass 0.06; collision mesh filename=package://Valkyrie/urdf/model/meshes/legs/lj5.dae; visual mesh filename=package://Valkyrie/urdf/model/meshes/legs/lj5.dae
- added link leftElbowPitchLink, mass 1.83; collision mesh filename=package://Valkyrie/urdf/model/meshes/arms/aj4_left.dae; visual mesh filename=package://Valkyrie/urdf/model/meshes/arms/aj4_left.dae
- added link leftFoot, mass 3.255; collision box size=0.27 0.16 0.064; collision sphere radius=0.0
- added link leftForearmLink, mass 2.476; collision mesh filename=package://Valkyrie/urdf/model/meshes/arms/aj5_left.dae; visual mesh filename=package://Valkyrie/urdf/model/meshes/arms/aj5_left.dae
- added link leftHipPitchLink, mass 10.2; collision mesh filename=package://Valkyrie/urdf/model/meshes/legs/lj3_left.dae; visual mesh filename=package://Valkyrie/urdf/model/meshes/legs/lj3_left.dae
- added link leftHipRollLink, mass 3.665; collision mesh filename=package://Valkyrie/urdf/model/meshes/legs/lj2_left.dae; visual mesh filename=package://Valkyrie/urdf/model/meshes/legs/lj2_left.dae
- added link leftHipYawLink, mass 2.39; collision mesh filename=package://Valkyrie/urdf/model/meshes/legs/lj1_left.dae; visual mesh filename=package://Valkyrie/urdf/model/meshes/legs/lj1_left.dae
- added link leftKneePitchLink, mass 6.6; collision mesh filename=package://Valkyrie/urdf/model/meshes/legs/lj4_left.dae; visual mesh filename=package://Valkyrie/urdf/model/meshes/legs/lj4_left.dae
- added link leftPalm, mass 0.712; collision mesh filename=package://Valkyrie/urdf/model/meshes/arms/palm_left.dae; visual mesh filename=package://Valkyrie/urdf/model/meshes/arms/palm_left.dae
- added link leftShoulderPitchLink, mass 2.65; collision mesh filename=package://Valkyrie/urdf/model/meshes/arms/aj1_left.dae; visual mesh filename=package://Valkyrie/urdf/model/meshes/arms/aj1_left.dae
- added link leftShoulderRollLink, mass 3.97; collision mesh filename=package://Valkyrie/urdf/model/meshes/arms/aj2_left.dae; visual mesh filename=package://Valkyrie/urdf/model/meshes/arms/aj2_left.dae
- added link leftShoulderYawLink, mass 3.085; collision mesh filename=package://Valkyrie/urdf/model/meshes/arms/aj3_left.dae; visual mesh filename=package://Valkyrie/urdf/model/meshes/arms/aj3_left.dae
- added link leftWristRollLink, mass 0.14; collision mesh filename=package://Valkyrie/urdf/model/meshes/arms/aj6_left.dae; visual mesh filename=package://Valkyrie/urdf/model/meshes/arms/aj6_left.dae
- added link rightAnklePitchLink, mass 0.06; collision mesh filename=package://Valkyrie/urdf/model/meshes/legs/lj5.dae; visual mesh filename=package://Valkyrie/urdf/model/meshes/legs/lj5.dae
- added link rightElbowPitchLink, mass 1.83; collision mesh filename=package://Valkyrie/urdf/model/meshes/arms/aj4_right.dae; visual mesh filename=package://Valkyrie/urdf/model/meshes/arms/aj4_right.dae
- added link rightFoot, mass 3.255; collision box size=0.27 0.16 0.064; collision sphere radius=0.0
- added link rightForearmLink, mass 2.476; collision mesh filename=package://Valkyrie/urdf/model/meshes/arms/aj5_right.dae; visual mesh filename=package://Valkyrie/urdf/model/meshes/arms/aj5_right.dae
- added link rightHipPitchLink, mass 10.2; collision mesh filename=package://Valkyrie/urdf/model/meshes/legs/lj3_right.dae; visual mesh filename=package://Valkyrie/urdf/model/meshes/legs/lj3_right.dae
- added link rightHipRollLink, mass 3.665; collision mesh filename=package://Valkyrie/urdf/model/meshes/legs/lj2_right.dae; visual mesh filename=package://Valkyrie/urdf/model/meshes/legs/lj2_right.dae
- added link rightHipYawLink, mass 2.39; collision mesh filename=package://Valkyrie/urdf/model/meshes/legs/lj1_right.dae; visual mesh filename=package://Valkyrie/urdf/model/meshes/legs/lj1_right.dae
- added link rightKneePitchLink, mass 6.6; collision mesh filename=package://Valkyrie/urdf/model/meshes/legs/lj4_right.dae; visual mesh filename=package://Valkyrie/urdf/model/meshes/legs/lj4_right.dae
- added link rightPalm, mass 0.712; collision mesh filename=package://Valkyrie/urdf/model/meshes/arms/palm_right.dae; visual mesh filename=package://Valkyrie/urdf/model/meshes/arms/palm_right.dae
- added link rightShoulderPitchLink, mass 2.65; collision mesh filename=package://Valkyrie/urdf/model/meshes/arms/aj1_right.dae; visual mesh filename=package://Valkyrie/urdf/model/meshes/arms/aj1_right.dae
- added link rightShoulderRollLink, mass 3.97; collision mesh filename=package://Valkyrie/urdf/model/meshes/arms/aj2_right.dae; visual mesh filename=package://Valkyrie/urdf/model/meshes/arms/aj2_right.dae
- added link rightShoulderYawLink, mass 3.085; collision mesh filename=package://Valkyrie/urdf/model/meshes/arms/aj3_right.dae; visual mesh filename=package://Valkyrie/urdf/model/meshes/arms/aj3_right.dae
- added link rightWristRollLink, mass 0.14; collision mesh filename=package://Valkyrie/urdf/model/meshes/arms/aj6_right.dae; visual mesh filename=package://Valkyrie/urdf/model/meshes/arms/aj6_right.dae
- added link torso, mass 39.47; collision mesh filename=package://Valkyrie/urdf/model/meshes/torso/torso.dae; visual mesh filename=package://Valkyrie/urdf/model/meshes/torso/torso.dae
- added link torsoPitchLink, mass 0.1; collision mesh filename=package://Valkyrie/urdf/model/meshes/torso/torsopitch.dae; visual mesh filename=package://Valkyrie/urdf/model/meshes/torso/torsopitch.dae
- added link torsoYawLink, mass 0.5; collision mesh filename=package://Valkyrie/urdf/model/meshes/torso/torsoyaw.dae; visual mesh filename=package://Valkyrie/urdf/model/meshes/torso/torsoyaw.dae
Joints:
- removed joint back_bkx
- removed joint back_bky
- removed joint back_bkz
- removed joint l_arm_elx
- removed joint l_arm_ely
- removed joint l_arm_lwy
- removed joint l_arm_mwx
- removed joint l_arm_shx
- removed joint l_arm_shz
- removed joint l_arm_uwy
- removed joint l_leg_akx
- removed joint l_leg_aky
- removed joint l_leg_hpx
- removed joint l_leg_hpy
- removed joint l_leg_hpz
- removed joint l_leg_kny
- removed joint neck_ay
- removed joint r_arm_elx
- removed joint r_arm_ely
- removed joint r_arm_lwy
- removed joint r_arm_mwx
- removed joint r_arm_shx
- removed joint r_arm_shz
- removed joint r_arm_uwy
- removed joint r_leg_akx
- removed joint r_leg_aky
- removed joint r_leg_hpx
- removed joint r_leg_hpy
- removed joint r_leg_hpz
- removed joint r_leg_kny
- added joint leftAnklePitch: type revolute, parent leftKneePitchLink, child leftAnklePitchLink, origin xyz=-0.0102381 0.0 -0.40627 rpy=0.0 0.0 0.0, axis 0 1 0, limit lower=-1.8644 upper=1.875 effort=805 velocity=11
- added joint leftAnkleRoll: type revolute, parent leftAnklePitchLink, child leftFoot, origin xyz=0.0 0.0 0.0 rpy=0.0 0.0 0.0, axis 1 0 0, limit lower=-1.349 upper=1.348 effort=805 velocity=11
- added joint leftElbowPitch: type revolute, parent leftShoulderYawLink, child leftElbowPitchLink, origin xyz=0.0254 0.33 0.0 rpy=0.0 0.0 0.0, axis 0 0 1, limit lower=-2.174 upper=0.12 effort=65 velocity=11.5
- added joint leftForearmYaw: type revolute, parent leftElbowPitchLink, child leftForearmLink, origin xyz=-0.0254 0 0 rpy=0.0 0.0 0.0, axis 0 1 0, limit lower=-2.019 upper=3.14 effort=26 velocity=5
- added joint leftHipPitch: type revolute, parent leftHipRollLink, child leftHipPitchLink, origin xyz=0.0 0.0 -0.0609 rpy=0.0 0.0 0.0, axis 0 1 0, limit lower=-2.42 upper=1.619 effort=840 velocity=6.11
- added joint leftHipRoll: type revolute, parent leftHipYawLink, child leftHipRollLink, origin xyz=0.0 0.0 0.0 rpy=0.0 0.0 0.0, axis 1 0 0, limit lower=-0.467 upper=0.5515 effort=840 velocity=7
- added joint leftHipYaw: type revolute, parent pelvis, child leftHipYawLink, origin xyz=0.0 0.1016 -0.1853 rpy=0.0 0.0 0.0, axis 0 0 1, limit lower=-0.4141 upper=1.1 effort=840 velocity=5.89
- added joint leftKneePitch: type revolute, parent leftHipPitchLink, child leftKneePitchLink, origin xyz=0.000112225 0.0361046 -0.430959 rpy=0.0 0.0 0.0, axis 0 1 0, limit lower=-0.083 upper=2.057 effort=950 velocity=6.11
- added joint leftShoulderPitch: type revolute, parent torso, child leftShoulderPitchLink, origin xyz=-0.0316 0.0 0.2984 rpy=0.0 0.0 0.0, axis 0 1 0, limit lower=-2.85 upper=2.0 effort=190 velocity=5.89
- added joint leftShoulderRoll: type revolute, parent leftShoulderPitchLink, child leftShoulderRollLink, origin xyz=0.0 0.2499 0.0 rpy=0.0 0.0 0.0, axis 1 0 0, limit lower=-1.519 upper=1.266 effort=190 velocity=5.89
- added joint leftShoulderYaw: type revolute, parent leftShoulderRollLink, child leftShoulderYawLink, origin xyz=0.0 0.0 0.0 rpy=0.0 0.0 0.0, axis 0 1 0, limit lower=-3.1 upper=2.18 effort=65 velocity=11.5
- added joint leftWristPitch: type revolute, parent leftWristRollLink, child leftPalm, origin xyz=0.0 0.0 0.0 rpy=0.0 0.0 0.0, axis 0 0 1, limit lower=-0.36 upper=0.49 effort=14 velocity=1
- added joint leftWristRoll: type revolute, parent leftForearmLink, child leftWristRollLink, origin xyz=0.0 0.2871 0.0 rpy=0.0 0.0 0.0, axis 1 0 0, limit lower=-0.62 upper=0.625 effort=14 velocity=1
- added joint lowerNeckPitch: type revolute, parent torso, child lowerNeckPitchLink, origin xyz=0.0203518 0.0 0.33845 rpy=0.0 0.0 0.0, axis 0 1 0, limit lower=0 upper=1.162 effort=26 velocity=5
- added joint rightAnklePitch: type revolute, parent rightKneePitchLink, child rightAnklePitchLink, origin xyz=-0.0102381 0.0 -0.40627 rpy=0.0 0.0 0.0, axis 0 1 0, limit lower=-1.8644 upper=1.875 effort=805 velocity=11
- added joint rightAnkleRoll: type revolute, parent rightAnklePitchLink, child rightFoot, origin xyz=0.0 0.0 0.0 rpy=0.0 0.0 0.0, axis 1 0 0, limit lower=-1.349 upper=1.348 effort=805 velocity=11
- added joint rightElbowPitch: type revolute, parent rightShoulderYawLink, child rightElbowPitchLink, origin xyz=0.0254 -0.33 0.0 rpy=0.0 0.0 0.0, axis 0 0 1, limit lower=-0.12 upper=2.174 effort=65 velocity=11.5
- added joint rightForearmYaw: type revolute, parent rightElbowPitchLink, child rightForearmLink, origin xyz=-0.0254 0 0 rpy=0.0 0.0 0.0, axis 0 1 0, limit lower=-2.019 upper=3.14 effort=26 velocity=5
- added joint rightHipPitch: type revolute, parent rightHipRollLink, child rightHipPitchLink, origin xyz=0.0 0.0 -0.0609 rpy=0.0 0.0 0.0, axis 0 1 0, limit lower=-2.42 upper=1.619 effort=840 velocity=6.11
- added joint rightHipRoll: type revolute, parent rightHipYawLink, child rightHipRollLink, origin xyz=0.0 0.0 0.0 rpy=0.0 0.0 0.0, axis 1 0 0, limit lower=-0.5515 upper=0.467 effort=840 velocity=7
- added joint rightHipYaw: type revolute, parent pelvis, child rightHipYawLink, origin xyz=0.0 -0.1016 -0.1853 rpy=0.0 0.0 0.0, axis 0 0 1, limit lower=-1.1 upper=0.4141 effort=840 velocity=5.89
- added joint rightKneePitch: type revolute, parent rightHipPitchLink, child rightKneePitchLink, origin xyz=0.000112225 -0.0361046 -0.430959 rpy=0.0 0.0 0.0, axis 0 1 0, limit lower=-0.083 upper=2.057 effort=950 velocity=6.11
- added joint rightShoulderPitch: type revolute, parent torso, child rightShoulderPitchLink, origin xyz=-0.0316 0.0 0.2984 rpy=0.0 0.0 0.0, axis 0 1 0, limit lower=-2.85 upper=2.0 effort=190 velocity=5.89
- added joint rightShoulderRoll: type revolute, parent rightShoulderPitchLink, child rightShoulderRollLink, origin xyz=0.0 -0.2499 0.0 rpy=0.0 0.0 0.0, axis 1 0 0, limit lower=-1.266 upper=1.519 effort=190 velocity=5.89
- added joint rightShoulderYaw: type revolute, parent rightShoulderRollLink, child rightShoulderYawLink, origin xyz=0.0 0.0 0.0 rpy=0.0 0.0 0.0, axis 0 1 0, limit lower=-3.1 upper=2.18 effort=65 velocity=11.5
- added joint rightWristPitch: type revolute, parent rightWristRollLink, child rightPalm, origin xyz=0.0 0.0 0.0 rpy=0.0 0.0 0.0, axis 0 0 1, limit lower=-0.49 upper=0.36 effort=14 velocity=1
- added joint rightWristRoll: type revolute, parent rightForearmLink, child rightWristRollLink, origin xyz=0.0 -0.2871 0.0 rpy=0.0 0.0 0.0, axis 1 0 0, limit lower=-0.625 upper=0.62 effort=14 velocity=1
- added joint torsoPitch: type revolute, parent torsoYawLink, child torsoPitchLink, origin xyz=0.04191 0.0 0.0 rpy=0.0 0.0 0.0, axis 0 1 0, limit lower=-0.13 upper=0.666 effort=800 velocity=9
- added joint torsoRoll: type revolute, parent torsoPitchLink, child torso, origin xyz=0.0 0.0 0.0203 rpy=0.0 0.0 0.0, axis 1 0 0, limit lower=-0.23 upper=0.255 effort=800 velocity=9
- added joint torsoYaw: type revolute, parent pelvis, child torsoYawLink, origin xyz=0.0 0.0 0.0 rpy=0.0 0.0 0.0, axis 0 0 1, limit lower=-1.329 upper=1.181 effort=800 velocity=5.89
- joint l_hand_force_torque_joint: parent l_hand -> leftPalm
- joint leftCOP_Offset: parent l_foot -> leftFoot
- joint leftHazardCamera_Offset: parent utorso -> torso
- joint leftIndexFingerPitch1: parent l_hand -> leftPalm
- joint leftLegSixAxis_Offset: parent l_foot -> leftFoot
- joint leftMiddleFingerPitch1: parent l_hand -> leftPalm
- joint leftPinkyPitch1: parent l_hand -> leftPalm
- joint leftThumbRoll: parent l_hand -> leftPalm
- joint leftTorsoIMU_Offset: parent utorso -> torso
- joint r_hand_force_torque_joint: parent r_hand -> rightPalm
- joint rightCOP_Offset: parent r_foot -> rightFoot
- joint rightHazardCamera_Offset: parent utorso -> torso
- joint rightIndexFingerPitch1: parent r_hand -> rightPalm
- joint rightLegSixAxis_Offset: parent r_foot -> rightFoot
- joint rightMiddleFingerPitch1: parent r_hand -> rightPalm
- joint rightPinkyPitch1: parent r_hand -> rightPalm
- joint rightThumbRoll: parent r_hand -> rightPalm
- joint rightTorsoIMU_Offset: parent utorso -> torso

Commit message: resetting torque limits, walking still works fine

File: drake/examples/Valkyrie/urdf/urdf/valkyrie_A_sim_drake.urdf (robot description, URDF)
Before this commit: robot valkyrie, 87 links, 86 joints
Joints:
- joint leftAnklePitch: limit lower=-1.8644 upper=1.875 effort=805 velocity=11 -> lower=-1.8644 upper=1.875 effort=205 velocity=11
- joint leftAnkleRoll: limit lower=-1.349 upper=1.348 effort=805 velocity=11 -> lower=-1.349 upper=1.348 effort=205 velocity=11
- joint leftHipPitch: limit lower=-2.42 upper=1.619 effort=840 velocity=6.11 -> lower=-2.42 upper=1.619 effort=350 velocity=6.11
- joint leftHipRoll: limit lower=-0.467 upper=0.5515 effort=840 velocity=7 -> lower=-0.467 upper=0.5515 effort=350 velocity=7
- joint leftHipYaw: limit lower=-0.4141 upper=1.1 effort=840 velocity=5.89 -> lower=-0.4141 upper=1.1 effort=190 velocity=5.89
- joint leftKneePitch: limit lower=-0.083 upper=2.057 effort=950 velocity=6.11 -> lower=-0.083 upper=2.057 effort=350 velocity=6.11
- joint rightAnklePitch: limit lower=-1.8644 upper=1.875 effort=805 velocity=11 -> lower=-1.8644 upper=1.875 effort=205 velocity=11
- joint rightAnkleRoll: limit lower=-1.349 upper=1.348 effort=805 velocity=11 -> lower=-1.349 upper=1.348 effort=205 velocity=11
- joint rightHipPitch: limit lower=-2.42 upper=1.619 effort=840 velocity=6.11 -> lower=-2.42 upper=1.619 effort=350 velocity=6.11
- joint rightHipRoll: limit lower=-0.5515 upper=0.467 effort=840 velocity=7 -> lower=-0.5515 upper=0.467 effort=350 velocity=7
- joint rightHipYaw: limit lower=-1.1 upper=0.4141 effort=840 velocity=5.89 -> lower=-1.1 upper=0.4141 effort=190 velocity=5.89
- joint rightKneePitch: limit lower=-0.083 upper=2.057 effort=950 velocity=6.11 -> lower=-0.083 upper=2.057 effort=350 velocity=6.11
- joint torsoPitch: limit lower=-0.13 upper=0.666 effort=800 velocity=9 -> lower=-0.13 upper=0.666 effort=150 velocity=9
- joint torsoRoll: limit lower=-0.23 upper=0.255 effort=800 velocity=9 -> lower=-0.23 upper=0.255 effort=150 velocity=9
- joint torsoYaw: limit lower=-1.329 upper=1.181 effort=800 velocity=5.89 -> lower=-1.329 upper=1.181 effort=190 velocity=5.89
