Commit message: Creates obj with texture
Adding a .obj that has the texture file reference in it.
Prius_ackerman1.urdf now calls the prius.obj file instead of the .dae

File: drake/examples/Cars/prius/prius_ackerman1.urdf (robot description, URDF)
Before this commit: robot car, 17 links, 16 joints
Links:
- link body: geometry visual mesh filename=prius.obj scale=1
