Commit message: Changes to prius_ackerman.urdf
Changes the alpha channels to 1 for visual geometries.
Mesh used is an .obj which includes texture info.

File: drake/examples/Cars/prius/prius_ackerman.urdf (robot description, URDF)
Before this commit: robot car, 17 links, 16 joints
Links:
- link body: geometry visual mesh filename=prius.stl scale=1
Joints:
- joint body: origin xyz=.97 -.92 0 -> xyz=0 0 0
