Commit message: adds prius with textures

File: drake/examples/Cars/prius/prius.urdf (robot description, URDF)
Before this commit: robot car, 17 links, 16 joints
Links:
- link body: geometry visual mesh filename=prius.dae scale=1

Commit message: convert prius.urdf to use package syntax for the mesh filename
This also adds an empty package.xml so that the prius directory looks
like a package according to rospack.

File: drake/examples/Cars/prius/prius.urdf (robot description, URDF)
Before this commit: robot car, 17 links, 16 joints
Links:
- link body: geometry visual mesh filename=package://prius/prius.dae scale=1

Commit message: convert prius.urdf to use package syntax for the mesh filename
This also adds an empty package.xml so that the prius directory looks
like a package according to rospack.

File: drake/examples/Cars/prius/prius.urdf (robot description, URDF)
Before this commit: robot prius_1, 13 links, 12 joints
Links:
- link body: geometry visual mesh filename=package://prius.dae scale=1.0 1.0 1.0

Commit message: update names in prius.urdf

File: drake/examples/Cars/prius/prius.urdf (robot description, URDF)
Before this commit: robot car, 17 links, 16 joints
Links:
- removed link front_left_contact_point
- removed link front_right_contact_point
- removed link rear_left_contact_point
- removed link rear_right_contact_point
- added link front_left_wheel_center; visual sphere radius=.01
- added link front_right_wheel_center; visual sphere radius=.01
- added link rear_left_wheel_center; visual sphere radius=.01
- added link rear_right_wheel_center; visual sphere radius=.01
Joints:
- removed joint front_left_contact_sliding
- removed joint front_right_contact_sliding
- removed joint rear_left_contact_sliding
- removed joint rear_right_contact_sliding
- added joint front_left_suspension: type prismatic, parent left_hub, child front_left_wheel_center, origin xyz=0 .801993 0, axis 0 0 1, limit lower=0 upper=.323342
- added joint front_right_suspension: type prismatic, parent right_hub, child front_right_wheel_center, origin xyz=0 -0.801993 0, axis 0 0 1, limit lower=0 upper=.323342
- added joint rear_left_suspension: type prismatic, parent rear_axle, child rear_left_wheel_center, origin xyz=-1.409480 .801993 -0.323342, axis 0 0 1, limit lower=0 upper=0.34925
- added joint rear_right_suspension: type prismatic, parent rear_axle, child rear_right_wheel_center, origin xyz=-1.409480 -0.801993 -0.323342, axis 0 0 1, limit lower=0 upper=0.34925
- joint left_wheel_joint: parent front_left_contact_point -> front_left_wheel_center
- joint rear_left_wheel_joint: parent rear_left_contact_point -> rear_left_wheel_center
- joint rear_right_wheel_joint: parent rear_right_contact_point -> rear_right_wheel_center
- joint right_wheel_joint: parent front_right_contact_point -> front_right_wheel_center

Commit message: Removed slash in front of prius.dae mesh name. Tested to work on OSX.

File: drake/examples/Cars/prius/prius.urdf (robot description, URDF)
Before this commit: robot prius_1, 13 links, 12 joints
Links:
- link body: geometry visual mesh filename=prius.dae scale=1.0 1.0 1.0
