Commit message: convert prius.urdf to use package syntax for the mesh filename
This ensures that we have an example that tests drake support
for the package:// syntax for resource urls.

File: drake/examples/Cars/models/prius/prius.urdf (robot description, URDF)
Before this commit: robot prius_1, 13 links, 12 joints
Links:
- link body: geometry visual mesh filename=package://drake/examples/Cars/models/prius/prius.dae scale=1.0 1.0 1.0

Commit message: Modified Prius steering geometry to achieve a smaller turning radius.

File: drake/examples/Cars/models/prius/prius.urdf (robot description, URDF)
Before this commit: robot prius_1, 13 links, 12 joints
Links:
- link tie_rod: geometry visual box size=0.061842 0.91 0.030921
Joints:
- joint axle_tie_rod_arm: limit lower=-0.401426 upper=0.5 effort=0.0 velocity=0.0 -> lower=-0.7 upper=0.7 effort=0.0 velocity=0.0
- joint steering: limit lower=-0.401426 upper=0.5 effort=0.0 velocity=0.0 -> lower=-0.7 upper=0.7 effort=0.0 velocity=0.0

File: drake/examples/Cars/ros_packages/drake_cars_examples/models/drake_prius/xacro/drake_prius_base.xacro (robot description, xacro)
@@ -43,6 +43,7 @@
       <inertia ixx="0" ixy="0" ixz="0" iyy="0" iyz="0" izz="0"/>
     </inertial> -->
-    <visual name="__v2">
-      <origin rpy="0 0 0.46364" xyz="-0.1086 -0.0543 0"/>
+    <visual name="side_of_L">
+      <origin rpy="0 0 0.17012086" xyz="-0.1086 -0.0543 0"/>
+      <!-- <origin rpy="0 0 0.46364" xyz="-0.1086 -0.0543 0"/> -->
       <geometry>
         <box size="0.204637 0.061842 0.030921"/>
@@ -52,6 +53,6 @@
       </material>
     </visual>
-    <visual name="__v1">
-      <origin rpy="0 0 0" xyz="0 0.02228  0"/>
+    <visual name="bottom_of_L">
+      <origin rpy="0  0  0" xyz="0       0.02228  0"/>
       <geometry>
         <box size="0.061842 0.140955 0.030921"/>
@@ -87,5 +88,6 @@
       <origin rpy="0 0 0" xyz="0 -0.4085 0"/>
       <geometry>
-        <box size="0.061842 0.878847 0.030921"/>
+        <box size="0.061842 0.91 0.030921"/>
+        <!-- <box size="0.061842 0.878847 0.030921"/> -->
       </geometry>
       <material name="blue">
@@ -140,5 +142,5 @@
       <inertia ixx="0" ixy="0" ixz="0" iyy="0" iyz="0" izz="0"/>
     </inertial> -->
-    <visual name="v1">
+    <visual name="bottom_of_L">
       <origin rpy="0 0 0" xyz="0 -0.02228 0"/>
       <geometry>
@@ -149,6 +151,7 @@
       </material>
     </visual>
-    <visual name="v2">
-      <origin rpy="0 0 -0.46364" xyz="-0.1086 0.0543 0"/>
+    <visual name="side_of_L">
+      <origin rpy="0 0 -0.17012086" xyz="-0.1086 0.0543 0"/>
+      <!-- <origin rpy="0 0 -0.46364" xyz="-0.1086 0.0543 0"/> -->
       <geometry>
         <box size="0.204637 0.061842 0.030921"/>
@@ -333,5 +336,5 @@
     <origin rpy="0 0 0" xyz="0 0.49473 -0.03092"/>
     <axis xyz="0 0 1"/>
-    <limit effort="0.0" lower="-0.401426" upper="0.5" velocity="0.0"/>
+    <limit effort="0.0" lower="-0.7" upper="0.7" velocity="0.0"/>
   </joint>
   <joint name="left_hub" type="fixed">
@@ -361,5 +364,5 @@
     <origin rpy="0 0 0" xyz="0 -0.49473 -0.03092"/>
     <axis xyz="0 0 1"/>
-    <limit effort="0.0" lower="-0.401426" upper="0.5" velocity="0.0"/>
+    <limit effort="0.0" lower="-0.7" upper="0.7" velocity="0.0"/>
   </joint>
   <joint name="right_hub" type="fixed">
