Commit message: Added golfcart_tf_pubisher. Modified prius models by changing name of "body" link to be "chassis".

File: drake/examples/Cars/drake_catkin_workspace/src/drake_cars_examples/models/drake_prius/xacro/drake_prius_base.xacro (robot description, xacro)
@@ -311,5 +311,5 @@
     </visual>
   </link>
-  <link name="body">
+  <link name="chassis">
     <inertial>
       <mass value="5.42794"/>
@@ -401,7 +401,7 @@
     <limit effort="10000" velocity="10000"/>
   </joint>
-  <joint name="body" type="fixed">
+  <joint name="chassis" type="fixed">
     <parent link="chassis_floor"/>
-    <child link="body"/>
+    <child link="chassis"/>
     <origin rpy="0  0  0" xyz="0 0 0.006857999999999975226927518"/>
     <axis xyz="0  0  0"/>

File: drake/examples/Cars/models/prius/prius.urdf (robot description, URDF)
Before this commit: robot prius_1, 13 links, 12 joints
Links:
- removed link body
- added link chassis, mass 5.42794; visual mesh filename=prius.dae scale=1.0 1.0 1.0
Joints:
- removed joint body
- added joint chassis: type fixed, parent chassis_floor, child chassis, origin xyz=0 0 0.006857999999999975226927518 rpy=0  0  0, axis 0  0  0, limit lower=0 upper=0 effort=0 velocity=0
