Commit message: remove mesh ref from urdf

File: drake/examples/QPInverseDynamicsForHumanoids/valkyrie_sim_drake.urdf (robot description, URDF)
Before this commit: robot valkyrie, 84 links, 83 joints
Links:
- link hokuyo_link: geometry collision box size=0.08 0.06 0.04238; collision cylinder length=0.047 radius=0.024425
- link leftAnklePitchLink: geometry 
- link leftElbowPitchLink: geometry 
- link leftFoot: geometry collision box size=0.27 0.16 0.064; collision sphere radius=0.0
- link leftForearmLink: geometry 
- link leftHipPitchLink: geometry 
- link leftHipRollLink: geometry 
- link leftHipYawLink: geometry 
- link leftIndexFingerPitch1Link: geometry 
- link leftIndexFingerPitch2Link: geometry 
- link leftIndexFingerPitch3Link: geometry 
- link leftKneePitchLink: geometry 
- link leftMiddleFingerPitch1Link: geometry 
- link leftMiddleFingerPitch2Link: geometry 
- link leftMiddleFingerPitch3Link: geometry 
- link leftPalm: geometry 
- link leftPinkyPitch1Link: geometry 
- link leftPinkyPitch2Link: geometry 
- link leftPinkyPitch3Link: geometry 
- link leftShoulderPitchLink: geometry 
- link leftShoulderRollLink: geometry 
- link leftShoulderYawLink: geometry 
- link leftThumbPitch1Link: geometry 
- link leftThumbPitch2Link: geometry 
- link leftThumbPitch3Link: geometry 
- link leftThumbRollLink: geometry 
- link leftWristRollLink: geometry 
- link lowerNeckPitchLink: geometry 
- link neckYawLink: geometry 
- link pelvis: geometry 
- link rightAnklePitchLink: geometry 
- link rightElbowPitchLink: geometry 
- link rightFoot: geometry collision box size=0.27 0.16 0.064; collision sphere radius=0.0
- link rightForearmLink: geometry 
- link rightHipPitchLink: geometry 
- link rightHipRollLink: geometry 
- link rightHipYawLink: geometry 
- link rightIndexFingerPitch1Link: geometry 
- link rightIndexFingerPitch2Link: geometry 
- link rightIndexFingerPitch3Link: geometry 
- link rightKneePitchLink: geometry 
- link rightMiddleFingerPitch1Link: geometry 
- link rightMiddleFingerPitch2Link: geometry 
- link rightMiddleFingerPitch3Link: geometry 
- link rightPalm: geometry 
- link rightPinkyPitch1Link: geometry 
- link rightPinkyPitch2Link: geometry 
- link rightPinkyPitch3Link: geometry 
- link rightShoulderPitchLink: geometry 
- link rightShoulderRollLink: geometry 
- link rightShoulderYawLink: geometry 
- link rightThumbPitch1Link: geometry 
- link rightThumbPitch2Link: geometry 
- link rightThumbPitch3Link: geometry 
- link rightThumbRollLink: geometry 
- link rightWristRollLink: geometry 
- link torso: geometry 
- link torsoPitchLink: geometry 
- link torsoYawLink: geometry 
- link upperNeckPitchLink: geometry 
