Commit message: Added publishing of transform from world to world_link in multi_cars_on_plane simulation.

File: ros/drake_cars_examples/models/planar_world.xacro (robot description, xacro)
@@ -15,4 +15,7 @@
         <box size="500.0 500.0 2.0" />
       </geometry>
+        <material name="gray">
+          <color rgba="0.2 0.2 0.2 1" />
+        </material>
     </visual>
   </link>
