Commit message: Multi-model simulation and DrakeRosTfPublisher works!

File: ros/drake_cars_examples/models/drake_prius/xacro/drake_prius_free_in_world_2.xacro (robot description, xacro)
@@ -3,6 +3,6 @@
   <property name="world_pitch" value="0" />
   <property name="world_yaw" value="0" />
-  <property name="world_x" value="1" />
-  <property name="world_y" value="1" />
+  <property name="world_x" value="5" />
+  <property name="world_y" value="5" />
   <property name="world_z" value="1.2" />
   <xacro:include

File: ros/drake_cars_examples/models/drake_prius/xacro/drake_prius_free_in_world_3.xacro (robot description, xacro)
@@ -3,6 +3,6 @@
   <property name="world_pitch" value="0" />
   <property name="world_yaw" value="0" />
-  <property name="world_x" value="-1" />
-  <property name="world_y" value="1" />
+  <property name="world_x" value="-5" />
+  <property name="world_y" value="5" />
   <property name="world_z" value="1.2" />
   <xacro:include

File: ros/drake_cars_examples/models/drake_prius/xacro/drake_prius_free_in_world_4.xacro (robot description, xacro)
@@ -3,7 +3,7 @@
   <property name="world_pitch" value="0" />
   <property name="world_yaw" value="0" />
-  <property name="world_x" value="-1" />
-  <property name="world_y" value="-1" />
-  <property name="world_z" value="1.2" />
+  <property name="world_x" value="-5" />
+  <property name="world_y" value="-5" />
+  <property name="world_z" value="1.2"/>
   <xacro:include
       filename="$(find drake_cars_examples)/models/drake_prius/xacro/drake_prius_free_in_world_base.xacro" />

File: ros/drake_cars_examples/models/drake_prius/xacro/drake_prius_free_in_world_5.xacro (robot description, xacro)
@@ -3,6 +3,6 @@
   <property name="world_pitch" value="0" />
   <property name="world_yaw" value="0" />
-  <property name="world_x" value="1" />
-  <property name="world_y" value="-1" />
+  <property name="world_x" value="5" />
+  <property name="world_y" value="-5" />
   <property name="world_z" value="1.2" />
   <xacro:include

File: ros/drake_cars_examples/models/drake_prius/xacro/drake_prius_free_in_world_base.xacro (robot description, xacro)
@@ -8,5 +8,5 @@
     <inertial>
       <mass value="0" />
-      <origin rpy="${world_roll} ${world_pitch} ${world_yaw}"
+      <origin rpy="0 0 0"
               xyz="${world_x} ${world_y} ${world_z}" />
       <inertia ixx="0" ixy="0" ixz="0" iyy="0" iyz="0" izz="0" />
@@ -14,5 +14,6 @@
   </link>
   <joint name="virtual_floating_dofs" type="floating">
-    <origin rpy="0 0 0" xyz="0 0 0" />
+    <origin rpy="${world_roll} ${world_pitch} ${world_yaw}"
+            xyz="${world_x} ${world_y} ${world_z}" />
     <axis xyz="0 0 1" />
     <parent link="world" />

File: ros/drake_cars_examples/models/planar_world.xacro (robot description, xacro)
@@ -1,4 +1,4 @@
 <robot xmlns:xacro="http://www.ros.org/wiki/xacro" name="planar_world" >
-  <link name="world_link">
+  <link name="ground_plane">
     <!--
     Inertia data is arbitrary. Its purpose here is to evade the
@@ -11,12 +11,18 @@
     </inertial> -->
     <visual>
-      <origin xyz="0 0 -1.0" rpy="0 0 0" />
+      <origin xyz="0 0 -1" rpy="0 0 0" />
       <geometry>
-        <box size="500.0 500.0 2.0" />
+        <box size="40.0 40.0 2.0" />
       </geometry>
-        <material name="gray">
-          <color rgba="0.2 0.2 0.2 1" />
-        </material>
+      <material name="gray">
+        <color rgba="0.5 0.5 0.5 1" />
+      </material>
     </visual>
+    <collision name="world_link_collision">
+      <origin xyz="0 0 -1" rpy="0 0 0" />
+      <geometry>
+        <box size="40.0 40.0 2.0" />
+      </geometry>
+    </collision>
   </link>
 </robot>
