Commit message: format change

File: drake/examples/MechanicalTransmission/mechanical_transmission.urdf (robot description, URDF)
Before this commit: robot MechanicalTransmission, 3 links, 2 joints
Joints:
- joint joint1: mimic joint=joint2 multiplier=0.5 -> joint=joint2 multiplier=0.5 offset=1.0

Commit message: address Liang's comment

File: drake/examples/MechanicalTransmission/mechanical_transmission.urdf (robot description, URDF)
Before this commit: robot MechanicalTransmission, 3 links, 2 joints
Joints:
- joint joint2: parent base_link -> link1
