Commit message: updated valkyrie model files

File: drake/examples/Valkyrie_PT/val_description/other_urdf/valkyrie_sim_drake_simple.urdf (robot description, URDF)
Before this commit: robot valkyrie, 84 links, 83 joints
Links:
- removed link leftTorsoImu_Frame
- removed link pelvisMiddleImu_Frame
- removed link pelvisRearImu_Frame
- added link leftLegSixAxis_Frame, mass 1e-07
- added link leftPelvisIMU_Frame, mass 1e-07
- added link leftTorsoIMU_Frame, mass 1e-07
- added link rightLegSixAxis_Frame, mass 1e-07
- added link rightPelvisIMU_Frame, mass 1e-07
- added link rightTorsoIMU_Frame, mass 1e-07
- link head: geometry 
- link head_imu_link: geometry 
- link hokuyo_link: geometry 
- link l_hand_force_torque: geometry 
- link leftAnklePitchLink: mass 0.03 -> 0.06; geometry 
- link leftElbowPitchLink: geometry collision cylinder length=0.141 radius=0.061; visual cylinder length=0.141 radius=0.061
- link leftFoot: mass 2.27 -> 3.255; geometry collision box size=0.27 0.16 0.064; collision sphere radius=0.0
- link leftForearmLink: geometry collision cylinder length=0.22 radius=0.06; visual cylinder length=0.22 radius=0.06
- link leftHipPitchLink: geometry collision box size=0.22 0.08 0.254; collision box size=0.22 0.22 0.29
- link leftHipRollLink: geometry 
- link leftHipYawLink: geometry collision sphere radius=0.14; visual sphere radius=0.14
- link leftIndexFingerPitch1Link: geometry collision box size=0.015 0.04 0.025; visual box size=0.015 0.04 0.025
- link leftIndexFingerPitch2Link: geometry collision box size=0.015 0.03 0.020; visual box size=0.015 0.03 0.020
- link leftIndexFingerPitch3Link: geometry collision box size=0.015 0.022 0.017; visual box size=0.015 0.022 0.017
- link leftKneePitchLink: mass 6.2 -> 6.6; geometry collision box size=0.185 0.18 0.38; visual box size=0.185 0.18 0.38
- link leftMiddleFingerPitch1Link: geometry collision box size=0.015 0.04 0.025; visual box size=0.015 0.04 0.025
- link leftMiddleFingerPitch2Link: geometry collision box size=0.015 0.03 0.020; visual box size=0.015 0.03 0.020
- link leftMiddleFingerPitch3Link: geometry collision box size=0.015 0.022 0.017; visual box size=0.015 0.022 0.017
- link leftPalm: geometry collision box size=0.025 0.07 0.1; collision box size=0.03 0.12 0.1
- link leftPinkyPitch1Link: geometry collision box size=0.015 0.04 0.025; visual box size=0.015 0.04 0.025
- link leftPinkyPitch2Link: geometry collision box size=0.015 0.03 0.020; visual box size=0.015 0.03 0.020
- link leftPinkyPitch3Link: geometry collision box size=0.015 0.022 0.017; visual box size=0.015 0.022 0.017
- link leftShoulderPitchLink: geometry collision cylinder length=0.2 radius=0.08; visual cylinder length=0.2 radius=0.08
- link leftShoulderRollLink: geometry collision cylinder length=0.12 radius=0.075; visual cylinder length=0.12 radius=0.075
- link leftShoulderYawLink: geometry collision cylinder length=0.20 radius=0.075; visual cylinder length=0.20 radius=0.075
- link leftThumbPitch1Link: geometry collision box size=0.025 0.015 0.04; visual box size=0.025 0.015 0.04
- link leftThumbPitch2Link: geometry collision box size=0.020 0.015 0.03; visual box size=0.020 0.015 0.03
- link leftThumbPitch3Link: geometry collision box size=0.017 0.015 0.022; visual box size=0.017 0.015 0.022
- link leftThumbRollLink: geometry 
- link leftWristRollLink: geometry 
- link left_palm: geometry 
- link lowerNeckPitchLink: geometry 
- link neckYawLink: geometry 
- link pelvis: geometry collision cylinder length=0.18 radius=0.18; collision sphere radius=0.18
- link r_hand_force_torque: geometry 
- link rightAnklePitchLink: mass 0.03 -> 0.06; geometry 
- link rightElbowPitchLink: geometry collision cylinder length=0.141 radius=0.061; visual cylinder length=0.141 radius=0.061
- link rightFoot: mass 2.27 -> 3.255; geometry collision box size=0.27 0.16 0.064; collision sphere radius=0.0
- link rightForearmLink: geometry collision cylinder length=0.22 radius=0.06; visual cylinder length=0.22 radius=0.06
- link rightHipPitchLink: geometry collision box size=0.22 0.08 0.254; collision box size=0.22 0.22 0.29
- link rightHipRollLink: geometry 
- link rightHipYawLink: geometry collision sphere radius=0.14; visual sphere radius=0.14
- link rightIndexFingerPitch1Link: geometry collision box size=0.015 0.04 0.025; visual box size=0.015 0.04 0.025
- link rightIndexFingerPitch2Link: geometry collision box size=0.015 0.03 0.020; visual box size=0.015 0.03 0.020
- link rightIndexFingerPitch3Link: geometry collision box size=0.015 0.022 0.017; visual box size=0.015 0.022 0.017
- link rightKneePitchLink: mass 6.2 -> 6.6; geometry collision box size=0.185 0.18 0.38; visual box size=0.185 0.18 0.38
- link rightMiddleFingerPitch1Link: geometry collision box size=0.015 0.04 0.025; visual box size=0.015 0.04 0.025
- link rightMiddleFingerPitch2Link: geometry collision box size=0.015 0.03 0.020; visual box size=0.015 0.03 0.020
- link rightMiddleFingerPitch3Link: geometry collision box size=0.015 0.022 0.017; visual box size=0.015 0.022 0.017
- link rightPalm: geometry collision box size=0.025 0.07 0.1; collision box size=0.03 0.12 0.1
- link rightPinkyPitch1Link: geometry collision box size=0.015 0.04 0.025; visual box size=0.015 0.04 0.025
- link rightPinkyPitch2Link: geometry collision box size=0.015 0.03 0.020; visual box size=0.015 0.03 0.020
- link rightPinkyPitch3Link: geometry collision box size=0.015 0.022 0.017; visual box size=0.015 0.022 0.017
- link rightShoulderPitchLink: geometry collision cylinder length=0.2 radius=0.08; visual cylinder length=0.2 radius=0.08
- link rightShoulderRollLink: geometry collision cylinder length=0.12 radius=0.075; visual cylinder length=0.12 radius=0.075
- link rightShoulderYawLink: geometry collision cylinder length=0.20 radius=0.075; visual cylinder length=0.20 radius=0.075
- link rightThumbPitch1Link: geometry collision box size=0.025 0.015 0.04; visual box size=0.025 0.015 0.04
- link rightThumbPitch2Link: geometry collision box size=0.020 0.015 0.03; visual box size=0.020 0.015 0.03
- link rightThumbPitch3Link: geometry collision box size=0.017 0.015 0.022; visual box size=0.017 0.015 0.022
- link rightThumbRollLink: geometry 
- link rightWristRollLink: geometry 
- link right_palm: geometry 
- link torso: geometry collision box size=0.25 0.36 0.42; collision cylinder length=0.3 radius=0.15
- link torsoPitchLink: geometry 
- link torsoYawLink: geometry 
- link upperNeckPitchLink: mass 3.89 -> 4.59; geometry collision sphere radius=0.15; visual sphere radius=0.15
Joints:
- removed joint leftTorsoImu_Offset
- removed joint pelvisMiddleImu_Offset
- removed joint pelvisRearImu_Offset
- added joint leftLegSixAxis_Offset: type fixed, parent leftFoot, child leftLegSixAxis_Frame, origin xyz=0.0215646 0.0 -0.051054 rpy=3.14 0.0 -1.047, axis 0 0 1
- added joint leftPelvisIMU_Offset: type fixed, parent pelvis, child leftPelvisIMU_Frame, origin xyz=0.0515 0.115 -0.042 rpy=1.57 0 -1.274, axis 0 0 1
- added joint leftTorsoIMU_Offset: type fixed, parent torso, child leftTorsoIMU_Frame, origin xyz=-0.047 0.134 0.363 rpy=1.57 0.0 3.14, axis 0 0 1
- added joint rightLegSixAxis_Offset: type fixed, parent rightFoot, child rightLegSixAxis_Frame, origin xyz=0.0215646 0.0 -0.051054 rpy=3.14 0.0 -1.047, axis 0 0 1
- added joint rightPelvisIMU_Offset: type fixed, parent pelvis, child rightPelvisIMU_Frame, origin xyz=0.0515 -0.115 -0.042 rpy=-1.57 0.0 1.274, axis 0 0 1
- added joint rightTorsoIMU_Offset: type fixed, parent torso, child rightTorsoIMU_Frame, origin xyz=-0.047 -0.134 0.363 rpy=-1.57 0.0 3.14, axis 0 0 1
- joint hokuyo_joint: type continuous -> fixed
- joint l_hand_face_joint: origin xyz=0.06 0.0 -0.045 rpy=3.14159265359 0 1.57079632679 -> xyz=0.07 0.0 -0.08 rpy=3.14159265359 0 1.57079632679
- joint leftCOP_Offset: origin xyz=0.0189 0.0 -0.0783 rpy=0.0 0.0 0.0 -> xyz=0.0189 0.0 -0.0783 rpy=0.0 0.13 0.0
- joint leftIndexFingerPitch1: limit lower=-1.57 upper=-0.0 effort=10 velocity=1 -> (none); type revolute -> fixed
- joint leftIndexFingerPitch2: limit lower=-1.658 upper=-0.0 effort=10 velocity=1 -> (none); type revolute -> fixed
- joint leftIndexFingerPitch3: limit lower=-1.92 upper=-0.0 effort=10 velocity=1 -> (none); type revolute -> fixed
- joint leftMiddleFingerPitch1: limit lower=-1.658 upper=-0.0 effort=10 velocity=1 -> (none); type revolute -> fixed
- joint leftMiddleFingerPitch2: limit lower=-1.92 upper=-0.0 effort=10 velocity=1 -> (none); type revolute -> fixed
- joint leftMiddleFingerPitch3: limit lower=-1.57 upper=-0.0 effort=10 velocity=1 -> (none); type revolute -> fixed
- joint leftPinkyPitch1: limit lower=-1.57 upper=-0.0 effort=10 velocity=1 -> (none); type revolute -> fixed
- joint leftPinkyPitch2: limit lower=-1.658 upper=-0.0 effort=10 velocity=1 -> (none); type revolute -> fixed
- joint leftPinkyPitch3: limit lower=-1.92 upper=-0.0 effort=10 velocity=1 -> (none); type revolute -> fixed
- joint leftThumbPitch1: axis 1 0 0 -> 0 0 1; limit lower=-1.658 upper=-0.0 effort=10 velocity=1 -> (none); type revolute -> fixed
- joint leftThumbPitch2: axis 1 0 0 -> 0 0 1; limit lower=-1.92 upper=-0.0 effort=10 velocity=1 -> (none); type revolute -> fixed
- joint leftThumbPitch3: axis 1 0 0 -> 0 0 1; limit lower=-1.57 upper=-0.0 effort=10 velocity=1 -> (none); type revolute -> fixed
- joint leftThumbRoll: axis 0 1 0 -> 0 0 1; limit lower=0.0 upper=2.356 effort=10 velocity=1 -> (none); type revolute -> fixed
- joint r_hand_face_joint: origin xyz=0.06 0 0.045 rpy=0 0 -1.57079632679 -> xyz=0.07 0 0.08 rpy=0 0 -1.57079632679
- joint rightCOP_Offset: origin xyz=0.0189 0.0 -0.0783 rpy=0.0 0.0 0.0 -> xyz=0.0189 0.0 -0.0783 rpy=0.0 0.13 0.0
- joint rightIndexFingerPitch1: limit lower=0.0 upper=1.57 effort=10 velocity=1 -> (none); type revolute -> fixed
- joint rightIndexFingerPitch2: limit lower=0.0 upper=1.658 effort=10 velocity=1 -> (none); type revolute -> fixed
- joint rightIndexFingerPitch3: limit lower=0.0 upper=1.92 effort=10 velocity=1 -> (none); type revolute -> fixed
- joint rightMiddleFingerPitch1: limit lower=0.0 upper=1.658 effort=10 velocity=1 -> (none); type revolute -> fixed
- joint rightMiddleFingerPitch2: limit lower=0.0 upper=1.92 effort=10 velocity=1 -> (none); type revolute -> fixed
- joint rightMiddleFingerPitch3: limit lower=0.0 upper=1.57 effort=10 velocity=1 -> (none); type revolute -> fixed
- joint rightPinkyPitch1: limit lower=0.0 upper=1.57 effort=10 velocity=1 -> (none); type revolute -> fixed
- joint rightPinkyPitch2: limit lower=0.0 upper=1.658 effort=10 velocity=1 -> (none); type revolute -> fixed
- joint rightPinkyPitch3: limit lower=0.0 upper=1.92 effort=10 velocity=1 -> (none); type revolute -> fixed
- joint rightThumbPitch1: axis 1 0 0 -> 0 0 1; limit lower=0.0 upper=1.658 effort=10 velocity=1 -> (none); type revolute -> fixed
- joint rightThumbPitch2: axis 1 0 0 -> 0 0 1; limit lower=0.0 upper=1.92 effort=10 velocity=1 -> (none); type revolute -> fixed
- joint rightThumbPitch3: axis 1 0 0 -> 0 0 1; limit lower=0.0 upper=1.57 effort=10 velocity=1 -> (none); type revolute -> fixed
- joint rightThumbRoll: axis 0 1 0 -> 0 0 1; limit lower=0.0 upper=2.356 effort=10 velocity=1 -> (none); type revolute -> fixed
