Commit message: stuff works

File: drake/examples/kuka_iiwa_arm/models/objects/simple_cuboid.urdf (robot description, URDF)
Before this commit: robot simple_cuboid, 1 links, 0 joints
Links:
- link base_link: mass 1 -> 0.5; geometry collision box size=0.1 0.2 0.3; visual box size=0.1 0.2 0.3

File: drake/examples/kuka_iiwa_arm/models/objects/simple_cylinder.urdf (robot description, URDF)
Before this commit: robot simple_cylinder, 1 links, 0 joints
Links:
- link base_link: mass 1 -> 0.25
