Commit message: New models added

File: drake/examples/kuka_iiwa_arm/models/objects/block_for_pick_and_place_large_size.urdf (robot description, URDF)
Before this commit: robot simple_cuboid, 1 links, 0 joints
Links:
- link base_link: geometry collision box size=0.059 0.119 0.199; collision sphere radius=1e-7

File: drake/examples/kuka_iiwa_arm/models/objects/block_for_pick_and_place_mid_size.urdf (robot description, URDF)
Before this commit: robot simple_cuboid, 1 links, 0 joints
Links:
- link base_link: geometry collision box size=0.059 0.089 0.199; collision sphere radius=1e-7

Commit message: review comments addressed

File: drake/examples/kuka_iiwa_arm/models/objects/block_for_pick_and_place_large_size.urdf (robot description, URDF)
Before this commit: robot simple_cuboid, 1 links, 0 joints
Links:
- link base_link: geometry collision box size=0.059 0.119 0.199; collision sphere radius=1e-7
