Commit message: change name of base link and joint in iiwa urdf file
By convention, director wants the base joint to be named 'base'.
In the future we could add code to director to support arbitrary names.

File: drake/examples/kuka_iiwa_arm/urdf/iiwa14_no_collision.urdf (robot description, URDF)
Before this commit: robot iiwa14, 11 links, 10 joints
Links:
- removed link world
- added link base
Joints:
- removed joint world_iiwa_joint
- added joint base_joint: type fixed, parent world, child iiwa_link_0, origin xyz=0 0 0.0 rpy=0 0 0

Commit message: fix parent link in kuka urdf

File: drake/examples/kuka_iiwa_arm/urdf/iiwa14_no_collision.urdf (robot description, URDF)
Before this commit: robot iiwa14, 11 links, 10 joints
Joints:
- joint base_joint: parent world -> base

Commit message: simplified polytope mesh for link 7

File: drake/examples/kuka_iiwa_arm/urdf/iiwa14_no_collision.urdf (robot description, URDF)
Before this commit: robot iiwa14, 11 links, 10 joints
Links:
- link iiwa_link_7: geometry collision mesh filename=meshes/collision/link_7_polytope.obj; visual mesh filename=meshes/visual/link_7_polytope.obj

Commit message: review comments addressed

File: drake/examples/kuka_iiwa_arm/urdf/iiwa14_no_collision.urdf (robot description, URDF)
Before this commit: robot iiwa14, 11 links, 10 joints
Links:
- link iiwa_link_7: geometry collision mesh filename=meshes/collision/link_7_polytope.obj; visual mesh filename=meshes/visual/link_7.obj
