Commit message: review comments addressed

File: drake/examples/kuka_iiwa_arm/urdf/iiwa14_simplified_collision.urdf (robot description, URDF)
Before this commit: robot iiwa14, 11 links, 10 joints
Links:
- link iiwa_link_0: geometry visual mesh filename=meshes/visual/link_0.obj
- link iiwa_link_1: geometry visual mesh filename=meshes/visual/link_1.obj
- link iiwa_link_2: geometry visual mesh filename=meshes/visual/link_2.obj
- link iiwa_link_3: geometry visual mesh filename=meshes/visual/link_3.obj
- link iiwa_link_4: geometry visual mesh filename=meshes/visual/link_4.obj
- link iiwa_link_5: geometry visual mesh filename=meshes/visual/link_5.obj
- link iiwa_link_6: geometry visual mesh filename=meshes/visual/link_6.obj
- link iiwa_link_7: geometry collision mesh filename=meshes/collision/link_7_polytope.obj; visual mesh filename=meshes/visual/link_7.obj
