Commit message: Updated KUKA IIWA arm demo with C++ test.

File: drake/examples/kuka_iiwa_arm/urdf/iiwa14.urdf (robot description, URDF)
Before this commit: robot iiwa14, 11 links, 10 joints
Links:
- link iiwa_link_0: geometry collision mesh filename=meshes/collision/link_0.obj; visual mesh filename=meshes/visual/link_0.obj
- link iiwa_link_1: geometry collision mesh filename=meshes/collision/link_1.obj; visual mesh filename=meshes/visual/link_1.obj
- link iiwa_link_2: geometry collision mesh filename=meshes/collision/link_2.obj; visual mesh filename=meshes/visual/link_2.obj
- link iiwa_link_3: geometry collision mesh filename=meshes/collision/link_3.obj; visual mesh filename=meshes/visual/link_3.obj
- link iiwa_link_4: geometry collision mesh filename=meshes/collision/link_4.obj; visual mesh filename=meshes/visual/link_4.obj
- link iiwa_link_5: geometry collision mesh filename=meshes/collision/link_5.obj; visual mesh filename=meshes/visual/link_5.obj
- link iiwa_link_6: geometry collision mesh filename=meshes/collision/link_6.obj; visual mesh filename=meshes/visual/link_6.obj
- link iiwa_link_7: geometry collision mesh filename=meshes/collision/link_7.obj; visual mesh filename=meshes/visual/link_7.obj

Commit message: Removes collision elements to speed things up

File: drake/examples/kuka_iiwa_arm/urdf/iiwa14.urdf (robot description, URDF)
Before this commit: robot iiwa14, 11 links, 10 joints
Links:
- link iiwa_link_0: geometry visual mesh filename=meshes/visual/link_0.obj
- link iiwa_link_1: geometry visual mesh filename=meshes/visual/link_1.obj
- link iiwa_link_2: geometry visual mesh filename=meshes/visual/link_2.obj
- link iiwa_link_3: geometry visual mesh filename=meshes/visual/link_3.obj
- link iiwa_link_4: geometry visual mesh filename=meshes/visual/link_4.obj
- link iiwa_link_5: geometry visual mesh filename=meshes/visual/link_5.obj
- link iiwa_link_6: geometry visual mesh filename=meshes/visual/link_6.obj

Commit message: Use cylinders instead of meshes for some links, for processing speed. Leave meshes for links at end of arm, for model accuracy. Changed colors to better match reality. In our arm, only a part of the link is orange, and this colors the entire link orange, but its an improvement to see each link. Adding model.config for future work in Gazebo. Make friction coefficient and damping in rigid body plant match rbs.

File: drake/examples/kuka_iiwa_arm/urdf/iiwa14.urdf (robot description, URDF)
Before this commit: robot iiwa14, 11 links, 10 joints
Links:
- link iiwa_link_0: geometry collision cylinder length=0.17 radius=0.139; visual mesh filename=meshes/visual/link_0.obj
- link iiwa_link_1: geometry collision cylinder length=0.29 radius=0.101; visual mesh filename=meshes/visual/link_1.obj
- link iiwa_link_2: geometry collision cylinder length=0.29 radius=0.101; visual mesh filename=meshes/visual/link_2.obj
- link iiwa_link_3: geometry collision cylinder length=0.29 radius=0.092; visual mesh filename=meshes/visual/link_3.obj
- link iiwa_link_4: geometry collision cylinder length=0.25 radius=0.092; visual mesh filename=meshes/visual/link_4.obj
- link iiwa_link_5: geometry collision cylinder length=0.29 radius=0.07; visual mesh filename=meshes/visual/link_5.obj

Commit message: Adds iiwa model with no collision

File: drake/examples/kuka_iiwa_arm/urdf/iiwa14.urdf (robot description, URDF)
Before this commit: robot iiwa14, 11 links, 10 joints
Links:
- link iiwa_link_0: geometry collision cylinder length=0.17 radius=0.139; visual mesh filename=meshes/visual/link_0.obj
- link iiwa_link_1: geometry collision cylinder length=0.29 radius=0.101; visual mesh filename=meshes/visual/link_1.obj
- link iiwa_link_2: geometry collision cylinder length=0.29 radius=0.101; visual mesh filename=meshes/visual/link_2.obj
- link iiwa_link_3: geometry collision cylinder length=0.29 radius=0.092; visual mesh filename=meshes/visual/link_3.obj
- link iiwa_link_4: geometry collision cylinder length=0.25 radius=0.092; visual mesh filename=meshes/visual/link_4.obj
- link iiwa_link_5: geometry collision cylinder length=0.29 radius=0.07; visual mesh filename=meshes/visual/link_5.obj
- link iiwa_link_6: geometry collision mesh filename=meshes/collision/link_6.obj; visual mesh filename=meshes/visual/link_6.obj

Commit message: Update iiwa mass/interia values to behave in a slightly more realistic manner when fed recorded torques from a stationary arm.
(with thanks to Harvard Agile Robotics Lab, who I copied these values from)

File: drake/examples/kuka_iiwa_arm/urdf/iiwa14.urdf (robot description, URDF)
Before this commit: robot iiwa14, 11 links, 10 joints
Links:
- link iiwa_link_1: mass 4 -> 5.76
- link iiwa_link_2: mass 4 -> 6.35
- link iiwa_link_3: mass 3 -> 3.5
- link iiwa_link_4: mass 2.7 -> 3.5
- link iiwa_link_5: mass 1.7 -> 3.5
- link iiwa_link_7: mass 0.3 -> 1.2

File: drake/examples/kuka_iiwa_arm/urdf/iiwa14_simplified_collision.urdf (robot description, URDF)
Before this commit: robot iiwa14, 11 links, 10 joints
Links:
- link iiwa_link_1: mass 4 -> 5.76
- link iiwa_link_2: mass 4 -> 6.35
- link iiwa_link_3: mass 3 -> 3.5
- link iiwa_link_4: mass 2.7 -> 3.5
- link iiwa_link_5: mass 1.7 -> 3.5
- link iiwa_link_7: mass 0.3 -> 1.2
