Commit message: Tweaks to get Kuka arm running

File: drake/examples/KukaArm/urdf/iiwa14.urdf (robot description, URDF)
Before this commit: robot iiwa14, 11 links, 10 joints
Links:
- removed link world
- link iiwa_link_0: geometry collision cylinder length=0.17 radius=0.139; visual mesh filename=meshes/visual/link_0.obj
- link iiwa_link_1: geometry collision cylinder length=0.29 radius=0.101; visual mesh filename=meshes/visual/link_1.obj
- link iiwa_link_2: geometry collision cylinder length=0.29 radius=0.101; visual mesh filename=meshes/visual/link_2.obj
- link iiwa_link_3: geometry collision cylinder length=0.29 radius=0.092; visual mesh filename=meshes/visual/link_3.obj
- link iiwa_link_4: geometry collision cylinder length=0.25 radius=0.092; visual mesh filename=meshes/visual/link_4.obj
- link iiwa_link_5: geometry collision cylinder length=0.29 radius=0.07; visual mesh filename=meshes/visual/link_5.obj
- link iiwa_link_6: geometry collision mesh filename=meshes/collision/link_6.obj; visual mesh filename=meshes/visual/link_6.obj
- link iiwa_link_7: geometry collision mesh filename=meshes/collision/link_7.obj; visual mesh filename=meshes/visual/link_7.obj
Joints:
- joint world_iiwa_joint: parent world -> (none)

File: drake/examples/KukaArm/urdf/iiwa14_with_weight.urdf (robot description, URDF)
Before this commit: robot iiwa14, 12 links, 11 joints
Links:
- removed link world
Joints:
- joint world_iiwa_joint: parent world -> (none)

Commit message: added milk-on-a-shelf example. updated arm model/meshes. now uses proper collision detection between shelf and spherical approximation of the milk jug.

File: drake/examples/KukaArm/urdf/iiwa14.urdf (robot description, URDF)
Before this commit: robot iiwa14, 10 links, 10 joints
Links:
- added link base
- link iiwa_link_0: geometry visual mesh filename=meshes/visual/link_0.obj
- link iiwa_link_1: mass 4 -> 5.76; geometry visual mesh filename=meshes/visual/link_1.obj
- link iiwa_link_2: mass 4 -> 6.35; geometry visual mesh filename=meshes/visual/link_2.obj
- link iiwa_link_3: mass 3 -> 3.5; geometry visual mesh filename=meshes/visual/link_3.obj
- link iiwa_link_4: mass 2.7 -> 3.5; geometry visual mesh filename=meshes/visual/link_4.obj
- link iiwa_link_5: mass 1.7 -> 3.5; geometry visual mesh filename=meshes/visual/link_5.obj
- link iiwa_link_6: geometry visual mesh filename=meshes/visual/link_6.obj
- link iiwa_link_7: mass 0.3 -> 1.2
Joints:
- removed joint world_iiwa_joint
- added joint base_joint: type fixed, parent base, child iiwa_link_0, origin xyz=0 0 0.0 rpy=0 0 0
