Commit message: Moves kuka iiwa 14 model into drake/manipulation and made it xacro-generated.

File: drake/manipulation/models/iiwa_description/urdf/iiwa14_polytope_collision.urdf (robot description, URDF)
Before this commit: robot iiwa14, 11 links, 10 joints
Links:
- link iiwa_link_0: geometry visual mesh filename=../meshes/visual/link_0.obj
- link iiwa_link_1: geometry visual mesh filename=../meshes/visual/link_1.obj
- link iiwa_link_2: geometry visual mesh filename=../meshes/visual/link_2.obj
- link iiwa_link_3: geometry visual mesh filename=../meshes/visual/link_3.obj
- link iiwa_link_4: geometry visual mesh filename=../meshes/visual/link_4.obj
- link iiwa_link_5: geometry visual mesh filename=../meshes/visual/link_5.obj
- link iiwa_link_6: geometry visual mesh filename=../meshes/visual/link_6.obj
- link iiwa_link_7: geometry collision mesh filename=../meshes/collision/link_7_polytope.obj; visual mesh filename=../meshes/visual/link_7.obj
Joints:
- joint base_joint: origin xyz=0 0 0.0 rpy=0 0 0 -> xyz=0 0 0 rpy=0 0 0

File: drake/manipulation/models/iiwa_description/urdf/iiwa14_primitive_collision.urdf (robot description, URDF)
Before this commit: robot iiwa14, 11 links, 10 joints
Links:
- link iiwa_link_0: geometry collision cylinder length=0.17 radius=0.139; visual mesh filename=../meshes/visual/link_0.obj
- link iiwa_link_1: geometry collision cylinder length=0.29 radius=0.101; visual mesh filename=../meshes/visual/link_1.obj
- link iiwa_link_2: geometry collision cylinder length=0.29 radius=0.101; visual mesh filename=../meshes/visual/link_2.obj
- link iiwa_link_3: geometry collision cylinder length=0.29 radius=0.092; visual mesh filename=../meshes/visual/link_3.obj
- link iiwa_link_4: geometry collision cylinder length=0.25 radius=0.092; visual mesh filename=../meshes/visual/link_4.obj
- link iiwa_link_5: geometry collision cylinder length=0.29 radius=0.07; visual mesh filename=../meshes/visual/link_5.obj
- link iiwa_link_6: geometry collision mesh filename=../meshes/collision/link_6.obj; visual mesh filename=../meshes/visual/link_6.obj
- link iiwa_link_7: geometry collision mesh filename=../meshes/collision/link_7.obj; visual mesh filename=../meshes/visual/link_7.obj
Joints:
- joint base_joint: origin xyz=0 0 0.0 rpy=0 0 0 -> xyz=0 0 0 rpy=0 0 0
