Commit message: Adds a prefix to the iiwa xacro and an example of a dual-iiwa-arm model.

File: drake/manipulation/models/iiwa_description/urdf/iiwa.transmission.xacro (robot description, xacro)
@@ -1,78 +1,78 @@
 <?xml version="1.0"?>
 <robot xmlns:xacro="http://www.ros.org/wiki/xacro">
-  <xacro:macro name="iiwa_transmission" params="hardware_interface">
-    <transmission name="iiwa_tran_1">
+  <xacro:macro name="iiwa_transmission" params="hardware_interface robot_name">
+    <transmission name="${robot_name}_tran_1">
       <robotNamespace>/${robot_name}</robotNamespace>
       <type>transmission_interface/SimpleTransmission</type>
-      <joint name="iiwa_joint_1">
+      <joint name="${robot_name}_joint_1">
 	<hardwareInterface>${hardware_interface}</hardwareInterface>
       </joint>
-      <actuator name="iiwa_motor_1">
+      <actuator name="${robot_name}_motor_1">
 	<hardwareInterface>${hardware_interface}</hardwareInterface>
 	<mechanicalReduction>1</mechanicalReduction>
       </actuator>
     </transmission>
-    <transmission name="iiwa_tran_2">
+    <transmission name="${robot_name}_tran_2">
       <robotNamespace>/${robot_name}</robotNamespace>
       <type>transmission_interface/SimpleTransmission</type>
-      <joint name="iiwa_joint_2">
+      <joint name="${robot_name}_joint_2">
 	<hardwareInterface>${hardware_interface}</hardwareInterface>
       </joint>
-      <actuator name="iiwa_motor_2">
+      <actuator name="${robot_name}_motor_2">
 	<hardwareInterface>${hardware_interface}</hardwareInterface>
 	<mechanicalReduction>1</mechanicalReduction>
       </actuator>
     </transmission>
-    <transmission name="iiwa_tran_3">
+    <transmission name="${robot_name}_tran_3">
       <robotNamespace>/${robot_name}</robotNamespace>
       <type>transmission_interface/SimpleTransmission</type>
-      <joint name="iiwa_joint_3">
+      <joint name="${robot_name}_joint_3">
 	<hardwareInterface>${hardware_interface}</hardwareInterface>
       </joint>
-      <actuator name="iiwa_motor_3">
+      <actuator name="${robot_name}_motor_3">
 	<hardwareInterface>${hardware_interface}</hardwareInterface>
 	<mechanicalReduction>1</mechanicalReduction>
       </actuator>
     </transmission>
-    <transmission name="iiwa_tran_4">
+    <transmission name="${robot_name}_tran_4">
       <robotNamespace>/${robot_name}</robotNamespace>
       <type>transmission_interface/SimpleTransmission</type>
-      <joint name="iiwa_joint_4">
+      <joint name="${robot_name}_joint_4">
 	<hardwareInterface>${hardware_interface}</hardwareInterface>
       </joint>
-      <actuator name="iiwa_motor_4">
+      <actuator name="${robot_name}_motor_4">
 	<hardwareInterface>${hardware_interface}</hardwareInterface>
 	<mechanicalReduction>1</mechanicalReduction>
       </actuator>
     </transmission>
-    <transmission name="iiwa_tran_5">
+    <transmission name="${robot_name}_tran_5">
       <robotNamespace>/${robot_name}</robotNamespace>
       <type>transmission_interface/SimpleTransmission</type>
-      <joint name="iiwa_joint_5">
+      <joint name="${robot_name}_joint_5">
 	<hardwareInterface>${hardware_interface}</hardwareInterface>
       </joint>
-      <actuator name="iiwa_motor_5">
+      <actuator name="${robot_name}_motor_5">
 	<hardwareInterface>${hardware_interface}</hardwareInterface>
 	<mechanicalReduction>1</mechanicalReduction>
       </actuator>
     </transmission>
-    <transmission name="iiwa_tran_6">
+    <transmission name="${robot_name}_tran_6">
       <robotNamespace>/${robot_name}</robotNamespace>
       <type>transmission_interface/SimpleTransmission</type>
-      <joint name="iiwa_joint_6">
+      <joint name="${robot_name}_joint_6">
 	<hardwareInterface>${hardware_interface}</hardwareInterface>
       </joint>
-      <actuator name="iiwa_motor_6">
+      <actuator name="${robot_name}_motor_6">
 	<hardwareInterface>${hardware_interface}</hardwareInterface>
 	<mechanicalReduction>1</mechanicalReduction>
       </actuator>
     </transmission>
-    <transmission name="iiwa_tran_7">
+    <transmission name="${robot_name}_tran_7">
       <robotNamespace>/${robot_name}</robotNamespace>
       <type>transmission_interface/SimpleTransmission</type>
-      <joint name="iiwa_joint_7">
+      <joint name="${robot_name}_joint_7">
 	<hardwareInterface>${hardware_interface}</hardwareInterface>
       </joint>
-      <actuator name="iiwa_motor_7">
+      <actuator name="${robot_name}_motor_7">
 	<hardwareInterface>${hardware_interface}</hardwareInterface>
 	<mechanicalReduction>1</mechanicalReduction>

File: drake/manipulation/models/iiwa_description/urdf/iiwa14.xacro (robot description, xacro)
@@ -16,5 +16,5 @@
       params="parent hardware_interface robot_name collision_type *origin">
     <!--joint between {parent} and link_0-->
-    <joint name="${parent}_joint" type="fixed">
+    <joint name="${robot_name}_${parent}_joint" type="fixed">
       <xacro:insert_block name="origin"/>
       <parent link="${parent}"/>
@@ -414,11 +414,12 @@
       <origin rpy="0 -1.57079632679 0" xyz="0 0 0.045"/>
     </joint>
-    <link name="iiwa_link_ee">
-    </link>
-    <frame name="iiwa_frame_ee" link="iiwa_link_ee"
+    <link name="${robot_name}_link_ee">
+    </link>
+    <frame name="${robot_name}_frame_ee" link="${robot_name}_link_ee"
            xyz="0.09 0 0" rpy="3.14159265359 0 1.57079632679"/>
     <!--Extensions -->
     <xacro:iiwa_gazebo robot_name="${robot_name}" />
-    <xacro:iiwa_transmission hardware_interface="${hardware_interface}"/>
+    <xacro:iiwa_transmission hardware_interface="${hardware_interface}"
+        robot_name="${robot_name}"/>
   </xacro:macro>
 </robot>

File: drake/manipulation/models/iiwa_description/urdf/iiwa14_polytope_collision.urdf (robot description, URDF)
Before this commit: robot iiwa14, 11 links, 10 joints
Joints:
- removed joint base_joint
- added joint iiwa_base_joint: type fixed, parent base, child iiwa_link_0, origin xyz=0 0 0 rpy=0 0 0

File: drake/manipulation/models/iiwa_description/urdf/iiwa14_primitive_collision.urdf (robot description, URDF)
Before this commit: robot iiwa14, 11 links, 10 joints
Joints:
- removed joint base_joint
- added joint iiwa_base_joint: type fixed, parent base, child iiwa_link_0, origin xyz=0 0 0 rpy=0 0 0
