Commit message: Addressing platform reviewer comments

File: drake/manipulation/models/jaco_description/urdf/j2n6s300_col.urdf (robot description, URDF)
Before this commit: robot j2n6s300, 16 links, 15 joints
Links:
- removed link base_link
- added link root; collision box size=0 0 0; visual box size=0 0 0
- link j2n6s300_link_1: geometry collision cylinder length=0.06 radius=0.025; visual cylinder length=0.06 radius=0.025
- link j2n6s300_link_2: geometry collision cylinder length=0.3 radius=0.025; visual cylinder length=0.05 radius=0.01
- link j2n6s300_link_3: geometry collision cylinder length=0.17 radius=0.025; visual cylinder length=0.17 radius=0.025
- link j2n6s300_link_4: geometry collision cylinder length=0.01 radius=0.025; visual cylinder length=0.01 radius=0.025
- link j2n6s300_link_5: geometry collision cylinder length=0.01 radius=0.025; visual cylinder length=0.01 radius=0.025
- link j2n6s300_link_6: geometry collision cylinder length=0.01 radius=0.025; visual cylinder length=0.01 radius=0.025
- link j2n6s300_link_base: geometry collision cylinder length=0.075 radius=0.025; visual cylinder length=0.075 radius=0.025
- link j2n6s300_link_finger_1: geometry collision cylinder length=0.01 radius=0.01; visual cylinder length=0.01 radius=0.01
- link j2n6s300_link_finger_2: geometry collision cylinder length=0.01 radius=0.01; visual cylinder length=0.01 radius=0.01
- link j2n6s300_link_finger_3: geometry collision cylinder length=0.01 radius=0.01; visual cylinder length=0.01 radius=0.01
- link j2n6s300_link_finger_tip_1: geometry collision cylinder length=0.01 radius=0.01; visual cylinder length=0.01 radius=0.01
- link j2n6s300_link_finger_tip_2: geometry collision cylinder length=0.01 radius=0.01; visual cylinder length=0.01 radius=0.01
- link j2n6s300_link_finger_tip_3: geometry collision cylinder length=0.01 radius=0.01; visual cylinder length=0.01 radius=0.01
Joints:
- joint connect_root_and_world: child base_link -> root
- joint j2n6s300_joint_2: limit lower=0.523598775598 upper=5.75958653158 effort=2000 velocity=1 -> lower=-2.618 upper=2.613 effort=2000 velocity=1; origin xyz=0 0.0016 -0.11875 rpy=-1.57079632679 0 3.14159265359 -> xyz=0 0.0016 -0.11875 rpy=-1.57079632679 3.1415 3.14159265359
- joint j2n6s300_joint_3: limit lower=0.523598775598 upper=5.75958653158 effort=2000 velocity=1 -> lower=-2.618 upper=2.613 effort=2000 velocity=1; origin xyz=0 -0.410 0 rpy=0 3.14159265359 0 -> xyz=0 -0.410 0 rpy=0 3.14159265359 3.1415
- joint j2n6s300_joint_base: parent base_link -> root
