Commit message: Make tree compilation *optional* when parsing sdf/urdf files
This enables being able to programmatically modify collision filter groups
of parsed files. It does this by providing an optional flag that defers
tree compilation (which used to be a defacto step in parsing).

1. URDF and SDF parsers are updated to propagate the flags.
2. Testing is provided to confirm behavior.
3. Incidental corrections to providing collision filter group support in
   sdf parsing.
   a. The doxygen module on the subject has been updated.
   b. SDF specific semantics have been documented and tested.

File: multibody/collision/test/filter_groups_in_file.urdf (robot description, URDF)
Before this commit: robot simple_anchored, 4 links, 3 joints
Links:
- link sphereA: mass None -> 1
- link sphereB: mass None -> 1
- link sphereC: mass None -> 1
- link sphereD: mass None -> 1
