Commit message: Synthetic scene generation : Random Clutter

File: examples/kuka_iiwa_arm/models/objects/open_top_box.urdf (robot description, URDF)
Before this commit: robot open_top_box, 1 links, 0 joints
Links:
- link bin: geometry collision box size=0.01 0.52 0.3; collision box size=0.01 0.52 0.3
