Commit message: Update iiwa visual representation
This exposes the underlying geometry which includes the
kuka logo and "elbow" patches. It also merges
coincident vertices and computes per-vertex mesh
normals. It updates all sdf and urdf files to reference
the new objs.

NOTE: Although an OBJ file can support multiple
materials are data pipeline *can't*. As such, if
different meshes receive different materials, we
currently require them to be different meshes.

File: manipulation/models/iiwa_description/urdf/iiwa14_spheres_collision.urdf (robot description, URDF)
Before this commit: robot iiwa14, 11 links, 10 joints
Links:
- link iiwa_link_2: geometry collision sphere radius=0.06602481863; collision sphere radius=0.07959901601
- link iiwa_link_3: geometry collision sphere radius=0.06062598796; collision sphere radius=0.06602481863
- link iiwa_link_4: geometry collision sphere radius=0.05993984276; collision sphere radius=0.06644602201
- link iiwa_link_5: geometry collision sphere radius=0.05281876964; collision sphere radius=0.06644602201
- link iiwa_link_6: geometry collision sphere radius=0.06341754633; visual mesh filename=../meshes/visual/link_6_grey.obj

File: manipulation/models/iiwa_description/urdf/iiwa14_spheres_dense_collision.urdf (robot description, URDF)
Before this commit: robot iiwa14, 11 links, 10 joints
Links:
- link iiwa_link_2: geometry collision sphere radius=0.065; collision sphere radius=0.065
- link iiwa_link_3: geometry collision sphere radius=0.055; collision sphere radius=0.055
- link iiwa_link_4: geometry collision sphere radius=0.06; collision sphere radius=0.06
- link iiwa_link_5: geometry collision sphere radius=0.035; collision sphere radius=0.035
- link iiwa_link_6: geometry collision sphere radius=0.055; collision sphere radius=0.065

File: manipulation/models/iiwa_description/urdf/iiwa14_spheres_dense_elbow_collision.urdf (robot description, URDF)
Before this commit: robot iiwa14, 11 links, 10 joints
Links:
- link iiwa_link_2: geometry collision sphere radius=0.06602481863; collision sphere radius=0.07959901601
- link iiwa_link_3: geometry collision sphere radius=0.055; collision sphere radius=0.055
- link iiwa_link_4: geometry collision sphere radius=0.06; collision sphere radius=0.06
- link iiwa_link_5: geometry visual mesh filename=../meshes/visual/band.obj; visual mesh filename=../meshes/visual/kuka.obj
- link iiwa_link_6: geometry collision sphere radius=0.055; collision sphere radius=0.08
