Commit message: update xacro velocity calculation on degrees

File: manipulation/models/iiwa_description/urdf/dual_iiwa14_polytope_collision.urdf (robot description, URDF)
Before this commit: robot dual_iiwa14, 21 links, 20 joints
Joints:
- joint left_iiwa_joint_1: limit lower=-2.96705972839 upper=2.96705972839 effort=300 velocity=10 -> lower=-2.96705972839 upper=2.96705972839 effort=320 velocity=1.4835298641951802
- joint left_iiwa_joint_2: limit lower=-2.09439510239 upper=2.09439510239 effort=300 velocity=10 -> lower=-2.09439510239 upper=2.09439510239 effort=320 velocity=1.4835298641951802
- joint left_iiwa_joint_3: limit lower=-2.96705972839 upper=2.96705972839 effort=300 velocity=10 -> lower=-2.96705972839 upper=2.96705972839 effort=176 velocity=1.7453292519943295
- joint left_iiwa_joint_4: limit lower=-2.09439510239 upper=2.09439510239 effort=300 velocity=10 -> lower=-2.09439510239 upper=2.09439510239 effort=176 velocity=1.3089969389957472
- joint left_iiwa_joint_5: limit lower=-2.96705972839 upper=2.96705972839 effort=300 velocity=10 -> lower=-2.96705972839 upper=2.96705972839 effort=110 velocity=2.2689280275926285
- joint left_iiwa_joint_6: limit lower=-2.09439510239 upper=2.09439510239 effort=300 velocity=10 -> lower=-2.09439510239 upper=2.09439510239 effort=40 velocity=2.356194490192345
- joint left_iiwa_joint_7: limit lower=-3.05432619099 upper=3.05432619099 effort=300 velocity=10 -> lower=-3.05432619099 upper=3.05432619099 effort=40 velocity=2.356194490192345
- joint right_iiwa_joint_1: limit lower=-2.96705972839 upper=2.96705972839 effort=300 velocity=10 -> lower=-2.96705972839 upper=2.96705972839 effort=320 velocity=1.4835298641951802
- joint right_iiwa_joint_2: limit lower=-2.09439510239 upper=2.09439510239 effort=300 velocity=10 -> lower=-2.09439510239 upper=2.09439510239 effort=320 velocity=1.4835298641951802
- joint right_iiwa_joint_3: limit lower=-2.96705972839 upper=2.96705972839 effort=300 velocity=10 -> lower=-2.96705972839 upper=2.96705972839 effort=176 velocity=1.7453292519943295
- joint right_iiwa_joint_4: limit lower=-2.09439510239 upper=2.09439510239 effort=300 velocity=10 -> lower=-2.09439510239 upper=2.09439510239 effort=176 velocity=1.3089969389957472
- joint right_iiwa_joint_5: limit lower=-2.96705972839 upper=2.96705972839 effort=300 velocity=10 -> lower=-2.96705972839 upper=2.96705972839 effort=110 velocity=2.2689280275926285
- joint right_iiwa_joint_6: limit lower=-2.09439510239 upper=2.09439510239 effort=300 velocity=10 -> lower=-2.09439510239 upper=2.09439510239 effort=40 velocity=2.356194490192345
- joint right_iiwa_joint_7: limit lower=-3.05432619099 upper=3.05432619099 effort=300 velocity=10 -> lower=-3.05432619099 upper=3.05432619099 effort=40 velocity=2.356194490192345

File: manipulation/models/iiwa_description/urdf/iiwa14.xacro (robot description, xacro)
@@ -67,5 +67,5 @@
       <origin xyz="0 0 0.1575" rpy="0 0 0"/>
       <axis xyz="0 0 1"/>
-      <limit lower="${-170 * PI / 180}" upper="${170 * PI / 180}" effort="320" velocity="1.48353"/>
+      <limit lower="${-170 * PI / 180}" upper="${170 * PI / 180}" effort="320" velocity="${85 * PI / 180}"/>
       <safety_controller soft_lower_limit="${-168 * PI / 180}" soft_upper_limit="${168 * PI / 180}" k_position="${safety_controller_k_pos}" k_velocity="${safety_controller_k_vel}"/>
       <dynamics damping="${joint_damping}"/>
@@ -110,5 +110,5 @@
       <origin xyz="0 0 0.2025" rpy="${PI / 2}   0 ${PI}"/>
       <axis xyz="0 0 1"/>
-      <limit lower="${-120 * PI / 180}" upper="${120 * PI / 180}" effort="320" velocity="1.48353"/>
+      <limit lower="${-120 * PI / 180}" upper="${120 * PI / 180}" effort="320" velocity="${85 * PI / 180}"/>
       <safety_controller soft_lower_limit="${-118 * PI / 180}" soft_upper_limit="${118 * PI / 180}" k_position="${safety_controller_k_pos}" k_velocity="${safety_controller_k_vel}"/>
       <dynamics damping="${joint_damping}"/>
@@ -162,5 +162,5 @@
       <origin xyz="0 0.2045 0" rpy="${PI / 2} 0 ${PI}"/>
       <axis xyz="0 0 1"/>
-      <limit lower="${-170 * PI / 180}" upper="${170 * PI / 180}" effort="176" velocity="1.74533"/>
+      <limit lower="${-170 * PI / 180}" upper="${170 * PI / 180}" effort="176" velocity="${100 * PI / 180}"/>
       <safety_controller soft_lower_limit="${-118 * PI / 180}" soft_upper_limit="${118 * PI / 180}" k_position="${safety_controller_k_pos}" k_velocity="${safety_controller_k_vel}"/>
       <dynamics damping="${joint_damping}"/>
@@ -221,5 +221,5 @@
       <origin xyz="0 0 0.2155" rpy="${PI / 2} 0 0"/>
       <axis xyz="0 0 1"/>
-      <limit lower="${-120 * PI / 180}" upper="${120 * PI / 180}" effort="176" velocity="1.309"/>
+      <limit lower="${-120 * PI / 180}" upper="${120 * PI / 180}" effort="176" velocity="${75 * PI / 180}"/>
       <safety_controller soft_lower_limit="${-118 * PI / 180}" soft_upper_limit="${118 * PI / 180}" k_position="${safety_controller_k_pos}" k_velocity="${safety_controller_k_vel}"/>
       <dynamics damping="${joint_damping}"/>
@@ -273,5 +273,5 @@
       <origin xyz="0 0.1845 0" rpy="${-PI / 2} ${PI} 0"/>
       <axis xyz="0 0 1"/>
-      <limit lower="${-170 * PI / 180}" upper="${170 * PI / 180}" effort="110" velocity="2.26893"/>
+      <limit lower="${-170 * PI / 180}" upper="${170 * PI / 180}" effort="110" velocity="${130 * PI / 180}"/>
       <safety_controller soft_lower_limit="${-118 * PI / 180}" soft_upper_limit="${118 * PI / 180}" k_position="${safety_controller_k_pos}" k_velocity="${safety_controller_k_vel}"/>
       <dynamics damping="${joint_damping}"/>
@@ -332,5 +332,5 @@
       <origin xyz="0 0 0.2155" rpy="${PI / 2} 0 0"/>
       <axis xyz="0 0 1"/>
-      <limit lower="${-120 * PI / 180}" upper="${120 * PI / 180}" effort="40" velocity="2.35619"/>
+      <limit lower="${-120 * PI / 180}" upper="${120 * PI / 180}" effort="40" velocity="${135 * PI / 180}"/>
       <safety_controller soft_lower_limit="${-118 * PI / 180}" soft_upper_limit="${118 * PI / 180}" k_position="${safety_controller_k_pos}" k_velocity="${safety_controller_k_vel}"/>
       <dynamics damping="${joint_damping}"/>
@@ -386,5 +386,5 @@
       <origin xyz="0 0.081 0" rpy="${- PI / 2} ${PI} 0"/>
       <axis xyz="0 0 1"/>
-      <limit lower="${-175 * PI / 180}" upper="${175 * PI / 180}" effort="40" velocity="2.35619"/>
+      <limit lower="${-175 * PI / 180}" upper="${175 * PI / 180}" effort="40" velocity="${135 * PI / 180}"/>
       <safety_controller soft_lower_limit="${-173 * PI / 180}" soft_upper_limit="${173 * PI / 180}" k_position="${safety_controller_k_pos}" k_velocity="${safety_controller_k_vel}"/>
       <dynamics damping="${joint_damping}"/>

File: manipulation/models/iiwa_description/urdf/iiwa14_no_collision.urdf (robot description, URDF)
Before this commit: robot iiwa14, 11 links, 10 joints
Joints:
- joint iiwa_joint_1: limit lower=-2.96705972839 upper=2.96705972839 effort=320 velocity=1.39626 -> lower=-2.96705972839 upper=2.96705972839 effort=320 velocity=1.4835298641951802
- joint iiwa_joint_2: limit lower=-2.09439510239 upper=2.09439510239 effort=320 velocity=1.39626 -> lower=-2.09439510239 upper=2.09439510239 effort=320 velocity=1.4835298641951802
- joint iiwa_joint_3: limit lower=-2.96705972839 upper=2.96705972839 effort=176 velocity=1.74533 -> lower=-2.96705972839 upper=2.96705972839 effort=176 velocity=1.7453292519943295
- joint iiwa_joint_4: limit lower=-2.09439510239 upper=2.09439510239 effort=176 velocity=1.309 -> lower=-2.09439510239 upper=2.09439510239 effort=176 velocity=1.3089969389957472
- joint iiwa_joint_5: limit lower=-2.96705972839 upper=2.96705972839 effort=110 velocity=2.26893 -> lower=-2.96705972839 upper=2.96705972839 effort=110 velocity=2.9670597283903604
- joint iiwa_joint_6: limit lower=-2.09439510239 upper=2.09439510239 effort=40 velocity=2.35619 -> lower=-2.09439510239 upper=2.09439510239 effort=40 velocity=2.356194490192345
- joint iiwa_joint_7: limit lower=-3.05432619099 upper=3.05432619099 effort=40 velocity=2.35619 -> lower=-3.05432619099 upper=3.05432619099 effort=40 velocity=2.356194490192345

File: manipulation/models/iiwa_description/urdf/iiwa14_polytope_collision.urdf (robot description, URDF)
Before this commit: robot iiwa14, 11 links, 10 joints
Joints:
- joint iiwa_joint_1: limit lower=-2.96705972839 upper=2.96705972839 effort=300 velocity=10 -> lower=-2.96705972839 upper=2.96705972839 effort=320 velocity=1.4835298641951802
- joint iiwa_joint_2: limit lower=-2.09439510239 upper=2.09439510239 effort=300 velocity=10 -> lower=-2.09439510239 upper=2.09439510239 effort=320 velocity=1.4835298641951802
- joint iiwa_joint_3: limit lower=-2.96705972839 upper=2.96705972839 effort=300 velocity=10 -> lower=-2.96705972839 upper=2.96705972839 effort=176 velocity=1.7453292519943295
- joint iiwa_joint_4: limit lower=-2.09439510239 upper=2.09439510239 effort=300 velocity=10 -> lower=-2.09439510239 upper=2.09439510239 effort=176 velocity=1.3089969389957472
- joint iiwa_joint_5: limit lower=-2.96705972839 upper=2.96705972839 effort=300 velocity=10 -> lower=-2.96705972839 upper=2.96705972839 effort=110 velocity=2.2689280275926285
- joint iiwa_joint_6: limit lower=-2.09439510239 upper=2.09439510239 effort=300 velocity=10 -> lower=-2.09439510239 upper=2.09439510239 effort=40 velocity=2.356194490192345
- joint iiwa_joint_7: limit lower=-3.05432619099 upper=3.05432619099 effort=300 velocity=10 -> lower=-3.05432619099 upper=3.05432619099 effort=40 velocity=2.356194490192345

File: manipulation/models/iiwa_description/urdf/iiwa14_primitive_collision.urdf (robot description, URDF)
Before this commit: robot iiwa14, 11 links, 10 joints
Joints:
- joint iiwa_joint_1: limit lower=-2.96705972839 upper=2.96705972839 effort=300 velocity=10 -> lower=-2.96705972839 upper=2.96705972839 effort=320 velocity=1.4835298641951802
- joint iiwa_joint_2: limit lower=-2.09439510239 upper=2.09439510239 effort=300 velocity=10 -> lower=-2.09439510239 upper=2.09439510239 effort=320 velocity=1.4835298641951802
- joint iiwa_joint_3: limit lower=-2.96705972839 upper=2.96705972839 effort=300 velocity=10 -> lower=-2.96705972839 upper=2.96705972839 effort=176 velocity=1.7453292519943295
- joint iiwa_joint_4: limit lower=-2.09439510239 upper=2.09439510239 effort=300 velocity=10 -> lower=-2.09439510239 upper=2.09439510239 effort=176 velocity=1.3089969389957472
- joint iiwa_joint_5: limit lower=-2.96705972839 upper=2.96705972839 effort=300 velocity=10 -> lower=-2.96705972839 upper=2.96705972839 effort=110 velocity=2.2689280275926285
- joint iiwa_joint_6: limit lower=-2.09439510239 upper=2.09439510239 effort=300 velocity=10 -> lower=-2.09439510239 upper=2.09439510239 effort=40 velocity=2.356194490192345
- joint iiwa_joint_7: limit lower=-3.05432619099 upper=3.05432619099 effort=300 velocity=10 -> lower=-3.05432619099 upper=3.05432619099 effort=40 velocity=2.356194490192345

File: manipulation/models/iiwa_description/urdf/iiwa14_spheres_collision.urdf (robot description, URDF)
Before this commit: robot iiwa14, 11 links, 10 joints
Joints:
- joint iiwa_joint_1: limit lower=-2.96705972839 upper=2.96705972839 effort=320 velocity=1.48353 -> lower=-2.96705972839 upper=2.96705972839 effort=320 velocity=1.4835298641951802
- joint iiwa_joint_2: limit lower=-2.09439510239 upper=2.09439510239 effort=320 velocity=1.48353 -> lower=-2.09439510239 upper=2.09439510239 effort=320 velocity=1.4835298641951802
- joint iiwa_joint_3: limit lower=-2.96705972839 upper=2.96705972839 effort=176 velocity=1.74533 -> lower=-2.96705972839 upper=2.96705972839 effort=176 velocity=1.7453292519943295
- joint iiwa_joint_4: limit lower=-2.09439510239 upper=2.09439510239 effort=176 velocity=1.309 -> lower=-2.09439510239 upper=2.09439510239 effort=176 velocity=1.3089969389957472
- joint iiwa_joint_5: limit lower=-2.96705972839 upper=2.96705972839 effort=110 velocity=2.26893 -> lower=-2.96705972839 upper=2.96705972839 effort=110 velocity=2.2689280275926285
- joint iiwa_joint_6: limit lower=-2.09439510239 upper=2.09439510239 effort=40 velocity=2.35619 -> lower=-2.09439510239 upper=2.09439510239 effort=40 velocity=2.356194490192345
- joint iiwa_joint_7: limit lower=-3.05432619099 upper=3.05432619099 effort=40 velocity=2.35619 -> lower=-3.05432619099 upper=3.05432619099 effort=40 velocity=2.356194490192345

File: manipulation/models/iiwa_description/urdf/iiwa14_spheres_dense_collision.urdf (robot description, URDF)
Before this commit: robot iiwa14, 11 links, 10 joints
Joints:
- joint iiwa_joint_1: limit lower=-2.96705972839 upper=2.96705972839 effort=320 velocity=1.48353 -> lower=-2.96705972839 upper=2.96705972839 effort=320 velocity=1.4835298641951802
- joint iiwa_joint_2: limit lower=-2.09439510239 upper=2.09439510239 effort=320 velocity=1.48353 -> lower=-2.09439510239 upper=2.09439510239 effort=320 velocity=1.4835298641951802
- joint iiwa_joint_3: limit lower=-2.96705972839 upper=2.96705972839 effort=176 velocity=1.74533 -> lower=-2.96705972839 upper=2.96705972839 effort=176 velocity=1.7453292519943295
- joint iiwa_joint_4: limit lower=-2.09439510239 upper=2.09439510239 effort=176 velocity=1.309 -> lower=-2.09439510239 upper=2.09439510239 effort=176 velocity=1.3089969389957472
- joint iiwa_joint_5: limit lower=-2.96705972839 upper=2.96705972839 effort=110 velocity=2.26893 -> lower=-2.96705972839 upper=2.96705972839 effort=110 velocity=2.2689280275926285
- joint iiwa_joint_6: limit lower=-2.09439510239 upper=2.09439510239 effort=40 velocity=2.35619 -> lower=-2.09439510239 upper=2.09439510239 effort=40 velocity=2.356194490192345
- joint iiwa_joint_7: limit lower=-3.05432619099 upper=3.05432619099 effort=40 velocity=2.35619 -> lower=-3.05432619099 upper=3.05432619099 effort=40 velocity=2.356194490192345

File: manipulation/models/iiwa_description/urdf/iiwa14_spheres_dense_elbow_collision.urdf (robot description, URDF)
Before this commit: robot iiwa14, 11 links, 10 joints
Joints:
- joint iiwa_joint_1: limit lower=-2.96705972839 upper=2.96705972839 effort=320 velocity=1.48353 -> lower=-2.96705972839 upper=2.96705972839 effort=320 velocity=1.4835298641951802
- joint iiwa_joint_2: limit lower=-2.09439510239 upper=2.09439510239 effort=320 velocity=1.48353 -> lower=-2.09439510239 upper=2.09439510239 effort=320 velocity=1.4835298641951802
- joint iiwa_joint_3: limit lower=-2.96705972839 upper=2.96705972839 effort=176 velocity=1.74533 -> lower=-2.96705972839 upper=2.96705972839 effort=176 velocity=1.7453292519943295
- joint iiwa_joint_4: limit lower=-2.09439510239 upper=2.09439510239 effort=176 velocity=1.309 -> lower=-2.09439510239 upper=2.09439510239 effort=176 velocity=1.3089969389957472
- joint iiwa_joint_5: limit lower=-2.96705972839 upper=2.96705972839 effort=110 velocity=2.26893 -> lower=-2.96705972839 upper=2.96705972839 effort=110 velocity=2.2689280275926285
- joint iiwa_joint_6: limit lower=-2.09439510239 upper=2.09439510239 effort=40 velocity=2.35619 -> lower=-2.09439510239 upper=2.09439510239 effort=40 velocity=2.356194490192345
- joint iiwa_joint_7: limit lower=-3.05432619099 upper=3.05432619099 effort=40 velocity=2.35619 -> lower=-3.05432619099 upper=3.05432619099 effort=40 velocity=2.356194490192345

File: manipulation/models/iiwa_description/urdf/planar_iiwa14_spheres_dense_elbow_collision.urdf (robot description, URDF)
Before this commit: robot iiwa14, 10 links, 9 joints
Joints:
- joint iiwa_joint_2: limit lower=-2.09439510239 upper=2.09439510239 effort=320 velocity=1.48353 -> lower=-2.09439510239 upper=2.09439510239 effort=320 velocity=1.4835298641951802
- joint iiwa_joint_4: limit lower=-2.09439510239 upper=2.09439510239 effort=176 velocity=1.309 -> lower=-2.09439510239 upper=2.09439510239 effort=176 velocity=1.3089969389957472
- joint iiwa_joint_6: limit lower=-2.09439510239 upper=2.09439510239 effort=40 velocity=2.35619 -> lower=-2.09439510239 upper=2.09439510239 effort=40 velocity=2.356194490192345
