Commit message: adding joint limits kuka model tests

File: manipulation/models/iiwa_description/urdf/iiwa14_no_collision.urdf (robot description, URDF)
Before this commit: robot iiwa14, 11 links, 10 joints
Joints:
- joint iiwa_joint_5: limit lower=-2.96705972839 upper=2.96705972839 effort=110 velocity=2.9670597283903604 -> lower=-2.96705972839 upper=2.96705972839 effort=110 velocity=2.2689280275926285
