Commit message: Update iiwa visual representation
This exposes the underlying geometry which includes the
kuka logo and "elbow" patches. It also merges
coincident vertices and computes per-vertex mesh
normals. It updates all sdf and urdf files to reference
the new objs.

NOTE: Although an OBJ file can support multiple
materials are data pipeline *can't*. As such, if
different meshes receive different materials, we
currently require them to be different meshes.

File: manipulation/models/iiwa_description/urdf/iiwa14.xacro (robot description, xacro)
@@ -128,9 +128,16 @@
       </inertial>
       <visual>
-        <origin xyz="0 0 0" rpy="0 0 0"/>
-        <geometry>
-          <mesh filename="../meshes/visual/link_2.obj"/>
+        <origin rpy="0 0 0" xyz="0 0 0"/>
+        <geometry>
+          <mesh filename="../meshes/visual/link_2_orange.obj"/>
         </geometry>
         <material name="Orange"/>
+      </visual>
+      <visual>
+        <origin rpy="0 0 0" xyz="0 0 0"/>
+        <geometry>
+          <mesh filename="../meshes/visual/link_2_grey.obj"/>
+        </geometry>
+        <material name="Grey"/>
       </visual>
       <xacro:if value="${collision_type == 'mesh'}">
@@ -181,4 +188,18 @@
         <material name="Grey"/>
       </visual>
+      <visual>
+        <origin rpy="0 0 0" xyz="0 0 0"/>
+        <geometry>
+          <mesh filename="../meshes/visual/kuka.obj"/>
+        </geometry>
+        <material name="Black"/>
+      </visual>
+      <visual>
+        <origin rpy="0 0 0" xyz="0 0 0"/>
+        <geometry>
+          <mesh filename="../meshes/visual/band.obj"/>
+        </geometry>
+        <material name="Silver"/>
+      </visual>
       <xacro:if value="${collision_type == 'mesh'}">
         <collision>
@@ -222,9 +243,16 @@
       </inertial>
       <visual>
-        <origin xyz="0 0 0" rpy="0 0 0"/>
-        <geometry>
-          <mesh filename="../meshes/visual/link_4.obj"/>
+        <origin rpy="0 0 0" xyz="0 0 0"/>
+        <geometry>
+          <mesh filename="../meshes/visual/link_4_orange.obj"/>
         </geometry>
         <material name="Orange"/>
+      </visual>
+      <visual>
+        <origin rpy="0 0 0" xyz="0 0 0"/>
+        <geometry>
+          <mesh filename="../meshes/visual/link_4_grey.obj"/>
+        </geometry>
+        <material name="Grey"/>
       </visual>
       <xacro:if value="${collision_type == 'mesh'}">
@@ -275,4 +303,18 @@
         <material name="Grey"/>
       </visual>
+      <visual>
+        <origin rpy="0 0 0" xyz="0 0 0"/>
+        <geometry>
+          <mesh filename="../meshes/visual/kuka.obj"/>
+        </geometry>
+        <material name="Black"/>
+      </visual>
+      <visual>
+        <origin rpy="0 0 0" xyz="0 0 0"/>
+        <geometry>
+          <mesh filename="../meshes/visual/band.obj"/>
+        </geometry>
+        <material name="Silver"/>
+      </visual>
       <xacro:if value="${collision_type == 'mesh'}">
         <collision>
@@ -316,7 +358,14 @@
       </inertial>
       <visual>
-        <origin xyz="0 0 0" rpy="0 0 0"/>
-        <geometry>
-          <mesh filename="../meshes/visual/link_6.obj"/>
+        <origin rpy="0 0 0" xyz="0 0 0"/>
+        <geometry>Silver
+          <mesh filename="../meshes/visual/link_6_grey.obj"/>
+        </geometry>
+        <material name="Grey"/>
+      </visual>
+      <visual>
+        <origin rpy="0 0 0" xyz="0 0 0"/>
+        <geometry>
+          <mesh filename="../meshes/visual/link_6_orange.obj"/>
         </geometry>
         <material name="Orange"/>

File: manipulation/models/iiwa_description/urdf/iiwa14_polytope_collision.urdf (robot description, URDF)
Before this commit: robot iiwa14, 11 links, 10 joints
Links:
- link iiwa_link_2: geometry visual mesh filename=../meshes/visual/link_2_grey.obj; visual mesh filename=../meshes/visual/link_2_orange.obj
- link iiwa_link_3: geometry visual mesh filename=../meshes/visual/band.obj; visual mesh filename=../meshes/visual/kuka.obj
- link iiwa_link_4: geometry visual mesh filename=../meshes/visual/link_4_grey.obj; visual mesh filename=../meshes/visual/link_4_orange.obj
- link iiwa_link_5: geometry visual mesh filename=../meshes/visual/band.obj; visual mesh filename=../meshes/visual/kuka.obj
- link iiwa_link_6: geometry visual mesh filename=../meshes/visual/link_6_grey.obj; visual mesh filename=../meshes/visual/link_6_orange.obj

Commit message: update on velocity and effort for kuka iiwa14

File: manipulation/models/iiwa_description/urdf/iiwa14.xacro (robot description, xacro)
@@ -15,6 +15,4 @@
   <xacro:property name="safety_controller_k_vel" value="2"/>
   <xacro:property name="joint_damping" value="0.5"/>
-  <xacro:property name="max_effort" value="300"/>
-  <xacro:property name="max_velocity" value="10"/>
   <xacro:macro name="iiwa14" params="parent hardware_interface robot_name collision_type *origin">
     <!--joint between {parent} and link_0-->
@@ -69,5 +67,5 @@
       <origin xyz="0 0 0.1575" rpy="0 0 0"/>
       <axis xyz="0 0 1"/>
-      <limit lower="${-170 * PI / 180}" upper="${170 * PI / 180}" effort="${max_effort}" velocity="${max_velocity}"/>
+      <limit lower="${-170 * PI / 180}" upper="${170 * PI / 180}" effort="320" velocity="1.48353"/>
       <safety_controller soft_lower_limit="${-168 * PI / 180}" soft_upper_limit="${168 * PI / 180}" k_position="${safety_controller_k_pos}" k_velocity="${safety_controller_k_vel}"/>
       <dynamics damping="${joint_damping}"/>
@@ -112,5 +110,5 @@
       <origin xyz="0 0 0.2025" rpy="${PI / 2}   0 ${PI}"/>
       <axis xyz="0 0 1"/>
-      <limit lower="${-120 * PI / 180}" upper="${120 * PI / 180}" effort="${max_effort}" velocity="${max_velocity}"/>
+      <limit lower="${-120 * PI / 180}" upper="${120 * PI / 180}" effort="320" velocity="1.48353"/>
       <safety_controller soft_lower_limit="${-118 * PI / 180}" soft_upper_limit="${118 * PI / 180}" k_position="${safety_controller_k_pos}" k_velocity="${safety_controller_k_vel}"/>
       <dynamics damping="${joint_damping}"/>
@@ -164,5 +162,5 @@
       <origin xyz="0 0.2045 0" rpy="${PI / 2} 0 ${PI}"/>
       <axis xyz="0 0 1"/>
-      <limit lower="${-170 * PI / 180}" upper="${170 * PI / 180}" effort="${max_effort}" velocity="${max_velocity}"/>
+      <limit lower="${-170 * PI / 180}" upper="${170 * PI / 180}" effort="176" velocity="1.74533"/>
       <safety_controller soft_lower_limit="${-118 * PI / 180}" soft_upper_limit="${118 * PI / 180}" k_position="${safety_controller_k_pos}" k_velocity="${safety_controller_k_vel}"/>
       <dynamics damping="${joint_damping}"/>
@@ -223,5 +221,5 @@
       <origin xyz="0 0 0.2155" rpy="${PI / 2} 0 0"/>
       <axis xyz="0 0 1"/>
-      <limit lower="${-120 * PI / 180}" upper="${120 * PI / 180}" effort="${max_effort}" velocity="${max_velocity}"/>
+      <limit lower="${-120 * PI / 180}" upper="${120 * PI / 180}" effort="176" velocity="1.309"/>
       <safety_controller soft_lower_limit="${-118 * PI / 180}" soft_upper_limit="${118 * PI / 180}" k_position="${safety_controller_k_pos}" k_velocity="${safety_controller_k_vel}"/>
       <dynamics damping="${joint_damping}"/>
@@ -275,5 +273,5 @@
       <origin xyz="0 0.1845 0" rpy="${-PI / 2} ${PI} 0"/>
       <axis xyz="0 0 1"/>
-      <limit lower="${-170 * PI / 180}" upper="${170 * PI / 180}" effort="${max_effort}" velocity="${max_velocity}"/>
+      <limit lower="${-170 * PI / 180}" upper="${170 * PI / 180}" effort="110" velocity="2.26893"/>
       <safety_controller soft_lower_limit="${-118 * PI / 180}" soft_upper_limit="${118 * PI / 180}" k_position="${safety_controller_k_pos}" k_velocity="${safety_controller_k_vel}"/>
       <dynamics damping="${joint_damping}"/>
@@ -334,5 +332,5 @@
       <origin xyz="0 0 0.2155" rpy="${PI / 2} 0 0"/>
       <axis xyz="0 0 1"/>
-      <limit lower="${-120 * PI / 180}" upper="${120 * PI / 180}" effort="${max_effort}" velocity="${max_velocity}"/>
+      <limit lower="${-120 * PI / 180}" upper="${120 * PI / 180}" effort="40" velocity="2.35619"/>
       <safety_controller soft_lower_limit="${-118 * PI / 180}" soft_upper_limit="${118 * PI / 180}" k_position="${safety_controller_k_pos}" k_velocity="${safety_controller_k_vel}"/>
       <dynamics damping="${joint_damping}"/>
@@ -388,5 +386,5 @@
       <origin xyz="0 0.081 0" rpy="${- PI / 2} ${PI} 0"/>
       <axis xyz="0 0 1"/>
-      <limit lower="${-175 * PI / 180}" upper="${175 * PI / 180}" effort="${max_effort}" velocity="${max_velocity}"/>
+      <limit lower="${-175 * PI / 180}" upper="${175 * PI / 180}" effort="40" velocity="2.35619"/>
       <safety_controller soft_lower_limit="${-173 * PI / 180}" soft_upper_limit="${173 * PI / 180}" k_position="${safety_controller_k_pos}" k_velocity="${safety_controller_k_vel}"/>
       <dynamics damping="${joint_damping}"/>

File: manipulation/models/iiwa_description/urdf/iiwa14_no_collision.urdf (robot description, URDF)
Before this commit: robot iiwa14, 11 links, 10 joints
Joints:
- joint iiwa_joint_1: limit lower=-2.96705972839 upper=2.96705972839 effort=300 velocity=10 -> lower=-2.96705972839 upper=2.96705972839 effort=320 velocity=1.39626
- joint iiwa_joint_2: limit lower=-2.09439510239 upper=2.09439510239 effort=300 velocity=10 -> lower=-2.09439510239 upper=2.09439510239 effort=320 velocity=1.39626
- joint iiwa_joint_3: limit lower=-2.96705972839 upper=2.96705972839 effort=300 velocity=10 -> lower=-2.96705972839 upper=2.96705972839 effort=176 velocity=1.74533
- joint iiwa_joint_4: limit lower=-2.09439510239 upper=2.09439510239 effort=300 velocity=10 -> lower=-2.09439510239 upper=2.09439510239 effort=176 velocity=1.309
- joint iiwa_joint_5: limit lower=-2.96705972839 upper=2.96705972839 effort=300 velocity=10 -> lower=-2.96705972839 upper=2.96705972839 effort=110 velocity=2.26893
- joint iiwa_joint_6: limit lower=-2.09439510239 upper=2.09439510239 effort=300 velocity=10 -> lower=-2.09439510239 upper=2.09439510239 effort=40 velocity=2.35619
- joint iiwa_joint_7: limit lower=-3.05432619099 upper=3.05432619099 effort=300 velocity=10 -> lower=-3.05432619099 upper=3.05432619099 effort=40 velocity=2.35619

File: manipulation/models/iiwa_description/urdf/iiwa14_spheres_collision.urdf (robot description, URDF)
Before this commit: robot iiwa14, 11 links, 10 joints
Joints:
- joint iiwa_joint_1: limit lower=-2.96705972839 upper=2.96705972839 effort=300 velocity=10 -> lower=-2.96705972839 upper=2.96705972839 effort=320 velocity=1.48353
- joint iiwa_joint_2: limit lower=-2.09439510239 upper=2.09439510239 effort=300 velocity=10 -> lower=-2.09439510239 upper=2.09439510239 effort=320 velocity=1.48353
- joint iiwa_joint_3: limit lower=-2.96705972839 upper=2.96705972839 effort=300 velocity=10 -> lower=-2.96705972839 upper=2.96705972839 effort=176 velocity=1.74533
- joint iiwa_joint_4: limit lower=-2.09439510239 upper=2.09439510239 effort=300 velocity=10 -> lower=-2.09439510239 upper=2.09439510239 effort=176 velocity=1.309
- joint iiwa_joint_5: limit lower=-2.96705972839 upper=2.96705972839 effort=300 velocity=10 -> lower=-2.96705972839 upper=2.96705972839 effort=110 velocity=2.26893
- joint iiwa_joint_6: limit lower=-2.09439510239 upper=2.09439510239 effort=300 velocity=10 -> lower=-2.09439510239 upper=2.09439510239 effort=40 velocity=2.35619
- joint iiwa_joint_7: limit lower=-3.05432619099 upper=3.05432619099 effort=300 velocity=10 -> lower=-3.05432619099 upper=3.05432619099 effort=40 velocity=2.35619

File: manipulation/models/iiwa_description/urdf/iiwa14_spheres_dense_collision.urdf (robot description, URDF)
Before this commit: robot iiwa14, 11 links, 10 joints
Joints:
- joint iiwa_joint_1: limit lower=-2.96705972839 upper=2.96705972839 effort=300 velocity=10 -> lower=-2.96705972839 upper=2.96705972839 effort=320 velocity=1.48353
- joint iiwa_joint_2: limit lower=-2.09439510239 upper=2.09439510239 effort=300 velocity=10 -> lower=-2.09439510239 upper=2.09439510239 effort=320 velocity=1.48353
- joint iiwa_joint_3: limit lower=-2.96705972839 upper=2.96705972839 effort=300 velocity=10 -> lower=-2.96705972839 upper=2.96705972839 effort=176 velocity=1.74533
- joint iiwa_joint_4: limit lower=-2.09439510239 upper=2.09439510239 effort=300 velocity=10 -> lower=-2.09439510239 upper=2.09439510239 effort=176 velocity=1.309
- joint iiwa_joint_5: limit lower=-2.96705972839 upper=2.96705972839 effort=300 velocity=10 -> lower=-2.96705972839 upper=2.96705972839 effort=110 velocity=2.26893
- joint iiwa_joint_6: limit lower=-2.09439510239 upper=2.09439510239 effort=300 velocity=10 -> lower=-2.09439510239 upper=2.09439510239 effort=40 velocity=2.35619
- joint iiwa_joint_7: limit lower=-3.05432619099 upper=3.05432619099 effort=300 velocity=10 -> lower=-3.05432619099 upper=3.05432619099 effort=40 velocity=2.35619

File: manipulation/models/iiwa_description/urdf/iiwa14_spheres_dense_elbow_collision.urdf (robot description, URDF)
Before this commit: robot iiwa14, 11 links, 10 joints
Joints:
- joint iiwa_joint_1: limit lower=-2.96705972839 upper=2.96705972839 effort=300 velocity=10 -> lower=-2.96705972839 upper=2.96705972839 effort=320 velocity=1.48353
- joint iiwa_joint_2: limit lower=-2.09439510239 upper=2.09439510239 effort=300 velocity=10 -> lower=-2.09439510239 upper=2.09439510239 effort=320 velocity=1.48353
- joint iiwa_joint_3: limit lower=-2.96705972839 upper=2.96705972839 effort=300 velocity=10 -> lower=-2.96705972839 upper=2.96705972839 effort=176 velocity=1.74533
- joint iiwa_joint_4: limit lower=-2.09439510239 upper=2.09439510239 effort=300 velocity=10 -> lower=-2.09439510239 upper=2.09439510239 effort=176 velocity=1.309
- joint iiwa_joint_5: limit lower=-2.96705972839 upper=2.96705972839 effort=300 velocity=10 -> lower=-2.96705972839 upper=2.96705972839 effort=110 velocity=2.26893
- joint iiwa_joint_6: limit lower=-2.09439510239 upper=2.09439510239 effort=300 velocity=10 -> lower=-2.09439510239 upper=2.09439510239 effort=40 velocity=2.35619
- joint iiwa_joint_7: limit lower=-3.05432619099 upper=3.05432619099 effort=300 velocity=10 -> lower=-3.05432619099 upper=3.05432619099 effort=40 velocity=2.35619

File: manipulation/models/iiwa_description/urdf/planar_iiwa14_spheres_dense_elbow_collision.urdf (robot description, URDF)
Before this commit: robot iiwa14, 10 links, 9 joints
Joints:
- joint iiwa_joint_2: limit lower=-2.09439510239 upper=2.09439510239 effort=300 velocity=10 -> lower=-2.09439510239 upper=2.09439510239 effort=320 velocity=1.48353
- joint iiwa_joint_4: limit lower=-2.09439510239 upper=2.09439510239 effort=300 velocity=10 -> lower=-2.09439510239 upper=2.09439510239 effort=176 velocity=1.309
- joint iiwa_joint_6: limit lower=-2.09439510239 upper=2.09439510239 effort=300 velocity=10 -> lower=-2.09439510239 upper=2.09439510239 effort=40 velocity=2.35619

Commit message: Replace .obj references to .gltf

File: manipulation/models/iiwa_description/urdf/iiwa14.xacro (robot description, xacro)
@@ -31,5 +31,5 @@
         <origin xyz="0 0 0" rpy="0 0 0"/>
         <geometry>
-          <mesh filename="package://drake_models/iiwa_description/meshes/iiwa14/visual/link_0.obj"/>
+          <mesh filename="package://drake_models/iiwa_description/meshes/iiwa14/visual/link_0.gltf"/>
         </geometry>
         <material name="Grey"/>
@@ -82,5 +82,5 @@
         <origin xyz="0 0 0" rpy="0 0 0"/>
         <geometry>
-          <mesh filename="package://drake_models/iiwa_description/meshes/iiwa14/visual/link_1.obj"/>
+          <mesh filename="package://drake_models/iiwa_description/meshes/iiwa14/visual/link_1.gltf"/>
         </geometry>
         <material name="Grey"/>
@@ -129,5 +129,5 @@
         <origin rpy="0 0 0" xyz="0 0 0"/>
         <geometry>
-          <mesh filename="package://drake_models/iiwa_description/meshes/iiwa14/visual/link_2_orange.obj"/>
+          <mesh filename="package://drake_models/iiwa_description/meshes/iiwa14/visual/link_2_orange.gltf"/>
         </geometry>
         <material name="Orange"/>
@@ -136,5 +136,5 @@
         <origin rpy="0 0 0" xyz="0 0 0"/>
         <geometry>
-          <mesh filename="package://drake_models/iiwa_description/meshes/iiwa14/visual/link_2_grey.obj"/>
+          <mesh filename="package://drake_models/iiwa_description/meshes/iiwa14/visual/link_2_grey.gltf"/>
         </geometry>
         <material name="Grey"/>
@@ -183,5 +183,5 @@
         <origin xyz="0 0 0" rpy="0 0 0"/>
         <geometry>
-          <mesh filename="package://drake_models/iiwa_description/meshes/iiwa14/visual/link_3.obj"/>
+          <mesh filename="package://drake_models/iiwa_description/meshes/iiwa14/visual/link_3.gltf"/>
         </geometry>
         <material name="Grey"/>
@@ -244,5 +244,5 @@
         <origin rpy="0 0 0" xyz="0 0 0"/>
         <geometry>
-          <mesh filename="package://drake_models/iiwa_description/meshes/iiwa14/visual/link_4_orange.obj"/>
+          <mesh filename="package://drake_models/iiwa_description/meshes/iiwa14/visual/link_4_orange.gltf"/>
         </geometry>
         <material name="Orange"/>
@@ -251,5 +251,5 @@
         <origin rpy="0 0 0" xyz="0 0 0"/>
         <geometry>
-          <mesh filename="package://drake_models/iiwa_description/meshes/iiwa14/visual/link_4_grey.obj"/>
+          <mesh filename="package://drake_models/iiwa_description/meshes/iiwa14/visual/link_4_grey.gltf"/>
         </geometry>
         <material name="Grey"/>
@@ -298,5 +298,5 @@
         <origin xyz="0 0 0" rpy="0 0 0"/>
         <geometry>
-          <mesh filename="package://drake_models/iiwa_description/meshes/iiwa14/visual/link_5.obj"/>
+          <mesh filename="package://drake_models/iiwa_description/meshes/iiwa14/visual/link_5.gltf"/>
         </geometry>
         <material name="Grey"/>
@@ -359,12 +359,12 @@
         <origin rpy="0 0 0" xyz="0 0 0"/>
         <geometry>
-          <mesh filename="package://drake_models/iiwa_description/meshes/iiwa14/visual/link_6_grey.obj"/>
-        </geometry>
-        <material name="Grey"/>
-      </visual>
-      <visual>
-        <origin rpy="0 0 0" xyz="0 0 0"/>
-        <geometry>
-          <mesh filename="package://drake_models/iiwa_description/meshes/iiwa14/visual/link_6_orange.obj"/>
+          <mesh filename="package://drake_models/iiwa_description/meshes/iiwa14/visual/link_6_grey.gltf"/>
+        </geometry>
+        <material name="Grey"/>
+      </visual>
+      <visual>
+        <origin rpy="0 0 0" xyz="0 0 0"/>
+        <geometry>
+          <mesh filename="package://drake_models/iiwa_description/meshes/iiwa14/visual/link_6_orange.gltf"/>
         </geometry>
         <material name="Orange"/>
@@ -415,5 +415,5 @@
         <origin xyz="0 0 0" rpy="0 0 0"/>
         <geometry>
-          <mesh filename="package://drake_models/iiwa_description/meshes/iiwa14/visual/link_7.obj"/>
+          <mesh filename="package://drake_models/iiwa_description/meshes/iiwa14/visual/link_7.gltf"/>
         </geometry>
         <material name="Grey"/>

Commit message: Catch *.obj references outside `iiwa_description`

File: manipulation/models/iiwa_description/urdf/iiwa14.xacro (robot description, xacro)
@@ -190,5 +190,5 @@
         <origin rpy="0 0 0" xyz="0 0 0"/>
         <geometry>
-          <mesh filename="package://drake_models/iiwa_description/meshes/iiwa14/visual/kuka.obj"/>
+          <mesh filename="package://drake_models/iiwa_description/meshes/iiwa14/visual/kuka.gltf"/>
         </geometry>
         <material name="Black"/>
@@ -197,5 +197,5 @@
         <origin rpy="0 0 0" xyz="0 0 0"/>
         <geometry>
-          <mesh filename="package://drake_models/iiwa_description/meshes/iiwa14/visual/band.obj"/>
+          <mesh filename="package://drake_models/iiwa_description/meshes/iiwa14/visual/band.gltf"/>
         </geometry>
         <material name="Silver"/>
@@ -305,5 +305,5 @@
         <origin rpy="0 0 0" xyz="0 0 0"/>
         <geometry>
-          <mesh filename="package://drake_models/iiwa_description/meshes/iiwa14/visual/kuka.obj"/>
+          <mesh filename="package://drake_models/iiwa_description/meshes/iiwa14/visual/kuka.gltf"/>
         </geometry>
         <material name="Black"/>
@@ -312,5 +312,5 @@
         <origin rpy="0 0 0" xyz="0 0 0"/>
         <geometry>
-          <mesh filename="package://drake_models/iiwa_description/meshes/iiwa14/visual/band.obj"/>
+          <mesh filename="package://drake_models/iiwa_description/meshes/iiwa14/visual/band.gltf"/>
         </geometry>
         <material name="Silver"/>
