Commit message: Fix stray material tags on gltf in xacro file

File: manipulation/models/iiwa_description/urdf/iiwa14.xacro (robot description, xacro)
@@ -33,5 +33,4 @@
           <mesh filename="package://drake_models/iiwa_description/meshes/iiwa14/visual/link_0.gltf"/>
         </geometry>
-        <material name="Grey"/>
       </visual>
       <xacro:if value="${collision_type == 'mesh'}">
@@ -84,5 +83,4 @@
           <mesh filename="package://drake_models/iiwa_description/meshes/iiwa14/visual/link_1.gltf"/>
         </geometry>
-        <material name="Grey"/>
       </visual>
       <xacro:if value="${collision_type == 'mesh'}">
@@ -131,5 +129,4 @@
           <mesh filename="package://drake_models/iiwa_description/meshes/iiwa14/visual/link_2_orange.gltf"/>
         </geometry>
-        <material name="Orange"/>
       </visual>
       <visual>
@@ -138,5 +135,4 @@
           <mesh filename="package://drake_models/iiwa_description/meshes/iiwa14/visual/link_2_grey.gltf"/>
         </geometry>
-        <material name="Grey"/>
       </visual>
       <xacro:if value="${collision_type == 'mesh'}">
@@ -185,5 +181,4 @@
           <mesh filename="package://drake_models/iiwa_description/meshes/iiwa14/visual/link_3.gltf"/>
         </geometry>
-        <material name="Grey"/>
       </visual>
       <visual>
@@ -192,5 +187,4 @@
           <mesh filename="package://drake_models/iiwa_description/meshes/iiwa14/visual/kuka.gltf"/>
         </geometry>
-        <material name="Black"/>
       </visual>
       <visual>
@@ -199,5 +193,4 @@
           <mesh filename="package://drake_models/iiwa_description/meshes/iiwa14/visual/band.gltf"/>
         </geometry>
-        <material name="Silver"/>
       </visual>
       <xacro:if value="${collision_type == 'mesh'}">
@@ -246,5 +239,4 @@
           <mesh filename="package://drake_models/iiwa_description/meshes/iiwa14/visual/link_4_orange.gltf"/>
         </geometry>
-        <material name="Orange"/>
       </visual>
       <visual>
@@ -300,5 +292,4 @@
           <mesh filename="package://drake_models/iiwa_description/meshes/iiwa14/visual/link_5.gltf"/>
         </geometry>
-        <material name="Grey"/>
       </visual>
       <visual>
@@ -307,5 +298,4 @@
           <mesh filename="package://drake_models/iiwa_description/meshes/iiwa14/visual/kuka.gltf"/>
         </geometry>
-        <material name="Black"/>
       </visual>
       <visual>
@@ -314,5 +304,4 @@
           <mesh filename="package://drake_models/iiwa_description/meshes/iiwa14/visual/band.gltf"/>
         </geometry>
-        <material name="Silver"/>
       </visual>
       <xacro:if value="${collision_type == 'mesh'}">
@@ -361,5 +350,4 @@
           <mesh filename="package://drake_models/iiwa_description/meshes/iiwa14/visual/link_6_grey.gltf"/>
         </geometry>
-        <material name="Grey"/>
       </visual>
       <visual>
@@ -368,5 +356,4 @@
           <mesh filename="package://drake_models/iiwa_description/meshes/iiwa14/visual/link_6_orange.gltf"/>
         </geometry>
-        <material name="Orange"/>
       </visual>
       <xacro:if value="${collision_type == 'mesh'}">
@@ -417,5 +404,4 @@
           <mesh filename="package://drake_models/iiwa_description/meshes/iiwa14/visual/link_7.gltf"/>
         </geometry>
-        <material name="Grey"/>
       </visual>
       <xacro:if value="${collision_type == 'mesh'}">

Commit message: Update IIWA `.obj` references to `.gltf` (#21079)
[workspace] Upgrade drake_models to latest commit

Co-authored-by: Jeremy Nimmer <jeremy.nimmer@tri.global>

File: manipulation/models/iiwa_description/urdf/iiwa14.xacro (robot description, xacro)
@@ -31,7 +31,6 @@
         <origin xyz="0 0 0" rpy="0 0 0"/>
         <geometry>
-          <mesh filename="package://drake_models/iiwa_description/meshes/iiwa14/visual/link_0.obj"/>
-        </geometry>
-        <material name="Grey"/>
+          <mesh filename="package://drake_models/iiwa_description/meshes/iiwa14/visual/link_0.gltf"/>
+        </geometry>
       </visual>
       <xacro:if value="${collision_type == 'mesh'}">
@@ -82,7 +81,6 @@
         <origin xyz="0 0 0" rpy="0 0 0"/>
         <geometry>
-          <mesh filename="package://drake_models/iiwa_description/meshes/iiwa14/visual/link_1.obj"/>
-        </geometry>
-        <material name="Grey"/>
+          <mesh filename="package://drake_models/iiwa_description/meshes/iiwa14/visual/link_1.gltf"/>
+        </geometry>
       </visual>
       <xacro:if value="${collision_type == 'mesh'}">
@@ -129,14 +127,12 @@
         <origin rpy="0 0 0" xyz="0 0 0"/>
         <geometry>
-          <mesh filename="package://drake_models/iiwa_description/meshes/iiwa14/visual/link_2_orange.obj"/>
-        </geometry>
-        <material name="Orange"/>
-      </visual>
-      <visual>
-        <origin rpy="0 0 0" xyz="0 0 0"/>
-        <geometry>
-          <mesh filename="package://drake_models/iiwa_description/meshes/iiwa14/visual/link_2_grey.obj"/>
-        </geometry>
-        <material name="Grey"/>
+          <mesh filename="package://drake_models/iiwa_description/meshes/iiwa14/visual/link_2_orange.gltf"/>
+        </geometry>
+      </visual>
+      <visual>
+        <origin rpy="0 0 0" xyz="0 0 0"/>
+        <geometry>
+          <mesh filename="package://drake_models/iiwa_description/meshes/iiwa14/visual/link_2_grey.gltf"/>
+        </geometry>
       </visual>
       <xacro:if value="${collision_type == 'mesh'}">
@@ -183,21 +179,18 @@
         <origin xyz="0 0 0" rpy="0 0 0"/>
         <geometry>
-          <mesh filename="package://drake_models/iiwa_description/meshes/iiwa14/visual/link_3.obj"/>
-        </geometry>
-        <material name="Grey"/>
-      </visual>
-      <visual>
-        <origin rpy="0 0 0" xyz="0 0 0"/>
-        <geometry>
-          <mesh filename="package://drake_models/iiwa_description/meshes/iiwa14/visual/kuka.obj"/>
-        </geometry>
-        <material name="Black"/>
-      </visual>
-      <visual>
-        <origin rpy="0 0 0" xyz="0 0 0"/>
-        <geometry>
-          <mesh filename="package://drake_models/iiwa_description/meshes/iiwa14/visual/band.obj"/>
-        </geometry>
-        <material name="Silver"/>
+          <mesh filename="package://drake_models/iiwa_description/meshes/iiwa14/visual/link_3.gltf"/>
+        </geometry>
+      </visual>
+      <visual>
+        <origin rpy="0 0 0" xyz="0 0 0"/>
+        <geometry>
+          <mesh filename="package://drake_models/iiwa_description/meshes/iiwa14/visual/kuka.gltf"/>
+        </geometry>
+      </visual>
+      <visual>
+        <origin rpy="0 0 0" xyz="0 0 0"/>
+        <geometry>
+          <mesh filename="package://drake_models/iiwa_description/meshes/iiwa14/visual/band.gltf"/>
+        </geometry>
       </visual>
       <xacro:if value="${collision_type == 'mesh'}">
@@ -244,12 +237,11 @@
         <origin rpy="0 0 0" xyz="0 0 0"/>
         <geometry>
-          <mesh filename="package://drake_models/iiwa_description/meshes/iiwa14/visual/link_4_orange.obj"/>
-        </geometry>
-        <material name="Orange"/>
-      </visual>
-      <visual>
-        <origin rpy="0 0 0" xyz="0 0 0"/>
-        <geometry>
-          <mesh filename="package://drake_models/iiwa_description/meshes/iiwa14/visual/link_4_grey.obj"/>
+          <mesh filename="package://drake_models/iiwa_description/meshes/iiwa14/visual/link_4_orange.gltf"/>
+        </geometry>
+      </visual>
+      <visual>
+        <origin rpy="0 0 0" xyz="0 0 0"/>
+        <geometry>
+          <mesh filename="package://drake_models/iiwa_description/meshes/iiwa14/visual/link_4_grey.gltf"/>
         </geometry>
         <material name="Grey"/>
@@ -298,21 +290,18 @@
         <origin xyz="0 0 0" rpy="0 0 0"/>
         <geometry>
-          <mesh filename="package://drake_models/iiwa_description/meshes/iiwa14/visual/link_5.obj"/>
-        </geometry>
-        <material name="Grey"/>
-      </visual>
-      <visual>
-        <origin rpy="0 0 0" xyz="0 0 0"/>
-        <geometry>
-          <mesh filename="package://drake_models/iiwa_description/meshes/iiwa14/visual/kuka.obj"/>
-        </geometry>
-        <material name="Black"/>
-      </visual>
-      <visual>
-        <origin rpy="0 0 0" xyz="0 0 0"/>
-        <geometry>
-          <mesh filename="package://drake_models/iiwa_description/meshes/iiwa14/visual/band.obj"/>
-        </geometry>
-        <material name="Silver"/>
+          <mesh filename="package://drake_models/iiwa_description/meshes/iiwa14/visual/link_5.gltf"/>
+        </geometry>
+      </visual>
+      <visual>
+        <origin rpy="0 0 0" xyz="0 0 0"/>
+        <geometry>
+          <mesh filename="package://drake_models/iiwa_description/meshes/iiwa14/visual/kuka.gltf"/>
+        </geometry>
+      </visual>
+      <visual>
+        <origin rpy="0 0 0" xyz="0 0 0"/>
+        <geometry>
+          <mesh filename="package://drake_models/iiwa_description/meshes/iiwa14/visual/band.gltf"/>
+        </geometry>
       </visual>
       <xacro:if value="${collision_type == 'mesh'}">
@@ -359,14 +348,12 @@
         <origin rpy="0 0 0" xyz="0 0 0"/>
         <geometry>
-          <mesh filename="package://drake_models/iiwa_description/meshes/iiwa14/visual/link_6_grey.obj"/>
-        </geometry>
-        <material name="Grey"/>
-      </visual>
-      <visual>
-        <origin rpy="0 0 0" xyz="0 0 0"/>
-        <geometry>
-          <mesh filename="package://drake_models/iiwa_description/meshes/iiwa14/visual/link_6_orange.obj"/>
-        </geometry>
-        <material name="Orange"/>
+          <mesh filename="package://drake_models/iiwa_description/meshes/iiwa14/visual/link_6_grey.gltf"/>
+        </geometry>
+      </visual>
+      <visual>
+        <origin rpy="0 0 0" xyz="0 0 0"/>
+        <geometry>
+          <mesh filename="package://drake_models/iiwa_description/meshes/iiwa14/visual/link_6_orange.gltf"/>
+        </geometry>
       </visual>
       <xacro:if value="${collision_type == 'mesh'}">
@@ -415,7 +402,6 @@
         <origin xyz="0 0 0" rpy="0 0 0"/>
         <geometry>
-          <mesh filename="package://drake_models/iiwa_description/meshes/iiwa14/visual/link_7.obj"/>
-        </geometry>
-        <material name="Grey"/>
+          <mesh filename="package://drake_models/iiwa_description/meshes/iiwa14/visual/link_7.gltf"/>
+        </geometry>
       </visual>
       <xacro:if value="${collision_type == 'mesh'}">
