Commit message: Switch to element tag

File: multibody/parsing/test/urdf_parser_test/convex_and_nonconvex_test.urdf (robot description, URDF)
Before this commit: robot non_conflicting_materials_2, 1 links, 0 joints
Links:
- link base_link: geometry collision mesh filename=../tri_cube.obj scale=1.1 1.1 1.1; collision mesh filename=../tri_cube.obj scale=1.1 1.1 1.1
