Commit message: Support capsule in parsing urdf

File: multibody/parsing/test/urdf_parser_test/non_conflicting_materials_1.urdf (robot description, URDF)
Before this commit: robot non_conflicting_materials_1, 1 links, 0 joints
Links:
- link base_link: geometry visual box size=.2 .2 .2; visual capsule length=0.5 radius=0.2
