Commit message: Textured objects
Previously, the only textured objects allowed were for mesh objects and
the texture had to be the same name as the mesh file.

This opens the door to applying textures to any of the primitives.
Furthermore, the texture can be specified in either URDF or SDF (via a
custom drake tag).

The textures are used *only* in rendering (RenderEngine*). Currently,
arbitrary textures are *not* communicated to drake visualizer. The concept
is tested in examples/scene_graph/bouncing_ball_run_dynamics.cc -- the
balls now have rainbow textures.

Updates MBP so that when a "visual" geometry is introduced, pre-existing
('phong', 'diffuse_map') properties get passed along.

Finally, parsing infrastructure was modified to support deferred image
validation. (After all, an image can be specified in URDF/SDF but if it
isn't consumed in the system, missing the image isn't actually a problem.)

File: multibody/parsing/test/urdf_parser_test/non_conflicting_materials_2.urdf (robot description, URDF)
Before this commit: robot non_conflicting_materials_2, 1 links, 0 joints
Links:
- added link material_by_name, mass 1; visual sphere radius=0.1
