Commit message: [parsing] Fix mis-parse of collision filter groups
Closes: #16310

Previously, a typo'd element name caused only the first element of
`drake:ignored_collision_filter_group` within a group to be actually
processed.  This patch fixes the typo and extends the existing tests to
cover the error case. Regrettably, it does not attempt a more vigorous
test refactoring. That may happen in the near future.

File: multibody/parsing/test/urdf_parser_test/collision_filter_group_parsing_test.urdf (robot description, URDF)
Before this commit: robot collision_filter_group_parsing_test, 4 links, 3 joints
Links:
- added link link5, mass 1; collision sphere radius=0.40
- added link link6, mass 1; collision sphere radius=0.40
