Commit message: Parse joint effort limits from URDF
Fixes #12859

File: multibody/parsing/test/urdf_parser_test/joint_parsing_test.urdf (robot description, URDF)
Before this commit: robot joint_parsing_test, 4 links, 3 joints
Joints:
- joint prismatic_joint: limit lower=-2 upper=1 effort=100 velocity=5 -> lower=-2 upper=1 effort=0 velocity=5

Commit message: parsing: Added ball and universal joints to urdf parser
Also made parsing tests more complete

File: multibody/parsing/test/urdf_parser_test/joint_parsing_test.urdf (robot description, URDF)
Before this commit: robot joint_parsing_test, 4 links, 3 joints
Links:
- added link link5, mass 1
- added link link6, mass 1
Joints:
- added joint ball_joint: type ball, parent link4, child link5, origin xyz=0 0 0 rpy=0 0 0
- added joint universal_joint: type universal, parent link5, child link6, origin xyz=0 0 0 rpy=0 0 0

Commit message: Add URDF continuous joint parsing test

File: multibody/parsing/test/urdf_parser_test/joint_parsing_test.urdf (robot description, URDF)
Before this commit: robot joint_parsing_test, 7 links, 4 joints
Links:
- added link link8, mass 1
Joints:
- added joint continuous_joint: type continuous, parent link7, child link8, origin xyz=0 0 0 rpy=0 0 0, axis 0 0 1

Commit message: Parse screw joints in URDF
Signed-off-by: Steve Peters <scpeters@openrobotics.org>

File: multibody/parsing/test/urdf_parser_test/joint_parsing_test.urdf (robot description, URDF)
Before this commit: robot joint_parsing_test, 8 links, 5 joints
Links:
- added link link9, mass 1

Commit message: [parsing] Add support for URDF mimic element.
Implements parsing support for the `<mimic>` element in URDF. Towards #17663.

Users could have been using existing URDF models in Drake with mimic
tags that were ignored. Now those models will be simulated differently
if they are being simulated with DiscreteContactSolver::kSap.

File: multibody/parsing/test/urdf_parser_test/joint_parsing_test.urdf (robot description, URDF)
Before this commit: robot joint_parsing_test, 9 links, 5 joints
Links:
- added link link10, mass 1
Joints:
- added joint revolute_joint_with_mimic: type revolute, parent link9, child link10, axis 0 0 1, mimic joint=revolute_joint multiplier=1.23 offset=4.56

Commit message: [parsing] Fix URDF planar joint support
Support the correct, standard 'joint' spelling of planar joints. Since
Drake only supported the incorrect 'drake:joint' spelling for several
years, continue to accept that as well.

File: multibody/parsing/test/urdf_parser_test/joint_parsing_test.urdf (robot description, URDF)
Before this commit: robot joint_parsing_test, 9 links, 5 joints
Joints:
- added joint planar_joint: type planar, parent link6, child link7, origin xyz=0 0 0 rpy=0 0 0

Commit message: [parsing] Add parsing of custom drake:mimic tag for SDFormat
Also fixes a small bug in the URDF parser for <mimic> elements
that specify a joint that is defined after the <joint> the tag
is a member of.

File: multibody/parsing/test/urdf_parser_test/joint_parsing_test.urdf (robot description, URDF)
Before this commit: robot joint_parsing_test, 10 links, 7 joints
Links:
- added link link11, mass 1
Joints:
- added joint revolute_joint_to_mimic: type revolute, parent link10, child link11, axis 0 0 1
- joint revolute_joint_with_mimic: mimic joint=revolute_joint multiplier=1.23 offset=4.56 -> joint=revolute_joint_to_mimic multiplier=1.23 offset=4.56

Commit message: [multibody] Add URDF and SDF Parsing for Curvilinear Joints (#22196)
Adds tags and joint configuration structure to URDF and SDF parsers
for CurvilinearJoint.

File: multibody/parsing/test/urdf_parser_test/joint_parsing_test.urdf (robot description, URDF)
Before this commit: robot joint_parsing_test, 12 links, 9 joints
Links:
- added link link13, mass 1
- added link link14, mass 1
