Commit message: Increase joint position limits to match Kinova documentation

File: manipulation/models/jaco_description/urdf/j2s7s300.urdf (robot description, URDF)
Before this commit: robot j2s7s300, 16 links, 15 joints
Joints:
- joint j2s7s300_joint_1: limit lower=-6.28318530718 upper=6.28318530718 effort=2000 velocity=1 -> lower=-174.532925 upper=174.532925 effort=2000 velocity=1
- joint j2s7s300_joint_3: limit lower=-6.28318530718 upper=6.28318530718 effort=2000 velocity=1 -> lower=-174.532925 upper=174.532925 effort=2000 velocity=1
- joint j2s7s300_joint_5: limit lower=-6.28318530718 upper=6.28318530718 effort=2000 velocity=1 -> lower=-174.532925 upper=174.532925 effort=2000 velocity=1
- joint j2s7s300_joint_7: limit lower=-6.28318530718 upper=6.28318530718 effort=2000 velocity=1 -> lower=-174.532925 upper=174.532925 effort=2000 velocity=1

Commit message: Add numerical validation for shape specifications plus test

File: manipulation/models/jaco_description/urdf/j2s7s300.urdf (robot description, URDF)
Before this commit: robot j2s7s300, 16 links, 15 joints
Links:
- link base: geometry collision sphere radius=0; visual sphere radius=0
- link j2s7s300_end_effector: geometry collision sphere radius=0; visual sphere radius=0

Commit message: Checkpoint.

File: manipulation/models/jaco_description/urdf/j2s7s300.urdf (robot description, URDF)
Before this commit: robot j2s7s300, 16 links, 15 joints
Links:
- link base: geometry collision sphere radius=0; visual sphere radius=0
- link j2s7s300_end_effector: geometry collision sphere radius=0; visual sphere radius=0
Joints:
- joint j2s7s300_joint_1: limit lower=-6.28318530718 upper=6.28318530718 effort=2000 velocity=1 -> lower=-174.532925 upper=174.532925 effort=2000 velocity=1
- joint j2s7s300_joint_3: limit lower=-6.28318530718 upper=6.28318530718 effort=2000 velocity=1 -> lower=-174.532925 upper=174.532925 effort=2000 velocity=1
- joint j2s7s300_joint_5: limit lower=-6.28318530718 upper=6.28318530718 effort=2000 velocity=1 -> lower=-174.532925 upper=174.532925 effort=2000 velocity=1
- joint j2s7s300_joint_7: limit lower=-6.28318530718 upper=6.28318530718 effort=2000 velocity=1 -> lower=-174.532925 upper=174.532925 effort=2000 velocity=1
