Commit message: Add hand/arm only jaco 7dof models, along with sphere collision versions

File: manipulation/models/jaco_description/urdf/j2s7s300_arm.urdf (robot description, URDF)
Before this commit: robot j2s7s300, 16 links, 15 joints
Links:
- removed link j2s7s300_end_effector
- removed link j2s7s300_link_finger_1
- removed link j2s7s300_link_finger_2
- removed link j2s7s300_link_finger_3
- removed link j2s7s300_link_finger_tip_1
- removed link j2s7s300_link_finger_tip_2
- removed link j2s7s300_link_finger_tip_3
- link j2s7s300_link_7: mass 0.727 -> 0.001; geometry 
Joints:
- removed joint j2s7s300_joint_end_effector
- removed joint j2s7s300_joint_finger_1
- removed joint j2s7s300_joint_finger_2
- removed joint j2s7s300_joint_finger_3
- removed joint j2s7s300_joint_finger_tip_1
- removed joint j2s7s300_joint_finger_tip_2
- removed joint j2s7s300_joint_finger_tip_3

File: manipulation/models/jaco_description/urdf/j2s7s300_arm_sphere_collision.urdf (robot description, URDF)
Before this commit: robot j2s7s300, 16 links, 15 joints
Links:
- removed link j2s7s300_end_effector
- removed link j2s7s300_link_finger_1
- removed link j2s7s300_link_finger_2
- removed link j2s7s300_link_finger_3
- removed link j2s7s300_link_finger_tip_1
- removed link j2s7s300_link_finger_tip_2
- removed link j2s7s300_link_finger_tip_3
- link j2s7s300_link_1: geometry collision sphere radius=0.02; collision sphere radius=0.02
- link j2s7s300_link_2: geometry collision sphere radius=0.02; collision sphere radius=0.02
- link j2s7s300_link_3: geometry collision sphere radius=0.015; collision sphere radius=0.015
- link j2s7s300_link_4: geometry collision sphere radius=0.015; collision sphere radius=0.015
- link j2s7s300_link_5: geometry collision sphere radius=0.0325; collision sphere radius=0.035
- link j2s7s300_link_6: geometry collision sphere radius=0.035; collision sphere radius=0.035
- link j2s7s300_link_7: mass 0.727 -> 0.001; geometry 
- link j2s7s300_link_base: geometry collision sphere radius=0.045; collision sphere radius=0.045
Joints:
- removed joint j2s7s300_joint_end_effector
- removed joint j2s7s300_joint_finger_1
- removed joint j2s7s300_joint_finger_2
- removed joint j2s7s300_joint_finger_3
- removed joint j2s7s300_joint_finger_tip_1
- removed joint j2s7s300_joint_finger_tip_2
- removed joint j2s7s300_joint_finger_tip_3

File: manipulation/models/jaco_description/urdf/j2s7s300_sphere_collision.urdf (robot description, URDF)
Before this commit: robot j2s7s300, 16 links, 15 joints
Links:
- link j2s7s300_link_1: geometry collision sphere radius=0.02; collision sphere radius=0.02
- link j2s7s300_link_2: geometry collision sphere radius=0.02; collision sphere radius=0.02
- link j2s7s300_link_3: geometry collision sphere radius=0.015; collision sphere radius=0.015
- link j2s7s300_link_4: geometry collision sphere radius=0.015; collision sphere radius=0.015
- link j2s7s300_link_5: geometry collision sphere radius=0.0325; collision sphere radius=0.035
- link j2s7s300_link_6: geometry collision sphere radius=0.035; collision sphere radius=0.035
- link j2s7s300_link_7: geometry collision sphere radius=0.03; collision sphere radius=0.03
- link j2s7s300_link_base: geometry collision sphere radius=0.045; collision sphere radius=0.045
- link j2s7s300_link_finger_1: geometry collision sphere radius=0.013; collision sphere radius=0.014
- link j2s7s300_link_finger_2: geometry collision sphere radius=0.013; collision sphere radius=0.014
- link j2s7s300_link_finger_3: geometry collision sphere radius=0.013; collision sphere radius=0.014
- link j2s7s300_link_finger_tip_1: geometry collision sphere radius=0.01; collision sphere radius=0.01
- link j2s7s300_link_finger_tip_2: geometry collision sphere radius=0.01; collision sphere radius=0.01
- link j2s7s300_link_finger_tip_3: geometry collision sphere radius=0.01; collision sphere radius=0.01

Commit message: Add hand/arm only jaco 7dof models, along with sphere collision versions

File: manipulation/models/jaco_description/urdf/j2s7s300_arm.urdf (robot description, URDF)
Before this commit: robot j2s7s300, 16 links, 15 joints
Links:
- removed link j2s7s300_end_effector
- removed link j2s7s300_link_finger_1
- removed link j2s7s300_link_finger_2
- removed link j2s7s300_link_finger_3
- removed link j2s7s300_link_finger_tip_1
- removed link j2s7s300_link_finger_tip_2
- removed link j2s7s300_link_finger_tip_3
- link j2s7s300_link_7: mass 0.727 -> 0.001; geometry 
Joints:
- removed joint j2s7s300_joint_end_effector
- removed joint j2s7s300_joint_finger_1
- removed joint j2s7s300_joint_finger_2
- removed joint j2s7s300_joint_finger_3
- removed joint j2s7s300_joint_finger_tip_1
- removed joint j2s7s300_joint_finger_tip_2
- removed joint j2s7s300_joint_finger_tip_3

File: manipulation/models/jaco_description/urdf/j2s7s300_arm_sphere_collision.urdf (robot description, URDF)
Before this commit: robot j2s7s300, 16 links, 15 joints
Links:
- removed link j2s7s300_end_effector
- removed link j2s7s300_link_finger_1
- removed link j2s7s300_link_finger_2
- removed link j2s7s300_link_finger_3
- removed link j2s7s300_link_finger_tip_1
- removed link j2s7s300_link_finger_tip_2
- removed link j2s7s300_link_finger_tip_3
- link j2s7s300_link_1: geometry collision sphere radius=0.02; collision sphere radius=0.02
- link j2s7s300_link_2: geometry collision sphere radius=0.02; collision sphere radius=0.02
- link j2s7s300_link_3: geometry collision sphere radius=0.015; collision sphere radius=0.015
- link j2s7s300_link_4: geometry collision sphere radius=0.015; collision sphere radius=0.015
- link j2s7s300_link_5: geometry collision sphere radius=0.0325; collision sphere radius=0.035
- link j2s7s300_link_6: geometry collision sphere radius=0.035; collision sphere radius=0.035
- link j2s7s300_link_7: mass 0.727 -> 0.001; geometry 
- link j2s7s300_link_base: geometry collision sphere radius=0.045; collision sphere radius=0.045
Joints:
- removed joint j2s7s300_joint_end_effector
- removed joint j2s7s300_joint_finger_1
- removed joint j2s7s300_joint_finger_2
- removed joint j2s7s300_joint_finger_3
- removed joint j2s7s300_joint_finger_tip_1
- removed joint j2s7s300_joint_finger_tip_2
- removed joint j2s7s300_joint_finger_tip_3
