Commit message: Changed the code to support only j2s6s300 return incorrect joint number. Should 6 but it gives 7 I am using j2s6s300_sphere_collision.urdf as the modified file

File: manipulation/models/jaco_description/urdf/j2s6s300_sphere_collision.urdf (robot description, URDF)
Before this commit: robot j2s6s300, 16 links, 15 joints
Links:
- removed link world
- link j2s6s300_link_1: geometry collision mesh filename=../meshes/shoulder.dae; visual mesh filename=../meshes/ring_big.dae
- link j2s6s300_link_2: geometry collision mesh filename=../meshes/arm.dae; visual mesh filename=../meshes/arm.dae
- link j2s6s300_link_3: geometry collision mesh filename=../meshes/forearm.dae; visual mesh filename=../meshes/forearm.dae
- link j2s6s300_link_4: geometry collision mesh filename=../meshes/wrist_spherical_1.dae; visual mesh filename=../meshes/ring_small.dae
- link j2s6s300_link_5: geometry collision mesh filename=../meshes/wrist_spherical_2.dae; visual mesh filename=../meshes/ring_small.dae
- link j2s6s300_link_6: geometry collision mesh filename=../meshes/hand_3finger.dae; visual mesh filename=../meshes/hand_3finger.dae
- link j2s6s300_link_base: geometry collision mesh filename=../meshes/base.dae; visual mesh filename=../meshes/base.dae
- link j2s6s300_link_finger_1: geometry collision mesh filename=../meshes/finger_proximal.dae; visual mesh filename=../meshes/finger_proximal.dae
- link j2s6s300_link_finger_2: geometry collision mesh filename=../meshes/finger_proximal.dae; visual mesh filename=../meshes/finger_proximal.dae
- link j2s6s300_link_finger_3: geometry collision mesh filename=../meshes/finger_proximal.dae; visual mesh filename=../meshes/finger_proximal.dae
- link j2s6s300_link_finger_tip_1: geometry collision mesh filename=../meshes/finger_distal.dae; visual mesh filename=../meshes/finger_distal.dae
- link j2s6s300_link_finger_tip_2: geometry collision mesh filename=../meshes/finger_distal.dae; visual mesh filename=../meshes/finger_distal.dae
- link j2s6s300_link_finger_tip_3: geometry collision mesh filename=../meshes/finger_distal.dae; visual mesh filename=../finger_distal.dae
Joints:
- removed joint connect_root_and_world

Commit message: created a urdf file j2s6s300_sphere_collision.urdf from the j2s7s300_sphere_collision.urdf by removing joint 3 link 3 Found that the jaco_condstants.h was used to get the number joints using the simulator Even though the changes look correct the simulator run but does not look correct. Using the real arm the system goes nutty

File: manipulation/models/jaco_description/urdf/j2s6s300_sphere_collision.urdf (robot description, URDF)
Before this commit: robot j2s6s300, 15 links, 14 joints
Links:
- removed link j2s6s300_link_3
- added link j2s6s300_link_7, mass 0.727; collision sphere radius=0.03; collision sphere radius=0.03
- link base: geometry collision sphere radius=0; visual sphere radius=0
- link j2s6s300_end_effector: geometry collision sphere radius=0; visual sphere radius=0
- link j2s6s300_link_1: geometry collision sphere radius=0.02; collision sphere radius=0.02
- link j2s6s300_link_2: mass 0.99 -> 0.8447; geometry collision sphere radius=0.02; collision sphere radius=0.02
- link j2s6s300_link_4: mass 0.463 -> 0.6763; geometry collision sphere radius=0.015; collision sphere radius=0.015
- link j2s6s300_link_5: geometry collision sphere radius=0.0325; collision sphere radius=0.035
- link j2s6s300_link_6: mass 0.99 -> 0.463; geometry collision sphere radius=0.035; collision sphere radius=0.035
- link j2s6s300_link_base: geometry collision sphere radius=0.045; collision sphere radius=0.045
- link j2s6s300_link_finger_1: geometry collision sphere radius=0.013; collision sphere radius=0.014
- link j2s6s300_link_finger_2: geometry collision sphere radius=0.013; collision sphere radius=0.014
- link j2s6s300_link_finger_3: geometry collision sphere radius=0.013; collision sphere radius=0.014
- link j2s6s300_link_finger_tip_1: geometry collision sphere radius=0.01; collision sphere radius=0.01
- link j2s6s300_link_finger_tip_2: geometry collision sphere radius=0.01; collision sphere radius=0.01
- link j2s6s300_link_finger_tip_3: geometry collision sphere radius=0.01; collision sphere radius=0.01
Joints:
- removed joint j2s6s300_joint_3
- added joint j2s6s300_joint_7: type continuous, parent j2s6s300_link_6, child j2s6s300_link_7, origin xyz=0 0.10375 0 rpy=-1.57079632679 0 3.14159265359, axis 0 0 1, limit lower=-174.532925 upper=174.532925 effort=2000 velocity=1
- joint j2s6s300_joint_1: limit lower=-6.28318530718 upper=6.28318530718 effort=40 velocity=0.628318530718 -> lower=-174.532925 upper=174.532925 effort=2000 velocity=1
- joint j2s6s300_joint_2: limit lower=0.820304748437 upper=5.46288055874 effort=80 velocity=0.628318530718 -> lower=0.523598775598 upper=5.75958653158 effort=2000 velocity=1
- joint j2s6s300_joint_4: limit lower=-6.28318530718 upper=6.28318530718 effort=20 velocity=0.837758040957 -> lower=0.523598775598 upper=5.75958653158 effort=2000 velocity=1; origin xyz=0 0.2073 -0.0114 rpy=-1.57079632679 0 3.14159265359 -> xyz=0.0 -0.410 0.0 rpy=0.0  3.14159265359 0.0; parent j2s6s300_link_3 -> j2s6s300_link_2; type continuous -> revolute
- joint j2s6s300_joint_5: limit lower=0.523598775598 upper=5.75958653158 effort=20 velocity=0.837758040957 -> lower=-174.532925 upper=174.532925 effort=2000 velocity=1; origin xyz=0 0 -0.10375 rpy=1.57079632679 0 3.14159265359 -> xyz=0 0.2073 -0.0114 rpy=-1.57079632679 0 3.14159265359; type revolute -> continuous
- joint j2s6s300_joint_6: limit lower=-6.28318530718 upper=6.28318530718 effort=20 velocity=0.837758040957 -> lower=0.523598775598 upper=5.75958653158 effort=2000 velocity=1; origin xyz=0 0.10375 0 rpy=-1.57079632679 0 3.14159265359 -> xyz=0 0 -0.10375 rpy=1.57079632679 0 3.14159265359; type continuous -> revolute
- joint j2s6s300_joint_base: limit lower=0 upper=0 effort=0 velocity=0 -> lower=0 upper=0 effort=2000 velocity=1
- joint j2s6s300_joint_end_effector: origin xyz=0 0 -0.1600 rpy=3.14159265359 0 1.57079632679 -> xyz=0 0 -0.1600 rpy=3.14159265359 0 0; parent j2s6s300_link_6 -> j2s6s300_link_7
- joint j2s6s300_joint_finger_1: limit lower=0 upper=1.51 effort=2 velocity=1 -> lower=0 upper=2 effort=2000 velocity=1; parent j2s6s300_link_6 -> j2s6s300_link_7
- joint j2s6s300_joint_finger_2: limit lower=0 upper=1.51 effort=2 velocity=1 -> lower=0 upper=2 effort=2000 velocity=1; parent j2s6s300_link_6 -> j2s6s300_link_7
- joint j2s6s300_joint_finger_3: limit lower=0 upper=1.51 effort=2 velocity=1 -> lower=0 upper=2 effort=2000 velocity=1; parent j2s6s300_link_6 -> j2s6s300_link_7
- joint j2s6s300_joint_finger_tip_1: limit lower=0 upper=2 effort=2 velocity=1 -> lower=0 upper=2 effort=2000 velocity=1; type revolute -> fixed
- joint j2s6s300_joint_finger_tip_2: limit lower=0 upper=2 effort=2 velocity=1 -> lower=0 upper=2 effort=2000 velocity=1; type revolute -> fixed
- joint j2s6s300_joint_finger_tip_3: limit lower=0 upper=2 effort=2 velocity=1 -> lower=0 upper=2 effort=2000 velocity=1; type revolute -> fixed

Commit message: found a little error in the wrapper in the 3rd joint

File: manipulation/models/jaco_description/urdf/j2s6s300_sphere_collision.urdf (robot description, URDF)
Before this commit: robot j2s6s300, 15 links, 14 joints
Links:
- link j2s6s300_link_4: geometry collision sphere radius=0.015; collision sphere radius=0.015

Commit message: I used the j2s7s300_sperical_collision.urdf as reference for j2s6s300_sperical_collision.urdf I relabeled the links and joints in the file j2s6s300_sperical_collision.urdf to make it easier following logical by using link and joint number increment to be 1

File: manipulation/models/jaco_description/urdf/j2s6s300_sphere_collision.urdf (robot description, URDF)
Before this commit: robot j2s6s300, 15 links, 14 joints
Links:
- removed link j2s6s300_link_7
- added link j2s6s300_link_3, mass 0.6763; collision sphere radius=0.015; collision sphere radius=0.015
- link j2s6s300_link_4: mass 0.6763 -> 0.463; geometry collision sphere radius=0.0325; collision sphere radius=0.035
- link j2s6s300_link_5: geometry collision sphere radius=0.035; collision sphere radius=0.035
- link j2s6s300_link_6: mass 0.463 -> 0.727; geometry collision sphere radius=0.03; collision sphere radius=0.03
Joints:
- removed joint j2s6s300_joint_7
- added joint j2s6s300_joint_3: type revolute, parent j2s6s300_link_2, child j2s6s300_link_3, origin xyz=0.0 -0.410 0.0 rpy=0.0  3.14159265359 0.0, axis 0 0 1, limit lower=0.523598775598 upper=5.75958653158 effort=2000 velocity=1
- joint j2s6s300_joint_4: limit lower=0.523598775598 upper=5.75958653158 effort=2000 velocity=1 -> lower=-174.532925 upper=174.532925 effort=2000 velocity=1; origin xyz=0.0 -0.410 0.0 rpy=0.0  3.14159265359 0.0 -> xyz=0 0.2073 -0.0114 rpy=-1.57079632679 0 3.14159265359; parent j2s6s300_link_2 -> j2s6s300_link_3; type revolute -> continuous
- joint j2s6s300_joint_5: limit lower=-174.532925 upper=174.532925 effort=2000 velocity=1 -> lower=0.523598775598 upper=5.75958653158 effort=2000 velocity=1; origin xyz=0 0.2073 -0.0114 rpy=-1.57079632679 0 3.14159265359 -> xyz=0 0 -0.10375 rpy=1.57079632679 0 3.14159265359; type continuous -> revolute
- joint j2s6s300_joint_6: limit lower=0.523598775598 upper=5.75958653158 effort=2000 velocity=1 -> lower=-174.532925 upper=174.532925 effort=2000 velocity=1; origin xyz=0 0 -0.10375 rpy=1.57079632679 0 3.14159265359 -> xyz=0 0.10375 0 rpy=-1.57079632679 0 3.14159265359; type revolute -> continuous
- joint j2s6s300_joint_end_effector: parent j2s6s300_link_7 -> j2s6s300_link_6
- joint j2s6s300_joint_finger_1: parent j2s6s300_link_7 -> j2s6s300_link_6
- joint j2s6s300_joint_finger_2: parent j2s6s300_link_7 -> j2s6s300_link_6
- joint j2s6s300_joint_finger_3: parent j2s6s300_link_7 -> j2s6s300_link_6
