Commit message: Curate the urdf to remove gazebo related tags

File: examples/hsr/models/urdfs/hsrb4s.obj.urdf (robot description, URDF)
Before this commit: robot hsrb, 45 links, 44 joints
Links:
- link arm_flex_link: geometry collision mesh filename=../meshes/arm_v0/arm_flex.obj; visual mesh filename=../meshes/arm_v0/arm_flex_light.obj
- link arm_lift_link: geometry collision mesh filename=../meshes/arm_v0/shoulder.obj; visual mesh filename=../meshes/arm_v0/shoulder.obj
- link arm_roll_link: geometry collision mesh filename=../meshes/arm_v0/arm_roll.obj; visual mesh filename=../meshes/arm_v0/arm_roll_light.obj
- link base_link: geometry collision mesh filename=../meshes/base_v2/base.obj; visual mesh filename=../meshes/base_v2/base_light.obj
- link base_range_sensor_link: geometry collision mesh filename=../meshes/sensors/laser.obj; visual mesh filename=../meshes/sensors/laser.obj
- link hand_l_distal_link: geometry collision mesh filename=../meshes/hand_v0/l_distal.obj; visual mesh filename=../meshes/hand_v0/l_distal.obj
- link hand_l_spring_proximal_link: geometry collision mesh filename=../meshes/hand_v0/l_proximal.obj; visual mesh filename=../meshes/hand_v0/l_proximal.obj
- link hand_palm_link: geometry collision mesh filename=../meshes/hand_v0/palm.obj; visual mesh filename=../meshes/hand_v0/palm.obj
- link hand_r_distal_link: geometry collision mesh filename=../meshes/hand_v0/r_distal.obj; visual mesh filename=../meshes/hand_v0/r_distal.obj
- link hand_r_spring_proximal_link: geometry collision mesh filename=../meshes/hand_v0/r_proximal.obj; visual mesh filename=../meshes/hand_v0/r_proximal.obj
- link head_l_stereo_camera_link: geometry visual mesh filename=../meshes/sensors/head_camera.obj
- link head_pan_link: geometry collision mesh filename=../meshes/head_v1/head_pan.obj; visual mesh filename=../meshes/head_v1/head_pan.obj
- link head_r_stereo_camera_link: geometry visual mesh filename=../meshes/sensors/head_camera.obj
- link head_rgbd_sensor_link: geometry collision mesh filename=../meshes/sensors/rgbd.obj; visual mesh filename=../meshes/sensors/rgbd_light.obj
- link head_tilt_link: geometry collision mesh filename=../meshes/head_v1/head.obj; collision mesh filename=../meshes/head_v1/tablet.obj
- link torso_lift_link: geometry collision mesh filename=../meshes/torso_v0/torso.obj; visual mesh filename=../meshes/torso_v0/torso_light.obj
- link wrist_flex_link: geometry collision cylinder length=0.04 radius=0.017; visual cylinder length=0.02 radius=0.017
- link wrist_roll_link: geometry collision mesh filename=../meshes/wrist_v0/wrist_roll.obj; visual mesh filename=../meshes/wrist_v0/wrist_roll.obj
