Commit message: Add obj version of meshes

File: manipulation/models/franka_description/urdf/hand.urdf (robot description, URDF)
Before this commit: robot hand, 3 links, 2 joints
Links:
- link panda_hand: geometry collision cylinder length=0.1 radius=0.05; collision cylinder length=0.1 radius=0.07
- link panda_leftfinger: geometry visual mesh filename=package://franka_description/meshes/visual/finger.obj
- link panda_rightfinger: geometry visual mesh filename=package://franka_description/meshes/visual/finger.obj

File: manipulation/models/franka_description/urdf/panda_arm.urdf (robot description, URDF)
Before this commit: robot panda, 9 links, 8 joints
Links:
- link panda_link0: geometry collision cylinder length=0.03 radius=0.09; collision sphere radius=0.09
- link panda_link1: geometry collision cylinder length=0.2830 radius=0.09; collision sphere radius=0.09
- link panda_link2: geometry collision cylinder length=0.12 radius=0.09; collision sphere radius=0.09
- link panda_link3: geometry collision cylinder length=0.15 radius=0.09; collision sphere radius=0.09
- link panda_link4: geometry collision cylinder length=0.12 radius=0.09; collision sphere radius=0.09
- link panda_link5: geometry collision cylinder length=0.1 radius=0.09; collision cylinder length=0.14 radius=0.055
- link panda_link6: geometry collision cylinder length=0.08 radius=0.08; collision sphere radius=0.08
- link panda_link7: geometry collision cylinder length=0.14 radius=0.07; collision sphere radius=0.07

File: manipulation/models/franka_description/urdf/panda_arm_hand.urdf (robot description, URDF)
Before this commit: robot panda, 12 links, 11 joints
Links:
- link panda_hand: geometry collision cylinder length=0.1 radius=0.05; collision cylinder length=0.1 radius=0.07
- link panda_leftfinger: geometry visual mesh filename=package://franka_description/meshes/visual/finger.obj
- link panda_link0: geometry collision cylinder length=0.03 radius=0.09; collision sphere radius=0.09
- link panda_link1: geometry collision cylinder length=0.2830 radius=0.09; collision sphere radius=0.09
- link panda_link2: geometry collision cylinder length=0.12 radius=0.09; collision sphere radius=0.09
- link panda_link3: geometry collision cylinder length=0.15 radius=0.09; collision sphere radius=0.09
- link panda_link4: geometry collision cylinder length=0.12 radius=0.09; collision sphere radius=0.09
- link panda_link5: geometry collision cylinder length=0.1 radius=0.09; collision cylinder length=0.14 radius=0.055
- link panda_link6: geometry collision cylinder length=0.08 radius=0.08; collision sphere radius=0.08
- link panda_link7: geometry collision cylinder length=0.14 radius=0.07; collision sphere radius=0.07
- link panda_rightfinger: geometry visual mesh filename=package://franka_description/meshes/visual/finger.obj

Commit message: Add inertial properties

File: manipulation/models/franka_description/urdf/hand.urdf (robot description, URDF)
Before this commit: robot hand, 3 links, 2 joints
Links:
- link panda_hand: mass None -> 0.73
- link panda_leftfinger: mass None -> 0.1
- link panda_rightfinger: mass None -> 0.1

File: manipulation/models/franka_description/urdf/panda_arm.urdf (robot description, URDF)
Before this commit: robot panda, 9 links, 8 joints
Links:
- link panda_link0: mass None -> 2.92
- link panda_link1: mass None -> 2.74
- link panda_link2: mass None -> 2.74
- link panda_link3: mass None -> 2.38
- link panda_link4: mass None -> 2.38
- link panda_link5: mass None -> 2.74
- link panda_link6: mass None -> 1.55
- link panda_link7: mass None -> 0.54

File: manipulation/models/franka_description/urdf/panda_arm_hand.urdf (robot description, URDF)
Before this commit: robot panda, 12 links, 11 joints
Links:
- link panda_hand: mass None -> 0.73
- link panda_leftfinger: mass None -> 0.1
- link panda_link0: mass None -> 2.92
- link panda_link1: mass None -> 2.74
- link panda_link2: mass None -> 2.74
- link panda_link3: mass None -> 2.38
- link panda_link4: mass None -> 2.38
- link panda_link5: mass None -> 2.74
- link panda_link6: mass None -> 1.55
- link panda_link7: mass None -> 0.54
- link panda_rightfinger: mass None -> 0.1

Commit message: Shrink collision geometery significantly, convert to spheres.

File: manipulation/models/franka_description/urdf/hand.urdf (robot description, URDF)
Before this commit: robot hand, 3 links, 2 joints
Links:
- link panda_hand: geometry collision sphere radius=0.05; collision sphere radius=0.05
- link panda_leftfinger: geometry collision sphere radius=0.012; collision sphere radius=0.012
- link panda_rightfinger: geometry collision sphere radius=0.012; collision sphere radius=0.012

Commit message: Shrink collision geometery significantly, convert to spheres.

File: manipulation/models/franka_description/urdf/hand.urdf (robot description, URDF)
Before this commit: robot hand, 3 links, 2 joints
Links:
- link panda_hand: geometry collision sphere radius=0.05; collision sphere radius=0.05
- link panda_leftfinger: geometry collision sphere radius=0.012; visual mesh filename=package://franka_description/meshes/visual/finger.obj
- link panda_rightfinger: geometry collision sphere radius=0.012; visual mesh filename=package://franka_description/meshes/visual/finger.obj
