Commit message: [panda_arm] Upstream acc. limits and collision filtering from Anzu

File: manipulation/models/franka_description/urdf/panda_arm_hand.urdf (robot description, URDF)
Before this commit: robot panda, 12 links, 11 joints
Joints:
- joint panda_joint5: limit lower=-2.8973 upper=2.8973 effort=12 velocity=2.6100 -> lower=-2.8973 upper=2.8973 effort=12 velocity=2.610
