Commit message: comments from review

File: examples/multibody/strandbeest/model/LegAssembly.xacro (robot description, xacro)
@@ -95,5 +95,5 @@
       <child link="${prefix}_bar_i" />
     </joint>
-    <joint name="${prefix}_joint_k_i" type="revolute">
+    <joint name="${prefix}_joint_k_g" type="revolute">
       <axis xyz="0 1 0" />
       <parent link="${prefix}_bar_k" />
@@ -112,5 +112,5 @@
       <child link="${prefix}_bar_e" />
     </joint>
-    <joint name="${prefix}_joint_j_e" type="revolute">
+    <joint name="${prefix}_joint_j_b" type="revolute">
       <axis xyz="0 1 0" />
       <parent link="${prefix}_bar_j" />
@@ -119,5 +119,5 @@
       <limit lower="-1.9" upper="-1.0" effort="0" velocity="1000" />
     </joint>
-    <joint name="${prefix}_joint_e_f" type="revolute">
+    <joint name="${prefix}_joint_b_f" type="revolute">
       <axis xyz="0 1 0" />
       <parent link="${prefix}_bar_b" />

File: examples/multibody/strandbeest/model/Macros.xacro (robot description, xacro)
@@ -23,5 +23,5 @@
   <!-- Macro to create the inertial properties modelling pvc pipe -->
   <xacro:macro name="strandbeest_cylinder_inertial"
-      params="xyz rpy length radius">
+      params="xyz rpy length">
     <inertial>
       <origin xyz="${xyz}" rpy="${rpy}" />
@@ -55,5 +55,5 @@
       params="xyz rpy length radius material">
     <xacro:strandbeest_cylinder_inertial xyz="${xyz}" rpy="${rpy}"
-        length="${length}" radius="${radius}" />
+        length="${length}"/>
     <xacro:strandbeest_cylinder_visual xyz="${xyz}" rpy="${rpy}"
         length="${length}" radius="${radius}" material="${material}" />
