Commit message: wip: removal of warned-about elements

File: examples/multibody/strandbeest/model/Strandbeest.xacro (robot description, xacro)
@@ -68,5 +68,4 @@
     <joint name="joint_crossbar_crank"/>
     <actuator name="crossbar_crank_motor"/>
-    <mechanicalReduction>1</mechanicalReduction>
   </transmission>
   <!-- Macro to define a pair of legs at an offset along the crank shaft -->

File: examples/pr2/models/pr2_description/urdf/pr2_simplified.urdf (robot description, URDF)
Before this commit: robot pr2, 83 links, 83 joints
Joints:
- joint l_gripper_l_finger_tip_joint: mimic joint=l_gripper_l_finger_joint multiplier=1 offset=0 -> (none)
- joint l_gripper_l_parallel_root_joint: mimic joint=l_gripper_l_finger_joint multiplier=1 offset=0 -> (none)
- joint l_gripper_r_finger_joint: mimic joint=l_gripper_l_finger_joint multiplier=1 offset=0 -> (none)
- joint l_gripper_r_finger_tip_joint: mimic joint=l_gripper_l_finger_joint multiplier=1 offset=0 -> (none)
- joint l_gripper_r_parallel_root_joint: mimic joint=l_gripper_l_finger_joint multiplier=-1 offset=0 -> (none)
- joint r_gripper_l_finger_tip_joint: mimic joint=r_gripper_l_finger_joint multiplier=1 offset=0 -> (none)
- joint r_gripper_l_parallel_root_joint: mimic joint=r_gripper_l_finger_joint multiplier=1 offset=0 -> (none)
- joint r_gripper_r_finger_joint: mimic joint=r_gripper_l_finger_joint multiplier=1 offset=0 -> (none)
- joint r_gripper_r_finger_tip_joint: mimic joint=r_gripper_l_finger_joint multiplier=1 offset=0 -> (none)
- joint r_gripper_r_parallel_root_joint: mimic joint=r_gripper_l_finger_joint multiplier=-1 offset=0 -> (none)

File: manipulation/models/franka_description/urdf/hand.urdf (robot description, URDF)
Before this commit: robot hand, 3 links, 2 joints
Joints:
- joint panda_finger_joint2: mimic joint=panda_finger_joint1 -> (none)

File: manipulation/models/franka_description/urdf/panda_arm_hand.urdf (robot description, URDF)
Before this commit: robot panda, 12 links, 11 joints
Joints:
- joint panda_finger_joint2: mimic joint=panda_finger_joint1 -> (none)

Commit message: Adds option to model Strandbeest with constraints

File: examples/multibody/strandbeest/model/Strandbeest.xacro (robot description, xacro)
@@ -7,95 +7,97 @@
 -->
 <robot xmlns:drake="http://drake.mit.edu" xmlns:xsi="http://www.w3.org/2001/XMLSchema-instance" xmlns:xacro="http://ros.org/wiki/xacro" xsi:schemaLocation="../../doc/drakeURDF.xsd" name="Strandbeest">
-  <xacro:include filename="Macros.xacro"/>
-  <xacro:include filename="LegPair.xacro"/>
-  <!-- Materials -->
-  <material name="tri_red">
-    <color rgba="0.8 0 0 1"/>
-  </material>
-  <material name="tri_black">
-    <color rgba="0 0 0 1"/>
-  </material>
-  <material name="tri_grey">
-    <color rgba="0.6 0.6 0.6 1"/>
-  </material>
-  <!-- Fixed floor link for collision and walking -->
-  <link name="floor">
-    <inertial>
-      <origin rpy="0 0 0" xyz="0 0 0"/>
-      <mass value="1"/>
-      <inertia ixx="1" ixy="0" ixz="0" iyy="1" iyz="0" izz="1"/>
-    </inertial>
-    <visual>
-      <origin rpy="0 0 0" xyz="0 0 0"/>
-      <geometry>
-        <box size="10 10 1"/>
-      </geometry>
-      <material name="gray">
-        <color rgba=".4 .4 .4 1"/>
-      </material>
-    </visual>
-    <collision>
-      <origin rpy="0 0 0" xyz="0 0 0"/>
-      <geometry>
-        <box size="10 10 1"/>
-      </geometry>
-      <drake:proximity_properties>
-        <drake:mu_static value="1"/>
-        <drake:mu_dynamic value="0.6"/>
-      </drake:proximity_properties>
-    </collision>
-  </link>
-  <joint name="floor_weld" type="fixed">
-    <origin rpy="0 0 0" xyz="0 0 0.0"/>
-    <parent link="world"/>
-    <child link="floor"/>
-  </joint>
-  <!-- Links -->
-  <link name="crossbar">
-    <xacro:strandbeest_cylinder xyz="0 0 0" rpy="${pi/2} 0 0" length="1.2" radius="0.01" material="tri_black"/>
-  </link>
-  <link name="crank_axle">
-    <xacro:strandbeest_cylinder xyz="0 0 0" rpy="${pi/2} 0 0" length="1.2" radius="0.02" material="tri_red"/>
-  </link>
-  <!-- Joints -->
-  <joint name="joint_crossbar_crank" type="continuous">
-    <axis xyz="0 1 0"/>
-    <parent link="crossbar"/>
-    <child link="crank_axle"/>
-    <origin rpy="0 0 0" xyz="0 0 0.078"/>
-  </joint>
-  <transmission name="crossbar_crank_transmission" type="pr2_mechanism_model/SimpleTransmission">
-    <joint name="joint_crossbar_crank"/>
-    <actuator name="crossbar_crank_motor"/>
-    <mechanicalReduction>1</mechanicalReduction>
-  </transmission>
-  <!-- Macro to define a pair of legs at an offset along the crank shaft -->
-  <xacro:macro name="positioned_leg_pair" params="name offset angle">
-    <xacro:strandbeest_leg_pair prefix="${name}"/>
-    <joint name="${name}_joint_crossbar_l" type="fixed">
+  <xacro:macro name="strandbeest" params="with_constraints">
+    <xacro:include filename="Macros.xacro"/>
+    <xacro:include filename="LegPair.xacro"/>
+    <!-- Materials -->
+    <material name="tri_red">
+      <color rgba="0.8 0 0 1"/>
+    </material>
+    <material name="tri_black">
+      <color rgba="0 0 0 1"/>
+    </material>
+    <material name="tri_grey">
+      <color rgba="0.6 0.6 0.6 1"/>
+    </material>
+    <!-- Fixed floor link for collision and walking -->
+    <link name="floor">
+      <inertial>
+        <origin rpy="0 0 0" xyz="0 0 0"/>
+        <mass value="1"/>
+        <inertia ixx="1" ixy="0" ixz="0" iyy="1" iyz="0" izz="1"/>
+      </inertial>
+      <visual>
+        <origin rpy="0 0 0" xyz="0 0 0"/>
+        <geometry>
+          <box size="10 10 1"/>
+        </geometry>
+        <material name="gray">
+          <color rgba=".4 .4 .4 1"/>
+        </material>
+      </visual>
+      <collision>
+        <origin rpy="0 0 0" xyz="0 0 0"/>
+        <geometry>
+          <box size="10 10 1"/>
+        </geometry>
+        <drake:proximity_properties>
+          <drake:mu_static value="1"/>
+          <drake:mu_dynamic value="0.6"/>
+        </drake:proximity_properties>
+      </collision>
+    </link>
+    <joint name="floor_weld" type="fixed">
+      <origin rpy="0 0 0" xyz="0 0 0.0"/>
+      <parent link="world"/>
+      <child link="floor"/>
+    </joint>
+    <!-- Links -->
+    <link name="crossbar">
+      <xacro:strandbeest_cylinder xyz="0 0 0" rpy="${pi/2} 0 0" length="1.2" radius="0.01" material="tri_black"/>
+    </link>
+    <link name="crank_axle">
+      <xacro:strandbeest_cylinder xyz="0 0 0" rpy="${pi/2} 0 0" length="1.2" radius="0.02" material="tri_red"/>
+    </link>
+    <!-- Joints -->
+    <joint name="joint_crossbar_crank" type="continuous">
       <axis xyz="0 1 0"/>
       <parent link="crossbar"/>
-      <child link="${name}_bar_l"/>
-      <origin rpy="0 0 0" xyz="0 ${offset} 0"/>
+      <child link="crank_axle"/>
+      <origin rpy="0 0 0" xyz="0 0 0.078"/>
     </joint>
-    <joint name="${name}_joint_crank_axle_m" type="fixed">
-      <axis xyz="0 1 0"/>
-      <parent link="crank_axle"/>
-      <child link="${name}_bar_m"/>
-      <origin rpy="0 ${angle} 0" xyz="0 ${offset} 0"/>
-    </joint>
+    <transmission name="crossbar_crank_transmission" type="pr2_mechanism_model/SimpleTransmission">
+      <joint name="joint_crossbar_crank"/>
+      <actuator name="crossbar_crank_motor"/>
+      <mechanicalReduction>1</mechanicalReduction>
+    </transmission>
+    <!-- Macro to define a pair of legs at an offset along the crank shaft -->
+    <xacro:macro name="positioned_leg_pair" params="name offset angle">
+      <xacro:strandbeest_leg_pair prefix="${name}" with_constraints="${with_constraints}"/>
+      <joint name="${name}_joint_crossbar_l" type="fixed">
+        <axis xyz="0 1 0"/>
+        <parent link="crossbar"/>
+        <child link="${name}_bar_l"/>
+        <origin rpy="0 0 0" xyz="0 ${offset} 0"/>
+      </joint>
+      <joint name="${name}_joint_crank_axle_m" type="fixed">
+        <axis xyz="0 1 0"/>
+        <parent link="crank_axle"/>
+        <child link="${name}_bar_m"/>
+        <origin rpy="0 ${angle} 0" xyz="0 ${offset} 0"/>
+      </joint>
+    </xacro:macro>
+    <!-- Define the legs -->
+    <xacro:positioned_leg_pair name="pair01" offset="0.6" angle="0">
+    </xacro:positioned_leg_pair>
+    <xacro:positioned_leg_pair name="pair02" offset="0.36" angle="${2*pi/3}">
+    </xacro:positioned_leg_pair>
+    <xacro:positioned_leg_pair name="pair03" offset="0.12" angle="${4*pi/3}">
+    </xacro:positioned_leg_pair>
+    <xacro:positioned_leg_pair name="pair04" offset="-0.12" angle="${pi/3}">
+    </xacro:positioned_leg_pair>
+    <xacro:positioned_leg_pair name="pair05" offset="-0.36" angle="${3*pi/3}">
+    </xacro:positioned_leg_pair>
+    <xacro:positioned_leg_pair name="pair06" offset="-0.6" angle="${5*pi/3}">
+    </xacro:positioned_leg_pair>
   </xacro:macro>
-  <!-- Define the legs -->
-  <xacro:positioned_leg_pair name="pair01" offset="0.6" angle="0">
-  </xacro:positioned_leg_pair>
-  <xacro:positioned_leg_pair name="pair02" offset="0.36" angle="${2*pi/3}">
-  </xacro:positioned_leg_pair>
-  <xacro:positioned_leg_pair name="pair03" offset="0.12" angle="${4*pi/3}">
-  </xacro:positioned_leg_pair>
-  <xacro:positioned_leg_pair name="pair04" offset="-0.12" angle="${pi/3}">
-  </xacro:positioned_leg_pair>
-  <xacro:positioned_leg_pair name="pair05" offset="-0.36" angle="${3*pi/3}">
-  </xacro:positioned_leg_pair>
-  <xacro:positioned_leg_pair name="pair06" offset="-0.6" angle="${5*pi/3}">
-  </xacro:positioned_leg_pair>
 </robot>
