Commit message: Address Rick's comments.

File: examples/planar_gripper/planar_gripper.xacro (robot description, xacro)
@@ -63,5 +63,5 @@
         </visual>
       </link>
-      <joint name='finger${fnum}_ShoulderJoint' type='revolute'>
+      <joint name='finger${fnum}_BaseJoint' type='revolute'>
         <child>finger${fnum}_link1</child>
         <parent>finger${fnum}_base</parent>
@@ -70,5 +70,5 @@
           <limit>
             <!-- Drake parses a zero effort joint as an un-actuated joint. -->
-            <effort>100</effort>
+            <effort>75</effort>
             <lower>-1.57</lower>
             <upper>1.57</upper>
@@ -119,4 +119,16 @@
           </material>
         </visual>
+        <collision name='link2_collision'>
+          <pose>0 0 -${l2_length/2} 0 0 0</pose>
+          <geometry>
+            <cylinder>
+              <length>${l2_length}</length>
+              <radius>${l2_radius}</radius>
+            </cylinder>
+          </geometry>
+          <material>
+            <diffuse>1 0 0 1</diffuse>
+          </material>
+        </collision>
         <collision name='link2_pad_collision'>
           <pose>0 0 -${l2_length + sensor_stack_len + tip_radius} 0 0 0</pose>
@@ -139,5 +151,5 @@
         </visual>
       </link>
-      <joint name='finger${fnum}_ElbowJoint' type='revolute'>
+      <joint name='finger${fnum}_MidJoint' type='revolute'>
         <parent>finger${fnum}_link1</parent>
         <child>finger${fnum}_link2</child>
@@ -147,7 +159,5 @@
           <xyz>1 0 0</xyz>
           <limit>
-            <effort>100</effort>
-            <!-- No limit provided. sdformat defaults to -1, which we parse as
-                 an actuated joint. -->
+            <effort>75</effort>
             <lower>-1.57</lower>
             <upper>1.57</upper>

Commit message: Address Rick's comments.

File: examples/planar_gripper/planar_gripper.xacro (robot description, xacro)
@@ -63,5 +63,5 @@
         </visual>
       </link>
-      <joint name='finger${fnum}_ShoulderJoint' type='revolute'>
+      <joint name='finger${fnum}_BaseJoint' type='revolute'>
         <child>finger${fnum}_link1</child>
         <parent>finger${fnum}_base</parent>
@@ -70,5 +70,5 @@
           <limit>
             <!-- Drake parses a zero effort joint as an un-actuated joint. -->
-            <effort>100</effort>
+            <effort>75</effort>
             <lower>-1.57</lower>
             <upper>1.57</upper>
@@ -119,4 +119,16 @@
           </material>
         </visual>
+        <collision name='link2_collision'>
+          <pose>0 0 -${l2_length/2} 0 0 0</pose>
+          <geometry>
+            <cylinder>
+              <length>${l2_length}</length>
+              <radius>${l2_radius}</radius>
+            </cylinder>
+          </geometry>
+          <material>
+            <diffuse>1 0 0 1</diffuse>
+          </material>
+        </collision>
         <collision name='link2_pad_collision'>
           <pose>0 0 -${l2_length + sensor_stack_len + tip_radius} 0 0 0</pose>
@@ -139,5 +151,5 @@
         </visual>
       </link>
-      <joint name='finger${fnum}_ElbowJoint' type='revolute'>
+      <joint name='finger${fnum}_MidJoint' type='revolute'>
         <parent>finger${fnum}_link1</parent>
         <child>finger${fnum}_link2</child>
@@ -147,7 +159,5 @@
           <xyz>1 0 0</xyz>
           <limit>
-            <effort>100</effort>
-            <!-- No limit provided. sdformat defaults to -1, which we parse as
-                 an actuated joint. -->
+            <effort>75</effort>
             <lower>-1.57</lower>
             <upper>1.57</upper>
@@ -163,25 +173,4 @@
     <xacro:finger fnum="2" />
     <xacro:finger fnum="3" />
-    <!--<link name="finger1_ground">-->
-      <!--<pose>0 0 -${config_radius} 0 0 0</pose>-->
-    <!--</link>-->
-    <!--<joint name="finger1_weld" type="fixed">-->
-      <!--<child>finger1_base</child>-->
-      <!--<parent>finger1_ground</parent>-->
-    <!--</joint>-->
-    <!--<link name="finger2_ground">-->
-      <!--<pose>0 0 -${config_radius} ${config_angle} 0 0</pose>-->
-    <!--</link>-->
-    <!--<joint name="finger2_weld" type="fixed">-->
-      <!--<child>finger2_base</child>-->
-      <!--<parent>finger2_ground</parent>-->
-    <!--</joint>-->
-    <!--<link name="finger3_ground">-->
-      <!--<pose>0 0 -${config_radius} ${2*config_angle} 0 0</pose>-->
-    <!--</link>-->
-    <!--<joint name="finger3_weld" type="fixed">-->
-      <!--<child>finger3_base</child>-->
-      <!--<parent>finger3_ground</parent>-->
-    <!--</joint>-->
   </model>
 </sdf>

Commit message: Address Grant's comment.

File: examples/planar_gripper/planar_gripper.xacro (robot description, xacro)
@@ -13,6 +13,4 @@
     <xacro:property name="sensor_stack_len" value="0.001" />
     <xacro:property name="tip_radius" value="0.015" />
-    <!--<xacro:property name="config_radius" value="0.18" />-->
-    <!--<xacro:property name="config_angle" value="2.1" />-->
     <xacro:macro name="finger" params="fnum">
       <link name="finger${fnum}_base">

Commit message: Updates the planar_gripper model to match the hardware. Also updates the planar_brick.sdf model to match the 100x100x70 mm physical brick.

File: examples/planar_gripper/planar_gripper.xacro (robot description, xacro)
@@ -3,14 +3,19 @@
   <model name='planar_gripper'>
     <xacro:property name="base_dim" value=".08" />
-    <xacro:property name="l1_length" value="0.07" />
+    <xacro:property name="l1_length" value="0.085" />
     <xacro:property name="l1_radius" value="0.011" />
     <xacro:property name="l1_mass" value="0.1" />
     <xacro:property name="l1_inertia" value="0.0083" />
-    <xacro:property name="l2_length" value="0.07" />
+    <xacro:property name="l2_length" value="0.0403" />
     <xacro:property name="l2_radius" value="0.011" />
     <xacro:property name="l2_mass" value="0.1" />
     <xacro:property name="l2_inertia" value="0.0083" />
-    <xacro:property name="sensor_stack_len" value="0.001" />
-    <xacro:property name="tip_radius" value="0.015" />
+    <xacro:property name="sensor_length" value="0.0085" />
+    <xacro:property name="sensor_width" value="0.02" />
+    <xacro:property name="tip_adapter_length" value="0.0075" />
+    <xacro:property name="tip_adapter_radius" value="0.0145" />
+    <xacro:property name="tip_cylinder_length" value="0.0035" />
+    <xacro:property name="tip_cylinder_radius" value="0.01" />
+    <xacro:property name="tip_sphere_radius" value="0.015" />
     <xacro:macro name="finger" params="fnum">
       <link name="finger${fnum}_base">
@@ -106,46 +111,74 @@
           </material>
         </visual>
-        <visual name='link2_sensor'>
-          <pose>0 0 -${l2_length + sensor_stack_len} 0 0 0</pose>
+        <!--The link 2 collision element extends up to the sphere fingertip-->
+        <collision name='link2_collision'>
+          <pose>0 0 -${(l2_length + sensor_length + tip_adapter_length + tip_cylinder_length)/2} 0 0 0</pose>
+          <geometry>
+            <cylinder>
+              <length>${l2_length + sensor_length + tip_adapter_length + tip_cylinder_length}</length>
+              <radius>${l2_radius}</radius>
+            </cylinder>
+          </geometry>
+          <material>
+            <diffuse>1 0 1 1</diffuse>
+          </material>
+        </collision>
+        <visual name='link2_sensor_visual'>
+          <pose>0 0 -${l2_length + sensor_length/2.0} 0 0 0</pose>
+          <geometry>
+            <box>
+              <size>${sensor_width} ${sensor_width} ${sensor_length}</size>
+            </box>
+          </geometry>
+          <material>
+            <diffuse>.1 .1 .1 1</diffuse>
+          </material>
+        </visual>
+        <visual name="tip_adapter_visual">
+          <pose>0 0 -${l2_length + sensor_length + tip_adapter_length/2} 0 0 0</pose>
+          <geometry>
+            <cylinder>
+              <length>${tip_adapter_length}</length>
+              <radius>${tip_adapter_radius}</radius>
+            </cylinder>
+          </geometry>
+          <material>
+            <diffuse>.1 .1 .1 1</diffuse>
+          </material>
+        </visual>
+        <visual name="tip_cylinder_visual">
+          <pose>0 0 -${l2_length + sensor_length + tip_adapter_length + tip_cylinder_length/2} 0 0 0</pose>
+          <geometry>
+            <cylinder>
+              <length>${tip_cylinder_length}</length>
+              <radius>${tip_cylinder_radius}</radius>
+            </cylinder>
+          </geometry>
+          <material>
+            <diffuse>.1 .1 .1 1</diffuse>
+          </material>
+        </visual>
+        <visual name='tip_sphere_visual'>
+          <pose>0 0 -${l2_length + sensor_length + tip_adapter_length + tip_sphere_radius} 0 0 0</pose>
           <geometry>
             <sphere>
-              <radius>${l2_radius}</radius>
+              <radius>${tip_sphere_radius}</radius>
             </sphere>
           </geometry>
           <material>
-            <diffuse>.1 .1 .1 1</diffuse>
-          </material>
-        </visual>
-        <collision name='link2_collision'>
-          <pose>0 0 -${l2_length/2} 0 0 0</pose>
-          <geometry>
-            <cylinder>
-              <length>${l2_length}</length>
-              <radius>${l2_radius}</radius>
-            </cylinder>
-          </geometry>
-          <material>
-            <diffuse>1 0 0 1</diffuse>
+            <diffuse>1 1 1 1</diffuse>
+          </material>
+        </visual>
+        <collision name='tip_sphere_collision'>
+          <pose>0 0 -${l2_length + sensor_length + tip_adapter_length + tip_sphere_radius} 0 0 0</pose>
+          <geometry>
+            <sphere>
+              <radius>${tip_sphere_radius}</radius>
+            </sphere>
+          </geometry>
+          <material>
+            <diffuse>1 1 1 1</diffuse>
           </material>
         </collision>
-        <collision name='link2_pad_collision'>
-          <pose>0 0 -${l2_length + sensor_stack_len + tip_radius} 0 0 0</pose>
-          <geometry>
-            <sphere>
-              <radius>${tip_radius}</radius>
-            </sphere>
-          </geometry>
-        </collision>
-        <visual name='link2_pad_visual'>
-          <pose>0 0 -${l2_length + sensor_stack_len + tip_radius} 0 0 0</pose>
-          <geometry>
-            <sphere>
-              <radius>${tip_radius}</radius>
-            </sphere>
-          </geometry>
-          <material>
-            <diffuse>1 1 1 1</diffuse>
-          </material>
-        </visual>
       </link>
       <joint name='finger${fnum}_MidJoint' type='revolute'>

Commit message: Adds a weld joint to the planar_gripper fingers at the force sensor interface, splitting link 2 into two separate links.

File: examples/planar_gripper/planar_gripper.xacro (robot description, xacro)
@@ -2,4 +2,6 @@
 <sdf xmlns:xacro="http://www.ros.org/wiki/xacro" version='1.6'>
   <model name='planar_gripper'>
+    <!-- Link mass and inertia values are guesses (currently), calculated using
+         a uniform rod model, rotating about its center of mass. -->
     <xacro:property name="base_dim" value=".08" />
     <xacro:property name="l1_length" value="0.085" />
@@ -7,11 +9,11 @@
     <xacro:property name="l1_mass" value="0.1" />
     <xacro:property name="l1_inertia" value="0.0083" />
-    <xacro:property name="l2_length" value="0.0403" />
+    <xacro:property name="l2_length" value="0.040" />
     <xacro:property name="l2_radius" value="0.011" />
     <xacro:property name="l2_mass" value="0.1" />
     <xacro:property name="l2_inertia" value="0.0083" />
-    <xacro:property name="sensor_length" value="0.0085" />
+    <xacro:property name="sensor_length" value="0.005" />
     <xacro:property name="sensor_width" value="0.02" />
-    <xacro:property name="tip_adapter_length" value="0.0075" />
+    <xacro:property name="tip_adapter_length" value="0.0113" />
     <xacro:property name="tip_adapter_radius" value="0.0145" />
     <xacro:property name="tip_cylinder_length" value="0.0035" />
@@ -84,14 +86,9 @@
       </joint>
       <link name="finger${fnum}_link2">
-        <!-- The origin of the Link2 frame is defined to be coincident with
-       the origin of the x-z plane in the elbow joint frame. -->
+        <!-- The origin of the link2 frame is located at the MidJoint. -->
         <pose>0 0 -${l1_length} 0 0 0</pose>
         <inertial>
-          <pose>0 0 -${l2_length/2} 0 0 0</pose>
+          <pose>0 0 -${(l2_length + sensor_length + tip_adapter_length + tip_cylinder_length)/2} 0 0 0</pose>
           <mass>${l2_mass}</mass>
-          <!-- This inertia is based on a solid cylinder with
-               radius=1.0 meters and height=2.0 meters. -->
-          <!-- For this model we could make izz = 0 however, sdformat will throw
-               an exception. -->
           <inertia>
             <ixx>${l2_inertia}</ixx><iyy>${l2_inertia}</iyy><izz>5e-7</izz>
@@ -111,5 +108,6 @@
           </material>
         </visual>
-        <!--The link 2 collision element extends up to the sphere fingertip-->
+        <!--The link 2 collision element extends up to (but not including) the
+            sphere fingertip-->
         <collision name='link2_collision'>
           <pose>0 0 -${(l2_length + sensor_length + tip_adapter_length + tip_cylinder_length)/2} 0 0 0</pose>
@@ -124,5 +122,5 @@
           </material>
         </collision>
-        <visual name='link2_sensor_visual'>
+        <visual name='sensor_visual'>
           <pose>0 0 -${l2_length + sensor_length/2.0} 0 0 0</pose>
           <geometry>
@@ -132,53 +130,7 @@
           </geometry>
           <material>
-            <diffuse>.1 .1 .1 1</diffuse>
-          </material>
-        </visual>
-        <visual name="tip_adapter_visual">
-          <pose>0 0 -${l2_length + sensor_length + tip_adapter_length/2} 0 0 0</pose>
-          <geometry>
-            <cylinder>
-              <length>${tip_adapter_length}</length>
-              <radius>${tip_adapter_radius}</radius>
-            </cylinder>
-          </geometry>
-          <material>
-            <diffuse>.1 .1 .1 1</diffuse>
-          </material>
-        </visual>
-        <visual name="tip_cylinder_visual">
-          <pose>0 0 -${l2_length + sensor_length + tip_adapter_length + tip_cylinder_length/2} 0 0 0</pose>
-          <geometry>
-            <cylinder>
-              <length>${tip_cylinder_length}</length>
-              <radius>${tip_cylinder_radius}</radius>
-            </cylinder>
-          </geometry>
-          <material>
-            <diffuse>.1 .1 .1 1</diffuse>
-          </material>
-        </visual>
-        <visual name='tip_sphere_visual'>
-          <pose>0 0 -${l2_length + sensor_length + tip_adapter_length + tip_sphere_radius} 0 0 0</pose>
-          <geometry>
-            <sphere>
-              <radius>${tip_sphere_radius}</radius>
-            </sphere>
-          </geometry>
-          <material>
-            <diffuse>1 1 1 1</diffuse>
-          </material>
-        </visual>
-        <collision name='tip_sphere_collision'>
-          <pose>0 0 -${l2_length + sensor_length + tip_adapter_length + tip_sphere_radius} 0 0 0</pose>
-          <geometry>
-            <sphere>
-              <radius>${tip_sphere_radius}</radius>
-            </sphere>
-          </geometry>
-          <material>
-            <diffuse>1 1 1 1</diffuse>
-          </material>
-        </collision>
+            <diffuse>.8 .8 .8 1</diffuse>
+          </material>
+        </visual>
       </link>
       <joint name='finger${fnum}_MidJoint' type='revolute'>
@@ -200,4 +152,69 @@
         </axis>
       </joint>
+      <!-- The tip link mass/inertia values are already included in link 2,
+           which welds to this link. Hence, the values here are set to be
+           (effectively) zero. -->
+      <link name="finger${fnum}_tip_link">
+        <pose>0 0 -${l1_length + l2_length + sensor_length} 0 0 0</pose>
+        <inertial>
+          <pose>0 0 -${(tip_adapter_length + tip_cylinder_length)/2} 0 0 0</pose>
+          <mass>1e-7</mass>
+          <inertia>
+            <ixx>1e-7</ixx><iyy>1e-7</iyy><izz>1e-7</izz>
+            <ixy>0</ixy><ixz>0</ixz><iyz>0</iyz>
+          </inertia>
+        </inertial>
+        <visual name="tip_adapter_visual">
+          <pose>0 0 -${tip_adapter_length/2} 0 0 0</pose>
+          <geometry>
+            <cylinder>
+              <length>${tip_adapter_length}</length>
+              <radius>${tip_adapter_radius}</radius>
+            </cylinder>
+          </geometry>
+          <material>
+            <diffuse>.3 .3 .3 1</diffuse>
+          </material>
+        </visual>
+        <visual name="tip_cylinder_visual">
+          <pose>0 0 -${tip_adapter_length + tip_cylinder_length/2} 0 0 0</pose>
+          <geometry>
+            <cylinder>
+              <length>${tip_cylinder_length}</length>
+              <radius>${tip_cylinder_radius}</radius>
+            </cylinder>
+          </geometry>
+          <material>
+            <diffuse>.3 .3 .3 1</diffuse>
+          </material>
+        </visual>
+        <visual name='tip_sphere_visual'>
+          <pose>0 0 -${tip_adapter_length + tip_sphere_radius} 0 0 0</pose>
+          <geometry>
+            <sphere>
+              <radius>${tip_sphere_radius}</radius>
+            </sphere>
+          </geometry>
+          <material>
+            <diffuse>1 1 1 1</diffuse>
+          </material>
+        </visual>
+        <collision name='tip_sphere_collision'>
+          <pose>0 0 -${tip_adapter_length + tip_sphere_radius} 0 0 0</pose>
+          <geometry>
+            <sphere>
+              <radius>${tip_sphere_radius}</radius>
+            </sphere>
+          </geometry>
+          <material>
+            <diffuse>1 1 1 1</diffuse>
+          </material>
+        </collision>
+      </link>
+      <joint name='finger${fnum}_sensor_weldjoint' type='fixed'>
+        <parent>finger${fnum}_link2</parent>
+        <child>finger${fnum}_tip_link</child>
+        <pose>0 0 0 0 0 0</pose>
+      </joint>
     </xacro:macro>
     <xacro:finger fnum="1" />
