Commit message: Adds a weld joint to the planar_gripper fingers at the force sensor interface, splitting link 2 into two separate links. This allows reaction force measurement via MBP.
Also fixes a bug in the definition of finger orientations.

File: examples/planar_gripper/planar_gripper.xacro (robot description, xacro)
@@ -2,4 +2,6 @@
 <sdf xmlns:xacro="http://www.ros.org/wiki/xacro" version='1.6'>
   <model name='planar_gripper'>
+    <!-- Link mass and inertia values are guesses (currently), calculated using
+         a uniform rod model, rotating about its center of mass. -->
     <xacro:property name="base_dim" value=".08" />
     <xacro:property name="l1_length" value="0.085" />
@@ -7,11 +9,11 @@
     <xacro:property name="l1_mass" value="0.1" />
     <xacro:property name="l1_inertia" value="0.0083" />
-    <xacro:property name="l2_length" value="0.0403" />
+    <xacro:property name="l2_length" value="0.040" />
     <xacro:property name="l2_radius" value="0.011" />
     <xacro:property name="l2_mass" value="0.1" />
     <xacro:property name="l2_inertia" value="0.0083" />
-    <xacro:property name="sensor_length" value="0.0085" />
+    <xacro:property name="sensor_length" value="0.005" />
     <xacro:property name="sensor_width" value="0.02" />
-    <xacro:property name="tip_adapter_length" value="0.0075" />
+    <xacro:property name="tip_adapter_length" value="0.0113" />
     <xacro:property name="tip_adapter_radius" value="0.0145" />
     <xacro:property name="tip_cylinder_length" value="0.0035" />
@@ -84,14 +86,9 @@
       </joint>
       <link name="finger${fnum}_link2">
-        <!-- The origin of the Link2 frame is defined to be coincident with
-       the origin of the x-z plane in the elbow joint frame. -->
+        <!-- The origin of the link2 frame is located at the MidJoint. -->
         <pose>0 0 -${l1_length} 0 0 0</pose>
         <inertial>
-          <pose>0 0 -${l2_length/2} 0 0 0</pose>
+          <pose>0 0 -${(l2_length + sensor_length + tip_adapter_length + tip_cylinder_length)/2} 0 0 0</pose>
           <mass>${l2_mass}</mass>
-          <!-- This inertia is based on a solid cylinder with
-               radius=1.0 meters and height=2.0 meters. -->
-          <!-- For this model we could make izz = 0 however, sdformat will throw
-               an exception. -->
           <inertia>
             <ixx>${l2_inertia}</ixx><iyy>${l2_inertia}</iyy><izz>5e-7</izz>
@@ -111,5 +108,6 @@
           </material>
         </visual>
-        <!--The link 2 collision element extends up to the sphere fingertip-->
+        <!--The link 2 collision element extends up to (but not including) the
+            sphere fingertip-->
         <collision name='link2_collision'>
           <pose>0 0 -${(l2_length + sensor_length + tip_adapter_length + tip_cylinder_length)/2} 0 0 0</pose>
@@ -124,5 +122,5 @@
           </material>
         </collision>
-        <visual name='link2_sensor_visual'>
+        <visual name='sensor_visual'>
           <pose>0 0 -${l2_length + sensor_length/2.0} 0 0 0</pose>
           <geometry>
@@ -132,53 +130,7 @@
           </geometry>
           <material>
-            <diffuse>.1 .1 .1 1</diffuse>
-          </material>
-        </visual>
-        <visual name="tip_adapter_visual">
-          <pose>0 0 -${l2_length + sensor_length + tip_adapter_length/2} 0 0 0</pose>
-          <geometry>
-            <cylinder>
-              <length>${tip_adapter_length}</length>
-              <radius>${tip_adapter_radius}</radius>
-            </cylinder>
-          </geometry>
-          <material>
-            <diffuse>.1 .1 .1 1</diffuse>
-          </material>
-        </visual>
-        <visual name="tip_cylinder_visual">
-          <pose>0 0 -${l2_length + sensor_length + tip_adapter_length + tip_cylinder_length/2} 0 0 0</pose>
-          <geometry>
-            <cylinder>
-              <length>${tip_cylinder_length}</length>
-              <radius>${tip_cylinder_radius}</radius>
-            </cylinder>
-          </geometry>
-          <material>
-            <diffuse>.1 .1 .1 1</diffuse>
-          </material>
-        </visual>
-        <visual name='tip_sphere_visual'>
-          <pose>0 0 -${l2_length + sensor_length + tip_adapter_length + tip_sphere_radius} 0 0 0</pose>
-          <geometry>
-            <sphere>
-              <radius>${tip_sphere_radius}</radius>
-            </sphere>
-          </geometry>
-          <material>
-            <diffuse>1 1 1 1</diffuse>
-          </material>
-        </visual>
-        <collision name='tip_sphere_collision'>
-          <pose>0 0 -${l2_length + sensor_length + tip_adapter_length + tip_sphere_radius} 0 0 0</pose>
-          <geometry>
-            <sphere>
-              <radius>${tip_sphere_radius}</radius>
-            </sphere>
-          </geometry>
-          <material>
-            <diffuse>1 1 1 1</diffuse>
-          </material>
-        </collision>
+            <diffuse>.8 .8 .8 1</diffuse>
+          </material>
+        </visual>
       </link>
       <joint name='finger${fnum}_MidJoint' type='revolute'>
@@ -200,4 +152,71 @@
         </axis>
       </joint>
+      <!-- The tip link's mass/inertia values are already included in link 2,
+           which welds to this link. Hence, the values here are set to be
+           (effectively) zero. Note: This fingertip link and its corresponding
+           weld joint allows us to sense forces via MBP's reaction forces
+           output port. -->
+      <link name="finger${fnum}_tip_link">
+        <pose>0 0 -${l1_length + l2_length + sensor_length} 0 0 0</pose>
+        <inertial>
+          <pose>0 0 -${(tip_adapter_length + tip_cylinder_length)/2} 0 0 0</pose>
+          <mass>1e-7</mass>
+          <inertia>
+            <ixx>1e-7</ixx><iyy>1e-7</iyy><izz>1e-7</izz>
+            <ixy>0</ixy><ixz>0</ixz><iyz>0</iyz>
+          </inertia>
+        </inertial>
+        <visual name="tip_adapter_visual">
+          <pose>0 0 -${tip_adapter_length/2} 0 0 0</pose>
+          <geometry>
+            <cylinder>
+              <length>${tip_adapter_length}</length>
+              <radius>${tip_adapter_radius}</radius>
+            </cylinder>
+          </geometry>
+          <material>
+            <diffuse>.3 .3 .3 1</diffuse>
+          </material>
+        </visual>
+        <visual name="tip_cylinder_visual">
+          <pose>0 0 -${tip_adapter_length + tip_cylinder_length/2} 0 0 0</pose>
+          <geometry>
+            <cylinder>
+              <length>${tip_cylinder_length}</length>
+              <radius>${tip_cylinder_radius}</radius>
+            </cylinder>
+          </geometry>
+          <material>
+            <diffuse>.3 .3 .3 1</diffuse>
+          </material>
+        </visual>
+        <visual name='tip_sphere_visual'>
+          <pose>0 0 -${tip_adapter_length + tip_sphere_radius} 0 0 0</pose>
+          <geometry>
+            <sphere>
+              <radius>${tip_sphere_radius}</radius>
+            </sphere>
+          </geometry>
+          <material>
+            <diffuse>1 1 1 1</diffuse>
+          </material>
+        </visual>
+        <collision name='tip_sphere_collision'>
+          <pose>0 0 -${tip_adapter_length + tip_sphere_radius} 0 0 0</pose>
+          <geometry>
+            <sphere>
+              <radius>${tip_sphere_radius}</radius>
+            </sphere>
+          </geometry>
+          <material>
+            <diffuse>1 1 1 1</diffuse>
+          </material>
+        </collision>
+      </link>
+      <joint name='finger${fnum}_sensor_weldjoint' type='fixed'>
+        <parent>finger${fnum}_link2</parent>
+        <child>finger${fnum}_tip_link</child>
+        <pose>0 0 0 0 0 0</pose>
+      </joint>
     </xacro:macro>
     <xacro:finger fnum="1" />

Commit message: Updates planar gripper sim parameters to match hardware. Also, moved BrickFace and Finger enums to planar_gripper_common.

File: examples/planar_gripper/planar_gripper.xacro (robot description, xacro)
@@ -7,10 +7,20 @@
     <xacro:property name="l1_length" value="0.085" />
     <xacro:property name="l1_radius" value="0.011" />
-    <xacro:property name="l1_mass" value="0.1" />
-    <xacro:property name="l1_inertia" value="0.0083" />
+    <xacro:property name="l1_mass" value="0.449" />
+    <xacro:property name="l1_ixx" value="1.519282829" />
+    <xacro:property name="l1_iyy" value="1.519856854" />
+    <xacro:property name="l1_izz" value="0.0006529" />
+    <xacro:property name="l1_ixz" value="2.8883e-05" />
+    <xacro:property name="l1_ixy" value="0" />
+    <xacro:property name="l1_iyz" value="0" />
     <xacro:property name="l2_length" value="0.040" />
     <xacro:property name="l2_radius" value="0.011" />
-    <xacro:property name="l2_mass" value="0.1" />
-    <xacro:property name="l2_inertia" value="0.0083" />
+    <xacro:property name="l2_mass" value="0.104" />
+    <xacro:property name="l2_ixx" value="1.513503562" />
+    <xacro:property name="l2_iyy" value="1.513508314" />
+    <xacro:property name="l2_izz" value="1.2773e-05" />
+    <xacro:property name="l2_ixz" value="6.523e-06" />
+    <xacro:property name="l2_ixy" value="0" />
+    <xacro:property name="l2_iyz" value="0" />
     <xacro:property name="sensor_length" value="0.005" />
     <xacro:property name="sensor_width" value="0.02" />
@@ -40,6 +50,10 @@
           <mass>${l1_mass}</mass>
           <inertia>
-            <ixx>${l1_inertia}</ixx><iyy>${l1_inertia}</iyy><izz>5e-7</izz>
-            <ixy>0</ixy><ixz>0</ixz><iyz>0</iyz>
+            <ixx>${l1_ixx}</ixx>
+            <iyy>${l1_iyy}</iyy>
+            <izz>${l1_izz}</izz>
+            <ixz>${l1_ixz}</ixz>
+            <ixy>${l1_ixy}</ixy>
+            <iyz>${l1_iyz}</iyz>
           </inertia>
         </inertial>
@@ -92,6 +106,10 @@
           <mass>${l2_mass}</mass>
           <inertia>
-            <ixx>${l2_inertia}</ixx><iyy>${l2_inertia}</iyy><izz>5e-7</izz>
-            <ixy>0</ixy><ixz>0</ixz><iyz>0</iyz>
+            <ixx>${l2_ixx}</ixx>
+            <iyy>${l2_iyy}</iyy>
+            <izz>${l2_izz}</izz>
+            <ixz>${l2_ixz}</ixz>
+            <ixy>${l2_ixy}</ixy>
+            <iyz>${l2_iyz}</iyz>
           </inertia>
         </inertial>

Commit message: Mow over all XML files with xmllint

File: examples/planar_gripper/planar_gripper.xacro (robot description, xacro)
@@ -1,26 +1,26 @@
 <?xml version="1.0"?>
-<sdf xmlns:xacro="http://www.ros.org/wiki/xacro" version='1.6'>
-  <model name='planar_gripper'>
+<sdf xmlns:xacro="http://www.ros.org/wiki/xacro" version="1.6">
+  <model name="planar_gripper">
     <!-- Link mass and inertia values are guesses (currently), calculated using
          a uniform rod model, rotating about its center of mass. -->
-    <xacro:property name="base_dim" value=".08" />
-    <xacro:property name="l1_length" value="0.085" />
-    <xacro:property name="l1_radius" value="0.011" />
-    <xacro:property name="l1_mass" value="0.1" />
-    <xacro:property name="l1_inertia" value="0.0083" />
-    <xacro:property name="l2_length" value="0.040" />
-    <xacro:property name="l2_radius" value="0.011" />
-    <xacro:property name="l2_mass" value="0.1" />
-    <xacro:property name="l2_inertia" value="0.0083" />
-    <xacro:property name="sensor_length" value="0.005" />
-    <xacro:property name="sensor_width" value="0.02" />
-    <xacro:property name="tip_adapter_length" value="0.0113" />
-    <xacro:property name="tip_adapter_radius" value="0.0145" />
-    <xacro:property name="tip_cylinder_length" value="0.0035" />
-    <xacro:property name="tip_cylinder_radius" value="0.01" />
-    <xacro:property name="tip_sphere_radius" value="0.015" />
+    <xacro:property name="base_dim" value=".08"/>
+    <xacro:property name="l1_length" value="0.085"/>
+    <xacro:property name="l1_radius" value="0.011"/>
+    <xacro:property name="l1_mass" value="0.1"/>
+    <xacro:property name="l1_inertia" value="0.0083"/>
+    <xacro:property name="l2_length" value="0.040"/>
+    <xacro:property name="l2_radius" value="0.011"/>
+    <xacro:property name="l2_mass" value="0.1"/>
+    <xacro:property name="l2_inertia" value="0.0083"/>
+    <xacro:property name="sensor_length" value="0.005"/>
+    <xacro:property name="sensor_width" value="0.02"/>
+    <xacro:property name="tip_adapter_length" value="0.0113"/>
+    <xacro:property name="tip_adapter_radius" value="0.0145"/>
+    <xacro:property name="tip_cylinder_length" value="0.0035"/>
+    <xacro:property name="tip_cylinder_radius" value="0.01"/>
+    <xacro:property name="tip_sphere_radius" value="0.015"/>
     <xacro:macro name="finger" params="fnum">
       <link name="finger${fnum}_base">
-        <visual name='base_visual'>
+        <visual name="base_visual">
           <pose>0 0 0 0 0 0</pose>
           <geometry>
@@ -40,9 +40,13 @@
           <mass>${l1_mass}</mass>
           <inertia>
-            <ixx>${l1_inertia}</ixx><iyy>${l1_inertia}</iyy><izz>5e-7</izz>
-            <ixy>0</ixy><ixz>0</ixz><iyz>0</iyz>
+            <ixx>${l1_inertia}</ixx>
+            <iyy>${l1_inertia}</iyy>
+            <izz>5e-7</izz>
+            <ixy>0</ixy>
+            <ixz>0</ixz>
+            <iyz>0</iyz>
           </inertia>
         </inertial>
-        <visual name='link1_visual'>
+        <visual name="link1_visual">
           <pose>0 0 -${l1_length/2} 0 0 0</pose>
           <geometry>
@@ -56,5 +60,5 @@
           </material>
         </visual>
-        <visual name='link1_joint_visual'>
+        <visual name="link1_joint_visual">
           <pose>0 0 -${l1_length} 0 0 0</pose>
           <geometry>
@@ -68,5 +72,5 @@
         </visual>
       </link>
-      <joint name='finger${fnum}_BaseJoint' type='revolute'>
+      <joint name="finger${fnum}_BaseJoint" type="revolute">
         <child>finger${fnum}_link1</child>
         <parent>finger${fnum}_base</parent>
@@ -92,9 +96,13 @@
           <mass>${l2_mass}</mass>
           <inertia>
-            <ixx>${l2_inertia}</ixx><iyy>${l2_inertia}</iyy><izz>5e-7</izz>
-            <ixy>0</ixy><ixz>0</ixz><iyz>0</iyz>
+            <ixx>${l2_inertia}</ixx>
+            <iyy>${l2_inertia}</iyy>
+            <izz>5e-7</izz>
+            <ixy>0</ixy>
+            <ixz>0</ixz>
+            <iyz>0</iyz>
           </inertia>
         </inertial>
-        <visual name='link2_visual'>
+        <visual name="link2_visual">
           <pose>0 0 -${l2_length/2} 0 0 0</pose>
           <geometry>
@@ -110,5 +118,5 @@
         <!--The link 2 collision element extends up to (but not including) the
             sphere fingertip-->
-        <collision name='link2_collision'>
+        <collision name="link2_collision">
           <pose>0 0 -${(l2_length + sensor_length + tip_adapter_length + tip_cylinder_length)/2} 0 0 0</pose>
           <geometry>
@@ -121,5 +129,5 @@
           </material>
         </collision>
-        <visual name='sensor_visual'>
+        <visual name="sensor_visual">
           <pose>0 0 -${l2_length + sensor_length/2.0} 0 0 0</pose>
           <geometry>
@@ -133,5 +141,5 @@
         </visual>
       </link>
-      <joint name='finger${fnum}_MidJoint' type='revolute'>
+      <joint name="finger${fnum}_MidJoint" type="revolute">
         <parent>finger${fnum}_link1</parent>
         <child>finger${fnum}_link2</child>
@@ -162,6 +170,10 @@
           <mass>1e-7</mass>
           <inertia>
-            <ixx>1e-7</ixx><iyy>1e-7</iyy><izz>1e-7</izz>
-            <ixy>0</ixy><ixz>0</ixz><iyz>0</iyz>
+            <ixx>1e-7</ixx>
+            <iyy>1e-7</iyy>
+            <izz>1e-7</izz>
+            <ixy>0</ixy>
+            <ixz>0</ixz>
+            <iyz>0</iyz>
           </inertia>
         </inertial>
@@ -190,5 +202,5 @@
           </material>
         </visual>
-        <visual name='tip_sphere_visual'>
+        <visual name="tip_sphere_visual">
           <pose>0 0 -${tip_adapter_length + tip_sphere_radius} 0 0 0</pose>
           <geometry>
@@ -201,5 +213,5 @@
           </material>
         </visual>
-        <collision name='tip_sphere_collision'>
+        <collision name="tip_sphere_collision">
           <pose>0 0 -${tip_adapter_length + tip_sphere_radius} 0 0 0</pose>
           <geometry>
@@ -213,5 +225,5 @@
         </collision>
       </link>
-      <joint name='finger${fnum}_sensor_weldjoint' type='fixed'>
+      <joint name="finger${fnum}_sensor_weldjoint" type="fixed">
         <parent>finger${fnum}_link2</parent>
         <child>finger${fnum}_tip_link</child>
@@ -219,7 +231,7 @@
       </joint>
     </xacro:macro>
-    <xacro:finger fnum="1" />
-    <xacro:finger fnum="2" />
-    <xacro:finger fnum="3" />
+    <xacro:finger fnum="1"/>
+    <xacro:finger fnum="2"/>
+    <xacro:finger fnum="3"/>
   </model>
 </sdf>
