Commit message: Use package instead of relative path for allegro model files

File: manipulation/models/allegro_hand_description/urdf/allegro_hand_description_left.urdf (robot description, URDF)
Before this commit: robot allegro_hand_left, 22 links, 21 joints
Links:
- link link_0: geometry collision box size=0.0196 0.0275 0.0164; visual mesh filename=package://allegro_hand_description/meshes/link_0.0.obj
- link link_1: geometry collision box size=0.0196 0.0275 0.054; visual mesh filename=package://allegro_hand_description/meshes/link_1.0.obj
- link link_10: geometry collision box size=0.0196 0.0275 0.0384; visual mesh filename=package://allegro_hand_description/meshes/link_2.0.obj
- link link_11: geometry collision box size=0.0196 0.0275 0.0267; visual mesh filename=package://allegro_hand_description/meshes/link_3.0.obj
- link link_11_tip: geometry collision sphere radius=0.012; visual mesh filename=package://allegro_hand_description/meshes/link_3.0_tip.obj
- link link_12: geometry collision box size=0.0358 0.034 0.0455; visual mesh filename=package://allegro_hand_description/meshes/link_12.0_left.obj
- link link_13: geometry collision box size=0.0196 0.0275 0.0177; visual mesh filename=package://allegro_hand_description/meshes/link_13.0.obj
- link link_14: geometry collision box size=0.0196 0.0275 0.0514; visual mesh filename=package://allegro_hand_description/meshes/link_14.0.obj
- link link_15: geometry collision box size=0.0196 0.0275 0.0423; visual mesh filename=package://allegro_hand_description/meshes/link_15.0.obj
- link link_15_tip: geometry collision sphere radius=0.012; visual mesh filename=package://allegro_hand_description/meshes/link_15.0_tip.obj
- link link_2: geometry collision box size=0.0196 0.0275 0.0384; visual mesh filename=package://allegro_hand_description/meshes/link_2.0.obj
- link link_3: geometry collision box size=0.0196 0.0275 0.0267; visual mesh filename=package://allegro_hand_description/meshes/link_3.0.obj
- link link_3_tip: geometry collision sphere radius=0.012; visual mesh filename=package://allegro_hand_description/meshes/link_3.0_tip.obj
- link link_4: geometry collision box size=0.0196 0.0275 0.0164; visual mesh filename=package://allegro_hand_description/meshes/link_0.0.obj
- link link_5: geometry collision box size=0.0196 0.0275 0.054; visual mesh filename=package://allegro_hand_description/meshes/link_1.0.obj
- link link_6: geometry collision box size=0.0196 0.0275 0.0384; visual mesh filename=package://allegro_hand_description/meshes/link_2.0.obj
- link link_7: geometry collision box size=0.0196 0.0275 0.0267; visual mesh filename=package://allegro_hand_description/meshes/link_3.0.obj
- link link_7_tip: geometry collision sphere radius=0.012; visual mesh filename=package://allegro_hand_description/meshes/link_3.0_tip.obj
- link link_8: geometry collision box size=0.0196 0.0275 0.0164; visual mesh filename=package://allegro_hand_description/meshes/link_0.0.obj
- link link_9: geometry collision box size=0.0196 0.0275 0.054; visual mesh filename=package://allegro_hand_description/meshes/link_1.0.obj
- link palm_link: geometry collision box size=0.0408 0.1130 0.095; visual mesh filename=package://allegro_hand_description/meshes/base_link_left.obj

File: manipulation/models/allegro_hand_description/urdf/allegro_hand_description_right.urdf (robot description, URDF)
Before this commit: robot allegro_hand_right, 22 links, 21 joints
Links:
- link link_0: geometry collision box size=0.0196 0.0275 0.0164; visual mesh filename=package://allegro_hand_description/meshes/link_0.0.obj
- link link_1: geometry collision box size=0.0196 0.0275 0.054; visual mesh filename=package://allegro_hand_description/meshes/link_1.0.obj
- link link_10: geometry collision box size=0.0196 0.0275 0.0384; visual mesh filename=package://allegro_hand_description/meshes/link_2.0.obj
- link link_11: geometry collision box size=0.0196 0.0275 0.0267; visual mesh filename=package://allegro_hand_description/meshes/link_3.0.obj
- link link_11_tip: geometry collision sphere radius=0.012; visual mesh filename=package://allegro_hand_description/meshes/link_3.0_tip.obj
- link link_12: geometry collision box size=0.0358 0.034 0.0455; visual mesh filename=package://allegro_hand_description/meshes/link_12.0_right.o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
- link link_13: geometry collision box size=0.0196 0.0275 0.0177; visual mesh filename=package://allegro_hand_description/meshes/link_13.0.obj
- link link_14: geometry collision box size=0.0196 0.0275 0.0514; visual mesh filename=package://allegro_hand_description/meshes/link_14.0.obj
- link link_15: geometry collision box size=0.0196 0.0275 0.0423; visual mesh filename=package://allegro_hand_description/meshes/link_15.0.obj
- link link_15_tip: geometry collision sphere radius=0.012; visual mesh filename=package://allegro_hand_description/meshes/link_15.0_tip.obj
- link link_2: geometry collision box size=0.0196 0.0275 0.0384; visual mesh filename=package://allegro_hand_description/meshes/link_2.0.obj
- link link_3: geometry collision box size=0.0196 0.0275 0.0267; visual mesh filename=package://allegro_hand_description/meshes/link_3.0.obj
- link link_3_tip: geometry collision sphere radius=0.012; visual mesh filename=package://allegro_hand_description/meshes/link_3.0_tip.obj
- link link_4: geometry collision box size=0.0196 0.0275 0.0164; visual mesh filename=package://allegro_hand_description/meshes/link_0.0.obj
- link link_5: geometry collision box size=0.0196 0.0275 0.054; visual mesh filename=package://allegro_hand_description/meshes/link_1.0.obj
- link link_6: geometry collision box size=0.0196 0.0275 0.0384; visual mesh filename=package://allegro_hand_description/meshes/link_2.0.obj
- link link_7: geometry collision box size=0.0196 0.0275 0.0267; visual mesh filename=package://allegro_hand_description/meshes/link_3.0.obj
- link link_7_tip: geometry collision sphere radius=0.012; visual mesh filename=package://allegro_hand_description/meshes/link_3.0_tip.obj
- link link_8: geometry collision box size=0.0196 0.0275 0.0164; visual mesh filename=package://allegro_hand_description/meshes/link_0.0.obj
- link link_9: geometry collision box size=0.0196 0.0275 0.054; visual mesh filename=package://allegro_hand_description/meshes/link_1.0.obj
- link palm_link: geometry collision box size=0.0408 0.1130 0.095; visual mesh filename=package://allegro_hand_description/meshes/base_link.obj
