Commit message: [parsing] Warn about unsupported URDF features
Closes: #16783
Closes: #16181

Based on study of the ROS documentation and urdfdom module sources, add
warnings for ignored URDF features. Implementation is similar to the
in-progress mujoco parser, with an eye to future integration of diagnostics
there.

Adjust tests for existing files that emit new warnings, and add explicit
tests for each of the added warning types.

File: examples/pr2/models/pr2_description/urdf/pr2_simplified.urdf (robot description, URDF)
Before this commit: robot pr2, 83 links, 83 joints
Joints:
- joint l_gripper_l_finger_tip_joint: mimic joint=l_gripper_l_finger_joint multiplier=1 offset=0 -> (none)
- joint l_gripper_l_parallel_root_joint: mimic joint=l_gripper_l_finger_joint multiplier=1 offset=0 -> (none)
- joint l_gripper_r_finger_joint: mimic joint=l_gripper_l_finger_joint multiplier=1 offset=0 -> (none)
- joint l_gripper_r_finger_tip_joint: mimic joint=l_gripper_l_finger_joint multiplier=1 offset=0 -> (none)
- joint l_gripper_r_parallel_root_joint: mimic joint=l_gripper_l_finger_joint multiplier=-1 offset=0 -> (none)
- joint r_gripper_l_finger_tip_joint: mimic joint=r_gripper_l_finger_joint multiplier=1 offset=0 -> (none)
- joint r_gripper_l_parallel_root_joint: mimic joint=r_gripper_l_finger_joint multiplier=1 offset=0 -> (none)
- joint r_gripper_r_finger_joint: mimic joint=r_gripper_l_finger_joint multiplier=1 offset=0 -> (none)
- joint r_gripper_r_finger_tip_joint: mimic joint=r_gripper_l_finger_joint multiplier=1 offset=0 -> (none)
- joint r_gripper_r_parallel_root_joint: mimic joint=r_gripper_l_finger_joint multiplier=-1 offset=0 -> (none)

File: manipulation/models/franka_description/urdf/hand.urdf (robot description, URDF)
Before this commit: robot hand, 3 links, 2 joints
Joints:
- joint panda_finger_joint2: mimic joint=panda_finger_joint1 -> (none)

File: manipulation/models/franka_description/urdf/panda_arm_hand.urdf (robot description, URDF)
Before this commit: robot panda, 12 links, 11 joints
Joints:
- joint panda_finger_joint2: mimic joint=panda_finger_joint1 -> (none)
