Commit message: fix: increase the accuracy of the joint angles

File: multibody/plant/test/inverse_dynamics_R.urdf (robot description, URDF)
Before this commit: robot R, 4 links, 3 joints
Joints:
- joint joint_1: limit lower=0 upper=3.14159 effort=0 velocity=0 -> lower=0 upper=3.14159265358979323846 effort=0 velocity=0; origin xyz=0.0 0 0.0 rpy=1.5708 0.0 0 -> xyz=0.0 0 0.0 rpy=1.5707963267948966 0.0 0
- joint joint_e: origin xyz=1 0.0 0 rpy=3.14159 -1.5708 0 -> xyz=1 0.0 0 rpy=3.14159265358979323846 -1.5707963267948966 0
