Commit message: [multibody] Remove unused brittle mesh paths from unit test

File: multibody/plant/test/atlas_with_fixed_joints.urdf (robot description, URDF)
Before this commit: robot atlas, 70 links, 69 joints
Links:
- link head: geometry 
- link hokuyo_link: geometry 
- link l_clav: geometry 
- link l_foot: geometry collision sphere radius=0.0; collision sphere radius=0.0
- link l_larm: geometry 
- link l_lfarm: geometry 
- link l_lglut: geometry 
- link l_lleg: geometry 
- link l_scap: geometry 
- link l_talus: geometry 
- link l_uarm: geometry 
- link l_ufarm: geometry 
- link l_uglut: geometry 
- link l_uleg: geometry 
- link left_palm: geometry 
- link ltorso: geometry 
- link mtorso: geometry 
- link pelvis: geometry 
- link r_clav: geometry 
- link r_foot: geometry collision sphere radius=0.0; collision sphere radius=0.0
- link r_larm: geometry 
- link r_lfarm: geometry 
- link r_lglut: geometry 
- link r_lleg: geometry 
- link r_scap: geometry 
- link r_talus: geometry 
- link r_uarm: geometry 
- link r_ufarm: geometry 
- link r_uglut: geometry 
- link r_uleg: geometry 
- link right_palm: geometry 
- link utorso: geometry 
