Commit message: [multibody] Move all benchmarks into one place
These were all written prior to our guidance to add benchmarks using a
certain folder structure.

File: multibody/benchmarking/cassie_v2.urdf (robot description, URDF)
Before this commit: robot cassie, 23 links, 22 joints
Links:
- link heel_spring_left: geometry visual mesh filename=heel-spring.obj
- link heel_spring_right: geometry visual mesh filename=heel-spring.obj
- link hip_left: geometry visual mesh filename=agility/left_hip.obj
- link hip_right: geometry visual mesh filename=agility/right_hip.obj
- link knee_left: geometry visual mesh filename=knee-output.obj
- link knee_right: geometry visual mesh filename=knee-output-r.obj
- link knee_spring_left: geometry visual mesh filename=knee-spring.obj
- link knee_spring_right: geometry visual mesh filename=knee-spring.obj
- link pelvis: geometry visual mesh filename=pelvis.obj
- link shin_left: geometry visual mesh filename=agility/left_shin.obj
- link shin_right: geometry visual mesh filename=agility/right_shin.obj
- link tarsus_left: geometry visual mesh filename=tarsus.obj
- link tarsus_right: geometry visual mesh filename=tarsus-r.obj
- link thigh_left: geometry visual mesh filename=agility/left_thigh.obj
- link thigh_right: geometry visual mesh filename=agility/right_thigh.obj
- link toe_left: geometry collision sphere radius=0.0; collision sphere radius=0.0
- link toe_right: geometry collision sphere radius=0.0; collision sphere radius=0.0
- link yaw_left: geometry visual mesh filename=agility/left_yaw.obj
- link yaw_right: geometry visual mesh filename=agility/right_yaw.obj
