Commit message: Add scene_graph operations to MultibodyPlantSubgraph

File: multibody/parsing/test/sdf_parser_test/interface_api_test/arm.urdf (robot description, URDF)
Before this commit: robot arm, 2 links, 1 joints
Links:
- link L1: geometry collision sphere radius=0.2; visual box size=0.1 0.1 0.1

Commit message: [parsing] Enable multi-robot collision filter groups
Relevant to: #14785

This patch extends the parsing of collision filter groups so that collision
filters can be defined across multiple robots by using SDFormat model
composition.

Summary of changes:
 * add CollisionFilterGroupResolver, with unit test
 * port existing parser modules to use it
   * modernize a few sdf_parser errors
 * demonstrate multi-robot filters in sdf_parser_test

File: multibody/parsing/test/sdf_parser_test/interface_api_test/arm.urdf (robot description, URDF)
Before this commit: robot arm, 2 links, 1 joints
Links:
- link L1: geometry collision sphere radius=0.4
- link L2: geometry collision sphere radius=0.4

Commit message: Fix some of the tests with bad mass/inertia properties.

File: multibody/parsing/test/sdf_parser_test/interface_api_test/arm.urdf (robot description, URDF)
Before this commit: robot arm, 2 links, 1 joints
Links:
- link L2: mass None -> 1

Commit message: New default spatial inertia constructor which alleviates need for recently created function SpatialInertia::MakeTestCube().

File: multibody/parsing/test/sdf_parser_test/interface_api_test/arm.urdf (robot description, URDF)
Before this commit: robot arm, 2 links, 1 joints
Links:
- link L2: mass 1 -> None

Commit message: Address reviewer feedback.
Signed-off-by: Addisu Z. Taddese <addisu@openrobotics.org>

File: multibody/parsing/test/sdf_parser_test/interface_api_test/arm.urdf (robot description, URDF)
Before this commit: robot arm, 2 links, 1 joints
Links:
- link L1: geometry collision sphere radius=0.4
