Commit message: wip: urdf text cleanups

File: manipulation/models/tri_homecart/homecart_bimanual.urdf.xacro (robot description, xacro)
@@ -25,7 +25,5 @@
       respect to the robot arm origins.
   -->
-  <link name="homecart_base_link">
-    <origin xyz="0 0 0" rpy="0 0 0"/>
-  </link>
+  <link name="homecart_base_link"/>
   <xacro:property name="arm_mount_cantilever_length" value="0.254"/>
   <xacro:property name="arm_mount_cantilever_height" value="0.015"/>
@@ -105,7 +103,5 @@
       <child link="${side}arm_mount_stack_link"/>
     </joint>
-    <link name="${side}arm_base_link">
-      <origin xyz="0 0 0" rpy="0 0 0"/>
-    </link>
+    <link name="${side}arm_base_link"/>
     <joint name="${side}arm_base_joint" type="fixed">
       <origin xyz="0 0 ${num_plates*0.02}" rpy="0 0 0"/>
@@ -222,5 +218,5 @@
     </inertial>
     <visual>
-    <origin xyz="0 0 0" rpy="0 0 0"/>
+      <origin xyz="0 0 0" rpy="0 0 0"/>
       <geometry>
         <mesh filename="package://drake_models/tri_homecart/homecart_bimanual_upper_structure.obj"/>
