Commit message: [parsing] Use non-identity world weld in #21413 regression
Identity joint frames are elided (#24687), so the nested URDF repro
needs a non-identity origin to exercise GetRelativeBodyName.

File: multibody/parsing/test/sdf_parser_test/world_weld.urdf (robot description, URDF)
Before this commit: robot gripper_with_world_weld, 1 links, 1 joints
Joints:
- joint world_weld: origin (none) -> xyz=0 0 0.1 rpy=0 0 0
